Commit message: iai_adapters_description: simplified the fwk_fwa_050 mesh

File: iai_adapters_description/urdf/fwk_fwa_050.urdf.xacro (robot description, xacro)
@@ -14,5 +14,5 @@
         <geometry>
           <!-- these meshes were exported in mm, so scale back to m -->
-          <mesh filename="package://iai_adapters_description/meshes/fwk_fwa_050.stl" scale="0.001 0.001 0.001"/>
+          <mesh filename="package://iai_adapters_description/meshes/fwk_fwa_050_simple.stl" scale="0.001 0.001 0.001"/>
         </geometry>
         <material name="Grey"/>
