Commit message: added collada files for the torso changes scale in URDFs/xacros

File: iai_adapters_description/urdf/adapter_fwa050_wsg50.urdf.xacro (robot description, xacro)
@@ -14,5 +14,5 @@
         <geometry>
           <!-- these meshes were exported in mm, so scale back to m -->
-          <mesh filename="package://iai_adapters_description/meshes/adapter_fwa050_wsg50.stl" scale="0.001 0.001 0.001"/>
+          <mesh filename="package://iai_adapters_description/meshes/adapter_fwa050_wsg50.stl"/>
         </geometry>
         <material name="Grey"/>

File: iai_adapters_description/urdf/adapter_kms40_fwk050.urdf.xacro (robot description, xacro)
@@ -14,5 +14,5 @@
         <geometry>
           <!-- these meshes were exported in mm, so scale back to m -->
-          <mesh filename="package://iai_adapters_description/meshes/adapter_kms40_fwk050.stl" scale="0.001 0.001 0.001"/>
+          <mesh filename="package://iai_adapters_description/meshes/adapter_kms40_fwk050.stl"/>
         </geometry>
         <material name="Grey"/>

File: iai_adapters_description/urdf/fwk_fwa_050.urdf.xacro (robot description, xacro)
@@ -14,5 +14,5 @@
         <geometry>
           <!-- these meshes were exported in mm, so scale back to m -->
-          <mesh filename="package://iai_adapters_description/meshes/fwk_fwa_050_simple.stl" scale="0.001 0.001 0.001"/>
+          <mesh filename="package://iai_adapters_description/meshes/fwk_fwa_050_simple.stl"/>
         </geometry>
         <material name="Grey"/>

File: iai_boxy_base/robots/base.URDF (robot description, URDF)
Before this commit: robot base, 3 links, 2 joints
Links:
- link base_link: geometry collision mesh filename=package://iai_boxy_base/meshes/base_link.STL; visual mesh filename=package://iai_boxy_base/meshes/base_link.dae

File: iai_boxy_description/sensors/kinect.urdf.xacro (robot description, xacro)
@@ -14,5 +14,5 @@
         <origin xyz="-0.05 -0.17 -0.02" rpy="${M_PI/2.0} 0 ${M_PI/2.0}"/>
         <geometry>
-          <mesh filename="package://iai_boxy_description/meshes/sensors/68-04546_Kinect_Sensor--coarse.STL" scale="0.001 0.001 0.001" />
+          <mesh filename="package://iai_boxy_description/meshes/sensors/68-04546_Kinect_Sensor--coarse.STL"  />
         </geometry>
         <material name="gray">

File: iai_boxy_torso/robots/torso.URDF (robot description, URDF)
Before this commit: robot torso, 4 links, 3 joints
Links:
- link torso_base_link: geometry collision mesh filename=package://iai_boxy_torso/meshes/torso_base_link.STL; visual mesh filename=package://iai_boxy_torso/meshes/torso_base_link.dae
- link triangle_base_link: geometry collision mesh filename=package://iai_boxy_torso/meshes/triangle_base_link.STL; visual mesh filename=package://iai_boxy_torso/meshes/triangle_base_link.dae

File: iai_kinect2_description/urdf/kinect2.urdf.xacro (robot description, xacro)
@@ -19,5 +19,5 @@
         <geometry>
           <!-- these meshes were exported in mm, so scale back to m -->
-          <mesh filename="package://iai_kinect2_description/meshes/kinect2_origin_on_rgb_optical_frame.stl" scale="0.001 0.001 0.001"/>
+          <mesh filename="package://iai_kinect2_description/meshes/kinect2_origin_on_rgb_optical_frame.stl" />
         </geometry>
         <material name="Kinect2Grey"/>

File: iai_kms_40_description/urdf/kms_40.urdf.xacro (robot description, xacro)
@@ -14,5 +14,5 @@
         <origin rpy="0 0 0" xyz="0 0 0"/>
         <geometry>
-          <mesh filename="package://iai_kms_40_description/meshes/adapter_plate_iso50_kms40_weiss.stl" scale="0.001 0.001 0.001"/>
+          <mesh filename="package://iai_kms_40_description/meshes/adapter_plate_iso50_kms40_weiss.stl" />
         </geometry>
         <material name="Grey"/>
@@ -39,5 +39,5 @@
         <origin rpy="0 0 0" xyz="0 0 0"/>
         <geometry>
-          <mesh filename="package://iai_kms_40_description/meshes/kms40_simple.stl" scale="0.001 0.001 0.001"/>
+          <mesh filename="package://iai_kms_40_description/meshes/kms40_simple.stl" />
         </geometry>
         <material name="Grey"/>

File: iai_kuka_lwr4_description/urdf/kuka_lwr_arm.urdf.xacro (robot description, xacro)
@@ -30,5 +30,5 @@
         <geometry>
           <!-- for each mesh we have two versions, one Collada file with normals and colors, and one simpler STL. The collada file is in cm, and the STL in meters -->
-          <mesh filename="package://iai_kuka_lwr4_description/meshes/arm_base.dae" scale="100 100 100"/>
+          <mesh filename="package://iai_kuka_lwr4_description/meshes/arm_base.dae" />
 	  <!--mesh filename="package://iai_kuka_lwr4_description/meshes/arm_base.stl" scale="1 1 1"-->
         </geometry>
@@ -68,5 +68,5 @@
         <origin xyz="0 0 0" rpy="0 0 ${M_PI}"/>
         <geometry>
-          <mesh filename="package://iai_kuka_lwr4_description/meshes/arm_segment_a.dae" scale="100 100 100"/>
+          <mesh filename="package://iai_kuka_lwr4_description/meshes/arm_segment_a.dae" />
           <!--mesh filename="package://iai_kuka_lwr4_description/meshes/arm_segment_a.stl" scale="1 1 1"/-->
         </geometry>
@@ -111,5 +111,5 @@
         <origin xyz="0 0 0.2" rpy="${M_PI} 0 ${M_PI}"/>
         <geometry>
-          <mesh filename="package://iai_kuka_lwr4_description/meshes/arm_segment_b.dae" scale="100 100 100"/>
+          <mesh filename="package://iai_kuka_lwr4_description/meshes/arm_segment_b.dae" />
           <!--mesh filename="package://iai_kuka_lwr4_description/meshes/arm_segment_b.stl" scale="1 1 1"/-->
         </geometry>
@@ -154,5 +154,5 @@
         <origin xyz="0 0 0" rpy="0 0 0"/>
         <geometry>
-          <mesh filename="package://iai_kuka_lwr4_description/meshes/arm_segment_a.dae" scale="100 100 100"/>
+          <mesh filename="package://iai_kuka_lwr4_description/meshes/arm_segment_a.dae" />
           <!--mesh filename="package://iai_kuka_lwr4_description/meshes/arm_segment_a.stl" scale="1 1 1"/-->
         </geometry>
@@ -197,5 +197,5 @@
         <origin xyz="0 0 0.2" rpy="0 ${M_PI} ${M_PI}"/>
         <geometry>
-          <mesh filename="package://iai_kuka_lwr4_description/meshes/arm_segment_b.dae" scale="100 100 100"/>
+          <mesh filename="package://iai_kuka_lwr4_description/meshes/arm_segment_b.dae" />
           <!--mesh filename="package://iai_kuka_lwr4_description/meshes/arm_segment_b.stl" scale="1 1 1"/-->
         </geometry>
@@ -240,5 +240,5 @@
         <origin xyz="0 0 0" rpy="0 0 ${M_PI}"/>
         <geometry name="${name}_arm_5_geom">
-          <mesh filename="package://iai_kuka_lwr4_description/meshes/arm_segment_last.dae" scale="100 100 100"/>
+          <mesh filename="package://iai_kuka_lwr4_description/meshes/arm_segment_last.dae" />
           <!--mesh filename="package://iai_kuka_lwr4_description/meshes/arm_segment_last.stl" scale="1 1 1"/-->
         </geometry>
@@ -283,5 +283,5 @@
         <origin xyz="0 0 0" rpy="0 0 ${M_PI}"/>
         <geometry>
-          <mesh filename="package://iai_kuka_lwr4_description/meshes/arm_wrist.dae" scale="100 100 100"/>
+          <mesh filename="package://iai_kuka_lwr4_description/meshes/arm_wrist.dae" />
           <!--mesh filename="package://iai_kuka_lwr4_description/meshes/arm_wrist.stl" scale="1 1 1"/-->
         </geometry>
@@ -326,5 +326,5 @@
         <origin xyz="0 0 0.078" rpy="0 0 0"/>
         <geometry>
-          <mesh filename="package://iai_kuka_lwr4_description/meshes/arm_flanche.dae" scale="100 100 100"/>
+          <mesh filename="package://iai_kuka_lwr4_description/meshes/arm_flanche.dae" />
           <!--mesh filename="package://iai_kuka_lwr4_description/meshes/arm_flanche.stl" scale="1 1 1"/-->
         </geometry>

File: iai_wsg_50_description/urdf/wsg_50.urdf.xacro (robot description, xacro)
@@ -70,16 +70,16 @@
           <origin xyz="0.0 0 0" rpy="0 0 0" />
           <geometry>
-             <mesh filename="package://iai_wsg_50_description/meshes/GUIDE_WSG50_110.stl" scale="0.001 0.001 0.001"/>
-	     <!--box size="0.0175 0.03 0.024"/-->
-          </geometry>
-          <material name="black">
-		<color rgba="0 0 0 1"/>
-      	  </material>
-      </visual>
-      <collision>
-          <origin xyz="0 0 0" rpy="0 0 0" />
-          <geometry>
-	     <!--box size="0.0175 0.03 0.024"/-->
-             <mesh filename="package://iai_wsg_50_description/meshes/GUIDE_WSG50_110.stl" scale="0.001 0.001 0.001"/>
+             <mesh filename="package://iai_wsg_50_description/meshes/GUIDE_WSG50_110.stl" />
+	     <!--box size="0.0175 0.03 0.024"/-->
+          </geometry>
+          <material name="black">
+		<color rgba="0 0 0 1"/>
+      	  </material>
+      </visual>
+      <collision>
+          <origin xyz="0 0 0" rpy="0 0 0" />
+          <geometry>
+	     <!--box size="0.0175 0.03 0.024"/-->
+             <mesh filename="package://iai_wsg_50_description/meshes/GUIDE_WSG50_110.stl" />
          </geometry>
      </collision>
@@ -110,14 +110,14 @@
           <origin xyz="0.0 0 0" rpy="0 0 0" />
           <geometry>
-             <mesh filename="package://iai_wsg_50_description/meshes/WSG-FMF.stl" scale="0.001 0.001 0.001"/>
-          </geometry>
-          <material name="black">
-		<color rgba="0 0 0 1"/>
-      	  </material>
-      </visual>
-      <collision>
-          <origin xyz="0 0 0" rpy="0 0 0" />
-          <geometry>
-             <mesh filename="package://iai_wsg_50_description/meshes/WSG-FMF.stl" scale="0.001 0.001 0.001"/>
+             <mesh filename="package://iai_wsg_50_description/meshes/WSG-FMF.stl" />
+          </geometry>
+          <material name="black">
+		<color rgba="0 0 0 1"/>
+      	  </material>
+      </visual>
+      <collision>
+          <origin xyz="0 0 0" rpy="0 0 0" />
+          <geometry>
+             <mesh filename="package://iai_wsg_50_description/meshes/WSG-FMF.stl" />
          </geometry>
      </collision>
@@ -155,16 +155,16 @@
           <origin xyz="0.0 0 0" rpy="0 0 0" />
           <geometry>
-             <mesh filename="package://iai_wsg_50_description/meshes/GUIDE_WSG50_110.stl" scale="0.001 0.001 0.001"/>
-	     <!--box size="0.0175 0.03 0.024"/-->
-          </geometry>
-          <material name="black">
-		<color rgba="0 0 0 1"/>
-      	  </material>
-      </visual>
-      <collision>
-          <origin xyz="0 0 0" rpy="0 0 0" />
-          <geometry>
-	     <!--box size="0.0175 0.03 0.024"/-->
-             <mesh filename="package://iai_wsg_50_description/meshes/GUIDE_WSG50_110.stl" scale="0.001 0.001 0.001"/>
+             <mesh filename="package://iai_wsg_50_description/meshes/GUIDE_WSG50_110.stl" />
+	     <!--box size="0.0175 0.03 0.024"/-->
+          </geometry>
+          <material name="black">
+		<color rgba="0 0 0 1"/>
+      	  </material>
+      </visual>
+      <collision>
+          <origin xyz="0 0 0" rpy="0 0 0" />
+          <geometry>
+	     <!--box size="0.0175 0.03 0.024"/-->
+             <mesh filename="package://iai_wsg_50_description/meshes/GUIDE_WSG50_110.stl" />
          </geometry>
      </collision>
@@ -195,14 +195,14 @@
           <origin xyz="0.0 0 0" rpy="0 0 0" />
           <geometry>
-             <mesh filename="package://iai_wsg_50_description/meshes/WSG-FMF.stl" scale="0.001 0.001 0.001"/>
-          </geometry>
-          <material name="black">
-		<color rgba="0 0 0 1"/>
-      	  </material>
-      </visual>
-      <collision>
-          <origin xyz="0 0 0" rpy="0 0 0" />
-          <geometry>
-             <mesh filename="package://iai_wsg_50_description/meshes/WSG-FMF.stl" scale="0.001 0.001 0.001"/>
+             <mesh filename="package://iai_wsg_50_description/meshes/WSG-FMF.stl" />
+          </geometry>
+          <material name="black">
+		<color rgba="0 0 0 1"/>
+      	  </material>
+      </visual>
+      <collision>
+          <origin xyz="0 0 0" rpy="0 0 0" />
+          <geometry>
+             <mesh filename="package://iai_wsg_50_description/meshes/WSG-FMF.stl" />
          </geometry>
      </collision>

Commit message: Fixed Boxy's wrist adaptor descriptions. Now, they can cope with empty prefixes.

File: iai_adapters_description/urdf/adapter_fwa050_wsg50.urdf.xacro (robot description, xacro)
@@ -4,10 +4,10 @@
   <xacro:macro name="adapter_fwa050_wsg50_xacro" params="prefix parent *origin">
     <!-- Joint connecting the parent to our frame_in -->
-    <joint name="${prefix}_adapter_fwa050_wsg50_in_joint" type="fixed">
+    <joint name="${prefix}adapter_fwa050_wsg50_in_joint" type="fixed">
       <xacro:insert_block name="origin"/>
       <parent link="${parent}"/>
-      <child link="${prefix}_adapter_fwa050_wsg50_frame_in"/>
+      <child link="${prefix}adapter_fwa050_wsg50_frame_in"/>
     </joint>
-    <link name="${prefix}_adapter_fwa050_wsg50_frame_in">
+    <link name="${prefix}adapter_fwa050_wsg50_frame_in">
       <visual>
         <origin rpy="0 0 0" xyz="0 0 0"/>
@@ -20,12 +20,12 @@
     </link>
     <!-- Empty link just to get the frame out -->
-    <link name="${prefix}_adapter_fwa050_wsg50_frame_out"/>
+    <link name="${prefix}adapter_fwa050_wsg50_frame_out"/>
     <!-- joint positioning the frame_out -->
-    <joint name="${prefix}_adapter_fwa050_wsg50_trans_frame_out"
+    <joint name="${prefix}adapter_fwa050_wsg50_trans_frame_out"
            type="fixed">
       <origin xyz="0 0 0.01"
               rpy="0 0 0" />
-      <parent link="${prefix}_adapter_fwa050_wsg50_frame_in" />
-      <child link="${prefix}_adapter_fwa050_wsg50_frame_out" />
+      <parent link="${prefix}adapter_fwa050_wsg50_frame_in" />
+      <child link="${prefix}adapter_fwa050_wsg50_frame_out" />
       <axis xyz="0 0 0" />
     </joint>

File: iai_adapters_description/urdf/adapter_kms40_fwk050.urdf.xacro (robot description, xacro)
@@ -4,10 +4,10 @@
   <xacro:macro name="adapter_kms40_fwk050_xacro" params="prefix parent *origin">
     <!-- Joint connecting the parent to our frame_in -->
-    <joint name="${prefix}_adapter_kms40_fwk050_in_joint" type="fixed">
+    <joint name="${prefix}adapter_kms40_fwk050_in_joint" type="fixed">
       <xacro:insert_block name="origin"/>
       <parent link="${parent}"/>
-      <child link="${prefix}_adapter_kms40_fwk050_frame_in"/>
+      <child link="${prefix}adapter_kms40_fwk050_frame_in"/>
     </joint>
-    <link name="${prefix}_adapter_kms40_fwk050_frame_in">
+    <link name="${prefix}adapter_kms40_fwk050_frame_in">
       <visual>
         <origin rpy="0 0 0" xyz="0 0 0"/>
@@ -20,12 +20,12 @@
     </link>
     <!-- Empty link just to get the frame out -->
-    <link name="${prefix}_adapter_kms40_fwk050_frame_out"/>
+    <link name="${prefix}adapter_kms40_fwk050_frame_out"/>
     <!-- joint positioning the frame_out -->
-    <joint name="${prefix}_adapter_kms40_fwk050_trans_frame_out"
+    <joint name="${prefix}adapter_kms40_fwk050_trans_frame_out"
            type="fixed">
       <origin xyz="0 0 0.01"
               rpy="0 0 0" />
-      <parent link="${prefix}_adapter_kms40_fwk050_frame_in" />
-      <child link="${prefix}_adapter_kms40_fwk050_frame_out" />
+      <parent link="${prefix}adapter_kms40_fwk050_frame_in" />
+      <child link="${prefix}adapter_kms40_fwk050_frame_out" />
       <axis xyz="0 0 0" />
     </joint>

File: iai_adapters_description/urdf/fwk_fwa_050.urdf.xacro (robot description, xacro)
@@ -4,10 +4,10 @@
   <xacro:macro name="fwk_fwa_050_xacro" params="prefix parent *origin">
     <!-- Joint connecting the parent to our frame_in -->
-    <joint name="${prefix}_fwk_fwa_050_in_joint" type="fixed">
+    <joint name="${prefix}fwk_fwa_050_in_joint" type="fixed">
       <xacro:insert_block name="origin"/>
       <parent link="${parent}"/>
-      <child link="${prefix}_fwk_fwa_050_frame_in"/>
+      <child link="${prefix}fwk_fwa_050_frame_in"/>
     </joint>
-    <link name="${prefix}_fwk_fwa_050_frame_in">
+    <link name="${prefix}fwk_fwa_050_frame_in">
       <visual>
         <origin rpy="0 0 0" xyz="0 0 0"/>
@@ -20,12 +20,12 @@
     </link>
     <!-- Empty link just to get the frame out -->
-    <link name="${prefix}_fwk_fwa_050_frame_out"/>
+    <link name="${prefix}fwk_fwa_050_frame_out"/>
     <!-- joint positioning the frame_out -->
-    <joint name="${prefix}_fwk_fwa_050_trans_frame_out"
+    <joint name="${prefix}fwk_fwa_050_trans_frame_out"
            type="fixed">
       <origin xyz="0 0 0.0141"
               rpy="0 0 0" />
-      <parent link="${prefix}_fwk_fwa_050_frame_in" />
-      <child link="${prefix}_fwk_fwa_050_frame_out" />
+      <parent link="${prefix}fwk_fwa_050_frame_in" />
+      <child link="${prefix}fwk_fwa_050_frame_out" />
       <axis xyz="0 0 0" />
     </joint>

File: iai_boxy_description/urdf/boxy_description.urdf.xacro (robot description, xacro)
@@ -147,14 +147,14 @@
         </lwr4_cabling_adaptor>
         <!-- The following URDFs have frame_in / frame_out, so they are simply placed at their parent -->
-        <kms_40_xacro parent="left_arm_cabling_adaptor_link" prefix="left_arm">
+        <kms_40_xacro parent="left_arm_cabling_adaptor_link" prefix="left_arm_">
           <origin xyz="0 0 0" rpy="0 0 3.14159265359" />  <!--places the kms40 frame 13mm from the parent -->
         </kms_40_xacro>
-        <adapter_kms40_fwk050_xacro parent="left_arm_kms40_frame_out" prefix="left_arm">
+        <adapter_kms40_fwk050_xacro parent="left_arm_kms40_frame_out" prefix="left_arm_">
           <origin xyz="0 0 0" rpy="0 0 0" />
         </adapter_kms40_fwk050_xacro>
-        <fwk_fwa_050_xacro parent="left_arm_adapter_kms40_fwk050_frame_out" prefix="left_arm">
+        <fwk_fwa_050_xacro parent="left_arm_adapter_kms40_fwk050_frame_out" prefix="left_arm_">
           <origin xyz="0 0 0" rpy="0 0 0" />
         </fwk_fwa_050_xacro>
-        <adapter_fwa050_wsg50_xacro parent="left_arm_fwk_fwa_050_frame_out" prefix="left_arm">
+        <adapter_fwa050_wsg50_xacro parent="left_arm_fwk_fwa_050_frame_out" prefix="left_arm_">
           <origin xyz="0 0 0.0" rpy="0 0 0" />
         </adapter_fwa050_wsg50_xacro>
@@ -272,14 +272,14 @@
         </lwr4_cabling_adaptor>
         <!-- The following URDFs have frame_in / frame_out, so they are simply placed at their parent -->
-        <kms_40_xacro parent="right_arm_cabling_adaptor_link" prefix="right_arm">
+        <kms_40_xacro parent="right_arm_cabling_adaptor_link" prefix="right_arm_">
           <origin xyz="0 0 0" rpy="0 0 3.14159265359" />  <!--places the kms40 frame 13mm from the parent -->
         </kms_40_xacro>
-        <adapter_kms40_fwk050_xacro parent="right_arm_kms40_frame_out" prefix="right_arm">
+        <adapter_kms40_fwk050_xacro parent="right_arm_kms40_frame_out" prefix="right_arm_">
           <origin xyz="0 0 0" rpy="0 0 0" />
         </adapter_kms40_fwk050_xacro>
-        <fwk_fwa_050_xacro parent="right_arm_adapter_kms40_fwk050_frame_out" prefix="right_arm">
+        <fwk_fwa_050_xacro parent="right_arm_adapter_kms40_fwk050_frame_out" prefix="right_arm_">
           <origin xyz="0 0 0" rpy="0 0 0" />
         </fwk_fwa_050_xacro>
-        <adapter_fwa050_wsg50_xacro parent="right_arm_fwk_fwa_050_frame_out" prefix="right_arm">
+        <adapter_fwa050_wsg50_xacro parent="right_arm_fwk_fwa_050_frame_out" prefix="right_arm_">
           <origin xyz="0 0 0.0" rpy="0 0 0" />
         </adapter_fwa050_wsg50_xacro>

File: iai_kms_40_description/urdf/kms_40.urdf.xacro (robot description, xacro)
@@ -4,11 +4,11 @@
   <xacro:macro name="kms_40_xacro" params="prefix parent *origin">
     <!-- Joint connecting the parent to our frame_in -->
-    <joint name="${prefix}_adapter_iso50_kms40_joint" type="fixed">
+    <joint name="${prefix}adapter_iso50_kms40_joint" type="fixed">
       <xacro:insert_block name="origin"/>
       <parent link="${parent}"/>
-      <child link="${prefix}_adapter_iso50_kms40_frame_in"/>
+      <child link="${prefix}adapter_iso50_kms40_frame_in"/>
     </joint>
     <!-- link for the adapter plate -->
-    <link name="${prefix}_adapter_iso50_kms40_frame_in">
+    <link name="${prefix}adapter_iso50_kms40_frame_in">
       <visual>
         <origin rpy="0 0 0" xyz="0 0 0"/>
@@ -20,20 +20,20 @@
     </link>
     <!-- Empty link just to get the frame out -->
-    <link name="${prefix}_adapter_iso50_kms40_frame_out"/>
+    <link name="${prefix}adapter_iso50_kms40_frame_out"/>
     <!-- joint positioning the frame_out -->
-    <joint name="${prefix}_adapter_iso50_kms40_trans_frame_out" type="fixed">
+    <joint name="${prefix}adapter_iso50_kms40_trans_frame_out" type="fixed">
       <origin xyz="0 0 0.016" rpy="0 0 0" />
-      <parent link="${prefix}_adapter_iso50_kms40_frame_in" />
-      <child link="${prefix}_adapter_iso50_kms40_frame_out" />
+      <parent link="${prefix}adapter_iso50_kms40_frame_in" />
+      <child link="${prefix}adapter_iso50_kms40_frame_out" />
       <axis xyz="0 0 0" />
     </joint>
     <!-- Now joint connecting the actual kms40 sensor -->
-    <joint name="${prefix}_kms40_joint" type="fixed">
+    <joint name="${prefix}kms40_joint" type="fixed">
       <origin xyz="0 0 0" rpy="0 0 0" />
-      <parent link="${prefix}_adapter_iso50_kms40_frame_out"/>
-      <child link="${prefix}_kms40_frame_in"/>
+      <parent link="${prefix}adapter_iso50_kms40_frame_out"/>
+      <child link="${prefix}kms40_frame_in"/>
     </joint>
     <!-- Link for the kms40 sensor-->
-    <link name="${prefix}_kms40_frame_in">
+    <link name="${prefix}kms40_frame_in">
       <visual>
         <origin rpy="0 0 0" xyz="0 0 0"/>
@@ -46,10 +46,10 @@
     <!-- Empty link just to get the frame out -->
     <!-- This is also the reference frame for the force/torque data -->
-    <link name="${prefix}_kms40_frame_out"/>
+    <link name="${prefix}kms40_frame_out"/>
     <!-- joint positioning the frame_out -->
-    <joint name="${prefix}_kms40_trans_frame_out" type="fixed">
+    <joint name="${prefix}kms40_trans_frame_out" type="fixed">
       <origin xyz="0 0 0.027" rpy="0 0 0" />
-      <parent link="${prefix}_kms40_frame_in" />
-      <child link="${prefix}_kms40_frame_out" />
+      <parent link="${prefix}kms40_frame_in" />
+      <child link="${prefix}kms40_frame_out" />
       <axis xyz="0 0 0" />
     </joint>
