Commit message: [boxy urdf] added collision tags for the adapters and kms40:
it's freaky how in the collision mesh of Boxy the grippers are just floating in the air...
Basically, just copy pasted the visual tags for collision.
The other changes are only minor stuff like fixing indentation / removing trailing whitespace / breaking too long lines.

File: iai_adapters_description/urdf/adapter_fwa050_wsg50.urdf.xacro (robot description, xacro)
@@ -14,8 +14,18 @@
         <geometry>
           <!-- these meshes were exported in mm, so scale back to m -->
-          <mesh filename="package://iai_adapters_description/meshes/adapter_fwa050_wsg50.stl" scale="0.001 0.001 0.001"/>
+          <mesh filename="package://iai_adapters_description/meshes/adapter_fwa050_wsg50.stl"
+                scale="0.001 0.001 0.001"/>
         </geometry>
         <material name="Grey"/>
       </visual>
+      <collision>
+        <origin rpy="0 0 0" xyz="0 0 0"/>
+        <geometry>
+          <!-- these meshes were exported in mm, so scale back to m -->
+          <mesh filename="package://iai_adapters_description/meshes/adapter_fwa050_wsg50.stl"
+                scale="0.001 0.001 0.001"/>
+        </geometry>
+        <material name="Grey"/>
+      </collision>
     </link>
     <!-- Empty link just to get the frame out -->
@@ -24,6 +34,5 @@
     <joint name="${prefix}adapter_fwa050_wsg50_trans_frame_out"
            type="fixed">
-      <origin xyz="0 0 0.01"
-              rpy="0 0 0" />
+      <origin xyz="0 0 0.01" rpy="0 0 0" />
       <parent link="${prefix}adapter_fwa050_wsg50_frame_in" />
       <child link="${prefix}adapter_fwa050_wsg50_frame_out" />

File: iai_adapters_description/urdf/adapter_kms40_fwk050.urdf.xacro (robot description, xacro)
@@ -14,8 +14,18 @@
         <geometry>
           <!-- these meshes were exported in mm, so scale back to m -->
-          <mesh filename="package://iai_adapters_description/meshes/adapter_kms40_fwk050.stl" scale="0.001 0.001 0.001"/>
+          <mesh filename="package://iai_adapters_description/meshes/adapter_kms40_fwk050.stl"
+                scale="0.001 0.001 0.001"/>
         </geometry>
         <material name="Grey"/>
       </visual>
+      <collision>
+        <origin rpy="0 0 0" xyz="0 0 0"/>
+        <geometry>
+          <!-- these meshes were exported in mm, so scale back to m -->
+          <mesh filename="package://iai_adapters_description/meshes/adapter_kms40_fwk050.stl"
+                scale="0.001 0.001 0.001"/>
+        </geometry>
+        <material name="Grey"/>
+      </collision>
     </link>
     <!-- Empty link just to get the frame out -->
@@ -24,6 +34,5 @@
     <joint name="${prefix}adapter_kms40_fwk050_trans_frame_out"
            type="fixed">
-      <origin xyz="0 0 0.01"
-              rpy="0 0 0" />
+      <origin xyz="0 0 0.01" rpy="0 0 0" />
       <parent link="${prefix}adapter_kms40_fwk050_frame_in" />
       <child link="${prefix}adapter_kms40_fwk050_frame_out" />

File: iai_adapters_description/urdf/fwk_fwa_050.urdf.xacro (robot description, xacro)
@@ -14,8 +14,18 @@
         <geometry>
           <!-- these meshes were exported in mm, so scale back to m -->
-          <mesh filename="package://iai_adapters_description/meshes/fwk_fwa_050_simple.stl" scale="0.001 0.001 0.001"/>
+          <mesh filename="package://iai_adapters_description/meshes/fwk_fwa_050_simple.stl"
+                scale="0.001 0.001 0.001"/>
         </geometry>
         <material name="Grey"/>
       </visual>
+      <collision>
+        <origin rpy="0 0 0" xyz="0 0 0"/>
+        <geometry>
+          <!-- these meshes were exported in mm, so scale back to m -->
+          <mesh filename="package://iai_adapters_description/meshes/fwk_fwa_050_simple.stl"
+                scale="0.001 0.001 0.001"/>
+        </geometry>
+        <material name="Grey"/>
+      </collision>
     </link>
     <!-- Empty link just to get the frame out -->
@@ -24,6 +34,5 @@
     <joint name="${prefix}fwk_fwa_050_trans_frame_out"
            type="fixed">
-      <origin xyz="0 0 0.0141"
-              rpy="0 0 0" />
+      <origin xyz="0 0 0.0141" rpy="0 0 0" />
       <parent link="${prefix}fwk_fwa_050_frame_in" />
       <child link="${prefix}fwk_fwa_050_frame_out" />

File: iai_adapters_description/urdf/lwr4_cabling_adaptor.urdf.xacro (robot description, xacro)
@@ -6,5 +6,6 @@
     <joint name="${prefix}arm_cabling_adaptor_joint" type="fixed">
       <xacro:insert_block name="origin" />
-      <!--origin xyz="0 0 0.01" rpy="0 0 0"/-->  <!-- This places the link at the end of the plate (frame_out) -->
+      <!-- This places the link at the end of the plate (frame_out) -->
+      <!--origin xyz="0 0 0.01" rpy="0 0 0"/-->
       <parent link="${parent}"/>
       <child link="${prefix}cabling_adaptor_link"/>
@@ -12,5 +13,6 @@
     <link name="${prefix}cabling_adaptor_link">
       <visual>
-        <origin xyz="0 0 -0.005" rpy="0 0 0" />  <!-- The cylinder is placed at the center -->
+        <!-- The cylinder is placed at the center -->
+        <origin xyz="0 0 -0.005" rpy="0 0 0" />
         <geometry>
           <cylinder length="0.01" radius="0.0315"/>
@@ -20,4 +22,14 @@
         </material>
       </visual>
+      <collision>
+        <!-- The cylinder is placed at the center -->
+        <origin xyz="0 0 -0.005" rpy="0 0 0" />
+        <geometry>
+          <cylinder length="0.01" radius="0.0315"/>
+        </geometry>
+        <material name="Black">
+          <color rgba="0 0 0 1.0"/>
+        </material>
+      </collision>
     </link>
   </xacro:macro>

File: iai_kms_40_description/urdf/kms_40.urdf.xacro (robot description, xacro)
@@ -14,8 +14,17 @@
         <origin rpy="0 0 0" xyz="0 0 0"/>
         <geometry>
-          <mesh filename="package://iai_kms_40_description/meshes/adapter_plate_iso50_kms40_weiss.stl" scale="0.001 0.001 0.001"/>
+          <mesh filename="package://iai_kms_40_description/meshes/adapter_plate_iso50_kms40_weiss.stl"
+                scale="0.001 0.001 0.001"/>
         </geometry>
         <material name="Grey"/>
       </visual>
+      <collision>
+        <origin rpy="0 0 0" xyz="0 0 0"/>
+        <geometry>
+          <mesh filename="package://iai_kms_40_description/meshes/adapter_plate_iso50_kms40_weiss.stl"
+                scale="0.001 0.001 0.001"/>
+        </geometry>
+        <material name="Grey"/>
+      </collision>
     </link>
     <!-- Empty link just to get the frame out -->
@@ -39,8 +48,17 @@
         <origin rpy="0 0 0" xyz="0 0 0"/>
         <geometry>
-          <mesh filename="package://iai_kms_40_description/meshes/kms40_simple.stl" scale="0.001 0.001 0.001"/>
+          <mesh filename="package://iai_kms_40_description/meshes/kms40_simple.stl"
+                scale="0.001 0.001 0.001"/>
         </geometry>
         <material name="Grey"/>
       </visual>
+      <collision>
+        <origin rpy="0 0 0" xyz="0 0 0"/>
+        <geometry>
+          <mesh filename="package://iai_kms_40_description/meshes/kms40_simple.stl"
+                scale="0.001 0.001 0.001"/>
+        </geometry>
+        <material name="Grey"/>
+      </collision>
     </link>
     <!-- Empty link just to get the frame out -->
