Commit message: fixed kinnect position for openease...

File: iai_boxy_description/sensors/kinect.urdf.xacro (robot description, xacro)
@@ -12,7 +12,9 @@
                     on February 11th, 2015. They are not set in stone! If the calibration
                     changes you might have to touch them again. Sorry! -->
+	 <!--
         <origin xyz="-0.05 -0.17 -0.02" rpy="${M_PI/2.0} 0 ${M_PI/2.0}"/>
+	 -->
         <geometry>
-          <mesh filename="package://iai_boxy_description/meshes/sensors/68-04546_Kinect_Sensor--coarse.STL"  />
+          <mesh filename="package://iai_boxy_description/meshes/sensors/68-04546_Kinect_Sensor-coarse.dae"  />
         </geometry>
         <material name="gray">
