Commit message: fixed joint limits on the head (incl. velocity)

File: iai_schunk_pw070_v6/robots/pw070_v6.URDF (robot description, URDF)
Before this commit: robot pw070_v6, 4 links, 3 joints
Joints:
- joint head_pan_joint: limit lower=-6.28 upper=6.28 effort=0 velocity=0 -> lower=-1.57 upper=1.57 effort=0 velocity=0.75
- joint head_tilt_joint: limit lower=-3.14159 upper=3.14159 effort=0 velocity=0 -> lower=-1.3 upper=1.3 effort=0 velocity=0.8

Commit message: /pw070 -> Increase limits

File: iai_schunk_pw070_v6/robots/pw070_v6.URDF (robot description, URDF)
Before this commit: robot pw070_v6, 4 links, 3 joints
Joints:
- joint head_tilt_joint: limit lower=-1.3 upper=1.3 effort=0 velocity=0.8 -> lower=-1.6 upper=1.6 effort=0 velocity=0.8
