Commit message: Adding simplified (decimated) STL files for all the robot parts. Adding the decimated STL files to the collision description in all the URDF files.

File: iai_boxy_base/robots/base.URDF (robot description, URDF)
Before this commit: robot base, 3 links, 2 joints
Links:
- link base_link: geometry collision mesh filename=package://iai_boxy_base/meshes/base_link_simple.STL; visual mesh filename=package://iai_boxy_base/meshes/base_link.STL

File: iai_boxy_torso/robots/torso.URDF (robot description, URDF)
Before this commit: robot torso, 4 links, 3 joints
Links:
- link torso_base_link: geometry collision mesh filename=package://iai_boxy_torso/meshes/torso_base_link_simple.STL; visual mesh filename=package://iai_boxy_torso/meshes/torso_base_link.STL

File: iai_schunk_pw070_v6/robots/pw070_v6.URDF (robot description, URDF)
Before this commit: robot pw070_v6, 4 links, 3 joints
Links:
- link pw070_base_link: geometry collision mesh filename=package://iai_schunk_pw070_v6//meshes/pw070_base_link_simpl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; visual mesh filename=package://iai_schunk_pw070_v6//meshes/pw070_base_link.STL
- link pw070_box: geometry collision mesh filename=package://iai_schunk_pw070_v6//meshes/pw070_box_simple.STL; visual mesh filename=package://iai_schunk_pw070_v6//meshes/pw070_box.STL
- link pw070_plate: geometry collision mesh filename=package://iai_schunk_pw070_v6//meshes/pw070_plate_simple.STL; visual mesh filename=package://iai_schunk_pw070_v6//meshes/pw070_plate.STL

File: iai_weiss_wsg50/robots/weiss_wsg50.urdf (robot description, URDF)
Before this commit: robot weiss_wsg50, 1 links, 0 joints
Links:
- link gripper_base_link: geometry collision mesh filename=package://iai_weiss_wsg50/meshes/gripper_base_link_simple.S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; visual mesh filename=package://iai_weiss_wsg50/meshes/gripper_base_link.STL

Commit message: iai_boxy_base: improved mesh of the base
Moved the lasers to their real position.
Fixed the laser axes.
Added the bars for the head mounting.
Added the plate on top of the bars.
The black adapter plate (6mm) is still missing below the PTU.

Now you can clearly see that the head is not placed correctly in the URDF.
This will need fixing, but I have to be careful because it affects
the hand/eye calibration.

File: iai_boxy_base/robots/base.URDF (robot description, URDF)
Before this commit: robot base, 3 links, 2 joints
Links:
- link base_link: mass 70.4306942428661 -> 70.0210745907357
Joints:
- joint laser_reference_back_joint: axis 0 0 0 -> -1 0 0; origin xyz=-0.738426406871194 0.0504883651003683 0.157499999999995 rpy=-4.33428293429891E-15 4.09876906549633E-15 2.35619449019234 -> xyz=-0.69357 -0.506 0.1575 rpy=4.9333E-15 4.5082E-15 -2.3562
- joint laser_reference_front_joint: axis 0 0 0 -> -0.99849 0 -0.054862; origin xyz=0.235926406871192 -0.497427516941588 0.157500000000002 rpy=4.70027852409606E-15 -4.70862925338426E-15 -0.78539816339745 -> xyz=0.19107 0.0506 0.1575 rpy=-4.1881E-15 -4.2124E-15 0.7854

Commit message: reexported some malformed STLs + using DAE for base now

File: iai_boxy_base/robots/base.URDF (robot description, URDF)
Before this commit: robot base, 3 links, 2 joints
Links:
- link base_link: geometry collision mesh filename=package://iai_boxy_base/meshes/base_link_simple.STL; visual mesh filename=package://iai_boxy_base/meshes/base_link.dae
