Commit message: Changed transmission to old format

File: iai_ur_description/urdf/ur.transmission.xacro (robot description, xacro)
@@ -2,57 +2,45 @@
 <robot xmlns:xacro="http://www.ros.org/wiki/xacro">
   <xacro:macro name="ur_arm_transmission" params="prefix">
-    <transmission name="${prefix}shoulder_pan_trans">
-      <type>transmission_interface/SimpleTransmission</type>
-      <joint name="${prefix}shoulder_pan_joint">
-        <hardwareInterface>PositionJointInterface</hardwareInterface>
-      </joint>
-      <actuator name="${prefix}shoulder_pan_motor">
-        <mechanicalReduction>1</mechanicalReduction>
-      </actuator>
+    <transmission
+      name="${prefix}shoulder_pan_trans"
+      type="pr2_mechanism_model/SimpleTransmission">
+      <actuator name="${prefix}shoulder_pan_motor"/>
+      <joint name="${prefix}shoulder_pan_joint"/>
+      <mechanicalReduction>1.0</mechanicalReduction>
     </transmission>
-    <transmission name="${prefix}shoulder_lift_trans">
-      <type>transmission_interface/SimpleTransmission</type>
-      <joint name="${prefix}shoulder_lift_joint">
-        <hardwareInterface>PositionJointInterface</hardwareInterface>
-      </joint>
-      <actuator name="${prefix}shoulder_lift_motor">
-        <mechanicalReduction>1</mechanicalReduction>
-      </actuator>
+    <transmission
+      name="${prefix}shoulder_lift_trans"
+      type="pr2_mechanism_model/SimpleTransmission">
+      <actuator name="${prefix}shoulder_lift_motor"/>
+      <joint name="${prefix}shoulder_lift_joint"/>
+      <mechanicalReduction>1.0</mechanicalReduction>
     </transmission>
-    <transmission name="${prefix}elbow_trans">
-      <type>transmission_interface/SimpleTransmission</type>
-      <joint name="${prefix}elbow_joint">
-        <hardwareInterface>PositionJointInterface</hardwareInterface>
-      </joint>
-      <actuator name="${prefix}elbow_motor">
-        <mechanicalReduction>1</mechanicalReduction>
-      </actuator>
+    <transmission
+      name="${prefix}elbow_trans"
+      type="pr2_mechanism_model/SimpleTransmission">
+      <actuator name="${prefix}elbow_motor"/>
+      <joint name="${prefix}elbow_joint"/>
+      <mechanicalReduction>1.0</mechanicalReduction>
     </transmission>
-    <transmission name="${prefix}wrist_1_trans">
-      <type>transmission_interface/SimpleTransmission</type>
-      <joint name="${prefix}wrist_1_joint">
-        <hardwareInterface>PositionJointInterface</hardwareInterface>
-      </joint>
-      <actuator name="${prefix}wrist_1_motor">
-        <mechanicalReduction>1</mechanicalReduction>
-      </actuator>
+    <transmission
+      name="${prefix}wrist_1_trans"
+      type="pr2_mechanism_model/SimpleTransmission">
+      <actuator name="${prefix}wrist_1_motor"/>
+      <joint name="${prefix}wrist_1_joint"/>
+      <mechanicalReduction>1.0</mechanicalReduction>
     </transmission>
-    <transmission name="${prefix}wrist_2_trans">
-      <type>transmission_interface/SimpleTransmission</type>
-      <joint name="${prefix}wrist_2_joint">
-        <hardwareInterface>PositionJointInterface</hardwareInterface>
-      </joint>
-      <actuator name="${prefix}wrist_2_motor">
-        <mechanicalReduction>1</mechanicalReduction>
-      </actuator>
+    <transmission
+      name="${prefix}wrist_2_trans"
+      type="pr2_mechanism_model/SimpleTransmission">
+      <actuator name="${prefix}wrist_2_motor"/>
+      <joint name="${prefix}wrist_2_joint"/>
+      <mechanicalReduction>1.0</mechanicalReduction>
     </transmission>
-    <transmission name="${prefix}wrist_3_trans">
-      <type>transmission_interface/SimpleTransmission</type>
-      <joint name="${prefix}wrist_3_joint">
-        <hardwareInterface>PositionJointInterface</hardwareInterface>
-      </joint>
-      <actuator name="${prefix}wrist_3_motor">
-        <mechanicalReduction>1</mechanicalReduction>
-      </actuator>
+    <transmission
+      name="${prefix}wrist_3_trans"
+      type="pr2_mechanism_model/SimpleTransmission">
+      <actuator name="${prefix}wrist_3_motor"/>
+      <joint name="${prefix}wrist_3_joint"/>
+      <mechanicalReduction>1.0</mechanicalReduction>
     </transmission>
   </xacro:macro>
