Commit message: Added a mounting joint to ur3-macro.

File: iai_ur_description/urdf/ur3.urdf.xacro (robot description, xacro)
@@ -52,5 +52,10 @@
     </inertial>
   </xacro:macro>
-  <xacro:macro name="ur3_robot" params="prefix joint_limited">
+  <xacro:macro name="ur3_robot" params="prefix parent joint_limited *origin">
+    <joint name="${prefix}mounting_joint" type="fixed">
+      <parent link="${parent}" />
+      <child link="${prefix}base_link" />
+      <insert_block name="origin"/>
+    </joint>
     <link name="${prefix}base_link" >
       <visual>

Commit message: Modify UR3 limited URDF

File: iai_ur_description/urdf/ur3.urdf.xacro (robot description, xacro)
@@ -242,4 +242,5 @@
       <xacro:if value="${joint_limited}">
         <limit lower="${-pi}" upper="${pi}" effort="54.0" velocity="3.2"/>
+				<limit lower="${-1.5*pi}" upper="${1.5*pi}" effort="54.0" velocity="3.2"/>
       </xacro:if>
       <dynamics damping="0.0" friction="0.0"/>

Commit message: Changing UR3 last joint limits

File: iai_ur_description/urdf/ur3.urdf.xacro (robot description, xacro)
@@ -241,5 +241,5 @@
       </xacro:unless>
       <xacro:if value="${joint_limited}">
-				<limit lower="${-1.5 * pi}" upper="${1.5 * pi}" effort="54.0" velocity="3.2"/>
+				<limit lower="${-1 * pi}" upper="${1 * pi}" effort="54.0" velocity="3.2"/>
       </xacro:if>
       <dynamics damping="0.0" friction="0.0"/>
