Commit message: Renamed package ur_description into iai_ur_description.

File: iai_ur_description/urdf/ur10.urdf.xacro (robot description, xacro)
@@ -5,6 +5,6 @@
   Contributers: Jimmy Da Silva, Ajit Krisshna N L, Muhammad Asif Rana
 -->
-  <xacro:include filename="$(find ur_description)/urdf/ur.transmission.xacro" />
-  <xacro:include filename="$(find ur_description)/urdf/ur.gazebo.xacro" />
+  <xacro:include filename="$(find iai_ur_description)/urdf/ur.transmission.xacro" />
+  <xacro:include filename="$(find iai_ur_description)/urdf/ur.gazebo.xacro" />
   <property name="pi" value="3.14159265" />
   <!-- Inertia parameters -->
@@ -57,13 +57,13 @@
       <visual>
         <geometry>
-          <mesh filename="package://ur_description/meshes/ur10/visual/base.dae"/>
-        </geometry>
-        <material name="LightGrey">
-          <color rgba="0.7 0.7 0.7 1.0"/>
-        </material>
-      </visual>
-      <collision>
-        <geometry>
-          <mesh filename="package://ur_description/meshes/ur10/collision/base.stl"/>
+          <mesh filename="package://iai_ur_description/meshes/ur10/visual/base.dae"/>
+        </geometry>
+        <material name="LightGrey">
+          <color rgba="0.7 0.7 0.7 1.0"/>
+        </material>
+      </visual>
+      <collision>
+        <geometry>
+          <mesh filename="package://iai_ur_description/meshes/ur10/collision/base.stl"/>
         </geometry>
       </collision>
@@ -88,13 +88,13 @@
       <visual>
         <geometry>
-          <mesh filename="package://ur_description/meshes/ur10/visual/shoulder.dae"/>
-        </geometry>
-        <material name="LightGrey">
-          <color rgba="0.7 0.7 0.7 1.0"/>
-        </material>
-      </visual>
-      <collision>
-        <geometry>
-          <mesh filename="package://ur_description/meshes/ur10/collision/shoulder.stl"/>
+          <mesh filename="package://iai_ur_description/meshes/ur10/visual/shoulder.dae"/>
+        </geometry>
+        <material name="LightGrey">
+          <color rgba="0.7 0.7 0.7 1.0"/>
+        </material>
+      </visual>
+      <collision>
+        <geometry>
+          <mesh filename="package://iai_ur_description/meshes/ur10/collision/shoulder.stl"/>
         </geometry>
       </collision>
@@ -119,13 +119,13 @@
       <visual>
         <geometry>
-          <mesh filename="package://ur_description/meshes/ur10/visual/upperarm.dae"/>
-        </geometry>
-        <material name="LightGrey">
-          <color rgba="0.7 0.7 0.7 1.0"/>
-        </material>
-      </visual>
-      <collision>
-        <geometry>
-          <mesh filename="package://ur_description/meshes/ur10/collision/upperarm.stl"/>
+          <mesh filename="package://iai_ur_description/meshes/ur10/visual/upperarm.dae"/>
+        </geometry>
+        <material name="LightGrey">
+          <color rgba="0.7 0.7 0.7 1.0"/>
+        </material>
+      </visual>
+      <collision>
+        <geometry>
+          <mesh filename="package://iai_ur_description/meshes/ur10/collision/upperarm.stl"/>
         </geometry>
       </collision>
@@ -150,13 +150,13 @@
       <visual>
          <geometry>
-          <mesh filename="package://ur_description/meshes/ur10/visual/forearm.dae"/>
-        </geometry>
-        <material name="LightGrey">
-          <color rgba="0.7 0.7 0.7 1.0"/>
-        </material>
-      </visual>
-      <collision>
-        <geometry>
-          <mesh filename="package://ur_description/meshes/ur10/collision/forearm.stl"/>
+          <mesh filename="package://iai_ur_description/meshes/ur10/visual/forearm.dae"/>
+        </geometry>
+        <material name="LightGrey">
+          <color rgba="0.7 0.7 0.7 1.0"/>
+        </material>
+      </visual>
+      <collision>
+        <geometry>
+          <mesh filename="package://iai_ur_description/meshes/ur10/collision/forearm.stl"/>
         </geometry>
       </collision>
@@ -181,13 +181,13 @@
       <visual>
         <geometry>
-          <mesh filename="package://ur_description/meshes/ur10/visual/wrist1.dae"/>
-        </geometry>
-        <material name="LightGrey">
-          <color rgba="0.7 0.7 0.7 1.0"/>
-        </material>
-      </visual>
-      <collision>
-        <geometry>
-          <mesh filename="package://ur_description/meshes/ur10/collision/wrist1.stl"/>
+          <mesh filename="package://iai_ur_description/meshes/ur10/visual/wrist1.dae"/>
+        </geometry>
+        <material name="LightGrey">
+          <color rgba="0.7 0.7 0.7 1.0"/>
+        </material>
+      </visual>
+      <collision>
+        <geometry>
+          <mesh filename="package://iai_ur_description/meshes/ur10/collision/wrist1.stl"/>
         </geometry>
       </collision>
@@ -212,13 +212,13 @@
       <visual>
         <geometry>
-          <mesh filename="package://ur_description/meshes/ur10/visual/wrist2.dae"/>
-        </geometry>
-        <material name="LightGrey">
-          <color rgba="0.7 0.7 0.7 1.0"/>
-        </material>
-      </visual>
-      <collision>
-        <geometry>
-          <mesh filename="package://ur_description/meshes/ur10/collision/wrist2.stl"/>
+          <mesh filename="package://iai_ur_description/meshes/ur10/visual/wrist2.dae"/>
+        </geometry>
+        <material name="LightGrey">
+          <color rgba="0.7 0.7 0.7 1.0"/>
+        </material>
+      </visual>
+      <collision>
+        <geometry>
+          <mesh filename="package://iai_ur_description/meshes/ur10/collision/wrist2.stl"/>
         </geometry>
       </collision>
@@ -243,13 +243,13 @@
       <visual>
         <geometry>
-          <mesh filename="package://ur_description/meshes/ur10/visual/wrist3.dae"/>
-        </geometry>
-        <material name="LightGrey">
-          <color rgba="0.7 0.7 0.7 1.0"/>
-        </material>
-      </visual>
-      <collision>
-        <geometry>
-          <mesh filename="package://ur_description/meshes/ur10/collision/wrist3.stl"/>
+          <mesh filename="package://iai_ur_description/meshes/ur10/visual/wrist3.dae"/>
+        </geometry>
+        <material name="LightGrey">
+          <color rgba="0.7 0.7 0.7 1.0"/>
+        </material>
+      </visual>
+      <collision>
+        <geometry>
+          <mesh filename="package://iai_ur_description/meshes/ur10/collision/wrist3.stl"/>
         </geometry>
       </collision>

File: iai_ur_description/urdf/ur10_joint_limited_robot.urdf.xacro (robot description, xacro)
@@ -1,11 +1,11 @@
 <?xml version="1.0"?>
 <robot xmlns:xacro="http://www.ros.org/wiki/xacro"
-       name="ur3" >
+       name="ur10" >
   <!-- common stuff -->
-  <xacro:include filename="$(find ur_description)/urdf/common.gazebo.xacro" />
-  <!-- ur3 -->
-  <xacro:include filename="$(find ur_description)/urdf/ur3.urdf.xacro" />
+  <xacro:include filename="$(find iai_ur_description)/urdf/common.gazebo.xacro" />
+  <!-- ur10 -->
+  <xacro:include filename="$(find iai_ur_description)/urdf/ur10.urdf.xacro" />
   <!-- arm -->
-  <xacro:ur3_robot prefix="" joint_limited="false"/>
+  <xacro:ur10_robot prefix="" joint_limited="true"/>
   <link name="world" />
   <joint name="world_joint" type="fixed">

File: iai_ur_description/urdf/ur10_robot.urdf.xacro (robot description, xacro)
@@ -1,11 +1,11 @@
 <?xml version="1.0"?>
 <robot xmlns:xacro="http://www.ros.org/wiki/xacro"
-       name="ur5" >
+       name="ur10" >
   <!-- common stuff -->
-  <xacro:include filename="$(find ur_description)/urdf/common.gazebo.xacro" />
-  <!-- ur5 -->
-  <xacro:include filename="$(find ur_description)/urdf/ur5.urdf.xacro" />
+  <xacro:include filename="$(find iai_ur_description)/urdf/common.gazebo.xacro" />
+  <!-- ur10 -->
+  <xacro:include filename="$(find iai_ur_description)/urdf/ur10.urdf.xacro" />
   <!-- arm -->
-  <xacro:ur5_robot prefix="" joint_limited="false"/>
+  <xacro:ur10_robot prefix="" joint_limited="false"/>
   <link name="world" />
   <joint name="world_joint" type="fixed">

File: iai_ur_description/urdf/ur3.urdf.xacro (robot description, xacro)
@@ -4,6 +4,6 @@
   Author: Felix Messmer
 -->
-  <xacro:include filename="$(find ur_description)/urdf/ur.transmission.xacro" />
-  <xacro:include filename="$(find ur_description)/urdf/ur.gazebo.xacro" />
+  <xacro:include filename="$(find iai_ur_description)/urdf/ur.transmission.xacro" />
+  <xacro:include filename="$(find iai_ur_description)/urdf/ur.gazebo.xacro" />
   <property name="pi" value="3.14159265" />
   <!-- Inertia parameters -->
@@ -56,13 +56,13 @@
       <visual>
         <geometry>
-          <mesh filename="package://ur_description/meshes/ur3/visual/base.dae"/>
-        </geometry>
-        <material name="LightGrey">
-          <color rgba="0.7 0.7 0.7 1.0"/>
-        </material>
-      </visual>
-      <collision>
-        <geometry>
-          <mesh filename="package://ur_description/meshes/ur3/collision/base.stl"/>
+          <mesh filename="package://iai_ur_description/meshes/ur3/visual/base.dae"/>
+        </geometry>
+        <material name="LightGrey">
+          <color rgba="0.7 0.7 0.7 1.0"/>
+        </material>
+      </visual>
+      <collision>
+        <geometry>
+          <mesh filename="package://iai_ur_description/meshes/ur3/collision/base.stl"/>
         </geometry>
       </collision>
@@ -87,13 +87,13 @@
       <visual>
         <geometry>
-          <mesh filename="package://ur_description/meshes/ur3/visual/shoulder.dae"/>
-        </geometry>
-        <material name="LightGrey">
-          <color rgba="0.7 0.7 0.7 1.0"/>
-        </material>
-      </visual>
-      <collision>
-        <geometry>
-          <mesh filename="package://ur_description/meshes/ur3/collision/shoulder.stl"/>
+          <mesh filename="package://iai_ur_description/meshes/ur3/visual/shoulder.dae"/>
+        </geometry>
+        <material name="LightGrey">
+          <color rgba="0.7 0.7 0.7 1.0"/>
+        </material>
+      </visual>
+      <collision>
+        <geometry>
+          <mesh filename="package://iai_ur_description/meshes/ur3/collision/shoulder.stl"/>
         </geometry>
       </collision>
@@ -118,13 +118,13 @@
       <visual>
         <geometry>
-          <mesh filename="package://ur_description/meshes/ur3/visual/upperarm.dae"/>
-        </geometry>
-        <material name="LightGrey">
-          <color rgba="0.7 0.7 0.7 1.0"/>
-        </material>
-      </visual>
-      <collision>
-        <geometry>
-          <mesh filename="package://ur_description/meshes/ur3/collision/upperarm.stl"/>
+          <mesh filename="package://iai_ur_description/meshes/ur3/visual/upperarm.dae"/>
+        </geometry>
+        <material name="LightGrey">
+          <color rgba="0.7 0.7 0.7 1.0"/>
+        </material>
+      </visual>
+      <collision>
+        <geometry>
+          <mesh filename="package://iai_ur_description/meshes/ur3/collision/upperarm.stl"/>
         </geometry>
       </collision>
@@ -149,13 +149,13 @@
       <visual>
          <geometry>
-          <mesh filename="package://ur_description/meshes/ur3/visual/forearm.dae"/>
-        </geometry>
-        <material name="LightGrey">
-          <color rgba="0.7 0.7 0.7 1.0"/>
-        </material>
-      </visual>
-      <collision>
-        <geometry>
-          <mesh filename="package://ur_description/meshes/ur3/collision/forearm.stl"/>
+          <mesh filename="package://iai_ur_description/meshes/ur3/visual/forearm.dae"/>
+        </geometry>
+        <material name="LightGrey">
+          <color rgba="0.7 0.7 0.7 1.0"/>
+        </material>
+      </visual>
+      <collision>
+        <geometry>
+          <mesh filename="package://iai_ur_description/meshes/ur3/collision/forearm.stl"/>
         </geometry>
       </collision>
@@ -180,13 +180,13 @@
       <visual>
         <geometry>
-          <mesh filename="package://ur_description/meshes/ur3/visual/wrist1.dae"/>
-        </geometry>
-        <material name="LightGrey">
-          <color rgba="0.7 0.7 0.7 1.0"/>
-        </material>
-      </visual>
-      <collision>
-        <geometry>
-          <mesh filename="package://ur_description/meshes/ur3/collision/wrist1.stl"/>
+          <mesh filename="package://iai_ur_description/meshes/ur3/visual/wrist1.dae"/>
+        </geometry>
+        <material name="LightGrey">
+          <color rgba="0.7 0.7 0.7 1.0"/>
+        </material>
+      </visual>
+      <collision>
+        <geometry>
+          <mesh filename="package://iai_ur_description/meshes/ur3/collision/wrist1.stl"/>
         </geometry>
       </collision>
@@ -211,13 +211,13 @@
       <visual>
         <geometry>
-          <mesh filename="package://ur_description/meshes/ur3/visual/wrist2.dae"/>
-        </geometry>
-        <material name="LightGrey">
-          <color rgba="0.7 0.7 0.7 1.0"/>
-        </material>
-      </visual>
-      <collision>
-        <geometry>
-          <mesh filename="package://ur_description/meshes/ur3/collision/wrist2.stl"/>
+          <mesh filename="package://iai_ur_description/meshes/ur3/visual/wrist2.dae"/>
+        </geometry>
+        <material name="LightGrey">
+          <color rgba="0.7 0.7 0.7 1.0"/>
+        </material>
+      </visual>
+      <collision>
+        <geometry>
+          <mesh filename="package://iai_ur_description/meshes/ur3/collision/wrist2.stl"/>
         </geometry>
       </collision>
@@ -242,13 +242,13 @@
       <visual>
         <geometry>
-          <mesh filename="package://ur_description/meshes/ur3/visual/wrist3.dae"/>
-        </geometry>
-        <material name="LightGrey">
-          <color rgba="0.7 0.7 0.7 1.0"/>
-        </material>
-      </visual>
-      <collision>
-        <geometry>
-          <mesh filename="package://ur_description/meshes/ur3/collision/wrist3.stl"/>
+          <mesh filename="package://iai_ur_description/meshes/ur3/visual/wrist3.dae"/>
+        </geometry>
+        <material name="LightGrey">
+          <color rgba="0.7 0.7 0.7 1.0"/>
+        </material>
+      </visual>
+      <collision>
+        <geometry>
+          <mesh filename="package://iai_ur_description/meshes/ur3/collision/wrist3.stl"/>
         </geometry>
       </collision>

File: iai_ur_description/urdf/ur3_joint_limited_robot.urdf.xacro (robot description, xacro)
@@ -1,11 +1,11 @@
 <?xml version="1.0"?>
 <robot xmlns:xacro="http://www.ros.org/wiki/xacro"
-       name="ur10" >
+       name="ur3" >
   <!-- common stuff -->
-  <xacro:include filename="$(find ur_description)/urdf/common.gazebo.xacro" />
-  <!-- ur10 -->
-  <xacro:include filename="$(find ur_description)/urdf/ur10.urdf.xacro" />
+  <xacro:include filename="$(find iai_ur_description)/urdf/common.gazebo.xacro" />
+  <!-- ur3 -->
+  <xacro:include filename="$(find iai_ur_description)/urdf/ur3.urdf.xacro" />
   <!-- arm -->
-  <xacro:ur10_robot prefix="" joint_limited="false"/>
+  <xacro:ur3_robot prefix="" joint_limited="true"/>
   <link name="world" />
   <joint name="world_joint" type="fixed">

File: iai_ur_description/urdf/ur3_robot.urdf.xacro (robot description, xacro)
@@ -1,11 +1,11 @@
 <?xml version="1.0"?>
 <robot xmlns:xacro="http://www.ros.org/wiki/xacro"
-       name="ur10" >
+       name="ur3" >
   <!-- common stuff -->
-  <xacro:include filename="$(find ur_description)/urdf/common.gazebo.xacro" />
-  <!-- ur10 -->
-  <xacro:include filename="$(find ur_description)/urdf/ur10.urdf.xacro" />
+  <xacro:include filename="$(find iai_ur_description)/urdf/common.gazebo.xacro" />
+  <!-- ur3 -->
+  <xacro:include filename="$(find iai_ur_description)/urdf/ur3.urdf.xacro" />
   <!-- arm -->
-  <xacro:ur10_robot prefix="" joint_limited="true"/>
+  <xacro:ur3_robot prefix="" joint_limited="false"/>
   <link name="world" />
   <joint name="world_joint" type="fixed">

File: iai_ur_description/urdf/ur5.urdf.xacro (robot description, xacro)
@@ -1,6 +1,6 @@
 <?xml version="1.0"?>
 <robot xmlns:xacro="http://www.ros.org/wiki/xacro">
-  <xacro:include filename="$(find ur_description)/urdf/ur.transmission.xacro" />
-  <xacro:include filename="$(find ur_description)/urdf/ur.gazebo.xacro" />
+  <xacro:include filename="$(find iai_ur_description)/urdf/ur.transmission.xacro" />
+  <xacro:include filename="$(find iai_ur_description)/urdf/ur.gazebo.xacro" />
   <property name="pi" value="3.14159265" />
   <!-- Inertia parameters -->
@@ -72,13 +72,13 @@
       <visual>
         <geometry>
-          <mesh filename="package://ur_description/meshes/ur5/visual/base.dae" />
-        </geometry>
-        <material name="LightGrey">
-          <color rgba="0.7 0.7 0.7 1.0"/>
-        </material>
-      </visual>
-      <collision>
-        <geometry>
-          <mesh filename="package://ur_description/meshes/ur5/collision/base.stl" />
+          <mesh filename="package://iai_ur_description/meshes/ur5/visual/base.dae" />
+        </geometry>
+        <material name="LightGrey">
+          <color rgba="0.7 0.7 0.7 1.0"/>
+        </material>
+      </visual>
+      <collision>
+        <geometry>
+          <mesh filename="package://iai_ur_description/meshes/ur5/collision/base.stl" />
         </geometry>
       </collision>
@@ -103,13 +103,13 @@
       <visual>
         <geometry>
-          <mesh filename="package://ur_description/meshes/ur5/visual/shoulder.dae" />
-        </geometry>
-        <material name="LightGrey">
-          <color rgba="0.7 0.7 0.7 1.0"/>
-        </material>
-      </visual>
-      <collision>
-        <geometry>
-          <mesh filename="package://ur_description/meshes/ur5/collision/shoulder.stl" />
+          <mesh filename="package://iai_ur_description/meshes/ur5/visual/shoulder.dae" />
+        </geometry>
+        <material name="LightGrey">
+          <color rgba="0.7 0.7 0.7 1.0"/>
+        </material>
+      </visual>
+      <collision>
+        <geometry>
+          <mesh filename="package://iai_ur_description/meshes/ur5/collision/shoulder.stl" />
         </geometry>
       </collision>
@@ -134,13 +134,13 @@
       <visual>
         <geometry>
-          <mesh filename="package://ur_description/meshes/ur5/visual/upperarm.dae" />
-        </geometry>
-        <material name="LightGrey">
-          <color rgba="0.7 0.7 0.7 1.0"/>
-        </material>
-      </visual>
-      <collision>
-        <geometry>
-          <mesh filename="package://ur_description/meshes/ur5/collision/upperarm.stl" />
+          <mesh filename="package://iai_ur_description/meshes/ur5/visual/upperarm.dae" />
+        </geometry>
+        <material name="LightGrey">
+          <color rgba="0.7 0.7 0.7 1.0"/>
+        </material>
+      </visual>
+      <collision>
+        <geometry>
+          <mesh filename="package://iai_ur_description/meshes/ur5/collision/upperarm.stl" />
         </geometry>
       </collision>
@@ -165,13 +165,13 @@
       <visual>
         <geometry>
-          <mesh filename="package://ur_description/meshes/ur5/visual/forearm.dae" />
-        </geometry>
-        <material name="LightGrey">
-          <color rgba="0.7 0.7 0.7 1.0"/>
-        </material>
-      </visual>
-      <collision>
-        <geometry>
-          <mesh filename="package://ur_description/meshes/ur5/collision/forearm.stl" />
+          <mesh filename="package://iai_ur_description/meshes/ur5/visual/forearm.dae" />
+        </geometry>
+        <material name="LightGrey">
+          <color rgba="0.7 0.7 0.7 1.0"/>
+        </material>
+      </visual>
+      <collision>
+        <geometry>
+          <mesh filename="package://iai_ur_description/meshes/ur5/collision/forearm.stl" />
         </geometry>
       </collision>
@@ -196,13 +196,13 @@
       <visual>
         <geometry>
-          <mesh filename="package://ur_description/meshes/ur5/visual/wrist1.dae" />
-        </geometry>
-        <material name="LightGrey">
-          <color rgba="0.7 0.7 0.7 1.0"/>
-        </material>
-      </visual>
-      <collision>
-        <geometry>
-          <mesh filename="package://ur_description/meshes/ur5/collision/wrist1.stl" />
+          <mesh filename="package://iai_ur_description/meshes/ur5/visual/wrist1.dae" />
+        </geometry>
+        <material name="LightGrey">
+          <color rgba="0.7 0.7 0.7 1.0"/>
+        </material>
+      </visual>
+      <collision>
+        <geometry>
+          <mesh filename="package://iai_ur_description/meshes/ur5/collision/wrist1.stl" />
         </geometry>
       </collision>
@@ -227,13 +227,13 @@
       <visual>
         <geometry>
-          <mesh filename="package://ur_description/meshes/ur5/visual/wrist2.dae" />
-        </geometry>
-        <material name="LightGrey">
-          <color rgba="0.7 0.7 0.7 1.0"/>
-        </material>
-      </visual>
-      <collision>
-        <geometry>
-          <mesh filename="package://ur_description/meshes/ur5/collision/wrist2.stl" />
+          <mesh filename="package://iai_ur_description/meshes/ur5/visual/wrist2.dae" />
+        </geometry>
+        <material name="LightGrey">
+          <color rgba="0.7 0.7 0.7 1.0"/>
+        </material>
+      </visual>
+      <collision>
+        <geometry>
+          <mesh filename="package://iai_ur_description/meshes/ur5/collision/wrist2.stl" />
         </geometry>
       </collision>
@@ -258,13 +258,13 @@
       <visual>
         <geometry>
-          <mesh filename="package://ur_description/meshes/ur5/visual/wrist3.dae" />
-        </geometry>
-        <material name="LightGrey">
-          <color rgba="0.7 0.7 0.7 1.0"/>
-        </material>
-      </visual>
-      <collision>
-        <geometry>
-          <mesh filename="package://ur_description/meshes/ur5/collision/wrist3.stl" />
+          <mesh filename="package://iai_ur_description/meshes/ur5/visual/wrist3.dae" />
+        </geometry>
+        <material name="LightGrey">
+          <color rgba="0.7 0.7 0.7 1.0"/>
+        </material>
+      </visual>
+      <collision>
+        <geometry>
+          <mesh filename="package://iai_ur_description/meshes/ur5/collision/wrist3.stl" />
         </geometry>
       </collision>

File: iai_ur_description/urdf/ur5_joint_limited_robot.urdf.xacro (robot description, xacro)
@@ -1,11 +1,11 @@
 <?xml version="1.0"?>
 <robot xmlns:xacro="http://www.ros.org/wiki/xacro"
-       name="ur3" >
+       name="ur5" >
   <!-- common stuff -->
-  <xacro:include filename="$(find ur_description)/urdf/common.gazebo.xacro" />
-  <!-- ur3 -->
-  <xacro:include filename="$(find ur_description)/urdf/ur3.urdf.xacro" />
+  <xacro:include filename="$(find iai_ur_description)/urdf/common.gazebo.xacro" />
+  <!-- ur5 -->
+  <xacro:include filename="$(find iai_ur_description)/urdf/ur5.urdf.xacro" />
   <!-- arm -->
-  <xacro:ur3_robot prefix="" joint_limited="true"/>
+  <xacro:ur5_robot prefix="" joint_limited="true"/>
   <link name="world" />
   <joint name="world_joint" type="fixed">
