Commit message: Added missing cabling adaptor plate to urdf-description of KUKA LWR4+ arm.

File: iai_kuka_lwr4_description/urdf/kuka_lwr_arm.urdf.xacro (robot description, xacro)
@@ -352,4 +352,18 @@
       </inertial>
     </link>
+    <joint name="${name}_cabling_adaptor_joint" type="fixed">
+      <origin xyz="0 0 0.005" rpy="0 0 0"/>
+      <parent link="${name}_arm_flange_link"/>
+      <child link="${name}_cabling_adaptor_link"/>
+    </joint>
+    <link name="${name}_cabling_adaptor_link">
+      <visual>
+        <origin rpy="0 0 0" xyz="0 0 0"/>
+        <geometry>
+          <cylinder length="0.01" radius="0.0315"/>
+        </geometry>
+        <material name="Black"/>
+      </visual>
+    </link>
     <!-- joint name="${name}_arm_hand_fixed_joint" type="fixed">
       <origin xyz="${-right * 0.075} -0.075 -0.016"

Commit message: Renaming cabling-adoptor of KUKA LWR 4+ for consistency.

File: iai_kuka_lwr4_description/urdf/kuka_lwr_arm.urdf.xacro (robot description, xacro)
@@ -352,10 +352,10 @@
       </inertial>
     </link>
-    <joint name="${name}_cabling_adaptor_joint" type="fixed">
+    <joint name="${name}_arm_cabling_adaptor_joint" type="fixed">
       <origin xyz="0 0 0.005" rpy="0 0 0"/>
       <parent link="${name}_arm_flange_link"/>
-      <child link="${name}_cabling_adaptor_link"/>
-    </joint>
-    <link name="${name}_cabling_adaptor_link">
+      <child link="${name}_arm_cabling_adaptor_link"/>
+    </joint>
+    <link name="${name}_arm_cabling_adaptor_link">
       <visual>
         <origin rpy="0 0 0" xyz="0 0 0"/>

Commit message: Small comment for a fix on the LWR4 model

File: iai_kuka_lwr4_description/urdf/kuka_lwr_arm.urdf.xacro (robot description, xacro)
@@ -352,6 +352,7 @@
       </inertial>
     </link>
+    <!-- Many Kuka LWR4s are equipped with a little plate to let the cables go out sideways -->
     <joint name="${name}_arm_cabling_adaptor_joint" type="fixed">
-      <origin xyz="0 0 0.005" rpy="0 0 0"/>
+      <origin xyz="0 0 0.005" rpy="0 0 0"/>  <!--FIXME: this puts the link in the center of the adapter, instead of the end -->
       <parent link="${name}_arm_flange_link"/>
       <child link="${name}_arm_cabling_adaptor_link"/>

Commit message: kuka_lwr4 description: changed to red (UniHB) color. Also now using the Collada files for better viewing (with normals).
Also changed the collada files to have red color.

File: iai_kuka_lwr4_description/urdf/kuka_lwr_arm.urdf.xacro (robot description, xacro)
@@ -29,7 +29,9 @@
         <origin xyz="0 0 0" rpy="0 0 0"/>
         <geometry>
-          <mesh filename="package://iai_kuka_lwr4_description/meshes/arm_base.stl"/>
-        </geometry>
-        <material name="Orange"/>
+          <!-- for each mesh we have two versions, one Collada file with normals and colors, and one simpler STL. The collada file is in cm, and the STL in meters -->
+          <mesh filename="package://iai_kuka_lwr4_description/meshes/arm_base.dae" scale="100 100 100"/>
+	  <!--mesh filename="package://iai_kuka_lwr4_description/meshes/arm_base.stl" scale="1 1 1"-->
+        </geometry>
+        <material name="UniHB-Red"/>
       </visual>
       <collision>
@@ -66,7 +68,8 @@
         <origin xyz="0 0 0" rpy="0 0 ${M_PI}"/>
         <geometry>
-          <mesh filename="package://iai_kuka_lwr4_description/meshes/arm_segment_a.stl"/>
-        </geometry>
-        <material name="Orange"/>
+          <mesh filename="package://iai_kuka_lwr4_description/meshes/arm_segment_a.dae" scale="100 100 100"/>
+          <!--mesh filename="package://iai_kuka_lwr4_description/meshes/arm_segment_a.stl" scale="1 1 1"/-->
+        </geometry>
+        <material name="UniHB-Red"/>
       </visual>
       <collision>
@@ -108,7 +111,8 @@
         <origin xyz="0 0 0.2" rpy="${M_PI} 0 ${M_PI}"/>
         <geometry>
-          <mesh filename="package://iai_kuka_lwr4_description/meshes/arm_segment_b.stl"/>
-        </geometry>
-        <material name="Orange"/>
+          <mesh filename="package://iai_kuka_lwr4_description/meshes/arm_segment_b.dae" scale="100 100 100"/>
+          <!--mesh filename="package://iai_kuka_lwr4_description/meshes/arm_segment_b.stl" scale="1 1 1"/-->
+        </geometry>
+        <material name="UniHB-Red"/>
       </visual>
       <collision>
@@ -150,7 +154,8 @@
         <origin xyz="0 0 0" rpy="0 0 0"/>
         <geometry>
-          <mesh filename="package://iai_kuka_lwr4_description/meshes/arm_segment_a.stl"/>
-        </geometry>
-        <material name="Orange"/>
+          <mesh filename="package://iai_kuka_lwr4_description/meshes/arm_segment_a.dae" scale="100 100 100"/>
+          <!--mesh filename="package://iai_kuka_lwr4_description/meshes/arm_segment_a.stl" scale="1 1 1"/-->
+        </geometry>
+        <material name="UniHB-Red"/>
       </visual>
       <collision>
@@ -192,7 +197,8 @@
         <origin xyz="0 0 0.2" rpy="0 ${M_PI} ${M_PI}"/>
         <geometry>
-          <mesh filename="package://iai_kuka_lwr4_description/meshes/arm_segment_b.stl"/>
-        </geometry>
-        <material name="Orange"/>
+          <mesh filename="package://iai_kuka_lwr4_description/meshes/arm_segment_b.dae" scale="100 100 100"/>
+          <!--mesh filename="package://iai_kuka_lwr4_description/meshes/arm_segment_b.stl" scale="1 1 1"/-->
+        </geometry>
+        <material name="UniHB-Red"/>
       </visual>
       <collision>
@@ -234,7 +240,8 @@
         <origin xyz="0 0 0" rpy="0 0 ${M_PI}"/>
         <geometry name="${name}_arm_5_geom">
-          <mesh filename="package://iai_kuka_lwr4_description/meshes/arm_segment_last.stl"/>
-        </geometry>
-        <material name="Orange"/>
+          <mesh filename="package://iai_kuka_lwr4_description/meshes/arm_segment_last.dae" scale="100 100 100"/>
+          <!--mesh filename="package://iai_kuka_lwr4_description/meshes/arm_segment_last.stl" scale="1 1 1"/-->
+        </geometry>
+        <material name="UniHB-Red"/>
       </visual>
       <collision>
@@ -276,5 +283,6 @@
         <origin xyz="0 0 0" rpy="0 0 ${M_PI}"/>
         <geometry>
-          <mesh filename="package://iai_kuka_lwr4_description/meshes/arm_wrist.stl"/>
+          <mesh filename="package://iai_kuka_lwr4_description/meshes/arm_wrist.dae" scale="100 100 100"/>
+          <!--mesh filename="package://iai_kuka_lwr4_description/meshes/arm_wrist.stl" scale="1 1 1"/-->
         </geometry>
         <material name="Grey"/>
@@ -318,7 +326,8 @@
         <origin xyz="0 0 0.078" rpy="0 0 0"/>
         <geometry>
-          <mesh filename="package://iai_kuka_lwr4_description/meshes/arm_flanche.stl"/>
-        </geometry>
-        <material name="Grey"/>
+          <mesh filename="package://iai_kuka_lwr4_description/meshes/arm_flanche.dae" scale="100 100 100"/>
+          <!--mesh filename="package://iai_kuka_lwr4_description/meshes/arm_flanche.stl" scale="1 1 1"/-->
+        </geometry>
+        <material name="Black"/>
       </visual>
       <collision>

Commit message: fixed position issues for the arm

File: iai_kuka_lwr4_description/urdf/kuka_lwr_arm.urdf.xacro (robot description, xacro)
@@ -66,7 +66,9 @@
       </inertial>
       <visual>
-        <origin xyz="0 0 0" rpy="0 0 ${M_PI}"/>
-        <geometry>
-          <mesh filename="package://iai_kuka_lwr4_description/meshes/arm_segment_a.dae" />
+	<!--
+        <origin xyz="0 0 0" rpy="0 0 ${M_PI}"/>
+	-->
+        <geometry>
+          <mesh filename="package://iai_kuka_lwr4_description/meshes/arm_seg_1.dae" />
           <!--mesh filename="package://iai_kuka_lwr4_description/meshes/arm_segment_a.stl" scale="1 1 1"/-->
         </geometry>
@@ -109,7 +111,9 @@
       </inertial>
       <visual>
+	<!--
         <origin xyz="0 0 0.2" rpy="${M_PI} 0 ${M_PI}"/>
-        <geometry>
-          <mesh filename="package://iai_kuka_lwr4_description/meshes/arm_segment_b.dae" />
+	-->
+        <geometry>
+          <mesh filename="package://iai_kuka_lwr4_description/meshes/arm_seg_2.dae" />
           <!--mesh filename="package://iai_kuka_lwr4_description/meshes/arm_segment_b.stl" scale="1 1 1"/-->
         </geometry>
@@ -154,5 +158,5 @@
         <origin xyz="0 0 0" rpy="0 0 0"/>
         <geometry>
-          <mesh filename="package://iai_kuka_lwr4_description/meshes/arm_segment_a.dae" />
+          <mesh filename="package://iai_kuka_lwr4_description/meshes/arm_seg_3.dae" />
           <!--mesh filename="package://iai_kuka_lwr4_description/meshes/arm_segment_a.stl" scale="1 1 1"/-->
         </geometry>
@@ -195,7 +199,9 @@
       </inertial>
       <visual>
+	<!--
         <origin xyz="0 0 0.2" rpy="0 ${M_PI} ${M_PI}"/>
-        <geometry>
-          <mesh filename="package://iai_kuka_lwr4_description/meshes/arm_segment_b.dae" />
+	-->
+        <geometry>
+          <mesh filename="package://iai_kuka_lwr4_description/meshes/arm_seg_4.dae" />
           <!--mesh filename="package://iai_kuka_lwr4_description/meshes/arm_segment_b.stl" scale="1 1 1"/-->
         </geometry>
@@ -238,7 +244,9 @@
       </inertial>
       <visual>
-        <origin xyz="0 0 0" rpy="0 0 ${M_PI}"/>
+	<!--
+        <origin xyz="0 0 0" rpy="0 0 ${M_PI}"/>
+	-->
         <geometry name="${name}_arm_5_geom">
-          <mesh filename="package://iai_kuka_lwr4_description/meshes/arm_segment_last.dae" />
+          <mesh filename="package://iai_kuka_lwr4_description/meshes/arm_seg_last.dae" />
           <!--mesh filename="package://iai_kuka_lwr4_description/meshes/arm_segment_last.stl" scale="1 1 1"/-->
         </geometry>
@@ -281,7 +289,9 @@
       </inertial>
       <visual>
-        <origin xyz="0 0 0" rpy="0 0 ${M_PI}"/>
-        <geometry>
-          <mesh filename="package://iai_kuka_lwr4_description/meshes/arm_wrist.dae" />
+	<!--
+        <origin xyz="0 0 0" rpy="0 0 ${M_PI}"/>
+	-->
+        <geometry>
+          <mesh filename="package://iai_kuka_lwr4_description/meshes/arm_seg_wrist.dae" />
           <!--mesh filename="package://iai_kuka_lwr4_description/meshes/arm_wrist.stl" scale="1 1 1"/-->
         </geometry>
@@ -324,7 +334,9 @@
       </inertial>
       <visual>
+	<!--
         <origin xyz="0 0 0.078" rpy="0 0 0"/>
-        <geometry>
-          <mesh filename="package://iai_kuka_lwr4_description/meshes/arm_flanche.dae" />
+	-->
+        <geometry>
+          <mesh filename="package://iai_kuka_lwr4_description/meshes/arm_seg_flanche.dae" />
           <!--mesh filename="package://iai_kuka_lwr4_description/meshes/arm_flanche.stl" scale="1 1 1"/-->
         </geometry>

Commit message: Corrected limits according to the more restricted controller we use (BEASTY)

File: iai_kuka_lwr4_description/urdf/kuka_lwr_arm.urdf.xacro (robot description, xacro)
@@ -48,8 +48,8 @@
       <origin xyz="0 0 0.11" rpy="0 0 0"/>
       <axis xyz="0 0 1"/>
-      <limit lower="${-170 * M_PI / 180}" upper="${170 * M_PI / 180}"
+      <limit lower="${-150 * M_PI / 180}" upper="${150 * M_PI / 180}"
              effort="204" velocity="${arm_velocity_scale_factor * 110 * M_PI / 180}" />
-      <safety_controller soft_lower_limit="${-168 * M_PI / 180}"
-                         soft_upper_limit="${168 * M_PI / 180}"
+      <safety_controller soft_lower_limit="${-148 * M_PI / 180}"
+                         soft_upper_limit="${148 * M_PI / 180}"
                          k_position="${safety_controller_k_pos}"
                          k_velocity="${safety_controller_k_vel}"/>
@@ -91,8 +91,8 @@
       <origin xyz="0 0 0.20" rpy="0 0 0"/>
       <axis xyz="0 -1 0"/>
-      <limit lower="${-120 * M_PI / 180}" upper="${120 * M_PI / 180}"
+      <limit lower="${-107 * M_PI / 180}" upper="${107 * M_PI / 180}"
              effort="306" velocity="${arm_velocity_scale_factor * 110 * M_PI / 180}" />
-      <safety_controller soft_lower_limit="${-118 * M_PI / 180}"
-                         soft_upper_limit="${118 * M_PI / 180}"
+      <safety_controller soft_lower_limit="${-105 * M_PI / 180}"
+                         soft_upper_limit="${105 * M_PI / 180}"
                          k_position="${safety_controller_k_pos}"
                          k_velocity="${safety_controller_k_vel}"/>
@@ -134,8 +134,8 @@
       <origin xyz="0 0 0.20" rpy="0 0 0"/>
       <axis xyz="0 0 1"/>
-      <limit lower="${-170 * M_PI / 180}" upper="${170 * M_PI / 180}"
+      <limit lower="${-150 * M_PI / 180}" upper="${150 * M_PI / 180}"
              effort="204" velocity="${arm_velocity_scale_factor * 130 * M_PI / 180}" />
-      <safety_controller soft_lower_limit="${-168 * M_PI / 180}"
-                         soft_upper_limit="${168 * M_PI / 180}"
+      <safety_controller soft_lower_limit="${-148 * M_PI / 180}"
+                         soft_upper_limit="${148 * M_PI / 180}"
                          k_position="${safety_controller_k_pos}"
                          k_velocity="${safety_controller_k_vel}"/>
@@ -177,8 +177,8 @@
       <origin xyz="0 0 0.20" rpy="0 0 0"/>
       <axis xyz="0 1 0"/>
-      <limit lower="${-120 * M_PI / 180}" upper="${120 * M_PI / 180}"
+      <limit lower="${-107 * M_PI / 180}" upper="${107 * M_PI / 180}"
              effort="306" velocity="${arm_velocity_scale_factor * 130 * M_PI / 180}" />
-      <safety_controller soft_lower_limit="${-118 * M_PI / 180}"
-                         soft_upper_limit="${118 * M_PI / 180}"
+      <safety_controller soft_lower_limit="${-105 * M_PI / 180}"
+                         soft_upper_limit="${105 * M_PI / 180}"
                          k_position="${safety_controller_k_pos}"
                          k_velocity="${safety_controller_k_vel}"/>
@@ -220,8 +220,8 @@
       <origin xyz="0 0 0.20" rpy="0 0 0"/>
       <axis xyz="0 0 1"/>
-      <limit lower="${-170 * M_PI / 180}" upper="${170 * M_PI / 180}"
+      <limit lower="${-150 * M_PI / 180}" upper="${150 * M_PI / 180}"
              effort="204" velocity="${arm_velocity_scale_factor * 130 * M_PI / 180}" />
-      <safety_controller soft_lower_limit="${-168 * M_PI / 180}"
-                         soft_upper_limit="${168 * M_PI / 180}"
+      <safety_controller soft_lower_limit="${-148 * M_PI / 180}"
+                         soft_upper_limit="${148 * M_PI / 180}"
                          k_position="${safety_controller_k_pos}"
                          k_velocity="${safety_controller_k_vel}"/>
@@ -263,8 +263,8 @@
       <origin xyz="0 0 0.19" rpy="0 0 0"/>
       <axis xyz="0 -1 0"/>
-      <limit lower="${-120 * M_PI / 180}" upper="${120 * M_PI / 180}"
+      <limit lower="${-115 * M_PI / 180}" upper="${115 * M_PI / 180}"
              effort="306" velocity="${arm_velocity_scale_factor * 180 * M_PI / 180}" />
-      <safety_controller soft_lower_limit="${-118 * M_PI / 180}"
-                         soft_upper_limit="${118 * M_PI / 180}"
+      <safety_controller soft_lower_limit="${-113 * M_PI / 180}"
+                         soft_upper_limit="${113 * M_PI / 180}"
                          k_position="${safety_controller_k_pos}"
                          k_velocity="${safety_controller_k_vel}"/>
@@ -306,8 +306,8 @@
       <origin xyz="0 0 0" rpy="0 0 0"/>
       <axis xyz="0 0 1"/>
-      <limit lower="${-170 * M_PI / 180}" upper="${170 * M_PI / 180}"
+      <limit lower="${-150 * M_PI / 180}" upper="${150 * M_PI / 180}"
              effort="204" velocity="${arm_velocity_scale_factor * 180 * M_PI / 180}" />
-      <safety_controller soft_lower_limit="${-168 * M_PI / 180}"
-                         soft_upper_limit="${168 * M_PI / 180}"
+      <safety_controller soft_lower_limit="${-148 * M_PI / 180}"
+                         soft_upper_limit="${148 * M_PI / 180}"
                          k_position="${safety_controller_k_pos}"
                          k_velocity="${safety_controller_k_vel}"/>

Commit message: Fixed missing tags in the URDF

File: iai_kuka_lwr4_description/urdf/kuka_lwr_arm.urdf.xacro (robot description, xacro)
@@ -55,4 +55,5 @@
                          k_velocity="${safety_controller_k_vel}"/>
       <dynamics damping="${joint_damping}"/>
+      <calibration rising="0.0"/>
       <parent link="calib_${name}_arm_base_link"/>
       <child link="${name}_arm_1_link"/>
@@ -98,4 +99,5 @@
                          k_velocity="${safety_controller_k_vel}"/>
       <dynamics damping="${joint_damping}"/>
+      <calibration rising="0.0"/>
       <parent link="${name}_arm_1_link"/>
       <child link="${name}_arm_2_link"/>
@@ -141,4 +143,5 @@
                          k_velocity="${safety_controller_k_vel}"/>
       <dynamics damping="${joint_damping}"/>
+      <calibration rising="0.0"/>
       <parent link="${name}_arm_2_link"/>
       <child link="${name}_arm_3_link"/>
@@ -184,4 +187,5 @@
                          k_velocity="${safety_controller_k_vel}"/>
       <dynamics damping="${joint_damping}"/>
+      <calibration rising="0.0"/>
       <parent link="${name}_arm_3_link"/>
       <child link="${name}_arm_4_link"/>
@@ -227,4 +231,5 @@
                          k_velocity="${safety_controller_k_vel}"/>
       <dynamics damping="${joint_damping}"/>
+      <calibration rising="0.0"/>
       <parent link="${name}_arm_4_link"/>
       <child link="${name}_arm_5_link"/>
@@ -270,4 +275,5 @@
                          k_velocity="${safety_controller_k_vel}"/>
       <dynamics damping="${joint_damping}"/>
+      <calibration rising="0.0"/>
       <parent link="${name}_arm_5_link"/>
       <child link="${name}_arm_6_link"/>
@@ -313,4 +319,5 @@
                          k_velocity="${safety_controller_k_vel}"/>
       <dynamics damping="${joint_damping}"/>
+      <calibration rising="0.0"/>
       <parent link="${name}_arm_6_link"/>
       <child link="${name}_arm_7_link"/>

File: iai_wsg_50_description/urdf/wsg_50.urdf.xacro (robot description, xacro)
@@ -180,7 +180,4 @@
      <parent link="${name}_gripper_right_link"/>
      <child link="${name}_finger_right_link" />
-     <dynamics friction="100" damping="100" />
-     <axis xyz="1 0 0"/>
-     <limit effort="100" velocity="100"/>
   </joint>
   <link name="${name}_finger_right_link">

Commit message: used .stl instead of .dae for kuka_lwr_arm.urdf

File: iai_kuka_lwr4_description/urdf/kuka_lwr_arm.urdf.xacro (robot description, xacro)
@@ -30,6 +30,6 @@
         <geometry>
           <!-- for each mesh we have two versions, one Collada file with normals and colors, and one simpler STL. The collada file is in cm, and the STL in meters -->
-          <mesh filename="package://iai_kuka_lwr4_description/meshes/arm_base.dae" scale="100 100 100"/>
-	  <!--mesh filename="package://iai_kuka_lwr4_description/meshes/arm_base.stl" scale="1 1 1"-->
+          <!-- <mesh filename="package://iai_kuka_lwr4_description/meshes/arm_base.dae" scale="100 100 100"/> -->
+	  		<mesh filename="package://iai_kuka_lwr4_description/meshes/arm_base.stl" scale="1 1 1"/>
         </geometry>
         <material name="UniHB-Red"/>
@@ -69,6 +69,6 @@
         <origin xyz="0 0 0" rpy="0 0 ${M_PI}"/>
         <geometry>
-          <mesh filename="package://iai_kuka_lwr4_description/meshes/arm_segment_a.dae" scale="100 100 100"/>
-          <!--mesh filename="package://iai_kuka_lwr4_description/meshes/arm_segment_a.stl" scale="1 1 1"/-->
+          <!-- <mesh filename="package://iai_kuka_lwr4_description/meshes/arm_segment_a.dae" scale="100 100 100"/> -->
+          <mesh filename="package://iai_kuka_lwr4_description/meshes/arm_segment_a.stl" scale="1 1 1"/>
         </geometry>
         <material name="UniHB-Red"/>
@@ -113,6 +113,6 @@
         <origin xyz="0 0 0.2" rpy="${M_PI} 0 ${M_PI}"/>
         <geometry>
-          <mesh filename="package://iai_kuka_lwr4_description/meshes/arm_segment_b.dae" scale="100 100 100"/>
-          <!--mesh filename="package://iai_kuka_lwr4_description/meshes/arm_segment_b.stl" scale="1 1 1"/-->
+          <!-- <mesh filename="package://iai_kuka_lwr4_description/meshes/arm_segment_b.dae" scale="100 100 100"/> -->
+          <mesh filename="package://iai_kuka_lwr4_description/meshes/arm_segment_b.stl" scale="1 1 1"/>
         </geometry>
         <material name="UniHB-Red"/>
@@ -157,6 +157,6 @@
         <origin xyz="0 0 0" rpy="0 0 0"/>
         <geometry>
-          <mesh filename="package://iai_kuka_lwr4_description/meshes/arm_segment_a.dae" scale="100 100 100"/>
-          <!--mesh filename="package://iai_kuka_lwr4_description/meshes/arm_segment_a.stl" scale="1 1 1"/-->
+          <!-- <mesh filename="package://iai_kuka_lwr4_description/meshes/arm_segment_a.dae" scale="100 100 100"/> -->
+          <mesh filename="package://iai_kuka_lwr4_description/meshes/arm_segment_a.stl" scale="1 1 1"/>
         </geometry>
         <material name="UniHB-Red"/>
@@ -201,6 +201,6 @@
         <origin xyz="0 0 0.2" rpy="0 ${M_PI} ${M_PI}"/>
         <geometry>
-          <mesh filename="package://iai_kuka_lwr4_description/meshes/arm_segment_b.dae" scale="100 100 100"/>
-          <!--mesh filename="package://iai_kuka_lwr4_description/meshes/arm_segment_b.stl" scale="1 1 1"/-->
+          <!-- <mesh filename="package://iai_kuka_lwr4_description/meshes/arm_segment_b.dae" scale="100 100 100"/> -->
+          <mesh filename="package://iai_kuka_lwr4_description/meshes/arm_segment_b.stl" scale="1 1 1"/>
         </geometry>
         <material name="UniHB-Red"/>
@@ -245,6 +245,6 @@
         <origin xyz="0 0 0" rpy="0 0 ${M_PI}"/>
         <geometry name="${name}_arm_5_geom">
-          <mesh filename="package://iai_kuka_lwr4_description/meshes/arm_segment_last.dae" scale="100 100 100"/>
-          <!--mesh filename="package://iai_kuka_lwr4_description/meshes/arm_segment_last.stl" scale="1 1 1"/-->
+          <!-- <mesh filename="package://iai_kuka_lwr4_description/meshes/arm_segment_last.dae" scale="100 100 100"/>  -->
+          <mesh filename="package://iai_kuka_lwr4_description/meshes/arm_segment_last.stl" scale="1 1 1"/>
         </geometry>
         <material name="UniHB-Red"/>
@@ -289,6 +289,6 @@
         <origin xyz="0 0 0" rpy="0 0 ${M_PI}"/>
         <geometry>
-          <mesh filename="package://iai_kuka_lwr4_description/meshes/arm_wrist.dae" scale="100 100 100"/>
-          <!--mesh filename="package://iai_kuka_lwr4_description/meshes/arm_wrist.stl" scale="1 1 1"/-->
+          <!-- <mesh filename="package://iai_kuka_lwr4_description/meshes/arm_wrist.dae" scale="100 100 100"/> -->
+          <mesh filename="package://iai_kuka_lwr4_description/meshes/arm_wrist.stl" scale="1 1 1"/>
         </geometry>
         <material name="Grey"/>
@@ -333,6 +333,6 @@
         <origin xyz="0 0 0.078" rpy="0 0 0"/>
         <geometry>
-          <mesh filename="package://iai_kuka_lwr4_description/meshes/arm_flanche.dae" scale="100 100 100"/>
-          <!--mesh filename="package://iai_kuka_lwr4_description/meshes/arm_flanche.stl" scale="1 1 1"/-->
+          <!-- <mesh filename="package://iai_kuka_lwr4_description/meshes/arm_flanche.dae" scale="100 100 100"/> -->
+          <mesh filename="package://iai_kuka_lwr4_description/meshes/arm_flanche.stl" scale="1 1 1"/>
         </geometry>
         <material name="Black"/>
