Commit message: kuka-lwr model: fix units
The collada files are in meters, so define the units to meter
 (the default for DAE anyway), and reset the scale to 1 1 1 in the URDF

File: iai_kuka_lwr4_description/urdf/kuka_lwr_arm.urdf.xacro (robot description, xacro)
@@ -30,5 +30,5 @@
         <geometry>
           <!-- for each mesh we have two versions, one Collada file with normals and colors, and one simpler STL. The collada file is in cm, and the STL in meters -->
-          <mesh filename="package://iai_kuka_lwr4_description/meshes/arm_base.dae" scale="100 100 100"/>
+          <mesh filename="package://iai_kuka_lwr4_description/meshes/arm_base.dae" scale="1 1 1"/>
 	  <!--mesh filename="package://iai_kuka_lwr4_description/meshes/arm_base.stl" scale="1 1 1"-->
         </geometry>
@@ -69,5 +69,5 @@
         <origin xyz="0 0 0" rpy="0 0 ${M_PI}"/>
         <geometry>
-          <mesh filename="package://iai_kuka_lwr4_description/meshes/arm_segment_a.dae" scale="100 100 100"/>
+          <mesh filename="package://iai_kuka_lwr4_description/meshes/arm_segment_a.dae" scale="1 1 1"/>
           <!--mesh filename="package://iai_kuka_lwr4_description/meshes/arm_segment_a.stl" scale="1 1 1"/-->
         </geometry>
@@ -113,5 +113,5 @@
         <origin xyz="0 0 0.2" rpy="${M_PI} 0 ${M_PI}"/>
         <geometry>
-          <mesh filename="package://iai_kuka_lwr4_description/meshes/arm_segment_b.dae" scale="100 100 100"/>
+          <mesh filename="package://iai_kuka_lwr4_description/meshes/arm_segment_b.dae" scale="1 1 1"/>
           <!--mesh filename="package://iai_kuka_lwr4_description/meshes/arm_segment_b.stl" scale="1 1 1"/-->
         </geometry>
@@ -157,5 +157,5 @@
         <origin xyz="0 0 0" rpy="0 0 0"/>
         <geometry>
-          <mesh filename="package://iai_kuka_lwr4_description/meshes/arm_segment_a.dae" scale="100 100 100"/>
+          <mesh filename="package://iai_kuka_lwr4_description/meshes/arm_segment_a.dae" scale="1 1 1"/>
           <!--mesh filename="package://iai_kuka_lwr4_description/meshes/arm_segment_a.stl" scale="1 1 1"/-->
         </geometry>
@@ -201,5 +201,5 @@
         <origin xyz="0 0 0.2" rpy="0 ${M_PI} ${M_PI}"/>
         <geometry>
-          <mesh filename="package://iai_kuka_lwr4_description/meshes/arm_segment_b.dae" scale="100 100 100"/>
+          <mesh filename="package://iai_kuka_lwr4_description/meshes/arm_segment_b.dae" scale="1 1 1"/>
           <!--mesh filename="package://iai_kuka_lwr4_description/meshes/arm_segment_b.stl" scale="1 1 1"/-->
         </geometry>
@@ -245,5 +245,5 @@
         <origin xyz="0 0 0" rpy="0 0 ${M_PI}"/>
         <geometry name="${name}_arm_5_geom">
-          <mesh filename="package://iai_kuka_lwr4_description/meshes/arm_segment_last.dae" scale="100 100 100"/>
+          <mesh filename="package://iai_kuka_lwr4_description/meshes/arm_segment_last.dae" scale="1 1 1"/>
           <!--mesh filename="package://iai_kuka_lwr4_description/meshes/arm_segment_last.stl" scale="1 1 1"/-->
         </geometry>
@@ -289,5 +289,5 @@
         <origin xyz="0 0 0" rpy="0 0 ${M_PI}"/>
         <geometry>
-          <mesh filename="package://iai_kuka_lwr4_description/meshes/arm_wrist.dae" scale="100 100 100"/>
+          <mesh filename="package://iai_kuka_lwr4_description/meshes/arm_wrist.dae" scale="1 1 1"/>
           <!--mesh filename="package://iai_kuka_lwr4_description/meshes/arm_wrist.stl" scale="1 1 1"/-->
         </geometry>
@@ -333,5 +333,5 @@
         <origin xyz="0 0 0.078" rpy="0 0 0"/>
         <geometry>
-          <mesh filename="package://iai_kuka_lwr4_description/meshes/arm_flanche.dae" scale="100 100 100"/>
+          <mesh filename="package://iai_kuka_lwr4_description/meshes/arm_flanche.dae" scale="1 1 1"/>
           <!--mesh filename="package://iai_kuka_lwr4_description/meshes/arm_flanche.stl" scale="1 1 1"/-->
         </geometry>

Commit message: Removed cabling adaptor from iai-kuka-lwr urdf.

File: iai_kuka_lwr4_description/urdf/kuka_lwr_arm.urdf.xacro (robot description, xacro)
@@ -368,26 +368,4 @@
       </inertial>
     </link>
-    <!-- Many Kuka LWR4s are equipped with a little plate to let the cables go out sideways -->
-    <joint name="${prefix}arm_cabling_adaptor_joint" type="fixed">
-      <origin xyz="0 0 0.01" rpy="0 0 0"/>  <!-- This places the link at the end of the plate (frame_out) -->
-      <parent link="${prefix}arm_flange_link"/>
-      <child link="${prefix}arm_cabling_adaptor_link"/>
-    </joint>
-    <link name="${prefix}arm_cabling_adaptor_link">
-      <visual>
-        <origin xyz="0 0 -0.005" rpy="0 0 0" />  <!-- The cylinder is placed at the center -->
-        <geometry>
-          <cylinder length="0.01" radius="0.0315"/>
-        </geometry>
-        <material name="Black"/>
-      </visual>
-    </link>
-    <!-- joint name="${prefix}arm_hand_fixed_joint" type="fixed">
-      <origin xyz="${-right * 0.075} -0.075 -0.016"
-              rpy="${0.5*right*M_PI} 0 ${(1.5 + 0.25*right)*M_PI}"/>
-      <parent link="${prefix}arm_7_link"/>
-      <child link="${prefix}arm_hand_link"/>
-    </joint>
-    <link name="${prefix}arm_hand_link" / -->
   </macro>
 </robot>

Commit message: Commented unnecessary material tags in kuka-xacro.

File: iai_kuka_lwr4_description/urdf/kuka_lwr_arm.urdf.xacro (robot description, xacro)
@@ -33,5 +33,5 @@
 	  <!--mesh filename="package://iai_kuka_lwr4_description/meshes/arm_base.stl" scale="1 1 1"-->
         </geometry>
-        <material name="UniHB-Red"/>
+        <!--material name="UniHB-Red"/-->
       </visual>
       <collision>
@@ -72,5 +72,5 @@
           <!--mesh filename="package://iai_kuka_lwr4_description/meshes/arm_segment_a.stl" scale="1 1 1"/-->
         </geometry>
-        <material name="UniHB-Red"/>
+        <!--material name="UniHB-Red"/-->
       </visual>
       <collision>
@@ -116,5 +116,5 @@
           <!--mesh filename="package://iai_kuka_lwr4_description/meshes/arm_segment_b.stl" scale="1 1 1"/-->
         </geometry>
-        <material name="UniHB-Red"/>
+        <!--material name="UniHB-Red"/-->
       </visual>
       <collision>
@@ -160,5 +160,5 @@
           <!--mesh filename="package://iai_kuka_lwr4_description/meshes/arm_segment_a.stl" scale="1 1 1"/-->
         </geometry>
-        <material name="UniHB-Red"/>
+        <!--material name="UniHB-Red"/-->
       </visual>
       <collision>
@@ -204,5 +204,5 @@
           <!--mesh filename="package://iai_kuka_lwr4_description/meshes/arm_segment_b.stl" scale="1 1 1"/-->
         </geometry>
-        <material name="UniHB-Red"/>
+        <!--material name="UniHB-Red"/-->
       </visual>
       <collision>
@@ -248,5 +248,5 @@
           <!--mesh filename="package://iai_kuka_lwr4_description/meshes/arm_segment_last.stl" scale="1 1 1"/-->
         </geometry>
-        <material name="UniHB-Red"/>
+        <!--material name="UniHB-Red"/-->
       </visual>
       <collision>
