Commit message: Separated URDF of kinect into its own package.

File: iai_kinect_description/urdf/kinect.urdf.xacro (robot description, xacro)
@@ -14,5 +14,5 @@
         <origin xyz="-0.05 -0.17 -0.02" rpy="${M_PI/2.0} 0 ${M_PI/2.0}"/>
         <geometry>
-          <mesh filename="package://iai_boxy_description/meshes/sensors/68-04546_Kinect_Sensor--coarse.STL" scale="0.001 0.001 0.001" />
+          <mesh filename="package://iai_kinect_description/meshes/68-04546_Kinect_Sensor--coarse.STL" scale="0.001 0.001 0.001" />
         </geometry>
         <material name="gray">

Commit message: Added collision mesh for the kinect

File: iai_kinect_description/urdf/kinect.urdf.xacro (robot description, xacro)
@@ -23,5 +23,5 @@
         <origin xyz="0.0 0.0 0" rpy="0 0 0"/>
         <geometry>
-        <sphere radius="0.0005"/>
+          <mesh filename="package:///iai_kinect_description/meshes/68-04546_Kinect_Sensor--coarse.STL" scale="0.001 0.001 0.001" />
         </geometry>
       </collision>

Commit message: fixed typo

File: iai_kinect_description/urdf/kinect.urdf.xacro (robot description, xacro)
@@ -23,5 +23,5 @@
         <origin xyz="0.0 0.0 0" rpy="0 0 0"/>
         <geometry>
-          <mesh filename="package:///iai_kinect_description/meshes/68-04546_Kinect_Sensor--coarse.STL" scale="0.001 0.001 0.001" />
+          <mesh filename="package://iai_kinect_description/meshes/68-04546_Kinect_Sensor--coarse.STL" scale="0.001 0.001 0.001" />
         </geometry>
       </collision>

Commit message: Collision mesh also has a rotation

File: iai_kinect_description/urdf/kinect.urdf.xacro (robot description, xacro)
@@ -21,5 +21,5 @@
       </visual>
       <collision>
-        <origin xyz="0.0 0.0 0" rpy="0 0 0"/>
+        <origin xyz="-0.05 -0.17 -0.02" rpy="${M_PI/2.0} 0 ${M_PI/2.0}"/>
         <geometry>
           <mesh filename="package://iai_kinect_description/meshes/68-04546_Kinect_Sensor--coarse.STL" scale="0.001 0.001 0.001" />
