Commit message: Replacing collision STL model

File: iai_boxy_description/robots/boxy_description.urdf (robot description, URDF)
Before this commit: robot boxy_description, 82 links, 81 joints
Links:
- link head_mount_kinect2_rgb_optical_frame: geometry collision mesh filename=package://iai_kinect2_description/meshes/kinect2_origin_on_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 scale=0.001 0.001 0.001; visual mesh filename=package://iai_kinect2_description/meshes/kinect2_origin_on_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 scale=0.001 0.001 0.001
- link neck_adapter_iso50_kinect2_frame_in: geometry collision mesh filename=package://iai_adapter_iso50_kinect2_description/meshes/adap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 scale=1 1 1; visual mesh filename=package://iai_adapter_iso50_kinect2_description/meshes/adap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 scale=1 1 1
- link neck_look_target: geometry visual cylinder length=0.35 radius=0.03
- link shoulder_kinect_link: geometry collision mesh filename=package://iai_kinect_description/meshes/68-04546_Kinect_Sen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 scale=0.001 0.001 0.001; visual mesh filename=package://iai_kinect_description/meshes/68-04546_Kinect_Sen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 scale=0.001 0.001 0.001
Joints:
- joint neck_shoulder_pan_joint: limit lower=-3.14159265 upper=3.14159265 effort=330.0 velocity=2.16 -> lower=-4.712388975 upper=4.712388975 effort=330.0 velocity=2.16
- joint shoulder_kinect_joint: origin xyz=-0.00585394 -0.52064754 1.46001 rpy=0.01708077682636155 0.0085798647123734 -0.00929470452726490 -> xyz=0.0405394 -0.52064754 1.47001 rpy=0.01708077682636155 0.0085798647123734 -0.00929470452726490
