Commit message: Corrected calibration of left and right arm in urdf description of boxy robot.

File: iai_boxy_description/robots/boxy_description.urdf.xacro (robot description, xacro)
@@ -38,6 +38,5 @@
 	<xacro:include filename="$(find iai_boxy_torso)/robots/torso.URDF" />
 	<kuka_lwr_arm parent="triangle_arm_left_link" name="left">
-	<origin xyz="0 0 0"
-			rpy="0 0 0"/>
+          <origin xyz="0 0 0" rpy="0 0 1.047198"/>
 	</kuka_lwr_arm>
 	<xacro:include filename="$(find iai_weiss_wsg50)/robots/weiss_wsg50.urdf" />
@@ -50,6 +49,5 @@
 	<!-- /JOINT to connect the base with the torso -->
 	<kuka_lwr_arm parent="triangle_arm_right_link" name="right">
-	<origin xyz="0 0 0"
-			rpy="0 0 0"/>
+          <origin xyz="0 0 0" rpy="0 0 -1.047198"/>
 	</kuka_lwr_arm>
 </robot>

Commit message: Corrected frame names of arm base links in urdf of boxy robot.

File: iai_boxy_description/robots/boxy_description.urdf.xacro (robot description, xacro)
@@ -37,5 +37,5 @@
 	<!-- /JOINT to connect the base with the torso -->
 	<xacro:include filename="$(find iai_boxy_torso)/robots/torso.URDF" />
-	<kuka_lwr_arm parent="triangle_arm_left_link" name="left">
+	<kuka_lwr_arm parent="triangle_left_arm_link" name="left">
           <origin xyz="0 0 0" rpy="0 0 1.047198"/>
 	</kuka_lwr_arm>
@@ -48,5 +48,5 @@
 	</joint>
 	<!-- /JOINT to connect the base with the torso -->
-	<kuka_lwr_arm parent="triangle_arm_right_link" name="right">
+	<kuka_lwr_arm parent="triangle_right_arm_link" name="right">
           <origin xyz="0 0 0" rpy="0 0 -1.047198"/>
 	</kuka_lwr_arm>

File: iai_boxy_torso/robots/torso.URDF (robot description, URDF)
Before this commit: robot torso, 4 links, 3 joints
Links:
- removed link triangle_arm_left_link
- removed link triangle_arm_right_link
- added link triangle_left_arm_link
- added link triangle_right_arm_link
Joints:
- removed joint triangle_arm_left_joint
- removed joint triangle_arm_right_joint
- added joint triangle_left_arm_joint: type fixed, parent triangle_base_link, child triangle_left_arm_link, origin xyz=-0.239507442352261 -0.181209704131733 -0.137000000000002 rpy=2.61799387796333 -1.5707963267949 0, axis 0 0 0
- added joint triangle_right_arm_joint: type fixed, parent triangle_base_link, child triangle_right_arm_link, origin xyz=-0.365488160465715 -0.181209539931436 -0.137 rpy=2.61799387801966 1.5707963267949 0, axis 0 0 0

Commit message: Added wsg50 gripper to urdf and controllers

File: iai_boxy_description/robots/boxy_description.urdf.xacro (robot description, xacro)
@@ -3,4 +3,5 @@
 	<xacro:include filename="$(find iai_kuka_lwr4_description)/defs/materials.xml"/>
 	<xacro:include filename="$(find iai_kuka_lwr4_description)/urdf/kuka_lwr_arm.urdf.xacro"/>
+	<xacro:include filename="$(find wsg_50_simulation)/urdf/wsg_50.urdf.xacro"/>
 	<!-- Property definitions e.g. constants -->
 	<xacro:property name="head_joint_x" value="0.2" />
@@ -40,6 +41,6 @@
           <origin xyz="0 0 0" rpy="0 0 1.047198"/>
 	</kuka_lwr_arm>
+	<!-- Old gripper
 	<xacro:include filename="$(find iai_weiss_wsg50)/robots/weiss_wsg50.urdf" />
-	<!-- JOINT to connect the base with the torso -->
 	<joint name="left_hand_joint" type="fixed">
 		<origin xyz="0 0 0.08" rpy="0 0 0" />
@@ -47,7 +48,13 @@
 		<child link="gripper_base_link" />
 	</joint>
-	<!-- /JOINT to connect the base with the torso -->
+  -->
 	<kuka_lwr_arm parent="triangle_right_arm_link" name="right">
           <origin xyz="0 0 0" rpy="0 0 -1.047198"/>
 	</kuka_lwr_arm>
+	<wsg_50_xacro name="left_gripper" parent="left_arm_flange_link">
+		<origin xyz="0 0 0" rpy="0 0 0"/>
+	</wsg_50_xacro>
+	<wsg_50_xacro name="right_gripper" parent="right_arm_flange_link">
+		<origin xyz="0 0 0" rpy="0 0 0"/>
+	</wsg_50_xacro>
 </robot>

Commit message: Calibrated values for kinect2 on the pan/tilt unit, and eye/hand with the right kuka arm

File: iai_boxy_description/robots/boxy_description.urdf.xacro (robot description, xacro)
@@ -30,4 +30,21 @@
 	<!-- /JOINT to connect the base with the pw070 -->
 	<xacro:include filename="$(find iai_schunk_pw070_v6)/robots/pw070_v6.URDF" />
+	<!-- JOINT to place the kinect2 camera on the pw070 -->
+        <!-- Comes from tool_H_clink in the calibration
+             The quaternion was converted to RPY using python and KDL
+              halcon has quat: w x y z
+              kdl and tf_static_transform_publisher use: x y z w
+            So take the first number from the halcon quat and put it last for KDL.
+           import PyKDL as p; r2 = p.Rotation.Quaternion(-0.494547,0.491515,-0.506787,0.506955) ; r2.GetRPY()
+  answer: (-1.5431199762943342, -0.0029080109443817533, -1.5676362600579434) -->
+	<joint name="kinect2_joint" type="fixed">
+		<origin xyz="0.0402529 -0.0959434 0.0332714" rpy="-1.5431199762943342 -0.0029080109443817533 -1.5676362600579434" />
+		<parent link="pw070_frame_out" />
+		<child link="head_mount_kinect2_rgb_optical_frame" />
+	</joint>
+	<!-- JOINT to place the kinect2 camera on the pw070 -->
+        <!-- empty link for the rgb_optical_frame -->
+        <link name="head_mount_kinect2_rgb_optical_frame">
+        </link>
 	<!-- JOINT to connect the base with the torso -->
 	<joint name="torso_joint" type="fixed">
@@ -49,4 +66,5 @@
 	</joint>
   -->
+	<!--This is a 60deg rotation to calib_right_arm_base_link -->
 	<kuka_lwr_arm parent="triangle_right_arm_link" name="right">
           <origin xyz="0 0 0" rpy="0 0 -1.047198"/>

File: iai_boxy_torso/robots/torso.URDF (robot description, URDF)
Before this commit: robot torso, 4 links, 3 joints
Joints:
- joint triangle_base_joint: origin xyz=0.1 0.0175 0.58662489 rpy=-1.5708 -5.5511E-17 1.5708 -> xyz=0.0786889663592487 0.0986351579738104 0.906352096493862 rpy=4.70695928 6.28217403836 1.56327975371; parent torso_base_link -> base_link

Commit message: Refactored urdf of kms40 to have another parameter for its origin.

File: iai_boxy_description/robots/boxy_description.urdf.xacro (robot description, xacro)
@@ -71,5 +71,7 @@
           <origin xyz="0 0 0" rpy="0 0 -1.047198"/>
 	</kuka_lwr_arm>
-        <kms_40_xacro parent="right_arm_cabling_adaptor_link" prefix="right_arm"/>
+        <kms_40_xacro parent="right_arm_cabling_adaptor_link" prefix="right_arm">
+          <origin xyz="0 0 0.013" rpy="0 0 3.14159265359" />
+        </kms_40_xacro>
 	<!--wsg_50_xacro name="left_gripper" parent="left_arm_flange_link">
 		<origin xyz="0 0 0" rpy="0 0 0"/>

File: iai_kms_40_description/urdf/kms_40.urdf.xacro (robot description, xacro)
@@ -2,7 +2,7 @@
 <robot xmlns:xacro="http://ros.org/wiki/xacro"
        name="kms_40">
-  <xacro:macro name="kms_40_xacro" params="prefix parent">
+  <xacro:macro name="kms_40_xacro" params="prefix parent *origin">
     <joint name="${prefix}_kms40_adaptor_joint" type="fixed">
-      <origin xyz="0 0 0.013" rpy="0 0 3.14159265359" />
+      <insert_block name="origin"/>
       <parent link="${parent}"/>
       <child link="${prefix}_kms40_adaptor_link"/>

Commit message: Getting rid of commented legacy in boxy-description.

File: iai_boxy_description/robots/boxy_description.urdf.xacro (robot description, xacro)
@@ -59,12 +59,4 @@
           <origin xyz="0 0 0" rpy="0 0 1.047198"/>
 	</kuka_lwr_arm>
-	<!-- Old gripper
-	<xacro:include filename="$(find iai_weiss_wsg50)/robots/weiss_wsg50.urdf" />
-	<joint name="left_hand_joint" type="fixed">
-		<origin xyz="0 0 0.08" rpy="0 0 0" />
-		<parent link="left_arm_7_link" />
-		<child link="gripper_base_link" />
-	</joint>
-  -->
 	<!--This is a 60deg rotation to calib_right_arm_base_link -->
 	<kuka_lwr_arm parent="triangle_right_arm_link" name="right">

Commit message: Re-attached right wsg50 behind kms40 of boxy.

File: iai_boxy_description/robots/boxy_description.urdf.xacro (robot description, xacro)
@@ -59,4 +59,7 @@
           <origin xyz="0 0 0" rpy="0 0 1.047198"/>
 	</kuka_lwr_arm>
+	<!--wsg_50_xacro name="left_gripper" parent="left_arm_flange_link">
+		<origin xyz="0 0 0" rpy="0 0 0"/>
+	</wsg_50_xacro-->
 	<!--This is a 60deg rotation to calib_right_arm_base_link -->
 	<kuka_lwr_arm parent="triangle_right_arm_link" name="right">
@@ -66,9 +69,6 @@
           <origin xyz="0 0 0.013" rpy="0 0 3.14159265359" />
         </kms_40_xacro>
-	<!--wsg_50_xacro name="left_gripper" parent="left_arm_flange_link">
-		<origin xyz="0 0 0" rpy="0 0 0"/>
-	</wsg_50_xacro-->
-	<!--wsg_50_xacro name="right_gripper" parent="right_arm_flange_link">
-		<origin xyz="0 0 0" rpy="0 0 0"/>
-	</wsg_50_xacro-->
+        <wsg_50_xacro name="right_gripper" parent="right_arm_kms40_link">
+          <origin xyz="0 0 0.013" rpy="0 0 3.14159265359"/>
+	</wsg_50_xacro>
 </robot>

Commit message: Re-attached left wsg50 behind the cabling-adaptor of boxy.

File: iai_boxy_description/robots/boxy_description.urdf.xacro (robot description, xacro)
@@ -59,7 +59,7 @@
           <origin xyz="0 0 0" rpy="0 0 1.047198"/>
 	</kuka_lwr_arm>
-	<!--wsg_50_xacro name="left_gripper" parent="left_arm_flange_link">
-		<origin xyz="0 0 0" rpy="0 0 0"/>
-	</wsg_50_xacro-->
+	<wsg_50_xacro name="left_gripper" parent="left_arm_cabling_adaptor_link">
+          <origin xyz="0 0 0" rpy="0 0 0.005"/>
+	</wsg_50_xacro>
 	<!--This is a 60deg rotation to calib_right_arm_base_link -->
 	<kuka_lwr_arm parent="triangle_right_arm_link" name="right">

Commit message: Added shoulder-kinect to urdf of boxy.

File: iai_boxy_description/robots/boxy_description.urdf.xacro (robot description, xacro)
@@ -5,4 +5,5 @@
 	<xacro:include filename="$(find iai_wsg_50_description)/urdf/wsg_50.urdf.xacro"/>
 	<xacro:include filename="$(find iai_kms_40_description)/urdf/kms_40.urdf.xacro"/>
+	<xacro:include filename="$(find iai_boxy_description)/sensors/kinect.urdf.xacro"/>
 	<!-- Property definitions e.g. constants -->
 	<xacro:property name="head_joint_x" value="0.2" />
@@ -48,4 +49,13 @@
         <link name="head_mount_kinect2_rgb_optical_frame">
         </link>
+        <!-- shoulder kinect -->
+        <!-- ORIGINAL DATA FROM HALCON CALIBRATION:
+             from: base_link to: shoulder_kinect_link
+             translation: -0.135394 -0.00764754 1.54755 (xyz)
+             quaternion: 0.0177781 0.202257 -0.0472198 0.978032 (xyzw) -->
+        <kinect name="shoulder_kinect" parent="base_link">
+          <origin xyz="-0.135394 -0.00764754 1.54755"
+                  rpy="0.01708077682636155 0.4085798647123734 -0.09294704527264909"/>
+       </kinect>
 	<!-- JOINT to connect the base with the torso -->
 	<joint name="torso_joint" type="fixed">

Commit message: boxy_description: added the adapter plates after the force torque sensor

File: iai_boxy_description/robots/boxy_description.urdf.xacro (robot description, xacro)
@@ -6,4 +6,7 @@
 	<xacro:include filename="$(find iai_kms_40_description)/urdf/kms_40.urdf.xacro"/>
 	<xacro:include filename="$(find iai_boxy_description)/sensors/kinect.urdf.xacro"/>
+	<xacro:include filename="$(find iai_adapters_description)/urdf/adapter_fwa050_wsg50.urdf.xacro"/>
+	<xacro:include filename="$(find iai_adapters_description)/urdf/adapter_kms40_fwk050.urdf.xacro"/>
+	<xacro:include filename="$(find iai_adapters_description)/urdf/fwk_fwa_050.urdf.xacro"/>
 	<!-- Property definitions e.g. constants -->
 	<xacro:property name="head_joint_x" value="0.2" />
@@ -77,8 +80,18 @@
 	</kuka_lwr_arm>
         <kms_40_xacro parent="right_arm_cabling_adaptor_link" prefix="right_arm">
-          <origin xyz="0 0 0.013" rpy="0 0 3.14159265359" />
+          <origin xyz="0 0 0.013" rpy="0 0 3.14159265359" />  <!--places the kms40 frame 13mm from the parent -->
         </kms_40_xacro>
-        <wsg_50_xacro name="right_gripper" parent="right_arm_kms40_link">
-          <origin xyz="0 0 0.013" rpy="0 0 3.14159265359"/>
+        <!-- The following 3 URDFs have frame_in / frame_out, so they are simply placed at their parent -->
+        <adapter_kms40_fwk050_xacro parent="right_arm_kms40_link" prefix="right_arm">
+          <origin xyz="0 0 0.013" rpy="0 0 0" />
+        </adapter_kms40_fwk050_xacro>
+        <fwk_fwa_050_xacro parent="right_arm_adapter_kms40_fwk050_frame_out" prefix="right_arm">
+          <origin xyz="0 0 0" rpy="0 0 0" />
+        </fwk_fwa_050_xacro>
+        <adapter_fwa050_wsg50_xacro parent="right_arm_fwk_fwa_050_frame_out" prefix="right_arm">
+          <origin xyz="0 0 0.0" rpy="0 0 0" />
+        </adapter_fwa050_wsg50_xacro>
+        <wsg_50_xacro name="right_gripper" parent="right_arm_adapter_fwa050_wsg50_frame_out">
+          <origin xyz="0 0 0" rpy="0 0 3.14159265359"/>
 	</wsg_50_xacro>
 </robot>

Commit message: boxy_description: Add real meshes for the kms40. Redefine reference frames, using frame_in/frame_out

File: iai_boxy_description/robots/boxy_description.urdf.xacro (robot description, xacro)
@@ -79,10 +79,10 @@
           <origin xyz="0 0 0" rpy="0 0 -1.047198"/>
 	</kuka_lwr_arm>
+        <!-- The following URDFs have frame_in / frame_out, so they are simply placed at their parent -->
         <kms_40_xacro parent="right_arm_cabling_adaptor_link" prefix="right_arm">
-          <origin xyz="0 0 0.013" rpy="0 0 3.14159265359" />  <!--places the kms40 frame 13mm from the parent -->
+          <origin xyz="0 0 0" rpy="0 0 3.14159265359" />  <!--places the kms40 frame 13mm from the parent -->
         </kms_40_xacro>
-        <!-- The following 3 URDFs have frame_in / frame_out, so they are simply placed at their parent -->
-        <adapter_kms40_fwk050_xacro parent="right_arm_kms40_link" prefix="right_arm">
-          <origin xyz="0 0 0.013" rpy="0 0 0" />
+        <adapter_kms40_fwk050_xacro parent="right_arm_kms40_frame_out" prefix="right_arm">
+          <origin xyz="0 0 0" rpy="0 0 0" />
         </adapter_kms40_fwk050_xacro>
         <fwk_fwa_050_xacro parent="right_arm_adapter_kms40_fwk050_frame_out" prefix="right_arm">

File: iai_kms_40_description/urdf/kms_40.urdf.xacro (robot description, xacro)
@@ -3,46 +3,55 @@
        name="kms_40">
   <xacro:macro name="kms_40_xacro" params="prefix parent *origin">
-    <joint name="${prefix}_kms40_adaptor_joint" type="fixed">
+    <!-- Joint connecting the parent to our frame_in -->
+    <joint name="${prefix}_adapter_iso50_kms40_joint" type="fixed">
       <insert_block name="origin"/>
       <parent link="${parent}"/>
-      <child link="${prefix}_kms40_adaptor_link"/>
+      <child link="${prefix}_adapter_iso50_kms40_frame_in"/>
     </joint>
-    <link name="${prefix}_kms40_adaptor_link">
+    <!-- link for the adapter plate -->
+    <link name="${prefix}_adapter_iso50_kms40_frame_in">
       <visual>
         <origin rpy="0 0 0" xyz="0 0 0"/>
         <geometry>
-          <cylinder length="0.016" radius="0.0315"/>
+          <mesh filename="package://iai_kms_40_description/meshes/adapter_plate_iso50_kms40_weiss.stl" scale="0.001 0.001 0.001"/>
         </geometry>
         <material name="Grey"/>
       </visual>
     </link>
+    <!-- Empty link just to get the frame out -->
+    <link name="${prefix}_adapter_iso50_kms40_frame_out"/>
+    <!-- joint positioning the frame_out -->
+    <joint name="${prefix}_adapter_iso50_kms40_trans_frame_out" type="fixed">
+      <origin xyz="0 0 0.016" rpy="0 0 0" />
+      <parent link="${prefix}_adapter_iso50_kms40_frame_in" />
+      <child link="${prefix}_adapter_iso50_kms40_frame_out" />
+      <axis xyz="0 0 0" />
+    </joint>
+    <!-- Now joint connecting the actual kms40 sensor -->
     <joint name="${prefix}_kms40_joint" type="fixed">
-      <origin xyz="0 0 0.021" rpy="0 0 0" />
-      <parent link="${prefix}_kms40_adaptor_link"/>
-      <child link="${prefix}_kms40_link"/>
+      <origin xyz="0 0 0" rpy="0 0 0" />
+      <parent link="${prefix}_adapter_iso50_kms40_frame_out"/>
+      <child link="${prefix}_kms40_frame_in"/>
     </joint>
-    <link name="${prefix}_kms40_link">
+    <!-- Link for the kms40 sensor-->
+    <link name="${prefix}_kms40_frame_in">
       <visual>
         <origin rpy="0 0 0" xyz="0 0 0"/>
         <geometry>
-          <cylinder length="0.026" radius="0.033"/>
+          <mesh filename="package://iai_kms_40_description/meshes/kms40_simple.stl" scale="0.001 0.001 0.001"/>
         </geometry>
         <material name="Grey"/>
       </visual>
     </link>
-    <joint name="${prefix}_kms40_connector_joint" type="fixed">
-      <origin xyz="0.021 0 0" rpy="0 0 0" />
-      <parent link="${prefix}_kms40_link"/>
-      <child link="${prefix}_kms40_connector_link"/>
+    <!-- Empty link just to get the frame out -->
+    <!-- This is also the reference frame for the force/torque data -->
+    <link name="${prefix}_kms40_frame_out"/>
+    <!-- joint positioning the frame_out -->
+    <joint name="${prefix}_kms40_trans_frame_out" type="fixed">
+      <origin xyz="0 0 0.027" rpy="0 0 0" />
+      <parent link="${prefix}_kms40_frame_in" />
+      <child link="${prefix}_kms40_frame_out" />
+      <axis xyz="0 0 0" />
     </joint>
-    <link name="${prefix}_kms40_connector_link">
-      <visual>
-        <origin rpy="0 0 0" xyz="0 0 0"/>
-        <geometry>
-          <box size="0.042 0.038 0.0255"/>
-        </geometry>
-        <material name="Grey"/>
-      </visual>
-    </link>
   </xacro:macro>
 </robot>

File: iai_kuka_lwr4_description/urdf/kuka_lwr_arm.urdf.xacro (robot description, xacro)
@@ -354,5 +354,5 @@
     <!-- Many Kuka LWR4s are equipped with a little plate to let the cables go out sideways -->
     <joint name="${name}_arm_cabling_adaptor_joint" type="fixed">
-      <origin xyz="0 0 0.005" rpy="0 0 0"/>  <!--FIXME: this puts the link in the center of the adapter, instead of the end -->
+      <origin xyz="0 0 0.01" rpy="0 0 0"/>  <!-- This places the link at the end of the plate (frame_out) -->
       <parent link="${name}_arm_flange_link"/>
       <child link="${name}_arm_cabling_adaptor_link"/>
@@ -360,5 +360,5 @@
     <link name="${name}_arm_cabling_adaptor_link">
       <visual>
-        <origin rpy="0 0 0" xyz="0 0 0"/>
+        <origin xyz="0 0 -0.005" rpy="0 0 0" />  <!-- The cylinder is placed at the center -->
         <geometry>
           <cylinder length="0.01" radius="0.0315"/>

Commit message: iai_boxy_description: use the new URDF for the kinect2

File: iai_boxy_description/robots/boxy_description.urdf.xacro (robot description, xacro)
@@ -9,4 +9,5 @@
 	<xacro:include filename="$(find iai_adapters_description)/urdf/adapter_kms40_fwk050.urdf.xacro"/>
 	<xacro:include filename="$(find iai_adapters_description)/urdf/fwk_fwa_050.urdf.xacro"/>
+	<xacro:include filename="$(find iai_kinect2_description)/urdf/kinect2.urdf.xacro"/>
 	<!-- Property definitions e.g. constants -->
 	<xacro:property name="head_joint_x" value="0.2" />
@@ -35,21 +36,17 @@
 	<!-- /JOINT to connect the base with the pw070 -->
 	<xacro:include filename="$(find iai_schunk_pw070_v6)/robots/pw070_v6.URDF" />
-	<!-- JOINT to place the kinect2 camera on the pw070 -->
-        <!-- Comes from tool_H_clink in the calibration
+	<!-- Kinect2 -->
+        <!-- Pose comes from tool_H_clink in the calibration
              The quaternion was converted to RPY using python and KDL
-              halcon has quat: w x y z
-              kdl and tf_static_transform_publisher use: x y z w
-            So take the first number from the halcon quat and put it last for KDL.
-           import PyKDL as p; r2 = p.Rotation.Quaternion(-0.494547,0.491515,-0.506787,0.506955) ; r2.GetRPY()
-  answer: (-1.5431199762943342, -0.0029080109443817533, -1.5676362600579434) -->
-	<joint name="kinect2_joint" type="fixed">
+               halcon has quat: w x y z
+               kdl and tf_static_transform_publisher use: x y z w
+             So take the first number from the halcon quat and put it last for KDL.
+               import PyKDL as p; r2 = p.Rotation.Quaternion(-0.494547,0.491515,-0.506787,0.506955) ; r2.GetRPY()
+               answer: (-1.5431199762943342, -0.0029080109443817533, -1.5676362600579434) -->
+        <!-- The following kinect2_xacro defines the _kinect2_rgb_optical_frame
+        And includes the fixed joint to place the kinect on the pw070  -->
+        <kinect2_xacro parent="pw070_frame_out" prefix="head_mount">
 		<origin xyz="0.0402529 -0.0959434 0.0332714" rpy="-1.5431199762943342 -0.0029080109443817533 -1.5676362600579434" />
-		<parent link="pw070_frame_out" />
-		<child link="head_mount_kinect2_rgb_optical_frame" />
-	</joint>
-	<!-- JOINT to place the kinect2 camera on the pw070 -->
-        <!-- empty link for the rgb_optical_frame -->
-        <link name="head_mount_kinect2_rgb_optical_frame">
-        </link>
+        </kinect2_xacro>
         <!-- shoulder kinect -->
         <!-- ORIGINAL DATA FROM HALCON CALIBRATION:

Commit message: Finally mounted left gripper of boxy. Mirrored actual mounting transform.

File: iai_boxy_description/robots/boxy_description.urdf.xacro (robot description, xacro)
@@ -71,5 +71,5 @@
 	</kuka_lwr_arm>
 	<wsg_50_xacro name="left_gripper" parent="left_arm_cabling_adaptor_link">
-          <origin xyz="0 0 0" rpy="0 0 0.005"/>
+          <origin xyz="0 0 0" rpy="0 0 0.78539816339"/>
 	</wsg_50_xacro>
 	<!--This is a 60deg rotation to calib_right_arm_base_link -->

Commit message: Temporary addition of frames for the spoon (pizza experiment)

File: iai_boxy_description/robots/boxy_description.urdf.xacro (robot description, xacro)
@@ -93,3 +93,22 @@
           <origin xyz="0 0 0" rpy="0 0 3.14159265359"/>
 	</wsg_50_xacro>
+        <!-- Temporary place for the spoon frames -->
+	<link name="spoon_tip"/>
+	<link name="spoon_left_side"/>
+	<link name="spoon_right_side"/>
+	<joint name="spoon_tip_joint" type="fixed">
+		<origin xyz="0.0096 -0.0718 0.1214" rpy="0.7 0 0" />
+		<parent link="right_gripper_tool_frame" />
+		<child link="spoon_tip" />
+	</joint>
+	<joint name="spoon_left_side" type="fixed">
+		<origin xyz="-0.0325 0 -0.06" rpy="0 0 0" />
+		<parent link="spoon_tip" />
+		<child link="spoon_left_side" />
+	</joint>
+	<joint name="spoon_left_right" type="fixed">
+		<origin xyz="0.0325 0 -0.06" rpy="0 0 0" />
+		<parent link="spoon_tip" />
+		<child link="spoon_right_side" />
+	</joint>
 </robot>

Commit message: [iai_boxy_description] added tiny inertia to base footprint link:
the same way as PR2 has it.

File: iai_boxy_description/robots/boxy_description.urdf.xacro (robot description, xacro)
@@ -20,4 +20,22 @@
 	<xacro:include filename="$(find iai_boxy_base)/robots/base.URDF" />
 	<link name="base_footprint">
+    <inertial>
+      <mass value="1"/>
+      <origin xyz="0 0 0"/>
+      <inertia ixx="0.01" ixy="0" ixz="0" iyy="0.01" iyz="0" izz="0.01"/>
+    </inertial>
+    <visual>
+      <origin rpy="0 0 0" xyz="0 0 0"/>
+      <geometry>
+        <box size="0.01 0.01 0.01"/>
+      </geometry>
+      <material name="White"/>
+    </visual>
+    <collision>
+      <origin rpy="0 0 0" xyz="0 0 0.071"/>
+      <geometry>
+        <box size="0.001 0.001 0.001"/>
+      </geometry>
+    </collision>
 	</link>
 	<!-- JOINT to define base_footprint -->
