Commit message: Add a joint for the middle of the spoon (needed for pizza demo)

File: iai_boxy_description/robots/boxy_description.urdf.xacro (robot description, xacro)
@@ -115,4 +115,5 @@
 	<link name="spoon_left_side"/>
 	<link name="spoon_right_side"/>
+        <link name="spoon_middle"/>
 	<joint name="spoon_tip_joint" type="fixed">
 		<origin xyz="0.0096 -0.0718 0.1214" rpy="0.7 0 0" />
@@ -130,3 +131,8 @@
 		<child link="spoon_right_side" />
 	</joint>
+	<joint name="spoon_middle" type="fixed">
+		<origin xyz="0.0325 0.025 -0.05" rpy="0 0 0" />
+		<parent link="spoon_tip" />
+		<child link="spoon_middle" />
+	</joint>
 </robot>

Commit message: Boxy: Removed PW070, and added new adapter for UR3.

File: iai_boxy_description/robots/boxy_description.urdf.xacro (robot description, xacro)
@@ -9,4 +9,5 @@
 	<xacro:include filename="$(find iai_adapters_description)/urdf/adapter_kms40_fwk050.urdf.xacro"/>
 	<xacro:include filename="$(find iai_adapters_description)/urdf/fwk_fwa_050.urdf.xacro"/>
+	<xacro:include filename="$(find iai_adapters_description)/urdf/adapter_boxy_ur3.urdf.xacro"/>
 	<xacro:include filename="$(find iai_kinect2_description)/urdf/kinect2.urdf.xacro"/>
 	<!-- Property definitions e.g. constants -->
@@ -46,12 +47,19 @@
 	</joint>
 	<!-- /JOINT for base_footprint -->
+        <!-- NEW NECK ASSEMBLY -->
+        <!-- mounting plate of UR3 -->
+        <adapter_boxy_ur3_xacro prefix="neck" parent="base_link">
+          <origin xyz="0.214 -0.227 1.48" rpy="0 0 0" />
+        </adapter_boxy_ur3_xacro>
+        <!-- /NEW NECK ASSEMBLY -->
+        <!-- OLD NEW ASSEMBLY -->
 	<!-- JOINT to connect the base with the pw070 -->
-	<joint name="head_joint" type="fixed">
+	<!--joint name="head_joint" type="fixed">
 		<origin xyz="${head_joint_x} ${head_joint_y} ${head_joint_z}" rpy="0 0 0" />
 		<parent link="base_link" />
 		<child link="pw070_base_link" />
-	</joint>
+	</joint-->
 	<!-- /JOINT to connect the base with the pw070 -->
-	<xacro:include filename="$(find iai_schunk_pw070_v6)/robots/pw070_v6.URDF" />
+	<!--xacro:include filename="$(find iai_schunk_pw070_v6)/robots/pw070_v6.URDF" /-->
 	<!-- Kinect2 -->
         <!-- Pose comes from tool_H_clink in the calibration
@@ -64,7 +72,7 @@
         <!-- The following kinect2_xacro defines the _kinect2_rgb_optical_frame
         And includes the fixed joint to place the kinect on the pw070  -->
-        <kinect2_xacro parent="pw070_frame_out" prefix="head_mount">
+        <!--kinect2_xacro parent="pw070_frame_out" prefix="head_mount">
 		<origin xyz="0.0402529 -0.0959434 0.0332714" rpy="-1.5431199762943342 -0.0029080109443817533 -1.5676362600579434" />
-        </kinect2_xacro>
+        </kinect2_xacro-->
         <!-- shoulder kinect -->
         <!-- ORIGINAL DATA FROM HALCON CALIBRATION:

Commit message: Added ur3 neck to boxy.

File: iai_boxy_description/robots/boxy_description.urdf.xacro (robot description, xacro)
@@ -8,6 +8,7 @@
 	<xacro:include filename="$(find iai_adapters_description)/urdf/adapter_fwa050_wsg50.urdf.xacro"/>
 	<xacro:include filename="$(find iai_adapters_description)/urdf/adapter_kms40_fwk050.urdf.xacro"/>
-	<xacro:include filename="$(find iai_adapters_description)/urdf/fwk_fwa_050.urdf.xacro"/>
+        <xacro:include filename="$(find iai_adapters_description)/urdf/fwk_fwa_050.urdf.xacro"/>
 	<xacro:include filename="$(find iai_adapters_description)/urdf/adapter_boxy_ur3.urdf.xacro"/>
+        <xacro:include filename="$(find iai_ur_description)/urdf/ur3.urdf.xacro" />
 	<xacro:include filename="$(find iai_kinect2_description)/urdf/kinect2.urdf.xacro"/>
 	<!-- Property definitions e.g. constants -->
@@ -49,7 +50,11 @@
         <!-- NEW NECK ASSEMBLY -->
         <!-- mounting plate of UR3 -->
-        <adapter_boxy_ur3_xacro prefix="neck" parent="base_link">
+        <adapter_boxy_ur3_xacro prefix="neck_" parent="base_link">
           <origin xyz="0.214 -0.227 1.48" rpy="0 0 0" />
         </adapter_boxy_ur3_xacro>
+        <xacro:ur3_robot prefix="neck_" parent="neck_adapter_ur3_frame_out"
+                         joint_limited="true">
+          <origin xyz="0.0 0.0 0.0" rpy="0.0 0.0 0.0" />
+        </xacro:ur3_robot>
         <!-- /NEW NECK ASSEMBLY -->
         <!-- OLD NEW ASSEMBLY -->

Commit message: Cleaning boxy: Removing deprecated spoon frames from boxy urdf.

File: iai_boxy_description/robots/boxy_description.urdf.xacro (robot description, xacro)
@@ -124,28 +124,3 @@
           <origin xyz="0 0 0" rpy="0 0 3.14159265359"/>
 	</wsg_50_xacro>
-        <!-- Temporary place for the spoon frames -->
-	<link name="spoon_tip"/>
-	<link name="spoon_left_side"/>
-	<link name="spoon_right_side"/>
-        <link name="spoon_middle"/>
-	<joint name="spoon_tip_joint" type="fixed">
-		<origin xyz="0.0096 -0.0718 0.1214" rpy="0.7 0 0" />
-		<parent link="right_gripper_tool_frame" />
-		<child link="spoon_tip" />
-	</joint>
-	<joint name="spoon_left_side" type="fixed">
-		<origin xyz="-0.0325 0 -0.06" rpy="0 0 0" />
-		<parent link="spoon_tip" />
-		<child link="spoon_left_side" />
-	</joint>
-	<joint name="spoon_left_right" type="fixed">
-		<origin xyz="0.0325 0 -0.06" rpy="0 0 0" />
-		<parent link="spoon_tip" />
-		<child link="spoon_right_side" />
-	</joint>
-	<joint name="spoon_middle" type="fixed">
-		<origin xyz="0.0325 0.025 -0.05" rpy="0 0 0" />
-		<parent link="spoon_tip" />
-		<child link="spoon_middle" />
-	</joint>
 </robot>

Commit message: Boxy: Turned UR3 neck by 90deg. As mounted in reality.

File: iai_boxy_description/robots/boxy_description.urdf.xacro (robot description, xacro)
@@ -55,5 +55,5 @@
         <xacro:ur3_robot prefix="neck_" parent="neck_adapter_ur3_frame_out"
                          joint_limited="true">
-          <origin xyz="0.0 0.0 0.0" rpy="0.0 0.0 0.0" />
+          <origin xyz="0.0 0.0 0.0" rpy="0.0 0.0 -${M_PI/2.0}" />
         </xacro:ur3_robot>
         <!-- /NEW NECK ASSEMBLY -->

Commit message: First try with the kinect on the arm

File: iai_boxy_description/robots/boxy_description.urdf.xacro (robot description, xacro)
@@ -12,4 +12,5 @@
         <xacro:include filename="$(find iai_ur_description)/urdf/ur3.urdf.xacro" />
 	<xacro:include filename="$(find iai_kinect2_description)/urdf/kinect2.urdf.xacro"/>
+	<xacro:include filename="$(find iai_adapter_iso50_kinect2_description)/urdf/adapter_iso50_kinect2.urdf.xacro"/>
 	<!-- Property definitions e.g. constants -->
 	<xacro:property name="head_joint_x" value="0.2" />
@@ -57,4 +58,8 @@
           <origin xyz="0.0 0.0 0.0" rpy="0.0 0.0 -${M_PI/2.0}" />
         </xacro:ur3_robot>
+        <!-- The following URDF has frame_in / frame_out, so it is placed at the parent -->
+        <adapter_iso50_kinect2_xacro parent="neck_tool0" prefix="neck">
+          <origin xyz="0 0 0" rpy="0 0 -1.570795" />
+        </adapter_iso50_kinect2_xacro>
         <!-- /NEW NECK ASSEMBLY -->
         <!-- OLD NEW ASSEMBLY -->
@@ -77,7 +82,7 @@
         <!-- The following kinect2_xacro defines the _kinect2_rgb_optical_frame
         And includes the fixed joint to place the kinect on the pw070  -->
-        <!--kinect2_xacro parent="pw070_frame_out" prefix="head_mount">
+        <kinect2_xacro parent="neck_adapter_iso50_kinect2_frame_out" prefix="head_mount">
 		<origin xyz="0.0402529 -0.0959434 0.0332714" rpy="-1.5431199762943342 -0.0029080109443817533 -1.5676362600579434" />
-        </kinect2_xacro-->
+        </kinect2_xacro>
         <!-- shoulder kinect -->
         <!-- ORIGINAL DATA FROM HALCON CALIBRATION:

Commit message: kinect2 on neck: better approximate position/orientation

File: iai_boxy_description/robots/boxy_description.urdf.xacro (robot description, xacro)
@@ -83,5 +83,5 @@
         And includes the fixed joint to place the kinect on the pw070  -->
         <kinect2_xacro parent="neck_adapter_iso50_kinect2_frame_out" prefix="head_mount">
-		<origin xyz="0.0402529 -0.0959434 0.0332714" rpy="-1.5431199762943342 -0.0029080109443817533 -1.5676362600579434" />
+		<origin xyz="-0.02 0.10 0.02" rpy="-1.570795 0 1.570795" />
         </kinect2_xacro>
         <!-- shoulder kinect -->

Commit message: Boxy URDF: Fixed orientation of left gripper and position of neck

File: iai_boxy_description/robots/boxy_description.urdf.xacro (robot description, xacro)
@@ -52,5 +52,5 @@
         <!-- mounting plate of UR3 -->
         <adapter_boxy_ur3_xacro prefix="neck_" parent="base_link">
-          <origin xyz="0.214 -0.227 1.48" rpy="0 0 0" />
+          <origin xyz="0.175 -0.227 1.48" rpy="0 0 0" />
         </adapter_boxy_ur3_xacro>
         <xacro:ur3_robot prefix="neck_" parent="neck_adapter_ur3_frame_out"
@@ -107,5 +107,5 @@
 	</kuka_lwr_arm>
 	<wsg_50_xacro name="left_gripper" parent="left_arm_cabling_adaptor_link">
-          <origin xyz="0 0 0" rpy="0 0 0.78539816339"/>
+          <origin xyz="0 0 0" rpy="0 0 2.35619183661"/>
 	</wsg_50_xacro>
 	<!--This is a 60deg rotation to calib_right_arm_base_link -->
