Commit message: Correct prefix-behavior of lwr-urdf.

File: iai_boxy_description/robots/boxy_description.urdf.xacro (robot description, xacro)
@@ -103,5 +103,5 @@
 	<xacro:include filename="$(find iai_boxy_torso)/robots/torso.URDF" />
         <!--FIXME: triangle_left_arm_link should be rotated, and not the origin of the arm (which right now is calib_left_arm_base_link -->
-	<kuka_lwr_arm parent="triangle_left_arm_link" name="left">
+	<kuka_lwr_arm parent="triangle_left_arm_link" prefix="left_">
           <origin xyz="0 0 0" rpy="0 0 1.047198"/>
 	</kuka_lwr_arm>
@@ -110,5 +110,5 @@
 	</wsg_50_xacro>
 	<!--This is a 60deg rotation to calib_right_arm_base_link -->
-	<kuka_lwr_arm parent="triangle_right_arm_link" name="right">
+	<kuka_lwr_arm parent="triangle_right_arm_link" prefix="right_">
           <origin xyz="0 0 0" rpy="0 0 -1.047198"/>
 	</kuka_lwr_arm>

File: iai_boxy_description/robots/boxy_gutted_description.urdf.xacro (robot description, xacro)
@@ -56,5 +56,5 @@
 	<xacro:include filename="$(find iai_boxy_torso)/robots/torso.URDF" />
 	<!--This is a 60deg rotation to calib_right_arm_base_link -->
-	<kuka_lwr_arm parent="triangle_right_arm_link" name="right">
+	<kuka_lwr_arm parent="triangle_right_arm_link" prefix="right_">
           <origin xyz="0 0 0" rpy="0 0 -1.047198"/>
 	</kuka_lwr_arm>

File: iai_boxy_description/robots/old_boxy_description.urdf.xacro (robot description, xacro)
@@ -85,5 +85,5 @@
 	<xacro:include filename="$(find iai_boxy_torso)/robots/torso.URDF" />
         <!--FIXME: triangle_left_arm_link should be rotated, and not the origin of the arm (which right now is calib_left_arm_base_link -->
-	<kuka_lwr_arm parent="triangle_left_arm_link" name="left">
+	<kuka_lwr_arm parent="triangle_left_arm_link" prefix="left_">
           <origin xyz="0 0 0" rpy="0 0 1.047198"/>
 	</kuka_lwr_arm>
@@ -92,5 +92,5 @@
 	</wsg_50_xacro>
 	<!--This is a 60deg rotation to calib_right_arm_base_link -->
-	<kuka_lwr_arm parent="triangle_right_arm_link" name="right">
+	<kuka_lwr_arm parent="triangle_right_arm_link" prefix="right_">
           <origin xyz="0 0 0" rpy="0 0 -1.047198"/>
 	</kuka_lwr_arm>

File: iai_kuka_lwr4_description/robots/kuka_lwr_arm.urdf.xacro (robot description, xacro)
@@ -5,5 +5,5 @@
   <include filename="$(find iai_kuka_lwr4_description)/defs/materials.xml"/>
   <link name="base"/>
-  <kuka_lwr_arm parent="base" name="arm">
+  <kuka_lwr_arm parent="base" prefix="">
     <origin xyz="0 0 0" rpy="0 0 0"/>
   </kuka_lwr_arm>

File: iai_kuka_lwr4_description/urdf/kuka_lwr_arm.urdf.xacro (robot description, xacro)
@@ -13,11 +13,11 @@
   <property name="joint_damping" value="0.1" />
   <property name="arm_velocity_scale_factor" value="1"/>
-  <macro name="kuka_lwr_arm" params="parent name *origin">
-    <joint name="${parent}_${name}_arm_base_joint" type="fixed">
+  <macro name="kuka_lwr_arm" params="parent prefix *origin">
+    <joint name="${parent}_${prefix}arm_base_joint" type="fixed">
       <insert_block name="origin"/>
       <parent link="${parent}"/>
-      <child link="calib_${name}_arm_base_link"/>
-    </joint>
-    <link name="calib_${name}_arm_base_link">
+      <child link="calib_${prefix}arm_base_link"/>
+    </joint>
+    <link name="calib_${prefix}arm_base_link">
       <inertial>
         <mass value="${arm_elem_base_mass}"/>
@@ -42,8 +42,8 @@
       </collision>
     </link>
-    <gazebo reference="calib_${name}_arm_base_link">
-      <material value="kuka-lwr.material"/>
-    </gazebo>
-    <joint name="${name}_arm_0_joint" type="revolute">
+    <gazebo reference="calib_${prefix}arm_base_link">
+      <material value="kuka-lwr.material"/>
+    </gazebo>
+    <joint name="${prefix}arm_0_joint" type="revolute">
       <origin xyz="0 0 0.11" rpy="0 0 0"/>
       <axis xyz="0 0 1"/>
@@ -56,8 +56,8 @@
       <dynamics damping="${joint_damping}"/>
       <calibration rising="0.0"/>
-      <parent link="calib_${name}_arm_base_link"/>
-      <child link="${name}_arm_1_link"/>
-    </joint>
-    <link name="${name}_arm_1_link">
+      <parent link="calib_${prefix}arm_base_link"/>
+      <child link="${prefix}arm_1_link"/>
+    </joint>
+    <link name="${prefix}arm_1_link">
       <inertial>
         <mass value="${arm_elem_link_mass}"/>
@@ -81,13 +81,13 @@
       </collision>
     </link>
-    <gazebo reference="${name}_arm_1_link">
-      <material value="kuka-lwr.material"/>
-    </gazebo>
-    <transmission name="${name}_arm_0_trans" type="pr2_mechanism_model/SimpleTransmission">
-      <actuator name="${name}_arm_0_motor"/>
-      <joint name="${name}_arm_0_joint"/>
-      <mechanicalReduction>1.0</mechanicalReduction>
-    </transmission>
-    <joint name="${name}_arm_1_joint" type="revolute">
+    <gazebo reference="${prefix}arm_1_link">
+      <material value="kuka-lwr.material"/>
+    </gazebo>
+    <transmission name="${prefix}arm_0_trans" type="pr2_mechanism_model/SimpleTransmission">
+      <actuator name="${prefix}arm_0_motor"/>
+      <joint name="${prefix}arm_0_joint"/>
+      <mechanicalReduction>1.0</mechanicalReduction>
+    </transmission>
+    <joint name="${prefix}arm_1_joint" type="revolute">
       <origin xyz="0 0 0.20" rpy="0 0 0"/>
       <axis xyz="0 -1 0"/>
@@ -100,8 +100,8 @@
       <dynamics damping="${joint_damping}"/>
       <calibration rising="0.0"/>
-      <parent link="${name}_arm_1_link"/>
-      <child link="${name}_arm_2_link"/>
-    </joint>
-    <link name="${name}_arm_2_link">
+      <parent link="${prefix}arm_1_link"/>
+      <child link="${prefix}arm_2_link"/>
+    </joint>
+    <link name="${prefix}arm_2_link">
       <inertial>
         <mass value="${arm_elem_link_mass}"/>
@@ -125,13 +125,13 @@
       </collision>
     </link>
-    <gazebo reference="${name}_arm_2_link">
-      <material value="kuka-lwr.material"/>
-    </gazebo>
-    <transmission name="${name}_arm_1_trans" type="pr2_mechanism_model/SimpleTransmission">
-      <actuator name="${name}_arm_1_motor"/>
-      <joint name="${name}_arm_1_joint"/>
-      <mechanicalReduction>1.0</mechanicalReduction>
-    </transmission>
-    <joint name="${name}_arm_2_joint" type="revolute">
+    <gazebo reference="${prefix}arm_2_link">
+      <material value="kuka-lwr.material"/>
+    </gazebo>
+    <transmission name="${prefix}arm_1_trans" type="pr2_mechanism_model/SimpleTransmission">
+      <actuator name="${prefix}arm_1_motor"/>
+      <joint name="${prefix}arm_1_joint"/>
+      <mechanicalReduction>1.0</mechanicalReduction>
+    </transmission>
+    <joint name="${prefix}arm_2_joint" type="revolute">
       <origin xyz="0 0 0.20" rpy="0 0 0"/>
       <axis xyz="0 0 1"/>
@@ -144,8 +144,8 @@
       <dynamics damping="${joint_damping}"/>
       <calibration rising="0.0"/>
-      <parent link="${name}_arm_2_link"/>
-      <child link="${name}_arm_3_link"/>
-    </joint>
-    <link name="${name}_arm_3_link">
+      <parent link="${prefix}arm_2_link"/>
+      <child link="${prefix}arm_3_link"/>
+    </joint>
+    <link name="${prefix}arm_3_link">
       <inertial>
         <mass value="${arm_elem_link_mass}"/>
@@ -169,13 +169,13 @@
       </collision>
     </link>
-    <gazebo reference="${name}_arm_3_link">
-      <material value="kuka-lwr.material"/>
-    </gazebo>
-    <transmission name="${name}_arm_2_trans" type="pr2_mechanism_model/SimpleTransmission">
-      <actuator name="${name}_arm_2_motor"/>
-      <joint name="${name}_arm_2_joint"/>
-      <mechanicalReduction>1.0</mechanicalReduction>
-    </transmission>
-    <joint name="${name}_arm_3_joint" type="revolute">
+    <gazebo reference="${prefix}arm_3_link">
+      <material value="kuka-lwr.material"/>
+    </gazebo>
+    <transmission name="${prefix}arm_2_trans" type="pr2_mechanism_model/SimpleTransmission">
+      <actuator name="${prefix}arm_2_motor"/>
+      <joint name="${prefix}arm_2_joint"/>
+      <mechanicalReduction>1.0</mechanicalReduction>
+    </transmission>
+    <joint name="${prefix}arm_3_joint" type="revolute">
       <origin xyz="0 0 0.20" rpy="0 0 0"/>
       <axis xyz="0 1 0"/>
@@ -188,8 +188,8 @@
       <dynamics damping="${joint_damping}"/>
       <calibration rising="0.0"/>
-      <parent link="${name}_arm_3_link"/>
-      <child link="${name}_arm_4_link"/>
-    </joint>
-    <link name="${name}_arm_4_link">
+      <parent link="${prefix}arm_3_link"/>
+      <child link="${prefix}arm_4_link"/>
+    </joint>
+    <link name="${prefix}arm_4_link">
       <inertial>
         <mass value="${arm_elem_link_mass}"/>
@@ -213,13 +213,13 @@
       </collision>
     </link>
-    <gazebo reference="${name}_arm_4_link">
-      <material value="kuka-lwr.material"/>
-    </gazebo>
-    <transmission name="${name}_arm_3_trans" type="pr2_mechanism_model/SimpleTransmission">
-      <actuator name="${name}_arm_3_motor"/>
-      <joint name="${name}_arm_3_joint"/>
-      <mechanicalReduction>1.0</mechanicalReduction>
-    </transmission>
-    <joint name="${name}_arm_4_joint" type="revolute">
+    <gazebo reference="${prefix}arm_4_link">
+      <material value="kuka-lwr.material"/>
+    </gazebo>
+    <transmission name="${prefix}arm_3_trans" type="pr2_mechanism_model/SimpleTransmission">
+      <actuator name="${prefix}arm_3_motor"/>
+      <joint name="${prefix}arm_3_joint"/>
+      <mechanicalReduction>1.0</mechanicalReduction>
+    </transmission>
+    <joint name="${prefix}arm_4_joint" type="revolute">
       <origin xyz="0 0 0.20" rpy="0 0 0"/>
       <axis xyz="0 0 1"/>
@@ -232,8 +232,8 @@
       <dynamics damping="${joint_damping}"/>
       <calibration rising="0.0"/>
-      <parent link="${name}_arm_4_link"/>
-      <child link="${name}_arm_5_link"/>
-    </joint>
-    <link name="${name}_arm_5_link">
+      <parent link="${prefix}arm_4_link"/>
+      <child link="${prefix}arm_5_link"/>
+    </joint>
+    <link name="${prefix}arm_5_link">
       <inertial>
         <mass value="${arm_elem_link_mass}"/>
@@ -244,5 +244,5 @@
       <visual>
         <origin xyz="0 0 0" rpy="0 0 ${M_PI}"/>
-        <geometry name="${name}_arm_5_geom">
+        <geometry name="${prefix}arm_5_geom">
           <mesh filename="package://iai_kuka_lwr4_description/meshes/arm_segment_last.dae" scale="1 1 1"/>
           <!--mesh filename="package://iai_kuka_lwr4_description/meshes/arm_segment_last.stl" scale="1 1 1"/-->
@@ -257,13 +257,13 @@
       </collision>
     </link>
-    <gazebo reference="${name}_arm_5_link">
-      <material value="kuka-lwr.material"/>
-    </gazebo>
-    <transmission name="${name}_arm_4_trans" type="pr2_mechanism_model/SimpleTransmission">
-      <actuator name="${name}_arm_4_motor"/>
-      <joint name="${name}_arm_4_joint"/>
-      <mechanicalReduction>1.0</mechanicalReduction>
-    </transmission>
-    <joint name="${name}_arm_5_joint" type="revolute">
+    <gazebo reference="${prefix}arm_5_link">
+      <material value="kuka-lwr.material"/>
+    </gazebo>
+    <transmission name="${prefix}arm_4_trans" type="pr2_mechanism_model/SimpleTransmission">
+      <actuator name="${prefix}arm_4_motor"/>
+      <joint name="${prefix}arm_4_joint"/>
+      <mechanicalReduction>1.0</mechanicalReduction>
+    </transmission>
+    <joint name="${prefix}arm_5_joint" type="revolute">
       <origin xyz="0 0 0.19" rpy="0 0 0"/>
       <axis xyz="0 -1 0"/>
@@ -276,8 +276,8 @@
       <dynamics damping="${joint_damping}"/>
       <calibration rising="0.0"/>
-      <parent link="${name}_arm_5_link"/>
-      <child link="${name}_arm_6_link"/>
-    </joint>
-    <link name="${name}_arm_6_link">
+      <parent link="${prefix}arm_5_link"/>
+      <child link="${prefix}arm_6_link"/>
+    </joint>
+    <link name="${prefix}arm_6_link">
       <inertial>
         <mass value="${arm_elem_ball_link_mass}"/>
@@ -301,13 +301,13 @@
       </collision>
     </link>
-    <gazebo reference="${name}_arm_6_link">
-      <material value="kuka-lwr.material"/>
-    </gazebo>
-    <transmission name="${name}_arm_5_trans" type="pr2_mechanism_model/SimpleTransmission">
-      <actuator name="${name}_arm_5_motor"/>
-      <joint name="${name}_arm_5_joint"/>
-      <mechanicalReduction>1.0</mechanicalReduction>
-    </transmission>
-    <joint name="${name}_arm_6_joint" type="revolute">
+    <gazebo reference="${prefix}arm_6_link">
+      <material value="kuka-lwr.material"/>
+    </gazebo>
+    <transmission name="${prefix}arm_5_trans" type="pr2_mechanism_model/SimpleTransmission">
+      <actuator name="${prefix}arm_5_motor"/>
+      <joint name="${prefix}arm_5_joint"/>
+      <mechanicalReduction>1.0</mechanicalReduction>
+    </transmission>
+    <joint name="${prefix}arm_6_joint" type="revolute">
       <origin xyz="0 0 0" rpy="0 0 0"/>
       <axis xyz="0 0 1"/>
@@ -320,8 +320,8 @@
       <dynamics damping="${joint_damping}"/>
       <calibration rising="0.0"/>
-      <parent link="${name}_arm_6_link"/>
-      <child link="${name}_arm_7_link"/>
-    </joint>
-    <link name="${name}_arm_7_link">
+      <parent link="${prefix}arm_6_link"/>
+      <child link="${prefix}arm_7_link"/>
+    </joint>
+    <link name="${prefix}arm_7_link">
       <inertial>
         <mass value="${arm_elem_end_link_mass}"/>
@@ -345,20 +345,20 @@
       </collision>
     </link>
-    <gazebo reference="${name}_arm_7_link">
-      <material value="kuka-lwr.material"/>
-    </gazebo>
-    <transmission name="${name}_arm_6_trans" type="pr2_mechanism_model/SimpleTransmission">
-      <actuator name="${name}_arm_6_motor"/>
-      <joint name="${name}_arm_6_joint"/>
+    <gazebo reference="${prefix}arm_7_link">
+      <material value="kuka-lwr.material"/>
+    </gazebo>
+    <transmission name="${prefix}arm_6_trans" type="pr2_mechanism_model/SimpleTransmission">
+      <actuator name="${prefix}arm_6_motor"/>
+      <joint name="${prefix}arm_6_joint"/>
       <mechanicalReduction>1.0</mechanicalReduction>
     </transmission>
     <!--arm_7_link has the same pose as the TCP defined in the DLR Beasty controller:
        Center of the potato, with z-coming out towards the flange, and y going towards joint #6 -->
-    <joint name="${name}_arm_flange_joint" type="fixed">
+    <joint name="${prefix}arm_flange_joint" type="fixed">
       <origin xyz="0 0 0.078" rpy="0 0 0"/>
-      <parent link="${name}_arm_7_link"/>
-      <child link="${name}_arm_flange_link"/>
-    </joint>
-    <link name="${name}_arm_flange_link">
+      <parent link="${prefix}arm_7_link"/>
+      <child link="${prefix}arm_flange_link"/>
+    </joint>
+    <link name="${prefix}arm_flange_link">
       <inertial>
         <mass value="${arm_elem_flange_link_mass}"/>
@@ -369,10 +369,10 @@
     </link>
     <!-- Many Kuka LWR4s are equipped with a little plate to let the cables go out sideways -->
-    <joint name="${name}_arm_cabling_adaptor_joint" type="fixed">
+    <joint name="${prefix}arm_cabling_adaptor_joint" type="fixed">
       <origin xyz="0 0 0.01" rpy="0 0 0"/>  <!-- This places the link at the end of the plate (frame_out) -->
-      <parent link="${name}_arm_flange_link"/>
-      <child link="${name}_arm_cabling_adaptor_link"/>
-    </joint>
-    <link name="${name}_arm_cabling_adaptor_link">
+      <parent link="${prefix}arm_flange_link"/>
+      <child link="${prefix}arm_cabling_adaptor_link"/>
+    </joint>
+    <link name="${prefix}arm_cabling_adaptor_link">
       <visual>
         <origin xyz="0 0 -0.005" rpy="0 0 0" />  <!-- The cylinder is placed at the center -->
@@ -383,11 +383,11 @@
       </visual>
     </link>
-    <!-- joint name="${name}_arm_hand_fixed_joint" type="fixed">
+    <!-- joint name="${prefix}arm_hand_fixed_joint" type="fixed">
       <origin xyz="${-right * 0.075} -0.075 -0.016"
               rpy="${0.5*right*M_PI} 0 ${(1.5 + 0.25*right)*M_PI}"/>
-      <parent link="${name}_arm_7_link"/>
-      <child link="${name}_arm_hand_link"/>
-    </joint>
-    <link name="${name}_arm_hand_link" / -->
+      <parent link="${prefix}arm_7_link"/>
+      <child link="${prefix}arm_hand_link"/>
+    </joint>
+    <link name="${prefix}arm_hand_link" / -->
   </macro>
 </robot>

Commit message: Using lwr4-cabling-adaptor in Boxy description.

File: iai_boxy_description/robots/boxy_description.urdf.xacro (robot description, xacro)
@@ -5,4 +5,5 @@
 	<xacro:include filename="$(find iai_wsg_50_description)/urdf/wsg_50.urdf.xacro"/>
 	<xacro:include filename="$(find iai_kms_40_description)/urdf/kms_40.urdf.xacro"/>
+        <include filename="$(find iai_adapters_description)/urdf/lwr4_cabling_adaptor.urdf.xacro" />
 	<!--xacro:include filename="$(find iai_boxy_description)/sensors/kinect.urdf.xacro"/-->
 	<xacro:include filename="$(find iai_adapters_description)/urdf/adapter_fwa050_wsg50.urdf.xacro"/>
@@ -106,4 +107,7 @@
           <origin xyz="0 0 0" rpy="0 0 1.047198"/>
 	</kuka_lwr_arm>
+        <lwr4_cabling_adaptor parent="left_arm_flange_link" prefix="left_arm_">
+          <origin xyz="0 0 0.01" rpy="0 0 0"/>
+        </lwr4_cabling_adaptor>
 	<wsg_50_xacro name="left_gripper" parent="left_arm_cabling_adaptor_link">
           <origin xyz="0 0 0" rpy="0 0 2.35619183661"/>
@@ -113,4 +117,7 @@
           <origin xyz="0 0 0" rpy="0 0 -1.047198"/>
 	</kuka_lwr_arm>
+        <lwr4_cabling_adaptor parent="right_arm_flange_link" prefix="right_arm_">
+          <origin xyz="0 0 0.01" rpy="0 0 0"/>
+        </lwr4_cabling_adaptor>
         <!-- The following URDFs have frame_in / frame_out, so they are simply placed at their parent -->
         <kms_40_xacro parent="right_arm_cabling_adaptor_link" prefix="right_arm">

Commit message: Moving F/T sensor to the left arm

File: iai_boxy_description/robots/boxy_description.urdf.xacro (robot description, xacro)
@@ -110,7 +110,77 @@
           <origin xyz="0 0 0.01" rpy="0 0 0"/>
         </lwr4_cabling_adaptor>
-	<wsg_50_xacro name="left_gripper" parent="left_arm_cabling_adaptor_link">
+        <!-- The following URDFs have frame_in / frame_out, so they are simply placed at their parent -->
+        <kms_40_xacro parent="left_arm_cabling_adaptor_link" prefix="left_arm">
+          <origin xyz="0 0 0" rpy="0 0 3.14159265359" />  <!--places the kms40 frame 13mm from the parent -->
+        </kms_40_xacro>
+        <adapter_kms40_fwk050_xacro parent="left_arm_kms40_frame_out" prefix="left_arm">
+          <origin xyz="0 0 0" rpy="0 0 0" />
+        </adapter_kms40_fwk050_xacro>
+        <fwk_fwa_050_xacro parent="left_arm_adapter_kms40_fwk050_frame_out" prefix="left_arm">
+          <origin xyz="0 0 0" rpy="0 0 0" />
+        </fwk_fwa_050_xacro>
+        <adapter_fwa050_wsg50_xacro parent="left_arm_fwk_fwa_050_frame_out" prefix="left_arm">
+          <origin xyz="0 0 0.0" rpy="0 0 0" />
+        </adapter_fwa050_wsg50_xacro>
+        <wsg_50_xacro name="left_gripper" parent="left_arm_adapter_fwa050_wsg50_frame_out">
+          <origin xyz="0 0 0" rpy="0 0 3.14159265359"/>
+	</wsg_50_xacro>
+  <link name="left_wrist_optical_frame_x">
+    <inertial>
+      <mass value="1"/>
+      <origin xyz="0 0 0"/>
+      <inertia ixx="0.01" ixy="0" ixz="0" iyy="0.01" iyz="0" izz="0.01"/>
+    </inertial>
+    <visual>
+      <origin rpy="0 0 0" xyz="0 0 0"/>
+      <geometry>
+        <box size="0.01 0.01 0.01"/>
+      </geometry>
+      <material name="White"/>
+    </visual>
+    <collision>
+      <origin rpy="0 0 0" xyz="0 0 0.0"/>
+      <geometry>
+        <box size="0.001 0.001 0.001"/>
+      </geometry>
+    </collision>
+  </link>
+        <!-- JOINT to define base_footprint -->
+        <joint name="left_wrist_optical_joint_x" type="fixed">
+                <origin xyz="0.000836 -0.053028 0.073603" rpy="0.007552 6.274592 3.141201"/>
+                <parent link="left_gripper_base_link" />
+                <child link="left_wrist_optical_frame_x" />
+        </joint>
+        <!-- /JOINT for base_footprint -->
+  <link name="left_wrist_optical_frame">
+    <inertial>
+      <mass value="1"/>
+      <origin xyz="0 0 0"/>
+      <inertia ixx="0.01" ixy="0" ixz="0" iyy="0.01" iyz="0" izz="0.01"/>
+    </inertial>
+    <visual>
+      <origin rpy="0 0 0" xyz="0 0 0"/>
+      <geometry>
+        <box size="0.01 0.01 0.01"/>
+      </geometry>
+      <material name="White"/>
+    </visual>
+    <collision>
+      <origin rpy="0 0 0" xyz="0 0 0.0"/>
+      <geometry>
+        <box size="0.001 0.001 0.001"/>
+      </geometry>
+    </collision>
+  </link>
+        <!-- JOINT to define base_footprint -->
+        <joint name="left_wrist_optical_joint" type="fixed">
+                <origin xyz="0.0 0.0 0.0" rpy="0.0 0.0 3.141519"/>
+                <parent link="left_wrist_optical_frame_x" />
+                <child link="left_wrist_optical_frame" />
+        </joint>
+        <!-- /JOINT for base_footprint -->
+	<!--wsg_50_xacro name="left_gripper" parent="left_arm_cabling_adaptor_link">
           <origin xyz="0 0 0" rpy="0 0 2.35619183661"/>
-	</wsg_50_xacro>
+	</wsg_50_xacro-->
 	<!--This is a 60deg rotation to calib_right_arm_base_link -->
 	<kuka_lwr_arm parent="triangle_right_arm_link" prefix="right_">
