Commit message: Xacro of kuka-lwr has new parameter to specify which colored daes to use.

File: iai_boxy_description/robots/boxy_description.urdf.xacro (robot description, xacro)
@@ -104,5 +104,5 @@
 	<xacro:include filename="$(find iai_boxy_torso)/robots/torso.URDF" />
         <!--FIXME: triangle_left_arm_link should be rotated, and not the origin of the arm (which right now is calib_left_arm_base_link -->
-	<kuka_lwr_arm parent="triangle_left_arm_link" prefix="left_">
+	<kuka_lwr_arm parent="triangle_left_arm_link" prefix="left_" color_postfix="">
           <origin xyz="0 0 0" rpy="0 0 1.047198"/>
 	</kuka_lwr_arm>
@@ -184,5 +184,5 @@
 	</wsg_50_xacro-->
 	<!--This is a 60deg rotation to calib_right_arm_base_link -->
-	<kuka_lwr_arm parent="triangle_right_arm_link" prefix="right_">
+	<kuka_lwr_arm parent="triangle_right_arm_link" prefix="right_" color_postfix="">
           <origin xyz="0 0 0" rpy="0 0 -1.047198"/>
 	</kuka_lwr_arm>

File: iai_kuka_lwr4_description/robots/kuka_lwr_arm.urdf.xacro (robot description, xacro)
@@ -5,5 +5,5 @@
   <include filename="$(find iai_kuka_lwr4_description)/defs/materials.xml"/>
   <link name="base"/>
-  <kuka_lwr_arm parent="base" prefix="">
+  <kuka_lwr_arm parent="base" prefix="" color_postfix="_blue">
     <origin xyz="0 0 0" rpy="0 0 0"/>
   </kuka_lwr_arm>

File: iai_kuka_lwr4_description/urdf/kuka_lwr_arm.urdf.xacro (robot description, xacro)
@@ -13,5 +13,5 @@
   <property name="joint_damping" value="0.1" />
   <property name="arm_velocity_scale_factor" value="1"/>
-  <macro name="kuka_lwr_arm" params="parent prefix *origin">
+  <macro name="kuka_lwr_arm" params="parent prefix *origin color_postfix">
     <joint name="${parent}_${prefix}arm_base_joint" type="fixed">
       <insert_block name="origin"/>
@@ -30,5 +30,5 @@
         <geometry>
           <!-- for each mesh we have two versions, one Collada file with normals and colors, and one simpler STL. The collada file is in cm, and the STL in meters -->
-          <mesh filename="package://iai_kuka_lwr4_description/meshes/arm_base.dae" scale="1 1 1"/>
+          <mesh filename="package://iai_kuka_lwr4_description/meshes/arm_base${color_postfix}.dae" scale="1 1 1"/>
 	  <!--mesh filename="package://iai_kuka_lwr4_description/meshes/arm_base.stl" scale="1 1 1"-->
         </geometry>
@@ -69,5 +69,5 @@
         <origin xyz="0 0 0" rpy="0 0 ${M_PI}"/>
         <geometry>
-          <mesh filename="package://iai_kuka_lwr4_description/meshes/arm_segment_a.dae" scale="1 1 1"/>
+          <mesh filename="package://iai_kuka_lwr4_description/meshes/arm_segment_a${color_postfix}.dae" scale="1 1 1"/>
           <!--mesh filename="package://iai_kuka_lwr4_description/meshes/arm_segment_a.stl" scale="1 1 1"/-->
         </geometry>
@@ -113,5 +113,5 @@
         <origin xyz="0 0 0.2" rpy="${M_PI} 0 ${M_PI}"/>
         <geometry>
-          <mesh filename="package://iai_kuka_lwr4_description/meshes/arm_segment_b.dae" scale="1 1 1"/>
+          <mesh filename="package://iai_kuka_lwr4_description/meshes/arm_segment_b${color_postfix}.dae" scale="1 1 1"/>
           <!--mesh filename="package://iai_kuka_lwr4_description/meshes/arm_segment_b.stl" scale="1 1 1"/-->
         </geometry>
@@ -157,5 +157,5 @@
         <origin xyz="0 0 0" rpy="0 0 0"/>
         <geometry>
-          <mesh filename="package://iai_kuka_lwr4_description/meshes/arm_segment_a.dae" scale="1 1 1"/>
+          <mesh filename="package://iai_kuka_lwr4_description/meshes/arm_segment_a${color_postfix}.dae" scale="1 1 1"/>
           <!--mesh filename="package://iai_kuka_lwr4_description/meshes/arm_segment_a.stl" scale="1 1 1"/-->
         </geometry>
@@ -201,5 +201,5 @@
         <origin xyz="0 0 0.2" rpy="0 ${M_PI} ${M_PI}"/>
         <geometry>
-          <mesh filename="package://iai_kuka_lwr4_description/meshes/arm_segment_b.dae" scale="1 1 1"/>
+          <mesh filename="package://iai_kuka_lwr4_description/meshes/arm_segment_b${color_postfix}.dae" scale="1 1 1"/>
           <!--mesh filename="package://iai_kuka_lwr4_description/meshes/arm_segment_b.stl" scale="1 1 1"/-->
         </geometry>
@@ -245,5 +245,5 @@
         <origin xyz="0 0 0" rpy="0 0 ${M_PI}"/>
         <geometry name="${prefix}arm_5_geom">
-          <mesh filename="package://iai_kuka_lwr4_description/meshes/arm_segment_last.dae" scale="1 1 1"/>
+          <mesh filename="package://iai_kuka_lwr4_description/meshes/arm_segment_last${color_postfix}.dae" scale="1 1 1"/>
           <!--mesh filename="package://iai_kuka_lwr4_description/meshes/arm_segment_last.stl" scale="1 1 1"/-->
         </geometry>

Commit message: Updating boxy_ur3_test.launch and boxy URDF

File: iai_boxy_description/robots/boxy_description.urdf.xacro (robot description, xacro)
@@ -5,13 +5,14 @@
 	<xacro:include filename="$(find iai_wsg_50_description)/urdf/wsg_50.urdf.xacro"/>
 	<xacro:include filename="$(find iai_kms_40_description)/urdf/kms_40.urdf.xacro"/>
-        <include filename="$(find iai_adapters_description)/urdf/lwr4_cabling_adaptor.urdf.xacro" />
+    <xacro:include filename="$(find iai_adapters_description)/urdf/lwr4_cabling_adaptor.urdf.xacro" />
 	<!--xacro:include filename="$(find iai_boxy_description)/sensors/kinect.urdf.xacro"/-->
 	<xacro:include filename="$(find iai_adapters_description)/urdf/adapter_fwa050_wsg50.urdf.xacro"/>
 	<xacro:include filename="$(find iai_adapters_description)/urdf/adapter_kms40_fwk050.urdf.xacro"/>
-        <xacro:include filename="$(find iai_adapters_description)/urdf/fwk_fwa_050.urdf.xacro"/>
+    <xacro:include filename="$(find iai_adapters_description)/urdf/fwk_fwa_050.urdf.xacro"/>
 	<xacro:include filename="$(find iai_adapters_description)/urdf/adapter_boxy_ur3.urdf.xacro"/>
-        <xacro:include filename="$(find iai_ur_description)/urdf/ur3.urdf.xacro" />
+    <xacro:include filename="$(find iai_ur_description)/urdf/ur3.urdf.xacro" />
 	<xacro:include filename="$(find iai_kinect2_description)/urdf/kinect2.urdf.xacro"/>
 	<xacro:include filename="$(find iai_adapter_iso50_kinect2_description)/urdf/adapter_iso50_kinect2.urdf.xacro"/>
+	<xacro:include filename="$(find boxy_description_urdf)/kinect2_target.urdf.xacro"/>
 	<!-- Property definitions e.g. constants -->
 	<xacro:property name="head_joint_x" value="0.2" />
@@ -24,9 +25,4 @@
 	<xacro:include filename="$(find iai_boxy_base)/robots/base.URDF" />
 	<link name="base_footprint">
-    <inertial>
-      <mass value="1"/>
-      <origin xyz="0 0 0"/>
-      <inertia ixx="0.01" ixy="0" ixz="0" iyy="0.01" iyz="0" izz="0.01"/>
-    </inertial>
     <visual>
       <origin rpy="0 0 0" xyz="0 0 0"/>
@@ -56,5 +52,5 @@
         </adapter_boxy_ur3_xacro>
         <xacro:ur3_robot prefix="neck_" parent="neck_adapter_ur3_frame_out"
-                         joint_limited="false">
+                         joint_limited="true">
           <origin xyz="0.0 0.0 0.0" rpy="0.0 0.0 -${M_PI/2.0}" />
         </xacro:ur3_robot>
@@ -63,9 +59,12 @@
           <origin xyz="0 0 0" rpy="0 0 -1.570795" />
         </adapter_iso50_kinect2_xacro>
+		 <!-- Imaginary joint to determine where Kineckt2 is looking -->
+		<xacro:kinect2_target_xacro parent="neck_tool0" prefix="neck">
+			<pose xyz="0 0 0" rpy="0 0 0" />
+		</xacro:kinect2_target_xacro>
         <!-- /NEW NECK ASSEMBLY -->
         <!-- OLD NEW ASSEMBLY -->
 	<!-- JOINT to connect the base with the pw070 -->
 	<!--joint name="head_joint" type="fixed">
-		<origin xyz="${head_joint_x} ${head_joint_y} ${head_joint_z}" rpy="0 0 0" />
 		<parent link="base_link" />
 		<child link="pw070_base_link" />

Commit message: Modifying UR3_limited URDF limits to improve head behaviour.

File: iai_boxy_description/robots/boxy_description.urdf.xacro (robot description, xacro)
@@ -5,11 +5,11 @@
 	<xacro:include filename="$(find iai_wsg_50_description)/urdf/wsg_50.urdf.xacro"/>
 	<xacro:include filename="$(find iai_kms_40_description)/urdf/kms_40.urdf.xacro"/>
-    <xacro:include filename="$(find iai_adapters_description)/urdf/lwr4_cabling_adaptor.urdf.xacro" />
-	<!--xacro:include filename="$(find iai_boxy_description)/sensors/kinect.urdf.xacro"/-->
+  <xacro:include filename="$(find iai_adapters_description)/urdf/lwr4_cabling_adaptor.urdf.xacro" />
+	<xacro:include filename="$(find iai_kinect_description)/urdf/kinect.urdf.xacro"/>
 	<xacro:include filename="$(find iai_adapters_description)/urdf/adapter_fwa050_wsg50.urdf.xacro"/>
 	<xacro:include filename="$(find iai_adapters_description)/urdf/adapter_kms40_fwk050.urdf.xacro"/>
-    <xacro:include filename="$(find iai_adapters_description)/urdf/fwk_fwa_050.urdf.xacro"/>
+  <xacro:include filename="$(find iai_adapters_description)/urdf/fwk_fwa_050.urdf.xacro"/>
 	<xacro:include filename="$(find iai_adapters_description)/urdf/adapter_boxy_ur3.urdf.xacro"/>
-    <xacro:include filename="$(find iai_ur_description)/urdf/ur3.urdf.xacro" />
+  <xacro:include filename="$(find iai_ur_description)/urdf/ur3.urdf.xacro" />
 	<xacro:include filename="$(find iai_kinect2_description)/urdf/kinect2.urdf.xacro"/>
 	<xacro:include filename="$(find iai_adapter_iso50_kinect2_description)/urdf/adapter_iso50_kinect2.urdf.xacro"/>
@@ -90,8 +90,10 @@
              translation: -0.135394 -0.00764754 1.54755 (xyz)
              quaternion: 0.0177781 0.202257 -0.0472198 0.978032 (xyzw) -->
-        <!--kinect name="shoulder_kinect" parent="base_link">
-          <origin xyz="-0.135394 -0.00764754 1.54755"
-                  rpy="0.01708077682636155 0.4085798647123734 -0.09294704527264909"/>
-       </kinect-->
+        <kinect name="shoulder_kinect" parent="base_link">
+          <!--<origin xyz="-0.135394 -0.00764754 1.54755"
+                  rpy="0.01708077682636155 0.4085798647123734 -0.09294704527264909"/> -->
+					<origin xyz="0.0405394 -0.52064754 1.47001"
+                  rpy="0.01708077682636155 0.0085798647123734 -0.00929470452726490"/>
+       </kinect>
 	<!-- JOINT to connect the base with the torso -->
 	<joint name="torso_joint" type="fixed">

File: iai_boxy_torso/robots/torso.URDF (robot description, URDF)
Before this commit: robot torso, 4 links, 3 joints
Joints:
- joint triangle_base_joint: origin xyz=0.0786889663592487 0.0986351579738104 1.002352096493862 rpy=4.70695928 6.28217403836 1.56327975371 -> xyz=0.0786889663592487 0.0986351579738104 0.996332096493862 rpy=4.70695928 6.28217403836 1.56327975371

File: iai_kinect_description/urdf/kinect.urdf.xacro (robot description, xacro)
@@ -27,5 +27,5 @@
       </collision>
     </link>
-    <joint name="${name}_rgb_joint" type="fixed">
+    <!--<joint name="${name}_rgb_joint" type="fixed">
       <origin xyz="0.0 -0.045 0.0" rpy="0.0 0.0 0.0"/>
       <parent link="${name}_link"/>
@@ -50,5 +50,5 @@
       <child link="${name}_depth_optical_frame"/>
     </joint>
-    <link name="${name}_depth_optical_frame"/>
+    <link name="${name}_depth_optical_frame"/>-->
   </xacro:macro>
 </robot>

File: iai_ur_description/urdf/ur3.urdf.xacro (robot description, xacro)
@@ -85,5 +85,6 @@
       </xacro:unless>
       <xacro:if value="${joint_limited}">
-        <limit lower="${-pi}" upper="${pi}" effort="330.0" velocity="2.16"/>
+        <!--limit lower="${-pi}" upper="${pi}" effort="330.0" velocity="2.16"/-->
+				<limit lower="${-1.5*pi}" upper="${1.5*pi}" effort="330.0" velocity="2.16"/>
       </xacro:if>
       <dynamics damping="0.0" friction="0.0"/>

Commit message: Adding collision objects to boxy URDF, simplifying collision meshes of UR3

File: iai_boxy_description/robots/boxy_description.urdf.xacro (robot description, xacro)
@@ -147,4 +147,49 @@
     </collision>
   </link>
+    <!-- Box that limits the position of the head while planning -->
+			<link name="limit_box" >
+			  <visual>
+				  <origin rpy="0 0 0" xyz="0.25 -0.2 1.35"/>
+					<geometry>
+						<box size="0.01 0.01 0.01"/>
+					</geometry>
+					<material name="box_color">
+						<color rgba="0.2 0.2 0.2 1"/>
+					</material>
+			 	</visual>
+			 	<collision>
+        	<origin rpy="0 0 0" xyz="0.25 -0.2 1.35"/>
+        	<geometry>
+         		<box size="0.4 0.35 0.1"/>
+        	</geometry>
+      	</collision>
+		  </link>
+			<joint name="fixed_box" type="fixed">
+                <origin xyz="0.0 0.0 0.0" rpy="0.0 0.0 0.0"/>
+                <parent link="base_link" />
+                <child link="limit_box" />
+      </joint>
+			<link name="limit_box2" >
+			  <visual>
+				  <origin rpy="0 0 0" xyz="-0.2 -0.2 1.55"/>
+					<geometry>
+						<box size="0.01 0.01 0.01"/>
+					</geometry>
+					<material name="box_color">
+						<color rgba="0.2 0.2 0.2 1"/>
+					</material>
+			 	</visual>
+			 	<collision>
+        	<origin rpy="0 0 0" xyz="-0.2 -0.2 1.55"/>
+        	<geometry>
+         		<box size="0.25 0.40 0.15"/>
+        	</geometry>
+      	</collision>
+		  </link>
+			<joint name="fixed_box2" type="fixed">
+                <origin xyz="0.0 0.0 0.0" rpy="0.0 0.0 0.0"/>
+                <parent link="base_link" />
+                <child link="limit_box2" />
+      </joint>
         <!-- JOINT to define base_footprint -->
         <joint name="left_wrist_optical_joint_x" type="fixed">

File: iai_kinect2_look_target/urdf/kinect2_target.urdf.xacro (robot description, xacro)
@@ -23,4 +23,10 @@
 				</material>
 			</visual>
+			<collision>
+        <origin rpy="0 0 0" xyz="0 0 ${Length/2+.03}"/>
+        <geometry>
+          <cylinder length="${Length}" radius="${R}"/>
+        </geometry>
+      </collision>
 		</link>
 <!-- Joints at the end of the target, to allow any orientation -->

File: iai_kinect_description/urdf/kinect.urdf.xacro (robot description, xacro)
@@ -23,5 +23,5 @@
         <origin xyz="-0.05 -0.17 -0.02" rpy="${M_PI/2.0} 0 ${M_PI/2.0}"/>
         <geometry>
-          <mesh filename="package://iai_kinect_description/meshes/68-04546_Kinect_Sensor--coarse.STL" scale="0.001 0.001 0.001" />
+          <mesh filename="package://iai_kinect_description/meshes/68-04546_Kinect_Sensor--coarse_simple.STL" scale="0.001 0.001 0.001" />
         </geometry>
       </collision>

File: iai_ur_description/urdf/ur3.urdf.xacro (robot description, xacro)
@@ -117,5 +117,5 @@
       </xacro:unless>
       <xacro:if value="${joint_limited}">
-        <limit lower="${-pi}" upper="${pi}" effort="330.0" velocity="2.16"/>
+        <limit lower="${-1.2 * pi}" upper="${1.2 * pi}" effort="330.0" velocity="2.16"/>
       </xacro:if>
       <dynamics damping="0.0" friction="0.0"/>
@@ -148,5 +148,5 @@
       </xacro:unless>
       <xacro:if value="${joint_limited}">
-        <limit lower="${-pi}" upper="${pi}" effort="150.0" velocity="3.15"/>
+        <limit lower="${-1.2 * pi}" upper="${1.2 * pi}" effort="150.0" velocity="3.15"/>
       </xacro:if>
       <dynamics damping="0.0" friction="0.0"/>
@@ -179,5 +179,5 @@
       </xacro:unless>
       <xacro:if value="${joint_limited}">
-        <limit lower="${-pi}" upper="${pi}" effort="54.0" velocity="3.2"/>
+        <limit lower="${-1.3 * pi}" upper="${1.3 * pi}" effort="54.0" velocity="3.2"/>
       </xacro:if>
       <dynamics damping="0.0" friction="0.0"/>
@@ -210,5 +210,5 @@
       </xacro:unless>
       <xacro:if value="${joint_limited}">
-        <limit lower="${-pi}" upper="${pi}" effort="54.0" velocity="3.2"/>
+        <limit lower="${-1.3 * pi}" upper="${1.3 * pi}" effort="54.0" velocity="3.2"/>
       </xacro:if>
       <dynamics damping="0.0" friction="0.0"/>
@@ -241,6 +241,5 @@
       </xacro:unless>
       <xacro:if value="${joint_limited}">
-        <limit lower="${-pi}" upper="${pi}" effort="54.0" velocity="3.2"/>
-				<limit lower="${-1.5*pi}" upper="${1.5*pi}" effort="54.0" velocity="3.2"/>
+				<limit lower="${-1.5 * pi}" upper="${1.5 * pi}" effort="54.0" velocity="3.2"/>
       </xacro:if>
       <dynamics damping="0.0" friction="0.0"/>

Commit message: boxy_description: changes due to hand-eye calibration

File: iai_boxy_description/robots/boxy_description.urdf.xacro (robot description, xacro)
@@ -83,5 +83,8 @@
         And includes the fixed joint to place the kinect on the pw070  -->
         <kinect2_xacro parent="neck_adapter_iso50_kinect2_frame_out" prefix="head_mount">
-		<origin xyz="-0.02 0.10 0.02" rpy="-1.570795 0 1.570795" />
+                <!-- From CAD -->
+		<!--origin xyz="-0.02 0.10 0.02" rpy="-1.570795 0 1.570795" /-->
+                <!-- From Halcon calibration on 20160902 -->
+		<origin xyz="-0.031284 0.098627 0.023544" rpy="4.728550 6.279385 1.578295"/>
         </kinect2_xacro>
         <!-- shoulder kinect -->
@@ -106,5 +109,8 @@
         <!--FIXME: triangle_left_arm_link should be rotated, and not the origin of the arm (which right now is calib_left_arm_base_link -->
 	<kuka_lwr_arm parent="triangle_left_arm_link" prefix="left_" color_postfix="">
-          <origin xyz="0 0 0" rpy="0 0 1.047198"/>
+          <!-- From CAD -->
+          <!--origin xyz="0 0 0" rpy="0 0 1.047198"/-->
+          <!-- from calibration on 20160903 -->
+          <origin xyz="-0.006185 0.004080 -0.010726" rpy="6.276354 6.281653 1.074679"/>
 	</kuka_lwr_arm>
         <lwr4_cabling_adaptor parent="left_arm_flange_link" prefix="left_arm_">

Commit message: Change virtual links coming out of the kinect2 for planning to use kinect2_rgb_optical_frame instead of some frame of the arm

File: iai_boxy_description/robots/boxy_description.urdf.xacro (robot description, xacro)
@@ -60,5 +60,5 @@
         </adapter_iso50_kinect2_xacro>
 		 <!-- Imaginary joint to determine where Kineckt2 is looking -->
-		<xacro:kinect2_target_xacro parent="neck_tool0" prefix="neck">
+		<xacro:kinect2_target_xacro parent="head_mount_kinect2_rgb_optical_frame" prefix="neck">
 			<pose xyz="0 0 0" rpy="0 0 0" />
 		</xacro:kinect2_target_xacro>

File: iai_kinect2_look_target/urdf/kinect2_target.urdf.xacro (robot description, xacro)
@@ -9,6 +9,6 @@
 			<parent link="${parent}"/>
 			<child link="${prefix}_look_target"/>
-			<limit effort="1000.0" lower="0" upper="1.5" velocity="0.5"/>
-			<origin xyz="0 0.01 0" rpy="-1.5708 0 0" />
+			<limit effort="1000.0" lower="0" upper="3.5" velocity="0.5"/>
+			<origin xyz="0 0.0 0.2" rpy="0 0 0" />
 			<axis xyz="0 0 1" />
 		</joint>
@@ -32,5 +32,5 @@
 		<link name="${prefix}_obstacle">
 			<visual>
-				<origin rpy="0 1.5708 0" xyz="0 0 0.1"/>
+				<origin rpy="0 0.0 0" xyz="0 0 0.1"/>
 				<geometry>
 					<mesh filename="package://iai_kinect2_look_target/meshes/Cilinder.stl" scale="0.0001 0.0001 0.0001" />
@@ -41,5 +41,5 @@
 			</visual>
 			<collision>
-        <origin rpy="0 1.5707 0" xyz="0 0 0.1"/>
+        <origin rpy="0 0.0 0" xyz="0 0 0.1"/>
         <geometry>
           <mesh filename="package://iai_kinect2_look_target/meshes/Cilinder.stl" scale="0.01 0.01 0.01" />
@@ -60,5 +60,5 @@
 			<parent link="${parent}"/>
 			<child link="${prefix}_obstacle"/>
-			<origin xyz="0 0.01 0" rpy="-1.5708 0 0" />
+			<origin xyz="0 0.0 0.01" rpy="0 0 0" />
 			<axis xyz="0 0 1" />
 		</joint>

Commit message: Modelled odometry of Boxy as additional 3 joints.

File: iai_boxy_description/robots/boxy_description.urdf.xacro (robot description, xacro)
@@ -24,4 +24,35 @@
 	<!-- /Property definitions e.g. constants -->
 	<xacro:include filename="$(find iai_boxy_base)/robots/base.URDF" />
+        <!-- virtual joints to model odometry -->
+        <link name="odom" />
+        <joint name="odom_x_joint" type="prismatic">
+          <parent link="odom"/>
+          <child link="odom_x_frame"/>
+          <axis xyz="1 0 0"/>
+          <!-- limits chosen heuristically
+               velocity: slow walking speed is 3-4km/hour ~= 1m/s
+               effort: reach max speed within 1s, Boxy has a mass of 200kg, so Fmax=200kg*1m/s2 -->
+          <limit velocity="1" effort="200"/>
+        </joint>
+        <link name="odom_x_frame" />
+        <joint name="odom_y_joint" type="prismatic">
+          <parent link="odom_x_frame"/>
+          <child link="odom_y_frame"/>
+          <axis xyz="0 1 0"/>
+          <!-- limits chosen heuristically
+               velocity: slow walking speed is 3-4km/hour ~= 1m/s
+               effort: reach max speed within 1s, Boxy has a mass of 200kg, so Fmax=200kg*1m/s2 -->
+          <limit velocity="1" effort="200"/>
+        </joint>
+        <link name="odom_y_frame" />
+        <joint name="odom_z_joint" type="revolute">
+          <parent link="odom_y_frame"/>
+          <child link="base_footprint"/>
+          <axis xyz="0 0 1"/>
+          <!-- limits chosen heuristically
+               velocity: one slow complete turn around in 5-6s, so 6.2rad/6s ~= 1rad/s
+               effort: reach max speed within 1s, Boxy has a mass of 200kg and a diagonale of 1m, so Fmax=200kg*1m*1m/s2 -->
+          <limit velocity="1" effort="200"/>
+        </joint>
 	<link name="base_footprint">
     <visual>

Commit message: Fix: Made sure that boxy's odom joints are at least quasi-limited.

File: iai_boxy_description/robots/boxy_description.urdf.xacro (robot description, xacro)
@@ -31,7 +31,8 @@
           <axis xyz="1 0 0"/>
           <!-- limits chosen heuristically
+               lower/upper: +-1km to create a quasi limitless prismatic joint
                velocity: slow walking speed is 3-4km/hour ~= 1m/s
                effort: reach max speed within 1s, Boxy has a mass of 200kg, so Fmax=200kg*1m/s2 -->
-          <limit velocity="1" effort="200"/>
+          <limit lower="-1000" upper="1000" velocity="1" effort="200"/>
         </joint>
         <link name="odom_x_frame" />
@@ -41,10 +42,11 @@
           <axis xyz="0 1 0"/>
           <!-- limits chosen heuristically
+               lower/upper: +-1km to create a quasi limitless prismatic joint
                velocity: slow walking speed is 3-4km/hour ~= 1m/s
                effort: reach max speed within 1s, Boxy has a mass of 200kg, so Fmax=200kg*1m/s2 -->
-          <limit velocity="1" effort="200"/>
+          <limit lower="-1000" upper="1000" velocity="1" effort="200"/>
         </joint>
         <link name="odom_y_frame" />
-        <joint name="odom_z_joint" type="revolute">
+        <joint name="odom_z_joint" type="continuous">
           <parent link="odom_y_frame"/>
           <child link="base_footprint"/>
