Commit message: Remove neck limiting boxes from Boxy's URDF, adding them to boxy_description_vision_target

File: iai_boxy_description/robots/boxy_description_vision_target.urdf.xacro (robot description, xacro)
@@ -4,4 +4,5 @@
   <xacro:include filename="$(find iai_boxy_description)/urdf/boxy_description.urdf.xacro"/>
   <xacro:include filename="$(find iai_kinect2_look_target)/urdf/kinect2_target.urdf.xacro"/>
+  <xacro:include filename="$(find iai_kinect2_look_target)/urdf/limit_boxes.urdf.xacro"/>
   <!-- actual robot -->
   <boxy/>
@@ -10,3 +11,7 @@
     <pose xyz="0 0 0" rpy="0 0 0" />
   </xacro:kinect2_target_xacro>
+  <!-- Limit collision boxes to limit the Kineckt2 position -->
+  <xacro:limit_boxes_xacro parent="base_link" prefix="neck_collision">
+    <pose xyz="0 0 0" rpy="0 0 0" />
+  </xacro:limit_boxes_xacro>
 </robot>

File: iai_boxy_description/urdf/boxy_description.urdf.xacro (robot description, xacro)
@@ -182,49 +182,4 @@
     </collision>
   </link>
-    <!-- Box that limits the position of the head while planning -->
-			<link name="limit_box" >
-			  <visual>
-				  <origin rpy="0 0 0" xyz="0.25 -0.2 1.35"/>
-					<geometry>
-						<box size="0.01 0.01 0.01"/>
-					</geometry>
-					<material name="box_color">
-						<color rgba="0.2 0.2 0.2 1"/>
-					</material>
-			 	</visual>
-			 	<collision>
-        	<origin rpy="0 0 0" xyz="0.25 -0.2 1.35"/>
-        	<geometry>
-         		<box size="0.4 0.35 0.1"/>
-        	</geometry>
-      	</collision>
-		  </link>
-			<joint name="fixed_box" type="fixed">
-                <origin xyz="0.0 0.0 0.0" rpy="0.0 0.0 0.0"/>
-                <parent link="base_link" />
-                <child link="limit_box" />
-      </joint>
-			<link name="limit_box2" >
-			  <visual>
-				  <origin rpy="0 0 0" xyz="-0.2 -0.2 1.55"/>
-					<geometry>
-						<box size="0.01 0.01 0.01"/>
-					</geometry>
-					<material name="box_color">
-						<color rgba="0.2 0.2 0.2 1"/>
-					</material>
-			 	</visual>
-			 	<collision>
-        	<origin rpy="0 0 0" xyz="-0.2 -0.2 1.55"/>
-        	<geometry>
-         		<box size="0.25 0.40 0.15"/>
-        	</geometry>
-      	</collision>
-		  </link>
-			<joint name="fixed_box2" type="fixed">
-                <origin xyz="0.0 0.0 0.0" rpy="0.0 0.0 0.0"/>
-                <parent link="base_link" />
-                <child link="limit_box2" />
-      </joint>
         <!-- JOINT to define base_footprint -->
         <joint name="left_wrist_optical_joint_x" type="fixed">
