Commit message: Change the initial position and limits for the torso joint

File: iai_boxy_torso/robots/torso.URDF (robot description, URDF)
Before this commit: robot torso, 4 links, 3 joints
Joints:
- joint triangle_base_joint: limit lower=0 upper=0.636 effort=1000 velocity=2 -> lower=-0.586 upper=0 effort=1000 velocity=2; origin xyz=0.1 0.0175 0.00062489 rpy=-1.5708 -5.5511E-17 1.5708 -> xyz=0.1 0.0175 0.58662489 rpy=-1.5708 -5.5511E-17 1.5708

Commit message: Limit the speed of the torso in the URDF to 2cm/s

File: iai_boxy_torso/robots/torso.URDF (robot description, URDF)
Before this commit: robot torso, 4 links, 3 joints
Joints:
- joint triangle_base_joint: limit lower=-0.586 upper=0 effort=1000 velocity=2 -> lower=-0.586 upper=0 effort=0 velocity=0.02

Commit message: Correcting the initial position of triangle base (90.6 to 102.8 cm)

File: iai_boxy_torso/robots/torso.URDF (robot description, URDF)
Before this commit: robot torso, 4 links, 3 joints
Joints:
- joint triangle_base_joint: origin xyz=0.0786889663592487 0.0986351579738104 0.906352096493862 rpy=4.70695928 6.28217403836 1.56327975371 -> xyz=0.0786889663592487 0.0986351579738104 1.028352096493862 rpy=4.70695928 6.28217403836 1.56327975371

Commit message: Correcting the initial position of triangle base (90.6 to 100.2 cm)

File: iai_boxy_torso/robots/torso.URDF (robot description, URDF)
Before this commit: robot torso, 4 links, 3 joints
Joints:
- joint triangle_base_joint: origin xyz=0.0786889663592487 0.0986351579738104 1.028352096493862 rpy=4.70695928 6.28217403836 1.56327975371 -> xyz=0.0786889663592487 0.0986351579738104 1.002352096493862 rpy=4.70695928 6.28217403836 1.56327975371

Commit message: Changed original of triangle_base_joint to have translation along +Z and not -Y. Circumvents a problem of giskard parsing urdfs with kdl_parser.

File: iai_boxy_torso/robots/torso.URDF (robot description, URDF)
Before this commit: robot torso, 4 links, 3 joints
Joints:
- joint triangle_base_joint: axis 0 -1 0 -> 0 0 1; origin xyz=0.0786889663592487 0.0986351579738104 0.996332096493862 rpy=4.70695928 6.28217403836 1.56327975371 -> xyz=0.0786889663592487 0.0986351579738104 0.996332096493862 rpy=0 0 0
- joint triangle_left_arm_joint: origin xyz=-0.239507442352261 -0.181209704131733 -0.137000000000002 rpy=2.61799387796333 -1.5707963267949 0 -> xyz=0.134209 -0.240707 0.181709 rpy=1.046186267441739 0.005429697608281147 3.1340705895651766
- joint triangle_right_arm_joint: origin xyz=-0.365488160465715 -0.181209539931436 -0.137 rpy=2.61799387801966 1.5707963267949 0 -> xyz=0.133262 -0.366684 0.181581 rpy=1.0482088349514576 -0.00542969760828114 -0.0075220640246236
