Commit message: Adding URDF of the virtual link of the Kinect2

File: iai_kinect2_look_target/urdf/kinect2_target.urdf.xacro (robot description, xacro)
@@ -1,47 +1,51 @@
 <?xml version="1.0"?>
-<!-- This is a hand-made URDF XACRO file for pointing at the target of the Microsoft Kinect-2 sensor (Xbox ONE) -->
+<!-- This is a hand-made URDF XACRO file for simulating the position where the Microsoft Kinect-2 sensor is looking -->
 <!-- Copyright Universitaet Bremen - Instititute for Artificial Intelligence. Author: Minerva Vargas -->
 <!-- License: GPLv3+ -->
-<robot xmlns:xacro="http://www.ros.org/wiki/xacro" name="joint_target">
-<!-- This is an imaginary joint at the end of the Kinect2 that points at the target, with any orientation -->
- <xacro:macro name="kinect2_xacro">
-  <link name="target_base" />
-  <link name="target_3" />
-  <link name="target_2">
-	<visual>
-    	  <geometry>
-    	    <cylinder length="0.4" radius="0.1"/>
-    	  </geometry>
-    	  <material name="blue">
-    	    <color rgba="0 0 .8 1"/>
-    	  </material>
-    </visual>
-  </link>
-  <joint name="joint1" type="revolute">
-    <parent link="target_base"/>
-    <child link="target_2"/>
-	<limit effort="1000.0" lower="0" upper="3" velocity="0.5"/>
-	<origin xyz="0 0 0" rpy="0 0 1.57" />
-	<axis xyz="0 0 1" />
-  </joint>
+<robot xmlns:xacro="http://ros.org/wiki/xacro" name="kinect2_target">
+	<xacro:macro name="kinect2_target_xacro" params ="prefix parent *origin">
+		<joint name="${prefix}_joint_end" type="prismatic">
+			<xacro:insert_block name="origin"/>
+			<parent link="${parent}"/>
+			<child link="${prefix}_look_target"/>
+			<limit effort="1000.0" lower="0" upper="1.5" velocity="0.5"/>
+			<origin xyz="0 0.01 0" rpy="-1.5708 0 0" />
+			<axis xyz="0 0 1" />
+		</joint>
+		<link name="${prefix}_look_target">
+			<visual>
+				<origin rpy="0 0 0" xyz="0 0 ${Length/2+.03}"/>
+				<geometry>
+					<cylinder length="${Length}" radius="${R}"/>
+				</geometry>
+				<material name="blue">
+					<color rgba="0.2 0.2 0.7 1"/>
+				</material>
+			</visual>
+		</link>
 <!-- Joints at the end of the target, to allow any orientation -->
-  <joint name="head1" type="continuous">
-    <parent link="target_2"/>
-    <child link="target_3"/>
-	<origin xyz="0 0 0" rpy="0 0 0" />
-	<axis xyz="0 0 1" />
-  </joint>
-  <joint name="head2" type="continuous">
-    <parent link="target_2"/>
-    <child link="target_3"/>
-	<origin xyz="0 0 0" rpy="0 0 0" />
-	<axis xyz="0 1 0" />
-  </joint>
-  <joint name="head3" type="continuous">
-    <parent link="target_2"/>
-    <child link="target_3"/>
-	<origin xyz="0 0 0" rpy="0 0 0" />
-	<axis xyz="1 0 0" />
-  </joint>
- </xacro:macro>
+		<joint name="head1" type="continuous">
+			<parent link="${prefix}_look_target"/>
+			<child link="${prefix}_look_target_2"/>
+			<origin xyz="0 0 0" rpy="0 0 0" />
+			<axis xyz="0 0 1" />
+		</joint>
+		<joint name="head2" type="continuous">
+			<parent link="${prefix}_look_target_2"/>
+			<child link="${prefix}_look_target_3"/>
+			<origin xyz="0 0 0" rpy="0 0 0" />
+			<axis xyz="0 1 0" />
+		</joint>
+		<joint name="head3" type="continuous">
+			<parent link="${prefix}_look_target_3"/>
+			<child link="${prefix}_look_target_4"/>
+			<origin xyz="0 0 0" rpy="0 0 0" />
+			<axis xyz="1 0 0" />
+		</joint>
+		<link name="${prefix}_look_target_2"/>
+		<link name="${prefix}_look_target_3"/>
+		<link name="${prefix}_look_target_4"/>
+	</xacro:macro>
+	<xacro:property name="R" value="0.03" />
+	<xacro:property name="Length" value="0.35" />
 </robot>

Commit message: Adding virtual link in front of kinect2

File: iai_kinect2_look_target/urdf/kinect2_target.urdf.xacro (robot description, xacro)
@@ -30,4 +30,21 @@
       </collision>
 		</link>
+		<link name="${prefix}_obstacle">
+			<visual>
+				<origin rpy="0 1.5708 0" xyz="0 0 0.1"/>
+				<geometry>
+					<mesh filename="package://iai_kinect2_look_target/meshes/Cilinder.stl" scale="0.01 0.01 0.01" />
+				</geometry>
+				<material name="blue">
+					<color rgba="0.2 0.2 0.7 1"/>
+				</material>
+			</visual>
+			<collision>
+        <origin rpy="0 1.5707 0" xyz="0 0 0.1"/>
+        <geometry>
+          <mesh filename="package://iai_kinect2_look_target/meshes/Cilinder.stl" scale="0.01 0.01 0.01" />
+        </geometry>
+      </collision>
+		</link>
 <!-- Joints at the end of the target, to allow any orientation -->
 		<joint name="head1" type="continuous">
@@ -35,4 +52,10 @@
 			<child link="${prefix}_look_target_2"/>
 			<origin xyz="0 0 0" rpy="0 0 0" />
+			<axis xyz="0 0 1" />
+		</joint>
+		<joint name="head" type="fixed">
+			<parent link="${parent}"/>
+			<child link="${prefix}_obstacle"/>
+			<origin xyz="0 0.01 0" rpy="-1.5708 0 0" />
 			<axis xyz="0 0 1" />
 		</joint>
@@ -53,5 +76,5 @@
 		<link name="${prefix}_look_target_4"/>
 	</xacro:macro>
-	<xacro:property name="R" value="0.03" />
+	<xacro:property name="R" value="0.028" />
 	<xacro:property name="Length" value="0.35" />
 </robot>

Commit message: Hidding kinect virtual link

File: iai_kinect2_look_target/urdf/kinect2_target.urdf.xacro (robot description, xacro)
@@ -14,5 +14,5 @@
 		</joint>
 		<link name="${prefix}_look_target">
-			<visual>
+			<!--<visual>
 				<origin rpy="0 0 0" xyz="0 0 ${Length/2+.03}"/>
 				<geometry>
@@ -22,5 +22,5 @@
 					<color rgba="0.2 0.2 0.7 1"/>
 				</material>
-			</visual>
+			</visual>-->
 			<collision>
         <origin rpy="0 0 0" xyz="0 0 ${Length/2+.03}"/>
@@ -31,5 +31,5 @@
 		</link>
 		<link name="${prefix}_obstacle">
-			<visual>
+			<!--<visual>
 				<origin rpy="0 1.5708 0" xyz="0 0 0.1"/>
 				<geometry>
@@ -39,5 +39,5 @@
 					<color rgba="0.2 0.2 0.7 1"/>
 				</material>
-			</visual>
+			</visual>-->
 			<collision>
         <origin rpy="0 1.5707 0" xyz="0 0 0.1"/>

Commit message: Color of kinect virtual link

File: iai_kinect2_look_target/urdf/kinect2_target.urdf.xacro (robot description, xacro)
@@ -28,4 +28,7 @@
           <cylinder length="${Length}" radius="${R}"/>
         </geometry>
+				<material name="blue">
+					<color rgba="0.2 0.2 0.7 1"/>
+				</material>
       </collision>
 		</link>
@@ -45,4 +48,7 @@
           <mesh filename="package://iai_kinect2_look_target/meshes/Cilinder.stl" scale="0.01 0.01 0.01" />
         </geometry>
+				<material name="blue">
+					<color rgba="0.2 0.2 0.5 1"/>
+				</material>
       </collision>
 		</link>

Commit message: Color of kinect virtual link

File: iai_kinect2_look_target/urdf/kinect2_target.urdf.xacro (robot description, xacro)
@@ -14,13 +14,13 @@
 		</joint>
 		<link name="${prefix}_look_target">
-			<!--<visual>
+			<visual>
 				<origin rpy="0 0 0" xyz="0 0 ${Length/2+.03}"/>
 				<geometry>
-					<cylinder length="${Length}" radius="${R}"/>
+					<cylinder length="0.01" radius="0.01"/>
 				</geometry>
 				<material name="blue">
 					<color rgba="0.2 0.2 0.7 1"/>
 				</material>
-			</visual>-->
+			</visual>
 			<collision>
         <origin rpy="0 0 0" xyz="0 0 ${Length/2+.03}"/>
@@ -28,19 +28,13 @@
           <cylinder length="${Length}" radius="${R}"/>
         </geometry>
+      </collision>
+		</link>
+		<link name="${prefix}_obstacle">
+			<visual>
+				<origin rpy="0 1.5708 0" xyz="0 0 0.1"/>
 				<material name="blue">
 					<color rgba="0.2 0.2 0.7 1"/>
 				</material>
-      </collision>
-		</link>
-		<link name="${prefix}_obstacle">
-			<!--<visual>
-				<origin rpy="0 1.5708 0" xyz="0 0 0.1"/>
-				<geometry>
-					<mesh filename="package://iai_kinect2_look_target/meshes/Cilinder.stl" scale="0.01 0.01 0.01" />
-				</geometry>
-				<material name="blue">
-					<color rgba="0.2 0.2 0.7 1"/>
-				</material>
-			</visual>-->
+			</visual>
 			<collision>
         <origin rpy="0 1.5707 0" xyz="0 0 0.1"/>

Commit message: Correcting kinect virtual link

File: iai_kinect2_look_target/urdf/kinect2_target.urdf.xacro (robot description, xacro)
@@ -17,5 +17,5 @@
 				<origin rpy="0 0 0" xyz="0 0 ${Length/2+.03}"/>
 				<geometry>
-					<cylinder length="0.01" radius="0.01"/>
+					<cylinder length="0.001" radius="0.001"/>
 				</geometry>
 				<material name="blue">
@@ -33,4 +33,7 @@
 			<visual>
 				<origin rpy="0 1.5708 0" xyz="0 0 0.1"/>
+				<geometry>
+					<mesh filename="package://iai_kinect2_look_target/meshes/Cilinder.stl" scale="0.0001 0.0001 0.0001" />
+				</geometry>
 				<material name="blue">
 					<color rgba="0.2 0.2 0.7 1"/>

Commit message: Correcting orientation and size of dummy link.

File: iai_kinect2_look_target/urdf/kinect2_target.urdf.xacro (robot description, xacro)
@@ -24,5 +24,5 @@
 			</visual>
 			<collision>
-        <origin rpy="0 0 0" xyz="0 0 ${Length/2+.03}"/>
+        <origin rpy="0 0 0" xyz="0 0 0.02"/>
         <geometry>
           <cylinder length="${Length}" radius="${R}"/>
@@ -41,5 +41,5 @@
 			</visual>
 			<collision>
-        <origin rpy="0 0.0 0" xyz="0 0 0.1"/>
+        <origin rpy="0 1.5708 0" xyz="0 0 0.1"/>
         <geometry>
           <mesh filename="package://iai_kinect2_look_target/meshes/Cilinder.stl" scale="0.01 0.01 0.01" />
@@ -79,5 +79,5 @@
 		<link name="${prefix}_look_target_4"/>
 	</xacro:macro>
-	<xacro:property name="R" value="0.028" />
+	<xacro:property name="R" value="0.022" />
 	<xacro:property name="Length" value="0.35" />
 </robot>
