Commit message: Add collision mesh for the adapter of the kinect2 to the ur3

File: iai_adapter_iso50_kinect2_description/urdf/adapter_iso50_kinect2.urdf.xacro (robot description, xacro)
@@ -18,4 +18,10 @@
         <material name="Grey"/>
       </visual>
+      <collision>
+        <origin xyz="0 0 0" rpy="0 0 0" />
+        <geometry>
+          <mesh filename="package://iai_adapter_iso50_kinect2_description/meshes/adapter_iso50_kinect2.stl" scale="1 1 1" />
+        </geometry>
+      </collision>
     </link>
     <!-- Empty link just to get the frame out -->

Commit message: Add xacro: tags to the xacro files

File: iai_adapter_iso50_kinect2_description/urdf/adapter_iso50_kinect2.urdf.xacro (robot description, xacro)
@@ -5,5 +5,5 @@
     <!-- Joint connecting the parent to our frame_in -->
     <joint name="${prefix}_adapter_iso50_kinect2_joint" type="fixed">
-      <insert_block name="origin"/>
+      <xacro:insert_block name="origin"/>
       <parent link="${parent}"/>
       <child link="${prefix}_adapter_iso50_kinect2_frame_in"/>

File: iai_adapters_description/robots/lwr4_cabling_adaptor.urdf.xacro (robot description, xacro)
@@ -1,5 +1,5 @@
 <?xml version="1.0"?>
 <robot name="lwr4_cabling_adaptor">
-  <include filename="$(find iai_adapters_description)/urdf/lwr4_cabling_adaptor.urdf.xacro" />
+  <xacro:include filename="$(find iai_adapters_description)/urdf/lwr4_cabling_adaptor.urdf.xacro" />
   <link name="base_link"/>
   <lwr4_cabling_adaptor parent="base_link" prefix="">

File: iai_adapters_description/urdf/adapter_boxy_ur3.urdf.xacro (robot description, xacro)
@@ -6,5 +6,5 @@
     <!-- Joint connecting the parent to our frame_in -->
     <joint name="${prefix}adapter_ur3_in_joint" type="fixed">
-      <insert_block name="origin"/>
+      <xacro:insert_block name="origin"/>
       <parent link="${parent}"/>
       <child link="${prefix}adapter_ur3_frame_in"/>

File: iai_adapters_description/urdf/adapter_fwa050_wsg50.urdf.xacro (robot description, xacro)
@@ -5,5 +5,5 @@
     <!-- Joint connecting the parent to our frame_in -->
     <joint name="${prefix}_adapter_fwa050_wsg50_in_joint" type="fixed">
-      <insert_block name="origin"/>
+      <xacro:insert_block name="origin"/>
       <parent link="${parent}"/>
       <child link="${prefix}_adapter_fwa050_wsg50_frame_in"/>

File: iai_adapters_description/urdf/adapter_kms40_fwk050.urdf.xacro (robot description, xacro)
@@ -5,5 +5,5 @@
     <!-- Joint connecting the parent to our frame_in -->
     <joint name="${prefix}_adapter_kms40_fwk050_in_joint" type="fixed">
-      <insert_block name="origin"/>
+      <xacro:insert_block name="origin"/>
       <parent link="${parent}"/>
       <child link="${prefix}_adapter_kms40_fwk050_frame_in"/>

File: iai_adapters_description/urdf/fwk_fwa_050.urdf.xacro (robot description, xacro)
@@ -5,5 +5,5 @@
     <!-- Joint connecting the parent to our frame_in -->
     <joint name="${prefix}_fwk_fwa_050_in_joint" type="fixed">
-      <insert_block name="origin"/>
+      <xacro:insert_block name="origin"/>
       <parent link="${parent}"/>
       <child link="${prefix}_fwk_fwa_050_frame_in"/>

File: iai_adapters_description/urdf/lwr4_cabling_adaptor.urdf.xacro (robot description, xacro)
@@ -5,5 +5,5 @@
   <xacro:macro name="lwr4_cabling_adaptor" params="prefix parent *origin">
     <joint name="${prefix}arm_cabling_adaptor_joint" type="fixed">
-      <insert_block name="origin" />
+      <xacro:insert_block name="origin" />
       <!--origin xyz="0 0 0.01" rpy="0 0 0"/-->  <!-- This places the link at the end of the plate (frame_out) -->
       <parent link="${parent}"/>

File: iai_kinect2_description/urdf/kinect2.urdf.xacro (robot description, xacro)
@@ -10,5 +10,5 @@
     <!-- Joint connecting the parent to our frame_in -->
     <joint name="${prefix}_kinect2_in_joint" type="fixed">
-      <insert_block name="origin"/>
+      <xacro:insert_block name="origin"/>
       <parent link="${parent}"/>
       <child link="${prefix}_kinect2_rgb_optical_frame"/>

File: iai_kinect_description/urdf/kinect.urdf.xacro (robot description, xacro)
@@ -3,5 +3,5 @@
   <xacro:macro name="kinect" params="name parent *origin">
     <joint name="${name}_joint" type="fixed">
-      <insert_block name="origin"/>
+      <xacro:insert_block name="origin"/>
       <parent link="${parent}"/>
       <child link="${name}_link" />

File: iai_kms_40_description/urdf/kms_40.urdf.xacro (robot description, xacro)
@@ -5,5 +5,5 @@
     <!-- Joint connecting the parent to our frame_in -->
     <joint name="${prefix}_adapter_iso50_kms40_joint" type="fixed">
-      <insert_block name="origin"/>
+      <xacro:insert_block name="origin"/>
       <parent link="${parent}"/>
       <child link="${prefix}_adapter_iso50_kms40_frame_in"/>

File: iai_roller_description/urdf/iai_roller.urdf.xacro (robot description, xacro)
@@ -7,5 +7,5 @@
 <xacro:macro name="iai_roller" params="name parent *origin">
  <joint name="${name}_joint" type="fixed">
-    <insert_block name="origin"/>
+    <xacro:insert_block name="origin"/>
     <parent link="${parent}"/>
     <child link="${name}_base_link"/>

File: iai_ur_description/urdf/ur10.urdf.xacro (robot description, xacro)
@@ -7,45 +7,45 @@
   <xacro:include filename="$(find iai_ur_description)/urdf/ur.transmission.xacro" />
   <xacro:include filename="$(find iai_ur_description)/urdf/ur.gazebo.xacro" />
-  <property name="pi" value="3.14159265" />
+  <xacro:property name="pi" value="3.14159265" />
   <!-- Inertia parameters -->
-  <property name="base_mass" value="4.0" />  <!-- This mass might be incorrect -->
-  <property name="shoulder_mass" value="7.778" />
-  <property name="upper_arm_mass" value="12.93" />
-  <property name="forearm_mass" value="3.87" />
-  <property name="wrist_1_mass" value="1.96" />
-  <property name="wrist_2_mass" value="1.96" />
-  <property name="wrist_3_mass" value="0.202" />
+  <xacro:property name="base_mass" value="4.0" />  <!-- This mass might be incorrect -->
+  <xacro:property name="shoulder_mass" value="7.778" />
+  <xacro:property name="upper_arm_mass" value="12.93" />
+  <xacro:property name="forearm_mass" value="3.87" />
+  <xacro:property name="wrist_1_mass" value="1.96" />
+  <xacro:property name="wrist_2_mass" value="1.96" />
+  <xacro:property name="wrist_3_mass" value="0.202" />
   <!-- These parameters are borrowed from the urcontrol.conf file
        but are not verified for the correct permutation.
        The permutation was guessed by looking at the UR5 parameters.
        Serious use of these parameters needs further inspection. -->
-  <property name="shoulder_cog" value="0.00008 0.00244 -0.037" />
-  <property name="upper_arm_cog" value="0.00001 0.15061 0.38757" />
-  <property name="forearm_cog" value="-0.00012 0.06112 0.1984" />
-  <property name="wrist_1_cog" value="-0.00021 -0.00112 0.02269" />
-  <property name="wrist_2_cog" value="-0.00021 0.00112 0.002269" />
-  <property name="wrist_3_cog" value="0 -0.001156 -0.00149" />
+  <xacro:property name="shoulder_cog" value="0.00008 0.00244 -0.037" />
+  <xacro:property name="upper_arm_cog" value="0.00001 0.15061 0.38757" />
+  <xacro:property name="forearm_cog" value="-0.00012 0.06112 0.1984" />
+  <xacro:property name="wrist_1_cog" value="-0.00021 -0.00112 0.02269" />
+  <xacro:property name="wrist_2_cog" value="-0.00021 0.00112 0.002269" />
+  <xacro:property name="wrist_3_cog" value="0 -0.001156 -0.00149" />
   <!-- Kinematic model -->
   <!-- Properties from urcontrol.conf -->
-  <property name="ur10_d1" value="0.1273" />
-  <property name="ur10_a2" value="-0.612" />
-  <property name="ur10_a3" value="-0.5723" />
-  <property name="ur10_d4" value="0.163941" />
-  <property name="ur10_d5" value="0.1157" />
-  <property name="ur10_d6" value="0.0922" />
+  <xacro:property name="ur10_d1" value="0.1273" />
+  <xacro:property name="ur10_a2" value="-0.612" />
+  <xacro:property name="ur10_a3" value="-0.5723" />
+  <xacro:property name="ur10_d4" value="0.163941" />
+  <xacro:property name="ur10_d5" value="0.1157" />
+  <xacro:property name="ur10_d6" value="0.0922" />
   <!-- Arbitrary offsets for shoulder/elbow joints -->
-  <property name="shoulder_offset" value="0.220941" />  <!-- measured from model -->
-  <property name="elbow_offset" value="-0.1719" /> <!-- measured from model -->
+  <xacro:property name="shoulder_offset" value="0.220941" />  <!-- measured from model -->
+  <xacro:property name="elbow_offset" value="-0.1719" /> <!-- measured from model -->
   <!-- link lengths used in model -->
-  <property name="shoulder_height" value="${ur10_d1}" />
-  <property name="upper_arm_length" value="${-ur10_a2}" />
-  <property name="forearm_length" value="${-ur10_a3}" />
-  <property name="wrist_1_length" value="${ur10_d4 - elbow_offset - shoulder_offset}" />
-  <property name="wrist_2_length" value="${ur10_d5}" />
-  <property name="wrist_3_length" value="${ur10_d6}" />
+  <xacro:property name="shoulder_height" value="${ur10_d1}" />
+  <xacro:property name="upper_arm_length" value="${-ur10_a2}" />
+  <xacro:property name="forearm_length" value="${-ur10_a3}" />
+  <xacro:property name="wrist_1_length" value="${ur10_d4 - elbow_offset - shoulder_offset}" />
+  <xacro:property name="wrist_2_length" value="${ur10_d5}" />
+  <xacro:property name="wrist_3_length" value="${ur10_d6}" />
   <xacro:macro name="cylinder_inertial" params="radius length mass *origin">
     <inertial>
       <mass value="${mass}" />
-      <insert_block name="origin" />
+      <xacro:insert_block name="origin" />
       <inertia ixx="${0.0833333 * mass * (3 * radius * radius + length * length)}" ixy="0.0" ixz="0.0"
         iyy="${0.0833333 * mass * (3 * radius * radius + length * length)}" iyz="0.0"

File: iai_ur_description/urdf/ur3.urdf.xacro (robot description, xacro)
@@ -6,45 +6,45 @@
   <xacro:include filename="$(find iai_ur_description)/urdf/ur.transmission.xacro" />
   <xacro:include filename="$(find iai_ur_description)/urdf/ur.gazebo.xacro" />
-  <property name="pi" value="3.14159265" />
+  <xacro:property name="pi" value="3.14159265" />
   <!-- Inertia parameters -->
-  <property name="base_mass" value="2.0" />  <!-- This mass might be incorrect -->
-  <property name="shoulder_mass" value="2.0" />
-  <property name="upper_arm_mass" value="3.42" />
-  <property name="forearm_mass" value="1.26" />
-  <property name="wrist_1_mass" value="0.8" />
-  <property name="wrist_2_mass" value="0.8" />
-  <property name="wrist_3_mass" value="0.35" />
+  <xacro:property name="base_mass" value="2.0" />  <!-- This mass might be incorrect -->
+  <xacro:property name="shoulder_mass" value="2.0" />
+  <xacro:property name="upper_arm_mass" value="3.42" />
+  <xacro:property name="forearm_mass" value="1.26" />
+  <xacro:property name="wrist_1_mass" value="0.8" />
+  <xacro:property name="wrist_2_mass" value="0.8" />
+  <xacro:property name="wrist_3_mass" value="0.35" />
   <!-- These parameters are borrowed from the urcontrol.conf file
        but are not verified for the correct permutation.
        The permutation was guessed by looking at the UR5 parameters.
        Serious use of these parameters needs further inspection. -->
-  <property name="shoulder_cog" value="0.0 -0.02 0.0" />
-  <property name="upper_arm_cog" value="0.13 0.0 0.1157" />
-  <property name="forearm_cog" value="0.05 0.0 0.0238" />
-  <property name="wrist_1_cog" value="0.0 0.0 0.01" />
-  <property name="wrist_2_cog" value="0.0 0.0 0.01" />
-  <property name="wrist_3_cog" value="0.0 0.0 -0.02" />
+  <xacro:property name="shoulder_cog" value="0.0 -0.02 0.0" />
+  <xacro:property name="upper_arm_cog" value="0.13 0.0 0.1157" />
+  <xacro:property name="forearm_cog" value="0.05 0.0 0.0238" />
+  <xacro:property name="wrist_1_cog" value="0.0 0.0 0.01" />
+  <xacro:property name="wrist_2_cog" value="0.0 0.0 0.01" />
+  <xacro:property name="wrist_3_cog" value="0.0 0.0 -0.02" />
   <!-- Kinematic model -->
   <!-- Properties from urcontrol.conf -->
-  <property name="ur3_d1" value="0.1519" />
-  <property name="ur3_a2" value="-0.24365" />
-  <property name="ur3_a3" value="-0.21325" />
-  <property name="ur3_d4" value="0.11235" />
-  <property name="ur3_d5" value="0.08535" />
-  <property name="ur3_d6" value="0.0819" />
+  <xacro:property name="ur3_d1" value="0.1519" />
+  <xacro:property name="ur3_a2" value="-0.24365" />
+  <xacro:property name="ur3_a3" value="-0.21325" />
+  <xacro:property name="ur3_d4" value="0.11235" />
+  <xacro:property name="ur3_d5" value="0.08535" />
+  <xacro:property name="ur3_d6" value="0.0819" />
   <!-- Arbitrary offsets for shoulder/elbow joints -->
-  <property name="shoulder_offset" value="0.1198" />  <!-- measured from model -->
-  <property name="elbow_offset" value="-0.0925" /> <!-- measured from model -->
+  <xacro:property name="shoulder_offset" value="0.1198" />  <!-- measured from model -->
+  <xacro:property name="elbow_offset" value="-0.0925" /> <!-- measured from model -->
   <!-- link lengths used in model -->
-  <property name="shoulder_height" value="${ur3_d1}" />
-  <property name="upper_arm_length" value="${-ur3_a2}" />
-  <property name="forearm_length" value="${-ur3_a3}" />
-  <property name="wrist_1_length" value="${ur3_d4 - elbow_offset - shoulder_offset}" />
-  <property name="wrist_2_length" value="${ur3_d5}" />
-  <property name="wrist_3_length" value="${ur3_d6}" />
+  <xacro:property name="shoulder_height" value="${ur3_d1}" />
+  <xacro:property name="upper_arm_length" value="${-ur3_a2}" />
+  <xacro:property name="forearm_length" value="${-ur3_a3}" />
+  <xacro:property name="wrist_1_length" value="${ur3_d4 - elbow_offset - shoulder_offset}" />
+  <xacro:property name="wrist_2_length" value="${ur3_d5}" />
+  <xacro:property name="wrist_3_length" value="${ur3_d6}" />
   <xacro:macro name="cylinder_inertial" params="radius length mass *origin">
     <inertial>
       <mass value="${mass}" />
-      <insert_block name="origin" />
+      <xacro:insert_block name="origin" />
       <inertia ixx="${0.0833333 * mass * (3 * radius * radius + length * length)}" ixy="0.0" ixz="0.0"
         iyy="${0.0833333 * mass * (3 * radius * radius + length * length)}" iyz="0.0"
@@ -56,5 +56,5 @@
       <parent link="${parent}" />
       <child link="${prefix}base_link" />
-      <insert_block name="origin"/>
+      <xacro:insert_block name="origin"/>
     </joint>
     <link name="${prefix}base_link" >

File: iai_ur_description/urdf/ur5.urdf.xacro (robot description, xacro)
@@ -3,19 +3,19 @@
   <xacro:include filename="$(find iai_ur_description)/urdf/ur.transmission.xacro" />
   <xacro:include filename="$(find iai_ur_description)/urdf/ur.gazebo.xacro" />
-  <property name="pi" value="3.14159265" />
+  <xacro:property name="pi" value="3.14159265" />
   <!-- Inertia parameters -->
-  <property name="base_mass" value="4.0" />  <!-- This mass might be incorrect -->
-  <property name="shoulder_mass" value="3.7000" />
-  <property name="upper_arm_mass" value="8.3930" />
-  <property name="forearm_mass" value="2.2750" />
-  <property name="wrist_1_mass" value="1.2190" />
-  <property name="wrist_2_mass" value="1.2190" />
-  <property name="wrist_3_mass" value="0.1879" />
-  <property name="shoulder_cog" value="0.0 0.00193 -0.02561" />
-  <property name="upper_arm_cog" value="0.0 -0.024201 0.2125" />
-  <property name="forearm_cog" value="0.0 0.0265 0.11993" />
-  <property name="wrist_1_cog" value="0.0 0.110949 0.01634" />
-  <property name="wrist_2_cog" value="0.0 0.0018 0.11099" />
-  <property name="wrist_3_cog" value="0.0 0.001159 0.0" />
+  <xacro:property name="base_mass" value="4.0" />  <!-- This mass might be incorrect -->
+  <xacro:property name="shoulder_mass" value="3.7000" />
+  <xacro:property name="upper_arm_mass" value="8.3930" />
+  <xacro:property name="forearm_mass" value="2.2750" />
+  <xacro:property name="wrist_1_mass" value="1.2190" />
+  <xacro:property name="wrist_2_mass" value="1.2190" />
+  <xacro:property name="wrist_3_mass" value="0.1879" />
+  <xacro:property name="shoulder_cog" value="0.0 0.00193 -0.02561" />
+  <xacro:property name="upper_arm_cog" value="0.0 -0.024201 0.2125" />
+  <xacro:property name="forearm_cog" value="0.0 0.0265 0.11993" />
+  <xacro:property name="wrist_1_cog" value="0.0 0.110949 0.01634" />
+  <xacro:property name="wrist_2_cog" value="0.0 0.0018 0.11099" />
+  <xacro:property name="wrist_3_cog" value="0.0 0.001159 0.0" />
   <!-- Kinematic model -->
   <!-- Properties from urcontrol.conf -->
@@ -30,20 +30,20 @@
     center_of_mass = [ [0, -0.02561, 0.00193], [0.2125, 0, 0.11336], [0.11993, 0.0, 0.0265], [0, -0.0018, 0.01634], [0, 0.0018,0.01634], [0, 0, -0.001159] ]
   -->
-  <property name="ur5_d1" value="0.089159" />
-  <property name="ur5_a2" value="-0.42500" />
-  <property name="ur5_a3" value="-0.39225" />
-  <property name="ur5_d4" value="0.10915" />
-  <property name="ur5_d5" value="0.09465" />
-  <property name="ur5_d6" value="0.0823" />
+  <xacro:property name="ur5_d1" value="0.089159" />
+  <xacro:property name="ur5_a2" value="-0.42500" />
+  <xacro:property name="ur5_a3" value="-0.39225" />
+  <xacro:property name="ur5_d4" value="0.10915" />
+  <xacro:property name="ur5_d5" value="0.09465" />
+  <xacro:property name="ur5_d6" value="0.0823" />
   <!-- Arbitrary offsets for shoulder/elbow joints -->
-  <property name="shoulder_offset" value="0.13585" />  <!-- measured from model -->
-  <property name="elbow_offset" value="-0.1197" /> <!-- measured from model -->
+  <xacro:property name="shoulder_offset" value="0.13585" />  <!-- measured from model -->
+  <xacro:property name="elbow_offset" value="-0.1197" /> <!-- measured from model -->
   <!-- link lengths used in model -->
-  <property name="shoulder_height" value="${ur5_d1}" />
-  <property name="upper_arm_length" value="${-ur5_a2}" />
-  <property name="forearm_length" value="${-ur5_a3}" />
-  <property name="wrist_1_length" value="${ur5_d4 - elbow_offset - shoulder_offset}" />
-  <property name="wrist_2_length" value="${ur5_d5}" />
-  <property name="wrist_3_length" value="${ur5_d6}" />
+  <xacro:property name="shoulder_height" value="${ur5_d1}" />
+  <xacro:property name="upper_arm_length" value="${-ur5_a2}" />
+  <xacro:property name="forearm_length" value="${-ur5_a3}" />
+  <xacro:property name="wrist_1_length" value="${ur5_d4 - elbow_offset - shoulder_offset}" />
+  <xacro:property name="wrist_2_length" value="${ur5_d5}" />
+  <xacro:property name="wrist_3_length" value="${ur5_d6}" />
   <!--property name="shoulder_height" value="0.089159" /-->
   <!--property name="shoulder_offset" value="0.13585" /-->  <!-- shoulder_offset - elbow_offset + wrist_1_length = 0.10915 -->
@@ -54,13 +54,13 @@
   <!--property name="wrist_2_length" value="0.09465" /-->   <!-- In CAD this distance is 0.930, but in the spec it is 0.09465 -->
   <!--property name="wrist_3_length" value="0.0823" /-->
-  <property name="shoulder_radius" value="0.060" />   <!-- manually measured -->
-  <property name="upper_arm_radius" value="0.054" />  <!-- manually measured -->
-  <property name="elbow_radius" value="0.060" />      <!-- manually measured -->
-  <property name="forearm_radius" value="0.040" />    <!-- manually measured -->
-  <property name="wrist_radius" value="0.045" />      <!-- manually measured -->
+  <xacro:property name="shoulder_radius" value="0.060" />   <!-- manually measured -->
+  <xacro:property name="upper_arm_radius" value="0.054" />  <!-- manually measured -->
+  <xacro:property name="elbow_radius" value="0.060" />      <!-- manually measured -->
+  <xacro:property name="forearm_radius" value="0.040" />    <!-- manually measured -->
+  <xacro:property name="wrist_radius" value="0.045" />      <!-- manually measured -->
   <xacro:macro name="cylinder_inertial" params="radius length mass *origin">
     <inertial>
       <mass value="${mass}" />
-      <insert_block name="origin" />
+      <xacro:insert_block name="origin" />
       <inertia ixx="${0.0833333 * mass * (3 * radius * radius + length * length)}" ixy="0.0" ixz="0.0"
         iyy="${0.0833333 * mass * (3 * radius * radius + length * length)}" iyz="0.0"

File: iai_wsg_50_description/robots/wsg_50.urdf.xacro (robot description, xacro)
@@ -1,5 +1,5 @@
 <?xml version="1.0"?>
 <robot name="iai_wsg_50">
-  <include filename="$(find iai_wsg_50_description)/urdf/wsg_50.urdf.xacro"/>
+  <xacro:include filename="$(find iai_wsg_50_description)/urdf/wsg_50.urdf.xacro"/>
   <link name="base_link"/>
   <wsg_50_xacro name="gripper" parent="base_link">

File: iai_wsg_50_description/urdf/wsg_50.urdf.xacro (robot description, xacro)
@@ -7,5 +7,5 @@
 <xacro:macro name="wsg_50_xacro" params="name parent *origin">
  <joint name="${name}_anterior_gripper_joint" type="fixed">
-    <insert_block name="origin"/>
+    <xacro:insert_block name="origin"/>
     <parent link="${parent}"/>
     <child link="${name}_base_link"/>
