Commit message: Added map frame, and some colors to KMS meshes.

File: iai_table_robot_description/robots/ur5_table.urdf.xacro (robot description, xacro)
@@ -2,4 +2,9 @@
 <robot xmlns:xacro="http://www.ros.org/wiki/xacro" name="ur5_table_description">
   <xacro:include filename="$(find iai_table_robot_description)/urdf/ur5_table.urdf.xacro"/>
+  <link name="map"/>
   <ur5_table/>
+  <joint name="table_localization" type="fixed">
+    <parent link="map"/>
+    <child link="table_link"/>
+  </joint>
 </robot>

File: iai_table_robot_description/urdf/ur5_table.urdf.xacro (robot description, xacro)
@@ -10,4 +10,10 @@
   <material name="gray">
     <color rgba="0.56 0.67 0.67 1"/>
+  </material>
+  <material name="Silver">
+    <color rgba="1.0 1.0 1.0 1.0"/>
+  </material>
+  <material name="Grey">
+    <color rgba="0.7 0.7 0.7 1.0"/>
   </material>
   <xacro:property name="table_height" value="0.6077" />
@@ -38,5 +44,5 @@
           <mesh filename="package://iai_table_robot_description/meshes/base_to_optical_table.stl"/>
         </geometry>
-        <material name="gray"/>
+        <material name="Silver"/>
       </visual>
     </link>
