Commit message: Shrinked description of kms40 because the cabling adaptor is actually part of our LWR.

File: iai_kms_40_description/urdf/kms_40.urdf.xacro (robot description, xacro)
@@ -3,21 +3,7 @@
        name="kms_40">
   <xacro:macro name="kms_40_xacro" params="prefix parent">
-    <joint name="${prefix}_cabling_adaptor_joint" type="fixed">
-      <origin xyz="0 0 0.005" rpy="0 0 3.14159265359"/>
+    <joint name="${prefix}_kms40_adaptor_joint" type="fixed">
+      <origin xyz="0 0 0.013" rpy="0 0 3.14159265359" />
       <parent link="${parent}"/>
-      <child link="${prefix}_cabling_adaptor_link"/>
-    </joint>
-    <link name="${prefix}_cabling_adaptor_link">
-      <visual>
-        <origin rpy="0 0 0" xyz="0 0 0"/>
-        <geometry>
-          <cylinder length="0.01" radius="0.0315"/>
-        </geometry>
-        <material name="Black"/>
-      </visual>
-    </link>
-    <joint name="${prefix}_kms40_adaptor_joint" type="fixed">
-      <origin xyz="0 0 0.013" rpy="0 0 0" />
-      <parent link="${prefix}_cabling_adaptor_link"/>
       <child link="${prefix}_kms40_adaptor_link"/>
     </joint>
@@ -45,10 +31,10 @@
       </visual>
     </link>
-    <joint name="${prefix}_kms40_box_joint" type="fixed">
+    <joint name="${prefix}_kms40_connector_joint" type="fixed">
       <origin xyz="0.021 0 0" rpy="0 0 0" />
       <parent link="${prefix}_kms40_link"/>
-      <child link="${prefix}_kms40_box_link"/>
+      <child link="${prefix}_kms40_connector_link"/>
     </joint>
-    <link name="${prefix}_kms40_box_link">
+    <link name="${prefix}_kms40_connector_link">
       <visual>
         <origin rpy="0 0 0" xyz="0 0 0"/>

Commit message: twisted kms40 frame by 90°

File: iai_kms_40_description/urdf/kms_40.urdf.xacro (robot description, xacro)
@@ -30,5 +30,5 @@
     <!-- Now joint connecting the actual kms40 sensor -->
     <joint name="${prefix}kms40_joint" type="fixed">
-      <origin xyz="0 0 0" rpy="0 0 0" />
+      <origin xyz="0 0 0" rpy="0 0 3.14159265359" />
       <parent link="${prefix}adapter_iso50_kms40_frame_out"/>
       <child link="${prefix}kms40_frame_in"/>

Commit message: Revert change by previous commit.
The 180deg rotation should not be made here, instead it should happen in the file
that includes this xacro.

File: iai_kms_40_description/urdf/kms_40.urdf.xacro (robot description, xacro)
@@ -30,5 +30,5 @@
     <!-- Now joint connecting the actual kms40 sensor -->
     <joint name="${prefix}kms40_joint" type="fixed">
-      <origin xyz="0 0 0" rpy="0 0 3.14159265359" />
+      <origin xyz="0 0 0" rpy="0 0 0" />
       <parent link="${prefix}adapter_iso50_kms40_frame_out"/>
       <child link="${prefix}kms40_frame_in"/>
