Commit message: minor fix: naming convention and prefix missing
Few minors fix:
 * Name convention inconsistency for gripper model/controller implementation
   - renaming joint names, suffix for joint should be "_joint"
 * fix error wsg_50_msgs.msg module not found in boxy configurator script,
     maybe caused by a pkg renaming.

File: iai_wsg_50_description/urdf/wsg_50.urdf.xacro (robot description, xacro)
@@ -44,5 +44,5 @@
   </gazebo>
   <!-- GRIPPER LEFT -->
-  <joint name="${name}_base_joint_gripper_left" type="prismatic">
+  <joint name="${name}_base_gripper_left_joint" type="prismatic">
      <limit lower="-0.055" upper="-0.0027" effort="1.0" velocity="0.42"/>
      <origin xyz="0 0 0" rpy="0 0 0" />      <!--origin xyz="-0.0067 0 0.049" rpy="0 0 0" /-->
@@ -55,5 +55,5 @@
   <transmission name="${name}_base_trans_left" type="pr2_mechanism_model/SimpleTransmission">
      <actuator name="${name}_base_motor_left" />
-     <joint name="${name}_base_joint_gripper_left" />
+     <joint name="${name}_base_gripper_left_joint" />
      <mechanicalReduction>1</mechanicalReduction>
      <motorTorqueConstant>1</motorTorqueConstant>
@@ -129,5 +129,5 @@
   </gazebo>
   <!-- GRIPPER RIGHT -->
-  <joint name="${name}_base_joint_gripper_right" type="prismatic">
+  <joint name="${name}_base_gripper_right_joint" type="prismatic">
      <limit lower="0.0027" upper="0.055" effort="1.0" velocity="0.42"/>
      <origin xyz="0 0 0" rpy="0 0 3.14159" />
@@ -140,5 +140,5 @@
   <transmission name="${name}_base_trans_right" type="pr2_mechanism_model/SimpleTransmission">
      <actuator name="${name}_base_motor_right" />
-     <joint name="${name}_base_joint_gripper_right" />
+     <joint name="${name}_base_gripper_right_joint" />
      <mechanicalReduction>1</mechanicalReduction>
      <motorTorqueConstant>1</motorTorqueConstant>

Commit message: add link suffix

File: iai_wsg_50_description/urdf/wsg_50.urdf.xacro (robot description, xacro)
@@ -48,5 +48,5 @@
      <origin xyz="0 0 0" rpy="0 0 0" />      <!--origin xyz="-0.0067 0 0.049" rpy="0 0 0" /-->
      <parent link="${name}_base_link"/>
-     <child link="${name}_gripper_left" />
+     <child link="${name}_gripper_left_link" />
      <dynamics friction="100" damping="100" />
      <axis xyz="1 0 0"/>
@@ -59,32 +59,32 @@
      <motorTorqueConstant>1</motorTorqueConstant>
   </transmission>
-  <link name="${name}_gripper_left">
-      <inertial>
-          <mass value="0.1" />
-          <origin xyz="0 0 0" />
-      <inertia ixx="1.0" ixy="0.0" ixz="0.0"
-               iyy="1.0" iyz="0.0"
-               izz="1.0" />
-      </inertial>
-      <visual>
-          <origin xyz="0.0 0 0" rpy="0 0 0" />
-          <geometry>
-             <mesh filename="package://iai_wsg_50_description/meshes/GUIDE_WSG50_110.stl" scale="0.001 0.001 0.001"/>
-	     <!--box size="0.0175 0.03 0.024"/-->
-          </geometry>
-          <material name="black">
-		<color rgba="0 0 0 1"/>
-      	  </material>
-      </visual>
-      <collision>
-          <origin xyz="0 0 0" rpy="0 0 0" />
-          <geometry>
-	     <!--box size="0.0175 0.03 0.024"/-->
-             <mesh filename="package://iai_wsg_50_description/meshes/GUIDE_WSG50_110.stl" scale="0.001 0.001 0.001"/>
-         </geometry>
-     </collision>
-     <contact_coefficients kd="1.0" kp="1000.0" mu="0"/>
-  </link>
-  <gazebo reference="${name}_gripper_left">
+  <link name="${name}_gripper_left_link">
+      <inertial>
+          <mass value="0.1" />
+          <origin xyz="0 0 0" />
+      <inertia ixx="1.0" ixy="0.0" ixz="0.0"
+               iyy="1.0" iyz="0.0"
+               izz="1.0" />
+      </inertial>
+      <visual>
+          <origin xyz="0.0 0 0" rpy="0 0 0" />
+          <geometry>
+             <mesh filename="package://iai_wsg_50_description/meshes/GUIDE_WSG50_110.stl" scale="0.001 0.001 0.001"/>
+	     <!--box size="0.0175 0.03 0.024"/-->
+          </geometry>
+          <material name="black">
+		<color rgba="0 0 0 1"/>
+      	  </material>
+      </visual>
+      <collision>
+          <origin xyz="0 0 0" rpy="0 0 0" />
+          <geometry>
+	     <!--box size="0.0175 0.03 0.024"/-->
+             <mesh filename="package://iai_wsg_50_description/meshes/GUIDE_WSG50_110.stl" scale="0.001 0.001 0.001"/>
+         </geometry>
+     </collision>
+     <contact_coefficients kd="1.0" kp="1000.0" mu="0"/>
+  </link>
+  <gazebo reference="${name}_gripper_left_link">
     <material>Gazebo/Blue</material>
     <turnGravityOff>false</turnGravityOff>
@@ -93,11 +93,11 @@
   <joint name="${name}_guide_joint_finger_left" type="fixed">
      <origin xyz="0 0 0.023" rpy="0 0 0" />
-     <parent link="${name}_gripper_left"/>
-     <child link="${name}_finger_left" />
+     <parent link="${name}_gripper_left_link"/>
+     <child link="${name}_finger_left_link" />
      <dynamics friction="100" damping="100" />
      <axis xyz="1 0 0"/>
      <!-- <limit effort="100" velocity="100"/> -->
   </joint>
-  <link name="${name}_finger_left">
+  <link name="${name}_finger_left_link">
       <inertial>
           <mass value="0.1" />
@@ -133,5 +133,5 @@
      <origin xyz="0 0 0" rpy="0 0 3.14159" />
      <parent link="${name}_base_link"/>
-     <child link="${name}_gripper_right" />
+     <child link="${name}_gripper_right_link" />
      <axis xyz="-1 0 0"/>
      <dynamics friction="100" damping="100" />
@@ -144,5 +144,5 @@
      <motorTorqueConstant>1</motorTorqueConstant>
   </transmission>
-    <link name="${name}_gripper_right">
+    <link name="${name}_gripper_right_link">
       <inertial>
           <mass value="0.1" />
@@ -178,11 +178,11 @@
   <joint name="${name}_guide_joint_finger_right" type="fixed">
      <origin xyz="0 0 0.023" rpy="0 0 0" />
-     <parent link="${name}_gripper_right"/>
-     <child link="${name}_finger_right" />
+     <parent link="${name}_gripper_right_link"/>
+     <child link="${name}_finger_right_link" />
      <dynamics friction="100" damping="100" />
      <axis xyz="1 0 0"/>
      <limit effort="100" velocity="100"/>
   </joint>
-  <link name="${name}_finger_right">
+  <link name="${name}_finger_right_link">
       <inertial>
           <mass value="0.1" />

Commit message: Added a fixed tool-frame to the wsg50 description.

File: iai_wsg_50_description/urdf/wsg_50.urdf.xacro (robot description, xacro)
@@ -213,4 +213,10 @@
     <turnGravityOff>false</turnGravityOff>
   </gazebo>
+  <link name="${name}_tool_frame"/>
+  <joint name="${name}_tool_frame_joint" type="fixed">
+     <origin xyz="0 0 0.154" rpy="0 0 0" />
+     <parent link="${name}_base_link"/>
+     <child link="${name}_tool_frame" />
+  </joint>
 </xacro:macro>
 </robot>

Commit message: wsg50 gripper urdf now requires only one joint

File: iai_wsg_50_description/urdf/wsg_50.urdf.xacro (robot description, xacro)
@@ -45,4 +45,5 @@
   <!-- GRIPPER LEFT -->
   <joint name="${name}_base_gripper_left_joint" type="prismatic">
+     <mimic joint ="${name}_gripper_joint" multiplier="-0.5"/>
      <limit lower="-0.055" upper="-0.0027" effort="1.0" velocity="0.42"/>
      <origin xyz="0 0 0" rpy="0 0 0" />      <!--origin xyz="-0.0067 0 0.049" rpy="0 0 0" /-->
@@ -129,8 +130,8 @@
   </gazebo>
   <!-- GRIPPER RIGHT -->
-  <joint name="${name}_base_gripper_right_joint" type="prismatic">
-     <limit lower="0.0027" upper="0.055" effort="1.0" velocity="0.42"/>
+  <joint name="${name}_gripper_joint" type="prismatic">
+     <limit lower="0.0065" upper="0.109" effort="1.0" velocity="0.42"/>
      <origin xyz="0 0 0" rpy="0 0 3.14159" />
-     <parent link="${name}_base_link"/>
+     <parent link="${name}_gripper_left_link"/>
      <child link="${name}_gripper_right_link" />
      <axis xyz="-1 0 0"/>

Commit message: WSG50-description: Removing superfluous 'gripper' from name of gripper joint.

File: iai_wsg_50_description/urdf/wsg_50.urdf.xacro (robot description, xacro)
@@ -45,5 +45,5 @@
   <!-- GRIPPER LEFT -->
   <joint name="${name}_base_gripper_left_joint" type="prismatic">
-     <mimic joint ="${name}_gripper_joint" multiplier="-0.5"/>
+     <mimic joint ="${name}_joint" multiplier="-0.5"/>
      <limit lower="-0.055" upper="-0.0027" effort="1.0" velocity="0.42"/>
      <origin xyz="0 0 0" rpy="0 0 0" />      <!--origin xyz="-0.0067 0 0.049" rpy="0 0 0" /-->
@@ -130,5 +130,5 @@
   </gazebo>
   <!-- GRIPPER RIGHT -->
-  <joint name="${name}_gripper_joint" type="prismatic">
+  <joint name="${name}_joint" type="prismatic">
      <limit lower="0.0065" upper="0.109" effort="1.0" velocity="0.42"/>
      <origin xyz="0 0 0" rpy="0 0 3.14159" />

Commit message: moved gripper tool frame of wsg 50 urdf 1 cm closer to be between the fingers

File: iai_wsg_50_description/urdf/wsg_50.urdf.xacro (robot description, xacro)
@@ -213,5 +213,5 @@
   <link name="${name}_tool_frame"/>
   <joint name="${name}_tool_frame_joint" type="fixed">
-     <origin xyz="0 0 0.154" rpy="0 0 0" />
+     <origin xyz="0 0 0.144" rpy="0 0 0" />
      <parent link="${name}_base_link"/>
      <child link="${name}_tool_frame" />
