Commit message: fixed laser pos

File: iai_boxy_base_2/robots/base.URDF (robot description, URDF)
Before this commit: robot base, 4 links, 3 joints
Links:
- link base_link: geometry collision mesh filename=package://iai_boxy_base_2/meshes/base.stl; visual mesh filename=package://iai_boxy_base_2/meshes/base.stl
Joints:
- joint laser_reference_front_joint: origin xyz=0.1772 0.060745 0.150 rpy=0.0 0.0 0.7853975 -> xyz=0.1772 0.060215 0.149929 rpy=0.0 0.0 0.7853975

Commit message: added plate to iai boxy base 2

File: iai_boxy_base_2/robots/base.URDF (robot description, URDF)
Before this commit: robot base, 4 links, 3 joints
Links:
- added link plate; collision box size=0.6 0.553 0.02; visual box size=0.6 0.553 0.02
Joints:
- added joint plate_joint: type fixed, parent base_footprint, child plate, origin xyz=0.06 0.02 0.62 rpy=0 0 0

Commit message: added connection to odom to boxy base 2

File: iai_boxy_base_2/robots/base.URDF (robot description, URDF)
Before this commit: robot base, 5 links, 4 joints
Links:
- added link odom
- added link odom_x_frame
- added link odom_y_frame
Joints:
- added joint odom_x_joint: type prismatic, parent odom, child odom_x_frame, axis 1 0 0, limit lower=-1000 upper=1000 effort=200 velocity=1
- added joint odom_y_joint: type prismatic, parent odom_x_frame, child odom_y_frame, axis 0 1 0, limit lower=-1000 upper=1000 effort=200 velocity=1
- added joint odom_z_joint: type continuous, parent odom_y_frame, child base_footprint, axis 0 0 1, limit effort=200 velocity=1

Commit message: iai_boxy_base_2: place the base_footprint at the center of wheels, according to CAD

File: iai_boxy_base_2/robots/base.URDF (robot description, URDF)
Before this commit: robot base, 8 links, 7 joints
Joints:
- joint base_footprint_joint: origin xyz=0.36 0.25 0.16 rpy=0 0 0 -> xyz=0.25525 0.225 0.16 rpy=0 0 0

Commit message: Fix small error in Z and add explanation of numbers chosen for /base_footprint to /base_link

File: iai_boxy_base_2/robots/base.URDF (robot description, URDF)
Before this commit: robot base, 8 links, 7 joints
Joints:
- joint base_footprint_joint: origin xyz=0.25525 0.225 0.16 rpy=0 0 0 -> xyz=0.25525 0.225 0.1616 rpy=0 0 0

Commit message: base donbots plate a child of base_link instead of base_footprint

File: iai_boxy_base_2/robots/base.URDF (robot description, URDF)
Before this commit: robot base, 8 links, 7 joints
Joints:
- joint plate_joint: origin xyz=0.06 0.02 0.62 rpy=0 0 0 -> xyz=-0.300 -0.230 0.460 rpy=0 0 0; parent base_footprint -> base_link

Commit message: modified robots/iai_donbot2_with_refills_finger.xacro

File: iai_boxy_base_2/robots/base.URDF (robot description, URDF)
Before this commit: robot base, 8 links, 7 joints
Joints:
- joint odom_x_joint: limit lower=-1000 upper=1000 effort=200 velocity=1 -> lower=-1000 upper=1000 effort=200 velocity=0.1
- joint odom_y_joint: limit lower=-1000 upper=1000 effort=200 velocity=1 -> lower=-1000 upper=1000 effort=200 velocity=0.1
- joint odom_z_joint: limit effort=200 velocity=1 -> effort=200 velocity=0.2

File: iai_donbot_description/robots/iai_donbot2_with_refills_finger.xacro (robot description, xacro)
@@ -4,6 +4,12 @@
   <!-- <link name="map"/> -->
   <iai_donbot/>
-  <joint name="refills_finger" type="continuous">
+  <joint name="refills_tool_frame_joint" type="fixed">
     <parent link="gripper_tool_frame"/>
+    <child link="refills_tool_frame"/>
+    <origin xyz="0 0 0.012" rpy="0.0 0.0 0.0" />
+  </joint>
+  <link name="refills_tool_frame"/>
+  <joint name="refills_finger_joint" type="continuous">
+    <parent link="refills_tool_frame"/>
     <child link="refills_finger"/>
     <axis xyz="1 0 0"/>

Commit message: reverted accidentally committed changes to odom velocity boxy base 2

File: iai_boxy_base_2/robots/base.URDF (robot description, URDF)
Before this commit: robot base, 8 links, 7 joints
Joints:
- joint odom_x_joint: limit lower=-1000 upper=1000 effort=200 velocity=0.1 -> lower=-1000 upper=1000 effort=200 velocity=1
- joint odom_y_joint: limit lower=-1000 upper=1000 effort=200 velocity=0.1 -> lower=-1000 upper=1000 effort=200 velocity=1
- joint odom_z_joint: limit effort=200 velocity=0.2 -> effort=200 velocity=1

Commit message: [iai_boxy_base_2] added a decimated mesh for collisions

File: iai_boxy_base_2/robots/base.URDF (robot description, URDF)
Before this commit: robot base, 8 links, 7 joints
Links:
- link base_link: geometry collision mesh filename=package://iai_boxy_base_2/meshes/base_lowres.stl; visual mesh filename=package://iai_boxy_base_2/meshes/base.stl
