Commit message: Fix xacro warning

File: iai_boxy_base_2/robots/base.xacro (robot description, xacro)
@@ -39,5 +39,5 @@
 			<axis xyz="-1 0 0" />
 		</joint>
-		<if value="${odom}">
+		<xacro:if value="${odom}">
 			<link name="odom" />
 			<joint name="odom_x_joint" type="prismatic">
@@ -78,5 +78,5 @@
 				<limit velocity="1" effort="200" />
 			</joint>
-		</if>
+		</xacro:if>
 		<!-- Definition of base_footprint -> base_link -->
 		<link name="base_footprint">

File: iai_donbot_description/robots/iai_donbot.xacro (robot description, xacro)
@@ -19,15 +19,15 @@
 		<color rgba="1.0 1.0 0.0 1.0" />
 	</material>
-	<property name="base_link_to_table_top" value="0.47" />
-	<property name="table_length" value="0.6" />
-	<property name="table_width" value="0.553" />
-	<property name="ur5_prefix" value="ur5_" />
-	<property name="arm_mounting_plate_width" value="0.18" />
-	<property name="arm_mounting_plate_length" value="0.15" />
-	<property name="arm_mounting_plate_height" value="0.006" />
-	<property name="arm_mounting_plate_x_offset" value="0.0" />
-	<property name="arm_mounting_plate_y_offset" value="0.027" />
-	<property name="kms_mounting_plate_height" value="0.016" />
-	<arg name="transmission_hw_interface" default="hardware_interface/PositionJointInterface" />
+	<xacro:property name="base_link_to_table_top" value="0.47" />
+	<xacro:property name="table_length" value="0.6" />
+	<xacro:property name="table_width" value="0.553" />
+	<xacro:property name="ur5_prefix" value="ur5_" />
+	<xacro:property name="arm_mounting_plate_width" value="0.18" />
+	<xacro:property name="arm_mounting_plate_length" value="0.15" />
+	<xacro:property name="arm_mounting_plate_height" value="0.006" />
+	<xacro:property name="arm_mounting_plate_x_offset" value="0.0" />
+	<xacro:property name="arm_mounting_plate_y_offset" value="0.027" />
+	<xacro:property name="kms_mounting_plate_height" value="0.016" />
+	<xacro:arg name="transmission_hw_interface" default="hardware_interface/PositionJointInterface" />
 	<!-- common stuff -->
 	<xacro:include filename="$(find iai_ur_description)/urdf/common.gazebo.xacro" />
@@ -35,5 +35,5 @@
 	<xacro:include filename="$(find iai_ur_description)/urdf/ur5.urdf.xacro" />
 	<!-- arm -->
-	<arg name="kinematics_config" default="$(find iai_ur_description)/config/ur5_default.yaml" />
+	<xacro:arg name="kinematics_config" default="$(find iai_ur_description)/config/ur5_default.yaml" />
 	<xacro:macro name="iai_donbot" params="odom">
 		<xacro:base odom="${odom}"/>
@@ -74,19 +74,19 @@
 			<origin xyz="0 0 0" rpy="0 ${pi/2} 0" />
 		</joint>
-		<kms_40_xacro parent="kms_mounting_plate" prefix="">
+		<xacro:kms_40_xacro parent="kms_mounting_plate" prefix="">
 			<origin xyz="0 0 0" rpy="0 0 ${pi}" />
-		</kms_40_xacro>
-		<adapter_kms40_fwk050_xacro parent="kms40_frame_out" prefix="">
+		</xacro:kms_40_xacro>
+		<xacro:adapter_kms40_fwk050_xacro parent="kms40_frame_out" prefix="">
 			<origin xyz="0 0 0" rpy="0 0 0" />
-		</adapter_kms40_fwk050_xacro>
-		<fwk_fwa_050_xacro parent="adapter_kms40_fwk050_frame_out" prefix="">
+		</xacro:adapter_kms40_fwk050_xacro>
+		<xacro:fwk_fwa_050_xacro parent="adapter_kms40_fwk050_frame_out" prefix="">
 			<origin xyz="0 0 0" rpy="0 0 0" />
-		</fwk_fwa_050_xacro>
-		<adapter_fwa050_wsg50_xacro parent="fwk_fwa_050_frame_out" prefix="">
+		</xacro:fwk_fwa_050_xacro>
+		<xacro:adapter_fwa050_wsg50_xacro parent="fwk_fwa_050_frame_out" prefix="">
 			<origin xyz="0 0 0.0" rpy="0 0 0" />
-		</adapter_fwa050_wsg50_xacro>
-		<wsg_50_xacro name="gripper" parent="adapter_fwa050_wsg50_frame_out">
+		</xacro:adapter_fwa050_wsg50_xacro>
+		<xacro:wsg_50_xacro name="gripper" parent="adapter_fwa050_wsg50_frame_out">
 			<origin xyz="0 0 0" rpy="0 0 3.14159265359" />
-		</wsg_50_xacro>
+		</xacro:wsg_50_xacro>
 		<link name="camera_holder_link">
 			<visual>

Commit message: Add visual to laser reference so sdf parse works

File: iai_boxy_base_2/robots/base.xacro (robot description, xacro)
@@ -25,5 +25,11 @@
 			</collision>
 		</link>
-		<link name="laser_reference_front" />
+		<link name="laser_reference_front">
+			<visual>
+				<geometry>
+					<cylinder radius="0.001" length="0.005"/>
+				</geometry>
+			</visual>
+		</link>
 		<joint name="laser_reference_front_joint" type="fixed">
 			<origin xyz="0.1772 0.060215 0.149929" rpy="0.0 0.0 0.7853975" />
@@ -32,5 +38,11 @@
 			<axis xyz="0.0 0.0 0.0" />
 		</joint>
-		<link name="laser_reference_back" />
+		<link name="laser_reference_back">
+			<visual>
+				<geometry>
+					<cylinder radius="0.001" length="0.005"/>
+				</geometry>
+			</visual>
+		</link>
 		<joint name="laser_reference_back_joint" type="fixed">
 			<origin xyz="-0.69357 -0.506 0.1575" rpy="4.9333E-15 4.5082E-15 -2.3562" />

Commit message: Add wheels for boxy and options

File: iai_boxy_base_2/robots/base.xacro (robot description, xacro)
@@ -1,5 +1,5 @@
 <?xml version="1.0"?>
 <robot xmlns:xacro="http://www.ros.org/wiki/xacro">
-	<xacro:macro name="base" params="odom">
+	<xacro:macro name="base" params="odom with_wheels">
 		<link name="base_link">
 			<inertial>
@@ -25,4 +25,102 @@
 			</collision>
 		</link>
+		<xacro:if value="${with_wheels}">
+			<joint name="wheel_left_up_joint" type="revolute">
+				<limit lower="-1000.0" upper="1000.0" effort="200.0" velocity="1.0" />
+				<origin xyz="0.13 0.09 -0.06" rpy="0.0 0.0 0.0" />
+				<parent link="base_link" />
+				<child link="wheel_left_up" />
+				<axis xyz="0 1 0" />
+			</joint>
+			<link name="wheel_left_up">
+				<inertial>
+					<origin xyz="0 0 0" rpy="0 0 0" />
+					<mass value="2.0" />
+					<inertia ixx="0.01" ixy="0.0" ixz="0.0" iyy="0.01" iyz="0.0" izz="0.03" />
+				</inertial>
+				<visual>
+					<geometry>
+						<mesh filename="package://iai_boxy_base_2/meshes/wheel_left_up.stl" />
+					</geometry>
+				</visual>
+				<collision>
+					<geometry>
+						<mesh filename="package://iai_boxy_base_2/meshes/wheel_collision.stl" />
+					</geometry>
+				</collision>
+			</link>
+			<joint name="wheel_left_down_joint" type="revolute">
+				<limit lower="-1000.0" upper="1000.0" effort="200.0" velocity="1.0" />
+				<origin xyz="-0.648 0.09 -0.06" rpy="0.0 0.0 0.0" />
+				<parent link="base_link" />
+				<child link="wheel_left_down" />
+				<axis xyz="0 1 0" />
+			</joint>
+			<link name="wheel_left_down">
+				<inertial>
+					<origin xyz="0 0 0" rpy="0 0 0" />
+					<mass value="2.0" />
+					<inertia ixx="0.01" ixy="0.0" ixz="0.0" iyy="0.01" iyz="0.0" izz="0.03" />
+				</inertial>
+				<visual>
+					<geometry>
+						<mesh filename="package://iai_boxy_base_2/meshes/wheel_left_down.stl" />
+					</geometry>
+				</visual>
+				<collision>
+					<geometry>
+						<mesh filename="package://iai_boxy_base_2/meshes/wheel_collision.stl" />
+					</geometry>
+				</collision>
+			</link>
+			<joint name="wheel_right_up_joint" type="revolute">
+				<limit lower="-1000.0" upper="1000.0" effort="200.0" velocity="1.0" />
+				<origin xyz="0.13 -0.545 -0.06" rpy="0.0 0.0 0.0" />
+				<parent link="base_link" />
+				<child link="wheel_right_up" />
+				<axis xyz="0 1 0" />
+			</joint>
+			<link name="wheel_right_up">
+				<inertial>
+					<origin xyz="0 0 0" rpy="0 0 0" />
+					<mass value="2.0" />
+					<inertia ixx="0.01" ixy="0.0" ixz="0.0" iyy="0.01" iyz="0.0" izz="0.03" />
+				</inertial>
+				<visual>
+					<geometry>
+						<mesh filename="package://iai_boxy_base_2/meshes/wheel_right_up.stl" />
+					</geometry>
+				</visual>
+				<collision>
+					<geometry>
+						<mesh filename="package://iai_boxy_base_2/meshes/wheel_collision.stl" />
+					</geometry>
+				</collision>
+			</link>
+			<joint name="wheel_right_down_joint" type="revolute">
+				<limit lower="-1000.0" upper="1000.0" effort="200.0" velocity="1.0" />
+				<origin xyz="-0.648 -0.545 -0.06" rpy="0.0 0.0 0.0" />
+				<parent link="base_link" />
+				<child link="wheel_right_down" />
+				<axis xyz="0 1 0" />
+			</joint>
+			<link name="wheel_right_down">
+				<inertial>
+					<origin xyz="0 0 0" rpy="0 0 0" />
+					<mass value="2.0" />
+					<inertia ixx="0.01" ixy="0.0" ixz="0.0" iyy="0.01" iyz="0.0" izz="0.03" />
+				</inertial>
+				<visual>
+					<geometry>
+						<mesh filename="package://iai_boxy_base_2/meshes/wheel_right_down.stl" />
+					</geometry>
+				</visual>
+				<collision>
+					<geometry>
+						<mesh filename="package://iai_boxy_base_2/meshes/wheel_collision.stl" />
+					</geometry>
+				</collision>
+			</link>
+		</xacro:if>
 		<link name="laser_reference_front">
 			<visual>

File: iai_donbot_description/robots/iai_donbot.urdf.xacro (robot description, xacro)
@@ -3,5 +3,5 @@
   <xacro:include filename="$(find iai_donbot_description)/robots/iai_donbot.xacro"/>
   <!-- <link name="map"/> -->
-  <xacro:iai_donbot odom="True"/>
+  <xacro:iai_donbot odom="True" with_wheels="False" with_boxes="True"/>
   <!-- <joint name="table_localization" type="fixed">
     <parent link="map"/>

File: iai_donbot_description/robots/iai_donbot.xacro (robot description, xacro)
@@ -36,6 +36,6 @@
 	<!-- arm -->
 	<xacro:arg name="kinematics_config" default="$(find iai_ur_description)/config/ur5_default.yaml" />
-	<xacro:macro name="iai_donbot" params="odom">
-		<xacro:base odom="${odom}"/> <!-- create base -->
+	<xacro:macro name="iai_donbot" params="odom with_wheels with_boxes">
+		<xacro:base odom="${odom}" with_wheels="${with_wheels}"/> <!-- create base -->
 		<!--
 		<joint name="arm_mounting_plate_joint" type="fixed">
@@ -133,112 +133,114 @@
 		</joint>
 		<!-- boxes to cover up switches and stuff -->
-		<joint name="switches_joint" type="fixed">
-			<parent link="base_link" />
-			<child link="switches" />
-			<origin xyz="-0.66 -0.225 0.225" rpy="0 0 0" />
-		</joint>
-		<link name="switches">
-			<visual>
-				<geometry>
-					<box size="0.12 0.4 0.45" />
-				</geometry>
-				<material name="Silver" />
-			</visual>
-			<collision>
-				<geometry>
-					<box size="0.12 0.4 0.45" />
-				</geometry>
-				<material name="Silver" />
-			</collision>
-		</link>
-		<joint name="charger_joint" type="fixed">
-			<parent link="base_link" />
-			<child link="charger" />
-			<origin xyz="0.075 -0.225 0.19" rpy="0 0 0" />
-		</joint>
-		<link name="charger">
-			<visual>
-				<geometry>
-					<box size="0.15 0.3 0.38" />
-				</geometry>
-				<material name="Silver" />
-			</visual>
-			<collision>
-				<geometry>
-					<box size="0.15 0.3 0.38" />
-				</geometry>
-				<material name="Silver" />
-			</collision>
-		</link>
-		<joint name="e_stop_joint" type="fixed">
-			<parent link="base_link" />
-			<child link="e_stop" />
-			<origin xyz="-0.035 -0.0015 0.52" rpy="0 0 0" />
-		</joint>
-		<link name="e_stop">
-			<visual>
-				<geometry>
-					<box size="0.07 0.07 0.1" />
-				</geometry>
-				<material name="yellow" />
-			</visual>
-			<collision>
-				<geometry>
-					<box size="0.07 0.07 0.1" />
-				</geometry>
-				<material name="yellow" />
-			</collision>
-		</link>
-		<joint name="wlan_joint" type="fixed">
-			<parent link="base_link" />
-			<child link="wlan" />
-			<origin xyz="0.05 -0.225 0.405" rpy="0 -0.314 0" />
-		</joint>
-		<link name="wlan">
-			<visual>
-				<geometry>
-					<box size="0.25 0.14 0.05" />
-				</geometry>
-				<material name="Silver" />
-			</visual>
-			<collision>
-				<geometry>
-					<box size="0.25 0.14 0.05" />
-				</geometry>
-				<material name="Silver" />
-			</collision>
-		</link>
-		<joint name="ur5_touchpad_joint" type="fixed">
-			<parent link="base_link" />
-			<child link="ur5_touchpad" />
-			<origin xyz="-0.16 -0.5355 0.38" rpy="0 0 0" />
-		</joint>
-		<link name="ur5_touchpad">
-			<visual>
-				<geometry>
-					<box size="0.32 0.06 0.24" />
-				</geometry>
-				<material name="Silver" />
-			</visual>
-			<collision>
-				<geometry>
-					<box size="0.32 0.06 0.24" />
-				</geometry>
-				<material name="Silver" />
-			</collision>
-		</link>
-		<joint name="wrist_collision_joint" type="fixed">
-			<parent link="adapter_kms40_fwk050_frame_in" />
-			<child link="wrist_collision" />
-			<origin xyz="0 0 -0.005" rpy="0 0 0" />
-		</joint>
-		<link name="wrist_collision">
-			<collision>
-				<geometry>
-					<cylinder radius="0.04" length="0.08" />
-				</geometry>
-				<material name="Silver" />
-			</collision>
-		</link>
+		<xacro:if value="${with_boxes}">
+			<joint name="switches_joint" type="fixed">
+				<parent link="base_link" />
+				<child link="switches" />
+				<origin xyz="-0.66 -0.225 0.225" rpy="0 0 0" />
+			</joint>
+			<link name="switches">
+				<visual>
+					<geometry>
+						<box size="0.12 0.4 0.45" />
+					</geometry>
+					<material name="Silver" />
+				</visual>
+				<collision>
+					<geometry>
+						<box size="0.12 0.4 0.45" />
+					</geometry>
+					<material name="Silver" />
+				</collision>
+			</link>
+			<joint name="charger_joint" type="fixed">
+				<parent link="base_link" />
+				<child link="charger" />
+				<origin xyz="0.075 -0.225 0.19" rpy="0 0 0" />
+			</joint>
+			<link name="charger">
+				<visual>
+					<geometry>
+						<box size="0.15 0.3 0.38" />
+					</geometry>
+					<material name="Silver" />
+				</visual>
+				<collision>
+					<geometry>
+						<box size="0.15 0.3 0.38" />
+					</geometry>
+					<material name="Silver" />
+				</collision>
+			</link>
+			<joint name="e_stop_joint" type="fixed">
+				<parent link="base_link" />
+				<child link="e_stop" />
+				<origin xyz="-0.035 -0.0015 0.52" rpy="0 0 0" />
+			</joint>
+			<link name="e_stop">
+				<visual>
+					<geometry>
+						<box size="0.07 0.07 0.1" />
+					</geometry>
+					<material name="yellow" />
+				</visual>
+				<collision>
+					<geometry>
+						<box size="0.07 0.07 0.1" />
+					</geometry>
+					<material name="yellow" />
+				</collision>
+			</link>
+			<joint name="wlan_joint" type="fixed">
+				<parent link="base_link" />
+				<child link="wlan" />
+				<origin xyz="0.05 -0.225 0.405" rpy="0 -0.314 0" />
+			</joint>
+			<link name="wlan">
+				<visual>
+					<geometry>
+						<box size="0.25 0.14 0.05" />
+					</geometry>
+					<material name="Silver" />
+				</visual>
+				<collision>
+					<geometry>
+						<box size="0.25 0.14 0.05" />
+					</geometry>
+					<material name="Silver" />
+				</collision>
+			</link>
+			<joint name="ur5_touchpad_joint" type="fixed">
+				<parent link="base_link" />
+				<child link="ur5_touchpad" />
+				<origin xyz="-0.16 -0.5355 0.38" rpy="0 0 0" />
+			</joint>
+			<link name="ur5_touchpad">
+				<visual>
+					<geometry>
+						<box size="0.32 0.06 0.24" />
+					</geometry>
+					<material name="Silver" />
+				</visual>
+				<collision>
+					<geometry>
+						<box size="0.32 0.06 0.24" />
+					</geometry>
+					<material name="Silver" />
+				</collision>
+			</link>
+			<joint name="wrist_collision_joint" type="fixed">
+				<parent link="adapter_kms40_fwk050_frame_in" />
+				<child link="wrist_collision" />
+				<origin xyz="0 0 -0.005" rpy="0 0 0" />
+			</joint>
+			<link name="wrist_collision">
+				<collision>
+					<geometry>
+						<cylinder radius="0.04" length="0.08" />
+					</geometry>
+					<material name="Silver" />
+				</collision>
+			</link>
+		</xacro:if>
 	</xacro:macro>
 </robot>

Commit message: Fix Bugs

File: iai_boxy_base_2/robots/base.xacro (robot description, xacro)
@@ -199,5 +199,5 @@
 			</visual>
 			<collision>
-				<origin rpy="0 0 0" xyz="0 0 0.071" />
+				<origin rpy="0 0 0" xyz="0 0 0" />
 				<geometry>
 					<box size="0.001 0.001 0.001" />

File: iai_donbot_description/robots/iai_donbot_with_refills_finger.urdf.xacro (robot description, xacro)
@@ -4,5 +4,5 @@
   <!-- <xacro:include filename="$(find fingertip_description)/urdf/mod2_fingertip.urdf.xacro"/> -->
   <!-- <link name="map"/> -->
-  <xacro:iai_donbot odom="True"/>
+  <xacro:iai_donbot odom="True" with_wheels="True" with_boxes="False" />
   <joint name="refills_tool_frame_joint" type="fixed">
     <parent link="gripper_tool_frame"/>
