Commit message: Fix issues

File: iai_boxy_base_2/robots/base.xacro (robot description, xacro)
@@ -1,4 +1,7 @@
 <?xml version="1.0"?>
 <robot xmlns:xacro="http://www.ros.org/wiki/xacro">
+	<material name="grey">
+    <color rgba="0.792156862745098 0.819607843137255 0.933333333333333 1" />
+  </material>
 	<xacro:macro name="base" params="odom with_wheels">
 		<link name="base_link">
@@ -12,111 +15,117 @@
 				<geometry>
 					<!-- <mesh -->
-					<mesh filename="package://iai_boxy_base_2/meshes/base.stl" />
-				</geometry>
-				<material name="">
-					<color rgba="0.792156862745098 0.819607843137255 0.933333333333333 1" />
-				</material>
+					<mesh filename="package://iai_boxy_base_2/meshes/base_without_wheels.stl" />
+				</geometry>
+				<material name="grey"/>
 			</visual>
 			<collision>
 				<origin xyz="0 0 0" rpy="0 0 0" />
 				<geometry>
-					<mesh filename="package://iai_boxy_base_2/meshes/base_lowres.stl" />
+					<mesh filename="package://iai_boxy_base_2/meshes/base_without_wheels.stl" />
 				</geometry>
 			</collision>
 		</link>
 		<xacro:if value="${with_wheels}">
-			<joint name="wheel_left_up_joint" type="revolute">
+			<joint name="wheel_front_left_joint" type="revolute">
 				<limit lower="-1000.0" upper="1000.0" effort="200.0" velocity="1.0" />
 				<origin xyz="0.13 0.09 -0.06" rpy="0.0 0.0 0.0" />
 				<parent link="base_link" />
-				<child link="wheel_left_up" />
-				<axis xyz="0 1 0" />
-			</joint>
-			<link name="wheel_left_up">
-				<inertial>
-					<origin xyz="0 0 0" rpy="0 0 0" />
-					<mass value="2.0" />
-					<inertia ixx="0.01" ixy="0.0" ixz="0.0" iyy="0.01" iyz="0.0" izz="0.03" />
-				</inertial>
-				<visual>
-					<geometry>
-						<mesh filename="package://iai_boxy_base_2/meshes/wheel_left_up.stl" />
-					</geometry>
-				</visual>
-				<collision>
-					<geometry>
-						<mesh filename="package://iai_boxy_base_2/meshes/wheel_collision.stl" />
-					</geometry>
-				</collision>
-			</link>
-			<joint name="wheel_left_down_joint" type="revolute">
+				<child link="wheel_front_left" />
+				<axis xyz="0 1 0" />
+			</joint>
+			<link name="wheel_front_left">
+				<inertial>
+					<origin xyz="0 0 0" rpy="0 0 0" />
+					<mass value="2.0" />
+					<inertia ixx="0.01" ixy="0.0" ixz="0.0" iyy="0.01" iyz="0.0" izz="0.03" />
+				</inertial>
+				<visual>
+					<geometry>
+						<mesh filename="package://iai_boxy_base_2/meshes/wheel_front_left.stl" />
+					</geometry>
+					<material name="grey"/>
+				</visual>
+				<collision>
+					<origin xyz="0 0 0" rpy="${pi/2} 0 0" />
+					<geometry>
+						<cylinder radius="0.105" length="0.08"/>
+					</geometry>
+				</collision>
+			</link>
+			<joint name="wheel_back_left_joint" type="revolute">
 				<limit lower="-1000.0" upper="1000.0" effort="200.0" velocity="1.0" />
 				<origin xyz="-0.648 0.09 -0.06" rpy="0.0 0.0 0.0" />
 				<parent link="base_link" />
-				<child link="wheel_left_down" />
-				<axis xyz="0 1 0" />
-			</joint>
-			<link name="wheel_left_down">
-				<inertial>
-					<origin xyz="0 0 0" rpy="0 0 0" />
-					<mass value="2.0" />
-					<inertia ixx="0.01" ixy="0.0" ixz="0.0" iyy="0.01" iyz="0.0" izz="0.03" />
-				</inertial>
-				<visual>
-					<geometry>
-						<mesh filename="package://iai_boxy_base_2/meshes/wheel_left_down.stl" />
-					</geometry>
-				</visual>
-				<collision>
-					<geometry>
-						<mesh filename="package://iai_boxy_base_2/meshes/wheel_collision.stl" />
-					</geometry>
-				</collision>
-			</link>
-			<joint name="wheel_right_up_joint" type="revolute">
+				<child link="wheel_back_left" />
+				<axis xyz="0 1 0" />
+			</joint>
+			<link name="wheel_back_left">
+				<inertial>
+					<origin xyz="0 0 0" rpy="0 0 0" />
+					<mass value="2.0" />
+					<inertia ixx="0.01" ixy="0.0" ixz="0.0" iyy="0.01" iyz="0.0" izz="0.03" />
+				</inertial>
+				<visual>
+					<geometry>
+						<mesh filename="package://iai_boxy_base_2/meshes/wheel_back_left.stl" />
+					</geometry>
+					<material name="grey"/>
+				</visual>
+				<collision>
+					<origin xyz="0 0 0" rpy="${pi/2} 0 0" />
+					<geometry>
+						<cylinder radius="0.105" length="0.08"/>
+					</geometry>
+				</collision>
+			</link>
+			<joint name="wheel_front_right_joint" type="revolute">
 				<limit lower="-1000.0" upper="1000.0" effort="200.0" velocity="1.0" />
 				<origin xyz="0.13 -0.545 -0.06" rpy="0.0 0.0 0.0" />
 				<parent link="base_link" />
-				<child link="wheel_right_up" />
-				<axis xyz="0 1 0" />
-			</joint>
-			<link name="wheel_right_up">
-				<inertial>
-					<origin xyz="0 0 0" rpy="0 0 0" />
-					<mass value="2.0" />
-					<inertia ixx="0.01" ixy="0.0" ixz="0.0" iyy="0.01" iyz="0.0" izz="0.03" />
-				</inertial>
-				<visual>
-					<geometry>
-						<mesh filename="package://iai_boxy_base_2/meshes/wheel_right_up.stl" />
-					</geometry>
-				</visual>
-				<collision>
-					<geometry>
-						<mesh filename="package://iai_boxy_base_2/meshes/wheel_collision.stl" />
-					</geometry>
-				</collision>
-			</link>
-			<joint name="wheel_right_down_joint" type="revolute">
+				<child link="wheel_front_right" />
+				<axis xyz="0 1 0" />
+			</joint>
+			<link name="wheel_front_right">
+				<inertial>
+					<origin xyz="0 0 0" rpy="0 0 0" />
+					<mass value="2.0" />
+					<inertia ixx="0.01" ixy="0.0" ixz="0.0" iyy="0.01" iyz="0.0" izz="0.03" />
+				</inertial>
+				<visual>
+					<geometry>
+						<mesh filename="package://iai_boxy_base_2/meshes/wheel_front_right.stl" />
+					</geometry>
+					<material name="grey"/>
+				</visual>
+				<collision>
+					<origin xyz="0 0 0" rpy="${pi/2} 0 0" />
+					<geometry>
+						<cylinder radius="0.105" length="0.08"/>
+					</geometry>
+				</collision>
+			</link>
+			<joint name="wheel_back_right_joint" type="revolute">
 				<limit lower="-1000.0" upper="1000.0" effort="200.0" velocity="1.0" />
 				<origin xyz="-0.648 -0.545 -0.06" rpy="0.0 0.0 0.0" />
 				<parent link="base_link" />
-				<child link="wheel_right_down" />
-				<axis xyz="0 1 0" />
-			</joint>
-			<link name="wheel_right_down">
-				<inertial>
-					<origin xyz="0 0 0" rpy="0 0 0" />
-					<mass value="2.0" />
-					<inertia ixx="0.01" ixy="0.0" ixz="0.0" iyy="0.01" iyz="0.0" izz="0.03" />
-				</inertial>
-				<visual>
-					<geometry>
-						<mesh filename="package://iai_boxy_base_2/meshes/wheel_right_down.stl" />
-					</geometry>
-				</visual>
-				<collision>
-					<geometry>
-						<mesh filename="package://iai_boxy_base_2/meshes/wheel_collision.stl" />
+				<child link="wheel_back_right" />
+				<axis xyz="0 1 0" />
+			</joint>
+			<link name="wheel_back_right">
+				<inertial>
+					<origin xyz="0 0 0" rpy="0 0 0" />
+					<mass value="2.0" />
+					<inertia ixx="0.01" ixy="0.0" ixz="0.0" iyy="0.01" iyz="0.0" izz="0.03" />
+				</inertial>
+				<visual>
+					<geometry>
+						<mesh filename="package://iai_boxy_base_2/meshes/wheel_back_right.stl" />
+					</geometry>
+					<material name="grey"/>
+				</visual>
+				<collision>
+					<origin xyz="0 0 0" rpy="${pi/2} 0 0" />
+					<geometry>
+						<cylinder radius="0.105" length="0.08"/>
 					</geometry>
 				</collision>

File: iai_donbot_description/robots/iai_donbot_with_refills_finger.urdf.xacro (robot description, xacro)
@@ -4,5 +4,5 @@
   <!-- <xacro:include filename="$(find fingertip_description)/urdf/mod2_fingertip.urdf.xacro"/> -->
   <!-- <link name="map"/> -->
-  <xacro:iai_donbot odom="True" with_wheels="True" with_boxes="False" />
+  <xacro:iai_donbot odom="True" with_wheels="True" with_boxes="True" />
   <joint name="refills_tool_frame_joint" type="fixed">
     <parent link="gripper_tool_frame"/>

Commit message: Fix inertia so mujoco can read it

File: iai_boxy_base_2/robots/base.xacro (robot description, xacro)
@@ -38,5 +38,5 @@
 					<origin xyz="0 0 0" rpy="0 0 0" />
 					<mass value="2.0" />
-					<inertia ixx="0.01" ixy="0.0" ixz="0.0" iyy="0.01" iyz="0.0" izz="0.03" />
+					<inertia ixx="0.01" ixy="0.0" ixz="0.0" iyy="0.01" iyz="0.0" izz="0.01" />
 				</inertial>
 				<visual>
@@ -64,5 +64,5 @@
 					<origin xyz="0 0 0" rpy="0 0 0" />
 					<mass value="2.0" />
-					<inertia ixx="0.01" ixy="0.0" ixz="0.0" iyy="0.01" iyz="0.0" izz="0.03" />
+					<inertia ixx="0.01" ixy="0.0" ixz="0.0" iyy="0.01" iyz="0.0" izz="0.01" />
 				</inertial>
 				<visual>
@@ -90,5 +90,5 @@
 					<origin xyz="0 0 0" rpy="0 0 0" />
 					<mass value="2.0" />
-					<inertia ixx="0.01" ixy="0.0" ixz="0.0" iyy="0.01" iyz="0.0" izz="0.03" />
+					<inertia ixx="0.01" ixy="0.0" ixz="0.0" iyy="0.01" iyz="0.0" izz="0.01" />
 				</inertial>
 				<visual>
@@ -116,5 +116,5 @@
 					<origin xyz="0 0 0" rpy="0 0 0" />
 					<mass value="2.0" />
-					<inertia ixx="0.01" ixy="0.0" ixz="0.0" iyy="0.01" iyz="0.0" izz="0.03" />
+					<inertia ixx="0.01" ixy="0.0" ixz="0.0" iyy="0.01" iyz="0.0" izz="0.01" />
 				</inertial>
 				<visual>

Commit message: [boxy_base_2] lowres collision mesh for the base

File: iai_boxy_base_2/robots/base.xacro (robot description, xacro)
@@ -22,5 +22,5 @@
 				<origin xyz="0 0 0" rpy="0 0 0" />
 				<geometry>
-					<mesh filename="package://iai_boxy_base_2/meshes/base_without_wheels.stl" />
+					<mesh filename="package://iai_boxy_base_2/meshes/base_without_wheels_lowres.stl" />
 				</geometry>
 			</collision>

Commit message: turned donbots plate grey

File: iai_boxy_base_2/robots/base.xacro (robot description, xacro)
@@ -245,5 +245,5 @@
 					<box size="0.6 0.553 0.02" />
 				</geometry>
-				<material name="White" />
+				<material name="Grey" />
 			</visual>
 			<collision>
