Commit message: moved refills tool frame to the front because new fingers are longer

File: iai_donbot_description/robots/iai_donbot2_with_refills_finger.xacro (robot description, xacro)
@@ -7,5 +7,5 @@
     <parent link="gripper_tool_frame"/>
     <child link="refills_tool_frame"/>
-    <origin xyz="0 0 0.012" rpy="0.0 0.0 0.0" />
+    <origin xyz="0 0 0.037" rpy="0.0 0.0 0.0" />
   </joint>
   <link name="refills_tool_frame"/>

Commit message: added boxes for marcos fingers to donbot with marcos fingers urdf

File: iai_donbot_description/robots/iai_donbot2_with_refills_finger.xacro (robot description, xacro)
@@ -17,4 +17,42 @@
   </joint>
   <link name="refills_finger"/>
+  <joint name="marco_left_finger_joint" type="fixed">
+    <parent link="gripper_finger_left_link"/>
+    <child link="marco_left_finger_link"/>
+    <origin xyz="-0.004 0.0 0.115" rpy="0 0 0" />
+  </joint>
+  <link name="marco_left_finger_link">
+    <visual>
+      <geometry>
+        <box size="0.008 0.03 0.13"/>
+      </geometry>
+      <material name="gray"/>
+    </visual>
+    <collision>
+      <geometry>
+        <box size="0.008 0.03 0.13"/>
+      </geometry>
+      <material name="gray"/>
+    </collision>
+  </link>
+  <joint name="marco_right_finger_joint" type="fixed">
+    <parent link="gripper_finger_right_link"/>
+    <child link="marco_right_finger_link"/>
+    <origin xyz="-0.004 0.0 0.115" rpy="0 0 0" />
+  </joint>
+  <link name="marco_right_finger_link">
+    <visual>
+      <geometry>
+        <box size="0.008 0.03 0.13"/>
+      </geometry>
+      <material name="gray"/>
+    </visual>
+    <collision>
+      <geometry>
+        <box size="0.008 0.03 0.13"/>
+      </geometry>
+      <material name="gray"/>
+    </collision>
+  l</link>
   <!-- include the xacro file with the fingertip sensor description //
    instantiate one left fingertip pcb and one for the right

Commit message: fixed typo in donbot urdf

File: iai_donbot_description/robots/iai_donbot2_with_refills_finger.xacro (robot description, xacro)
@@ -54,5 +54,5 @@
       <material name="gray"/>
     </collision>
-  l</link>
+  </link>
   <!-- include the xacro file with the fingertip sensor description //
    instantiate one left fingertip pcb and one for the right
