Commit message: renamed refills scanner robot to donbot

File: iai_donbot_description/robots/iai_donbot.xacro (robot description, xacro)
@@ -28,5 +28,5 @@
   <xacro:property name="arm_mounting_plate_y_offset" value="0.02" />
   <xacro:property name="kms_mounting_plate_height" value="0.016" />
-  <xacro:macro name="refills_scanner_robot">
+  <xacro:macro name="iai_donbot">
     <base/>
 <!--     <joint name="arm_mounting_plate_joint" type="fixed">
@@ -80,5 +80,5 @@
       <visual>
         <geometry>
-          <mesh filename="package://refills_scanner_robot_description/meshes/refills_camera_holder_and_camera.stl" scale="1 1 1"/>
+          <mesh filename="package://donbot_description/meshes/refills_camera_holder_and_camera.stl" scale="1 1 1"/>
         </geometry>
         <material name="gray"/>

Commit message: more donbot renaming

File: iai_donbot_description/robots/iai_donbot.xacro (robot description, xacro)
@@ -80,5 +80,5 @@
       <visual>
         <geometry>
-          <mesh filename="package://donbot_description/meshes/refills_camera_holder_and_camera.stl" scale="1 1 1"/>
+          <mesh filename="package://iai_donbot_description/meshes/refills_camera_holder_and_camera.stl" scale="1 1 1"/>
         </geometry>
         <material name="gray"/>

File: iai_donbot_description/robots/iai_donbot2.xacro (robot description, xacro)
@@ -1,5 +1,5 @@
 <?xml version="1.0"?>
 <robot xmlns:xacro="http://www.ros.org/wiki/xacro" name="iai_donbot">
-  <xacro:include filename="$(find donbot_description)/robots/iai_donbot.xacro"/>
+  <xacro:include filename="$(find iai_donbot_description)/robots/iai_donbot.xacro"/>
   <!-- <link name="map"/> -->
   <iai_donbot/>

Commit message: iai donbot urdf update

File: iai_donbot_description/robots/iai_donbot.xacro (robot description, xacro)
@@ -96,4 +96,10 @@
       <origin xyz="0 -0.075 0.035" rpy="0.261799 0 ${pi}" />
     </joint>
+    <link name="realsense_link"/>
+    <joint name="gripper_to_realsense_joint" type="fixed">
+      <parent link="gripper_base_link" />
+      <child link="camera_link" />
+      <origin xyz="0.022 -0.0405 0.045" rpy="0 0 0" />
+    </joint>
   </xacro:macro>
 </robot>

Commit message: fixed rotation for rs_camera_link

File: iai_donbot_description/robots/iai_donbot.xacro (robot description, xacro)
@@ -96,9 +96,9 @@
       <origin xyz="0 -0.075 0.035" rpy="0.261799 0 ${pi}" />
     </joint>
-    <link name="realsense_link"/>
+    <link name="rs_camera_link"/>
     <joint name="gripper_to_realsense_joint" type="fixed">
       <parent link="gripper_base_link" />
-      <child link="camera_link" />
-      <origin xyz="0.022 -0.0405 0.045" rpy="0 0 0" />
+      <child link="rs_camera_link" />
+      <origin xyz="0.022 0.0405 0.045" rpy="-${pi/2} -${pi/2} 0" />
     </joint>
   </xacro:macro>

Commit message: changed some offsets in donbot xacro

File: iai_donbot_description/robots/iai_donbot.xacro (robot description, xacro)
@@ -100,5 +100,5 @@
       <parent link="gripper_base_link" />
       <child link="rs_camera_link" />
-      <origin xyz="0.022 0.0405 0.045" rpy="-${pi/2} -${pi/2} 0" />
+      <origin xyz="0.032 0.0405 0.045" rpy="-${pi/2} -${pi/2} 0" />
     </joint>
   </xacro:macro>

Commit message: Added a link with the results of the calibration RGB camera -> Intel Realsense camera (Alexis Maldonado)

File: iai_donbot_description/robots/iai_donbot.xacro (robot description, xacro)
@@ -94,11 +94,17 @@
       <parent link="gripper_base_link" />
       <child link="camera_link" />
-      <origin xyz="0 -0.075 0.035" rpy="0.261799 0 ${pi}" />
+      <origin xyz="0 -0.075 0.035" rpy="0.226892 0 ${pi}" />
+    </joint>
+    <link name="rs_camera_link_calib"/>
+    <joint name="wristcam_to_realsense_joint" type="fixed">
+      <parent link="camera_link" />
+      <child link="rs_camera_link_calib" />
+      <origin xyz="-0.017490 -0.106718 0.015236" rpy="6.057290 0.002513 0.003934" />
     </joint>
     <link name="rs_camera_link"/>
-    <joint name="gripper_to_realsense_joint" type="fixed">
-      <parent link="gripper_base_link" />
+    <joint name="orient_fix_realsense_joint" type="fixed">
+      <parent link="rs_camera_link_calib" />
       <child link="rs_camera_link" />
-      <origin xyz="0.032 0.0405 0.045" rpy="-${pi/2} -${pi/2} 0" />
+      <origin xyz="0.0 0.0 0.0" rpy="${pi/2.0} -${pi/2.0} 0.0" />
     </joint>
   </xacro:macro>

Commit message: Calibrated the pose of the Point Grey camera (Alexis Maldonado).

File: iai_donbot_description/robots/iai_donbot.xacro (robot description, xacro)
@@ -94,5 +94,5 @@
       <parent link="gripper_base_link" />
       <child link="camera_link" />
-      <origin xyz="0 -0.075 0.035" rpy="0.226892 0 ${pi}" />
+      <origin xyz="-0.001932 -0.059745 0.084023" rpy="0.217986 0.008285 3.153345" />
     </joint>
     <link name="rs_camera_link_calib"/>

Commit message: moved donbot arm slightly relative to base

File: iai_donbot_description/robots/iai_donbot.xacro (robot description, xacro)
@@ -26,5 +26,5 @@
   <xacro:property name="arm_mounting_plate_height" value="0.006" />
   <xacro:property name="arm_mounting_plate_x_offset" value="0.06" />
-  <xacro:property name="arm_mounting_plate_y_offset" value="0.02" />
+  <xacro:property name="arm_mounting_plate_y_offset" value="0.027" />
   <xacro:property name="kms_mounting_plate_height" value="0.016" />
   <xacro:macro name="iai_donbot">

Commit message: made donbots urdf a child of base_link

File: iai_donbot_description/robots/iai_donbot.xacro (robot description, xacro)
@@ -18,5 +18,5 @@
     <color rgba="0.7 0.7 0.7 1.0"/>
   </material>
-  <xacro:property name="table_height" value="0.63" />
+  <xacro:property name="base_link_to_table_top" value="0.47" />
   <xacro:property name="table_length" value="0.6" />
   <xacro:property name="table_width" value="0.553" />
@@ -25,5 +25,5 @@
   <xacro:property name="arm_mounting_plate_length" value="0.15" />
   <xacro:property name="arm_mounting_plate_height" value="0.006" />
-  <xacro:property name="arm_mounting_plate_x_offset" value="0.06" />
+  <xacro:property name="arm_mounting_plate_x_offset" value="0.0" />
   <xacro:property name="arm_mounting_plate_y_offset" value="0.027" />
   <xacro:property name="kms_mounting_plate_height" value="0.016" />
@@ -33,5 +33,5 @@
       <parent link="base_footprint"/>
       <child link="arm_mounting_plate"/>
-      <origin xyz="${-table_length+arm_mounting_plate_x_offset+arm_mounting_plate_length/2} ${-table_width+arm_mounting_plate_y_offset+arm_mounting_plate_width/2} ${table_height}"/>
+      <origin xyz="${-table_length+arm_mounting_plate_x_offset+arm_mounting_plate_length/2} ${-table_width+arm_mounting_plate_y_offset+arm_mounting_plate_width/2} ${base_link_to_table_top}"/>
     </joint>
     <link name="arm_mounting_plate">
@@ -45,7 +45,7 @@
     <xacro:ur5_robot prefix="${ur5_prefix}" joint_limited="false"/>
     <joint name="arm_base_mounting_joint" type="fixed">
-      <parent link="base_footprint" />
+      <parent link="base_link" />
       <child link="${ur5_prefix}base_link" />
-      <origin xyz="${-(table_length-arm_mounting_plate_length)/2+arm_mounting_plate_x_offset} ${-(table_width-arm_mounting_plate_length)/2+arm_mounting_plate_y_offset} ${table_height}" rpy="0.0 0.0 0.0" />
+      <origin xyz="-0.525 -0.424 0.470" rpy="0.0 0.0 0.0" />
     </joint>
     <link name="kms_mounting_plate">

Commit message: Alexis Maldonado: Adjust the URDF for the new 12mp camera on the wrist

File: iai_donbot_description/robots/iai_donbot.xacro (robot description, xacro)
@@ -90,13 +90,24 @@
       <origin xyz="0 0 0" rpy="0 0 ${pi}" />
     </joint>
+    <link name="fivemp_camera_link"/>
+    <joint name="gripper_to_fivemp_camera_joint" type="fixed">
+      <parent link="gripper_base_link" />
+      <child link="fivemp_camera_link" />
+      <origin xyz="-0.001932 -0.059745 0.084023" rpy="0.217986 0.008285 3.153345" />
+    </joint>
     <link name="camera_link"/>
     <joint name="gripper_to_camera_joint" type="fixed">
       <parent link="gripper_base_link" />
       <child link="camera_link" />
-      <origin xyz="-0.001932 -0.059745 0.084023" rpy="0.217986 0.008285 3.153345" />
+      <!--Calib_errors = [0.003425, 0.2069, 0.00611, 0.42678]
+          Calib_errors = median_pos_error(m), median_orient_error(deg), max_pos_error(m), max_orient_error(deg) -->
+      <!-- from base_link origin xyz="0.004174 -0.067273 0.062438" rpy="0.209203 0.001106 3.120208"/-->
+      <!-- from ur5_base_link origin xyz="0.002956 -0.066498 0.060947" rpy="0.204429 6.281375 3.127197"/-->
+      <!-- calib errors: 0.00311, 0.24373, 0.00688, 0.4558 -->
+      <origin xyz="0.002956 -0.066498 0.060947" rpy="0.204429 6.281375 3.127197" />
     </joint>
     <link name="rs_camera_link_calib"/>
     <joint name="wristcam_to_realsense_joint" type="fixed">
-      <parent link="camera_link" />
+      <parent link="fivemp_camera_link" />
       <child link="rs_camera_link_calib" />
       <origin xyz="-0.017490 -0.106718 0.015236" rpy="6.057290 0.002513 0.003934" />

Commit message: Alexis Maldonado : Fixed pose of the intel camera relative to the rgb camera

File: iai_donbot_description/robots/iai_donbot.xacro (robot description, xacro)
@@ -90,10 +90,4 @@
       <origin xyz="0 0 0" rpy="0 0 ${pi}" />
     </joint>
-    <link name="fivemp_camera_link"/>
-    <joint name="gripper_to_fivemp_camera_joint" type="fixed">
-      <parent link="gripper_base_link" />
-      <child link="fivemp_camera_link" />
-      <origin xyz="-0.001932 -0.059745 0.084023" rpy="0.217986 0.008285 3.153345" />
-    </joint>
     <link name="camera_link"/>
     <joint name="gripper_to_camera_joint" type="fixed">
@@ -107,15 +101,9 @@
       <origin xyz="0.002956 -0.066498 0.060947" rpy="0.204429 6.281375 3.127197" />
     </joint>
-    <link name="rs_camera_link_calib"/>
+    <link name="rs_camera_link"/>
     <joint name="wristcam_to_realsense_joint" type="fixed">
-      <parent link="fivemp_camera_link" />
-      <child link="rs_camera_link_calib" />
-      <origin xyz="-0.017490 -0.106718 0.015236" rpy="6.057290 0.002513 0.003934" />
-    </joint>
-    <link name="rs_camera_link"/>
-    <joint name="orient_fix_realsense_joint" type="fixed">
-      <parent link="rs_camera_link_calib" />
+      <parent link="camera_link" />
       <child link="rs_camera_link" />
-      <origin xyz="0.0 0.0 0.0" rpy="${pi/2.0} -${pi/2.0} 0.0" />
+      <origin xyz="-0.017993 -0.107556 0.017699" rpy="6.270618 4.930698 1.578454"/>
     </joint>
   </xacro:macro>

Commit message: donbots camera holder link now has a collision entry

File: iai_donbot_description/robots/iai_donbot.xacro (robot description, xacro)
@@ -84,4 +84,10 @@
         <material name="gray"/>
       </visual>
+      <collision>
+        <geometry>
+          <mesh filename="package://iai_donbot_description/meshes/refills_camera_holder_and_camera.stl" scale="1 1 1"/>
+        </geometry>
+        <material name="gray"/>
+      </collision>
     </link>
     <joint name="gripper_to_camera_holder_joint" type="fixed">

Commit message: added boxes to donbot urdf that cover switches, chargers etc

File: iai_donbot_description/robots/iai_donbot.xacro (robot description, xacro)
@@ -17,4 +17,7 @@
   <material name="Grey">
     <color rgba="0.7 0.7 0.7 1.0"/>
+  </material>
+  <material name="yellow">
+    <color rgba="1.0 1.0 0.0 1.0"/>
   </material>
   <xacro:property name="base_link_to_table_top" value="0.47" />
@@ -113,4 +116,100 @@
       <origin xyz="-0.017993 -0.107556 0.017699" rpy="6.270618 4.930698 1.578454"/>
     </joint>
+    <!-- boxes to cover up switches and stuff -->
+    <joint name="switches_joint" type="fixed">
+      <parent link="base_link" />
+      <child link="switches" />
+      <origin xyz="-0.66 -0.225 0.225" rpy="0 0 0" />
+    </joint>
+    <link name="switches">
+      <visual>
+        <geometry>
+          <box size="0.12 0.4 0.45"/>
+        </geometry>
+        <material name="Silver"/>
+      </visual>
+      <collision>
+        <geometry>
+          <box size="0.12 0.4 0.45"/>
+        </geometry>
+        <material name="Silver"/>
+      </collision>
+    </link>
+    <joint name="charger_joint" type="fixed">
+      <parent link="base_link" />
+      <child link="charger" />
+      <origin xyz="0.075 -0.225 0.19" rpy="0 0 0" />
+    </joint>
+    <link name="charger">
+      <visual>
+        <geometry>
+          <box size="0.15 0.3 0.38"/>
+        </geometry>
+        <material name="Silver"/>
+      </visual>
+      <collision>
+        <geometry>
+          <box size="0.15 0.3 0.38"/>
+        </geometry>
+        <material name="Silver"/>
+      </collision>
+    </link>
+    <joint name="e_stop_joint" type="fixed">
+      <parent link="base_link" />
+      <child link="e_stop" />
+      <origin xyz="-0.035 -0.0015 0.52" rpy="0 0 0" />
+    </joint>
+    <link name="e_stop">
+      <visual>
+        <geometry>
+          <box size="0.07 0.07 0.1"/>
+        </geometry>
+        <material name="yellow"/>
+      </visual>
+      <collision>
+        <geometry>
+          <box size="0.07 0.07 0.1"/>
+        </geometry>
+        <material name="yellow"/>
+      </collision>
+    </link>
+    <joint name="wlan_joint" type="fixed">
+      <parent link="base_link" />
+      <child link="wlan" />
+      <origin xyz="0.05 -0.225 0.405" rpy="0 -0.314 0" />
+    </joint>
+    <link name="wlan">
+      <visual>
+        <geometry>
+          <box size="0.25 0.14 0.05"/>
+        </geometry>
+        <material name="Silver"/>
+      </visual>
+      <collision>
+        <geometry>
+          <box size="0.25 0.14 0.05"/>
+        </geometry>
+        <material name="Silver"/>
+      </collision>
+    </link>
+    <joint name="ur5_touchpad_joint" type="fixed">
+      <parent link="base_link" />
+      <child link="ur5_touchpad" />
+      <origin xyz="-0.16 -0.5355 0.38" rpy="0 0 0" />
+    </joint>
+    <link name="ur5_touchpad">
+      <visual>
+        <geometry>
+          <box size="0.32 0.06 0.24"/>
+        </geometry>
+        <material name="Silver"/>
+      </visual>
+      <collision>
+        <geometry>
+          <box size="0.32 0.06 0.24"/>
+        </geometry>
+        <material name="Silver"/>
+      </collision>
+    </link>
   </xacro:macro>
 </robot>

Commit message: added collision cylinder to donbots wrist

File: iai_donbot_description/robots/iai_donbot.xacro (robot description, xacro)
@@ -212,4 +212,17 @@
       </collision>
     </link>
+    <joint name="wrist_collision_joint" type="fixed">
+      <parent link="adapter_kms40_fwk050_frame_in" />
+      <child link="wrist_collision" />
+      <origin xyz="0 0 -0.005" rpy="0 0 0" />
+    </joint>
+    <link name="wrist_collision">
+      <collision>
+        <geometry>
+          <cylinder radius="0.04" length="0.08"/>
+        </geometry>
+        <material name="Silver"/>
+      </collision>
+    </link>
   </xacro:macro>
 </robot>
