Commit message: Re-introduced odometry joints that got lost in merge commit.

File: iai_boxy_description/urdf/boxy_description.urdf.xacro (robot description, xacro)
@@ -24,4 +24,37 @@
 	<xacro:include filename="$(find iai_boxy_base)/robots/base.URDF" />
         <xacro:macro name="boxy">
+        <!-- virtual joints to model odometry -->
+        <link name="odom" />
+        <joint name="odom_x_joint" type="prismatic">
+          <parent link="odom"/>
+          <child link="odom_x_frame"/>
+          <axis xyz="1 0 0"/>
+         <!-- limits chosen heuristically
+              lower/upper: +-1km to create a quasi limitless prismatic joint
+              velocity: slow walking speed is 3-4km/hour ~= 1m/s
+              effort: reach max speed within 1s, Boxy has a mass of 200kg, so Fmax=200kg*1m/s2 -->
+          <limit lower="-1000" upper="1000" velocity="1" effort="200"/>
+        </joint>
+        <link name="odom_x_frame" />
+        <joint name="odom_y_joint" type="prismatic">
+          <parent link="odom_x_frame"/>
+          <child link="odom_y_frame"/>
+          <axis xyz="0 1 0"/>
+          <!-- limits chosen heuristically
+               lower/upper: +-1km to create a quasi limitless prismatic joint
+               velocity: slow walking speed is 3-4km/hour ~= 1m/s
+               effort: reach max speed within 1s, Boxy has a mass of 200kg, so Fmax=200kg*1m/s2 -->
+          <limit lower="-1000" upper="1000" velocity="1" effort="200"/>
+        </joint>
+        <link name="odom_y_frame" />
+        <joint name="odom_z_joint" type="continuous">
+          <parent link="odom_y_frame"/>
+          <child link="base_footprint"/>
+          <axis xyz="0 0 1"/>
+          <!-- limits chosen heuristically
+               velocity: one slow complete turn around in 5-6s, so 6.2rad/6s ~= 1rad/s
+               effort: reach max speed within 1s, Boxy has a mass of 200kg and a diagonale of 1m, so Fmax=200kg*1m*1m/s2 -->
+          <limit velocity="1" effort="200"/>
+        </joint>
 	<link name="base_footprint">
     <visual>

Commit message: Fix Boxy's URDF to orient the FT sensor right

File: iai_boxy_description/urdf/boxy_description.urdf.xacro (robot description, xacro)
@@ -148,5 +148,5 @@
         <!-- The following URDFs have frame_in / frame_out, so they are simply placed at their parent -->
         <kms_40_xacro parent="left_arm_cabling_adaptor_link" prefix="left_arm_">
-          <origin xyz="0 0 0" rpy="0 0 3.14159265359" />  <!--places the kms40 frame 13mm from the parent -->
+          <origin xyz="0 0 0" rpy="0 0 0" />  <!--places the kms40 frame 13mm from the parent -->
         </kms_40_xacro>
         <adapter_kms40_fwk050_xacro parent="left_arm_kms40_frame_out" prefix="left_arm_">
@@ -160,5 +160,5 @@
         </adapter_fwa050_wsg50_xacro>
         <wsg_50_xacro name="left_gripper" parent="left_arm_adapter_fwa050_wsg50_frame_out">
-          <origin xyz="0 0 0" rpy="0 0 3.14159265359"/>
+          <origin xyz="0 0 0" rpy="0 0 0"/>
 	</wsg_50_xacro>
   <link name="left_wrist_optical_frame_x">

Commit message: Remove the shoulder kinect

File: iai_boxy_description/urdf/boxy_description.urdf.xacro (robot description, xacro)
@@ -6,5 +6,5 @@
 	<xacro:include filename="$(find iai_kms_40_description)/urdf/kms_40.urdf.xacro"/>
   <xacro:include filename="$(find iai_adapters_description)/urdf/lwr4_cabling_adaptor.urdf.xacro" />
-	<xacro:include filename="$(find iai_kinect_description)/urdf/kinect.urdf.xacro"/>
+	<!--xacro:include filename="$(find iai_kinect_description)/urdf/kinect.urdf.xacro"/-->
 	<xacro:include filename="$(find iai_adapters_description)/urdf/adapter_fwa050_wsg50.urdf.xacro"/>
 	<xacro:include filename="$(find iai_adapters_description)/urdf/adapter_kms40_fwk050.urdf.xacro"/>
@@ -122,10 +122,8 @@
              translation: -0.135394 -0.00764754 1.54755 (xyz)
              quaternion: 0.0177781 0.202257 -0.0472198 0.978032 (xyzw) -->
-        <kinect name="shoulder_kinect" parent="base_link">
-          <!--<origin xyz="-0.135394 -0.00764754 1.54755"
-                  rpy="0.01708077682636155 0.4085798647123734 -0.09294704527264909"/> -->
-					<origin xyz="0.0405394 -0.52064754 1.47001"
+        <!--kinect name="shoulder_kinect" parent="base_link">
+		<origin xyz="0.0405394 -0.52064754 1.47001"
                   rpy="0.01708077682636155 0.0085798647123734 -0.00929470452726490"/>
-       </kinect>
+       </kinect-->
 	<!-- JOINT to connect the base with the torso -->
 	<joint name="torso_joint" type="fixed">
