Commit message: Update boxy urdf, use new ur3 xacro.

File: iai_boxy_description/urdf/boxy_description.urdf.xacro (robot description, xacro)
@@ -11,5 +11,5 @@
   <xacro:include filename="$(find iai_adapters_description)/urdf/fwk_fwa_050.urdf.xacro"/>
   <xacro:include filename="$(find iai_adapters_description)/urdf/adapter_boxy_ur3.urdf.xacro"/>
-  <xacro:include filename="$(find iai_ur_description)/urdf/ur3.urdf.xacro"/>
+  <xacro:include filename="$(find ur_description)/urdf/ur3.urdf.xacro"/>
   <xacro:include filename="$(find iai_kinect2_description)/urdf/kinect2.urdf.xacro"/>
   <xacro:include filename="$(find iai_adapter_iso50_kinect2_description)/urdf/adapter_iso50_kinect2.urdf.xacro"/>
@@ -83,48 +83,21 @@
     <!-- NEW NECK ASSEMBLY -->
     <!-- mounting plate of UR3 -->
-    <adapter_boxy_ur3_xacro prefix="neck_" parent="base_link">
+    <xacro:property name="ur3_prefix" value="neck_"/>
+    <adapter_boxy_ur3_xacro prefix="${ur3_prefix}" parent="base_link">
       <origin xyz="0.175 -0.227 1.48" rpy="0 0 0"/>
     </adapter_boxy_ur3_xacro>
-    <xacro:ur3_robot prefix="neck_" parent="neck_adapter_ur3_frame_out" joint_limited="true">
-      <origin xyz="0.0 0.0 0.0" rpy="0.0 0.0 -${M_PI/2.0}"/>
-    </xacro:ur3_robot>
+    <xacro:ur3_robot prefix="${ur3_prefix}" joint_limited="true" transmission_hw_interface="$(arg transmission_hw_interface)" kinematics_file="${load_yaml('$(arg kinematics_config)')}"/>
+    <joint name="${ur3_prefix}base_mounting_joint" type="fixed">
+      <parent link="${ur3_prefix}adapter_ur3_frame_out" />
+      <child link="${ur3_prefix}base_link" />
+      <origin xyz="0.0 0.0 0.0" rpy="0.0 0.0 -${M_PI/1.0}"/>
+    </joint>
     <!-- The following URDF has frame_in / frame_out, so it is placed at the parent -->
     <adapter_iso50_kinect2_xacro parent="neck_tool0" prefix="neck">
       <origin xyz="0 0 0" rpy="0 0 -1.570795"/>
     </adapter_iso50_kinect2_xacro>
-    <!-- /NEW NECK ASSEMBLY -->
-    <!-- OLD NEW ASSEMBLY -->
-    <!-- JOINT to connect the base with the pw070 -->
-    <!--joint name="head_joint" type="fixed">
-		<parent link="base_link" />
-		<child link="pw070_base_link" />
-	</joint-->
-    <!-- /JOINT to connect the base with the pw070 -->
-    <!--xacro:include filename="$(find iai_schunk_pw070_v6)/robots/pw070_v6.URDF" /-->
-    <!-- Kinect2 -->
-    <!-- Pose comes from tool_H_clink in the calibration
-             The quaternion was converted to RPY using python and KDL
-               halcon has quat: w x y z
-               kdl and tf_static_transform_publisher use: x y z w
-             So take the first number from the halcon quat and put it last for KDL.
-               import PyKDL as p; r2 = p.Rotation.Quaternion(-0.494547,0.491515,-0.506787,0.506955) ; r2.GetRPY()
-               answer: (-1.5431199762943342, -0.0029080109443817533, -1.5676362600579434) -->
-    <!-- The following kinect2_xacro defines the _kinect2_rgb_optical_frame
-        And includes the fixed joint to place the kinect on the pw070  -->
     <kinect2_xacro parent="neck_adapter_iso50_kinect2_frame_out" prefix="head_mount">
-      <!-- From CAD -->
-      <!--origin xyz="-0.02 0.10 0.02" rpy="-1.570795 0 1.570795" /-->
-      <!-- From Halcon calibration on 20160902 -->
       <origin xyz="-0.031284 0.098627 0.023544" rpy="4.728550 6.279385 1.578295"/>
     </kinect2_xacro>
-    <!-- shoulder kinect -->
-    <!-- ORIGINAL DATA FROM HALCON CALIBRATION:
-             from: base_link to: shoulder_kinect_link
-             translation: -0.135394 -0.00764754 1.54755 (xyz)
-             quaternion: 0.0177781 0.202257 -0.0472198 0.978032 (xyzw) -->
-    <!--kinect name="shoulder_kinect" parent="base_link">
-		<origin xyz="0.0405394 -0.52064754 1.47001"
-                  rpy="0.01708077682636155 0.0085798647123734 -0.00929470452726490"/>
-       </kinect-->
     <!-- JOINT to connect the base with the torso -->
     <joint name="torso_joint" type="fixed">

Commit message: Turn UR3 base link by 90 degree.

File: iai_boxy_description/urdf/boxy_description.urdf.xacro (robot description, xacro)
@@ -91,5 +91,5 @@
       <parent link="${ur3_prefix}adapter_ur3_frame_out" />
       <child link="${ur3_prefix}base_link" />
-      <origin xyz="0.0 0.0 0.0" rpy="0.0 0.0 -${M_PI/1.0}"/>
+      <origin xyz="0.0 0.0 0.0" rpy="0.0 0.0 -${M_PI/2.0}"/>
     </joint>
     <!-- The following URDF has frame_in / frame_out, so it is placed at the parent -->

Commit message: Update boxy related ur3 description and general ur urdfs.

File: iai_boxy_description/urdf/boxy_description.urdf.xacro (robot description, xacro)
@@ -11,5 +11,5 @@
   <xacro:include filename="$(find iai_adapters_description)/urdf/fwk_fwa_050.urdf.xacro"/>
   <xacro:include filename="$(find iai_adapters_description)/urdf/adapter_boxy_ur3.urdf.xacro"/>
-  <xacro:include filename="$(find ur_description)/urdf/ur3.urdf.xacro"/>
+  <xacro:include filename="$(find iai_ur_description)/urdf/ur3.urdf.xacro"/>
   <xacro:include filename="$(find iai_kinect2_description)/urdf/kinect2.urdf.xacro"/>
   <xacro:include filename="$(find iai_adapter_iso50_kinect2_description)/urdf/adapter_iso50_kinect2.urdf.xacro"/>

File: iai_ur_description/urdf/common.gazebo.xacro (robot description, xacro)
@@ -1,4 +1,4 @@
 <?xml version="1.0"?>
-<robot xmlns:xacro="http://www.ros.org/wiki/xacro">
+<robot xmlns:xacro="http://wiki.ros.org/xacro">
   <gazebo>
     <plugin name="ros_control" filename="libgazebo_ros_control.so">

File: iai_ur_description/urdf/ur.transmission.xacro (robot description, xacro)
@@ -1,46 +1,58 @@
 <?xml version="1.0"?>
-<robot xmlns:xacro="http://www.ros.org/wiki/xacro">
-  <xacro:macro name="ur_arm_transmission" params="prefix">
-    <transmission
-      name="${prefix}shoulder_pan_trans"
-      type="pr2_mechanism_model/SimpleTransmission">
-      <actuator name="${prefix}shoulder_pan_motor"/>
-      <joint name="${prefix}shoulder_pan_joint"/>
-      <mechanicalReduction>1.0</mechanicalReduction>
+<robot xmlns:xacro="http://wiki.ros.org/xacro">
+  <xacro:macro name="ur_arm_transmission" params="prefix hw_interface">
+    <transmission name="${prefix}shoulder_pan_trans">
+      <type>transmission_interface/SimpleTransmission</type>
+      <joint name="${prefix}shoulder_pan_joint">
+        <hardwareInterface>${hw_interface}</hardwareInterface>
+      </joint>
+      <actuator name="${prefix}shoulder_pan_motor">
+        <mechanicalReduction>1</mechanicalReduction>
+      </actuator>
     </transmission>
-    <transmission
-      name="${prefix}shoulder_lift_trans"
-      type="pr2_mechanism_model/SimpleTransmission">
-      <actuator name="${prefix}shoulder_lift_motor"/>
-      <joint name="${prefix}shoulder_lift_joint"/>
-      <mechanicalReduction>1.0</mechanicalReduction>
+    <transmission name="${prefix}shoulder_lift_trans">
+      <type>transmission_interface/SimpleTransmission</type>
+      <joint name="${prefix}shoulder_lift_joint">
+        <hardwareInterface>${hw_interface}</hardwareInterface>
+      </joint>
+      <actuator name="${prefix}shoulder_lift_motor">
+        <mechanicalReduction>1</mechanicalReduction>
+      </actuator>
     </transmission>
-    <transmission
-      name="${prefix}elbow_trans"
-      type="pr2_mechanism_model/SimpleTransmission">
-      <actuator name="${prefix}elbow_motor"/>
-      <joint name="${prefix}elbow_joint"/>
-      <mechanicalReduction>1.0</mechanicalReduction>
+    <transmission name="${prefix}elbow_trans">
+      <type>transmission_interface/SimpleTransmission</type>
+      <joint name="${prefix}elbow_joint">
+        <hardwareInterface>${hw_interface}</hardwareInterface>
+      </joint>
+      <actuator name="${prefix}elbow_motor">
+        <mechanicalReduction>1</mechanicalReduction>
+      </actuator>
     </transmission>
-    <transmission
-      name="${prefix}wrist_1_trans"
-      type="pr2_mechanism_model/SimpleTransmission">
-      <actuator name="${prefix}wrist_1_motor"/>
-      <joint name="${prefix}wrist_1_joint"/>
-      <mechanicalReduction>1.0</mechanicalReduction>
+    <transmission name="${prefix}wrist_1_trans">
+      <type>transmission_interface/SimpleTransmission</type>
+      <joint name="${prefix}wrist_1_joint">
+        <hardwareInterface>${hw_interface}</hardwareInterface>
+      </joint>
+      <actuator name="${prefix}wrist_1_motor">
+        <mechanicalReduction>1</mechanicalReduction>
+      </actuator>
     </transmission>
-    <transmission
-      name="${prefix}wrist_2_trans"
-      type="pr2_mechanism_model/SimpleTransmission">
-      <actuator name="${prefix}wrist_2_motor"/>
-      <joint name="${prefix}wrist_2_joint"/>
-      <mechanicalReduction>1.0</mechanicalReduction>
+    <transmission name="${prefix}wrist_2_trans">
+      <type>transmission_interface/SimpleTransmission</type>
+      <joint name="${prefix}wrist_2_joint">
+        <hardwareInterface>${hw_interface}</hardwareInterface>
+      </joint>
+      <actuator name="${prefix}wrist_2_motor">
+        <mechanicalReduction>1</mechanicalReduction>
+      </actuator>
     </transmission>
-    <transmission
-      name="${prefix}wrist_3_trans"
-      type="pr2_mechanism_model/SimpleTransmission">
-      <actuator name="${prefix}wrist_3_motor"/>
-      <joint name="${prefix}wrist_3_joint"/>
-      <mechanicalReduction>1.0</mechanicalReduction>
+    <transmission name="${prefix}wrist_3_trans">
+      <type>transmission_interface/SimpleTransmission</type>
+      <joint name="${prefix}wrist_3_joint">
+        <hardwareInterface>${hw_interface}</hardwareInterface>
+      </joint>
+      <actuator name="${prefix}wrist_3_motor">
+        <mechanicalReduction>1</mechanicalReduction>
+      </actuator>
     </transmission>
   </xacro:macro>
