Commit message: Update boxy related ur3 description and general ur urdfs.

File: iai_ur_description/urdf/ur3.urdf.xacro (robot description, xacro)
@@ -1,4 +1,4 @@
 <?xml version="1.0"?>
-<robot xmlns:xacro="http://www.ros.org/wiki/xacro">
+<robot xmlns:xacro="http://wiki.ros.org/xacro">
 <!--
   Author: Felix Messmer
@@ -6,41 +6,4 @@
   <xacro:include filename="$(find iai_ur_description)/urdf/ur.transmission.xacro" />
   <xacro:include filename="$(find iai_ur_description)/urdf/ur.gazebo.xacro" />
-  <xacro:property name="pi" value="3.14159265" />
-  <!-- Inertia parameters -->
-  <xacro:property name="base_mass" value="2.0" />  <!-- This mass might be incorrect -->
-  <xacro:property name="shoulder_mass" value="2.0" />
-  <xacro:property name="upper_arm_mass" value="3.42" />
-  <xacro:property name="forearm_mass" value="1.26" />
-  <xacro:property name="wrist_1_mass" value="0.8" />
-  <xacro:property name="wrist_2_mass" value="0.8" />
-  <xacro:property name="wrist_3_mass" value="0.35" />
-  <!-- These parameters are borrowed from the urcontrol.conf file
-       but are not verified for the correct permutation.
-       The permutation was guessed by looking at the UR5 parameters.
-       Serious use of these parameters needs further inspection. -->
-  <xacro:property name="shoulder_cog" value="0.0 -0.02 0.0" />
-  <xacro:property name="upper_arm_cog" value="0.13 0.0 0.1157" />
-  <xacro:property name="forearm_cog" value="0.05 0.0 0.0238" />
-  <xacro:property name="wrist_1_cog" value="0.0 0.0 0.01" />
-  <xacro:property name="wrist_2_cog" value="0.0 0.0 0.01" />
-  <xacro:property name="wrist_3_cog" value="0.0 0.0 -0.02" />
-  <!-- Kinematic model -->
-  <!-- Properties from urcontrol.conf -->
-  <xacro:property name="ur3_d1" value="0.1519" />
-  <xacro:property name="ur3_a2" value="-0.24365" />
-  <xacro:property name="ur3_a3" value="-0.21325" />
-  <xacro:property name="ur3_d4" value="0.11235" />
-  <xacro:property name="ur3_d5" value="0.08535" />
-  <xacro:property name="ur3_d6" value="0.0819" />
-  <!-- Arbitrary offsets for shoulder/elbow joints -->
-  <xacro:property name="shoulder_offset" value="0.1198" />  <!-- measured from model -->
-  <xacro:property name="elbow_offset" value="-0.0925" /> <!-- measured from model -->
-  <!-- link lengths used in model -->
-  <xacro:property name="shoulder_height" value="${ur3_d1}" />
-  <xacro:property name="upper_arm_length" value="${-ur3_a2}" />
-  <xacro:property name="forearm_length" value="${-ur3_a3}" />
-  <xacro:property name="wrist_1_length" value="${ur3_d4 - elbow_offset - shoulder_offset}" />
-  <xacro:property name="wrist_2_length" value="${ur3_d5}" />
-  <xacro:property name="wrist_3_length" value="${ur3_d6}" />
   <xacro:macro name="cylinder_inertial" params="radius length mass *origin">
     <inertial>
@@ -52,12 +15,43 @@
     </inertial>
   </xacro:macro>
-  <xacro:macro name="ur3_robot" params="prefix parent joint_limited *origin">
-    <joint name="${prefix}mounting_joint" type="fixed">
-      <parent link="${parent}" />
-      <child link="${prefix}base_link" />
-      <xacro:insert_block name="origin"/>
-    </joint>
+  <xacro:macro name="ur3_robot" params="prefix joint_limited
+    shoulder_pan_lower_limit:=${-pi}    shoulder_pan_upper_limit:=${pi}
+    shoulder_lift_lower_limit:=${-pi}    shoulder_lift_upper_limit:=${pi}
+    elbow_joint_lower_limit:=${-pi}    elbow_joint_upper_limit:=${pi}
+    wrist_1_lower_limit:=${-pi}    wrist_1_upper_limit:=${pi}
+    wrist_2_lower_limit:=${-pi}    wrist_2_upper_limit:=${pi}
+    wrist_3_lower_limit:=${-pi}    wrist_3_upper_limit:=${pi}
+    transmission_hw_interface:=hardware_interface/PositionJointInterface
+    safety_limits:=false safety_pos_margin:=0.15
+    safety_k_position:=20
+    kinematics_file">
+    <xacro:property name="__kinematics" value="${kinematics_file['kinematics']}"/>
+    <!-- Inertia parameters -->
+    <xacro:property name="base_mass" value="2.0" />  <!-- This mass might be incorrect -->
+    <xacro:property name="shoulder_mass" value="2.0" />
+    <xacro:property name="upper_arm_mass" value="3.42" />
+    <xacro:property name="forearm_mass" value="1.26" />
+    <xacro:property name="wrist_1_mass" value="0.8" />
+    <xacro:property name="wrist_2_mass" value="0.8" />
+    <xacro:property name="wrist_3_mass" value="0.35" />
+    <!-- These parameters are borrowed from the urcontrol.conf file
+        but are not verified for the correct permutation.
+        The permutation was guessed by looking at the UR5 parameters.
+        Serious use of these parameters needs further inspection. -->
+    <xacro:property name="shoulder_cog" value="0.0 -0.02 0.0" />
+    <xacro:property name="upper_arm_cog" value="0.13 0.0 0.1157" />
+    <xacro:property name="forearm_cog" value="0.05 0.0 0.0238" />
+    <xacro:property name="wrist_1_cog" value="0.0 0.0 0.01" />
+    <xacro:property name="wrist_2_cog" value="0.0 0.0 0.01" />
+    <xacro:property name="wrist_3_cog" value="0.0 0.0 -0.02" />
+    <!-- Arbitrary offsets for shoulder/elbow joints -->
+    <xacro:property name="shoulder_offset" value="0.1198" />  <!-- measured from model -->
+    <xacro:property name="elbow_offset" value="0.0275" /> <!-- measured from model -->
+    <xacro:property name="upper_arm_inertia_offset" value="0.12" />  <!-- measured from model -->
+    <!-- This is for compatibility reasons, as transformation between base and base_link was always 180 degree in the iai_ur_description -->
+    <xacro:property name="base_correction" value="${pi}" />
     <link name="${prefix}base_link" >
       <visual>
+        <origin xyz="0 0 0" rpy="0 0 ${base_correction}"/>
         <geometry>
           <mesh filename="package://iai_ur_description/meshes/ur3/visual/base.dae"/>
@@ -68,4 +62,5 @@
       </visual>
       <collision>
+        <origin xyz="0 0 0" rpy="0 0 ${base_correction}"/>
         <geometry>
           <mesh filename="package://iai_ur_description/meshes/ur3/collision/base.stl"/>
@@ -79,12 +74,17 @@
       <parent link="${prefix}base_link" />
       <child link = "${prefix}shoulder_link" />
-      <origin xyz="0.0 0.0 ${shoulder_height}" rpy="0.0 0.0 0.0" />
+      <origin xyz="${__kinematics['shoulder']['x']} ${__kinematics['shoulder']['y']} ${__kinematics['shoulder']['z']}" rpy="${__kinematics['shoulder']['roll']} ${__kinematics['shoulder']['pitch']} ${__kinematics['shoulder']['yaw'] + base_correction}" />
       <axis xyz="0 0 1" />
       <xacro:unless value="${joint_limited}">
         <limit lower="${-2.0 * pi}" upper="${2.0 * pi}" effort="330.0" velocity="2.16"/>
-      </xacro:unless>
-      <xacro:if value="${joint_limited}">
-        <!--limit lower="${-pi}" upper="${pi}" effort="330.0" velocity="2.16"/-->
-				<limit lower="${-1.5*pi}" upper="${1.5*pi}" effort="330.0" velocity="2.16"/>
+        <xacro:if value="${safety_limits}">
+          <safety_controller soft_lower_limit="${-2.0 * pi + safety_pos_margin}" soft_upper_limit="${2.0 * pi - safety_pos_margin}" k_position="${safety_k_position}" k_velocity="0.0"/>
+        </xacro:if>
+      </xacro:unless>
+      <xacro:if value="${joint_limited}">
+        <limit lower="${shoulder_pan_lower_limit}" upper="${shoulder_pan_upper_limit}" effort="330.0" velocity="2.16"/>
+        <xacro:if value="${safety_limits}">
+          <safety_controller soft_lower_limit="${shoulder_pan_lower_limit + safety_pos_margin}" soft_upper_limit="${shoulder_pan_upper_limit - safety_pos_margin}" k_position="${safety_k_position}" k_velocity="0.0"/>
+        </xacro:if>
       </xacro:if>
       <dynamics damping="0.0" friction="0.0"/>
@@ -92,4 +92,5 @@
     <link name="${prefix}shoulder_link">
       <visual>
+        <origin xyz="0 0 0" rpy="0 0 ${pi}"/>
         <geometry>
           <mesh filename="package://iai_ur_description/meshes/ur3/visual/shoulder.dae"/>
@@ -100,4 +101,5 @@
       </visual>
       <collision>
+        <origin xyz="0 0 0" rpy="0 0 ${pi}"/>
         <geometry>
           <mesh filename="package://iai_ur_description/meshes/ur3/collision/shoulder.stl"/>
@@ -111,11 +113,17 @@
       <parent link="${prefix}shoulder_link" />
       <child link = "${prefix}upper_arm_link" />
-      <origin xyz="0.0 ${shoulder_offset} 0.0" rpy="0.0 ${pi / 2.0} 0.0" />
-      <axis xyz="0 1 0" />
+      <origin xyz="${__kinematics['upper_arm']['x']} ${__kinematics['upper_arm']['y']} ${__kinematics['upper_arm']['z']}" rpy="${__kinematics['upper_arm']['roll']} ${__kinematics['upper_arm']['pitch']} ${__kinematics['upper_arm']['yaw']}" />
+      <axis xyz="0 0 1" />
       <xacro:unless value="${joint_limited}">
         <limit lower="${-2.0 * pi}" upper="${2.0 * pi}" effort="330.0" velocity="2.16"/>
-      </xacro:unless>
-      <xacro:if value="${joint_limited}">
-        <limit lower="${-1.2 * pi}" upper="${1.2 * pi}" effort="330.0" velocity="2.16"/>
+        <xacro:if value="${safety_limits}">
+          <safety_controller soft_lower_limit="${-2.0 * pi + safety_pos_margin}" soft_upper_limit="${2.0 * pi - safety_pos_margin}" k_position="${safety_k_position}" k_velocity="0.0"/>
+        </xacro:if>
+      </xacro:unless>
+      <xacro:if value="${joint_limited}">
+        <limit lower="${shoulder_lift_lower_limit}" upper="${shoulder_lift_upper_limit}" effort="330.0" velocity="2.16"/>
+        <xacro:if value="${safety_limits}">
+          <safety_controller soft_lower_limit="${shoulder_lift_lower_limit + safety_pos_margin}" soft_upper_limit="${shoulder_lift_upper_limit - safety_pos_margin}" k_position="${safety_k_position}" k_velocity="0.0"/>
+        </xacro:if>
       </xacro:if>
       <dynamics damping="0.0" friction="0.0"/>
@@ -123,4 +131,5 @@
     <link name="${prefix}upper_arm_link">
       <visual>
+        <origin xyz="0 0 ${shoulder_offset}" rpy="${pi/2} 0 ${-pi/2}"/>
         <geometry>
           <mesh filename="package://iai_ur_description/meshes/ur3/visual/upperarm.dae"/>
@@ -131,10 +140,11 @@
       </visual>
       <collision>
+        <origin xyz="0 0 ${shoulder_offset}" rpy="${pi/2} 0 ${-pi/2}"/>
         <geometry>
           <mesh filename="package://iai_ur_description/meshes/ur3/collision/upperarm.stl"/>
         </geometry>
       </collision>
-      <xacro:cylinder_inertial radius="0.075" length="${-ur3_a2}" mass="${upper_arm_mass}">
-        <origin xyz="0.0 0.0 ${-ur3_a2/2.0}" rpy="0 0 0" />
+      <xacro:cylinder_inertial radius="0.075" length="${-1*__kinematics['forearm']['x']}" mass="${upper_arm_mass}">
+        <origin xyz="${0.5*__kinematics['forearm']['x']} 0.0 ${upper_arm_inertia_offset}" rpy="0 ${pi/2} 0" />
       </xacro:cylinder_inertial>
     </link>
@@ -142,11 +152,17 @@
       <parent link="${prefix}upper_arm_link" />
       <child link = "${prefix}forearm_link" />
-      <origin xyz="0.0 ${elbow_offset} ${upper_arm_length}" rpy="0.0 0.0 0.0" />
-      <axis xyz="0 1 0" />
-      <xacro:unless value="${joint_limited}">
-        <limit lower="${-2.0 * pi}" upper="${2.0 * pi}" effort="150.0" velocity="3.15"/>
-      </xacro:unless>
-      <xacro:if value="${joint_limited}">
-        <limit lower="${-1.2 * pi}" upper="${1.2 * pi}" effort="150.0" velocity="3.15"/>
+      <origin xyz="${__kinematics['forearm']['x']} ${__kinematics['forearm']['y']} ${__kinematics['forearm']['z']}" rpy="${__kinematics['forearm']['roll']} ${__kinematics['forearm']['pitch']} ${__kinematics['forearm']['yaw']}" />
+      <axis xyz="0 0 1" />
+      <xacro:unless value="${joint_limited}">
+        <limit lower="${-pi}" upper="${pi}" effort="150.0" velocity="3.15"/>
+        <xacro:if value="${safety_limits}">
+          <safety_controller soft_lower_limit="${-2.0 * pi + safety_pos_margin}" soft_upper_limit="${2.0 * pi - safety_pos_margin}" k_position="${safety_k_position}" k_velocity="0.0"/>
+        </xacro:if>
+      </xacro:unless>
+      <xacro:if value="${joint_limited}">
+        <limit lower="${elbow_joint_lower_limit}" upper="${elbow_joint_upper_limit}" effort="150.0" velocity="3.15"/>
+        <xacro:if value="${safety_limits}">
+          <safety_controller soft_lower_limit="${elbow_joint_lower_limit + safety_pos_margin}" soft_upper_limit="${elbow_joint_upper_limit - safety_pos_margin}" k_position="${safety_k_position}" k_velocity="0.0"/>
+        </xacro:if>
       </xacro:if>
       <dynamics damping="0.0" friction="0.0"/>
@@ -154,5 +170,6 @@
     <link name="${prefix}forearm_link">
       <visual>
-         <geometry>
+        <origin xyz="0 0 ${elbow_offset}" rpy="${pi/2} 0 ${-pi/2}"/>
+        <geometry>
           <mesh filename="package://iai_ur_description/meshes/ur3/visual/forearm.dae"/>
         </geometry>
@@ -162,10 +179,11 @@
       </visual>
       <collision>
+        <origin xyz="0 0 ${elbow_offset}" rpy="${pi/2} 0 ${-pi/2}"/>
         <geometry>
           <mesh filename="package://iai_ur_description/meshes/ur3/collision/forearm.stl"/>
         </geometry>
       </collision>
-      <xacro:cylinder_inertial radius="0.075" length="${-ur3_a3}" mass="${forearm_mass}">
-        <origin xyz="0.0 0.0 ${-ur3_a3/2.0}" rpy="0 0 0" />
+      <xacro:cylinder_inertial radius="0.075" length="${-1*__kinematics['wrist_1']['x']}" mass="${forearm_mass}">
+        <origin xyz="${0.5*__kinematics['forearm']['x']} 0.0 ${elbow_offset}" rpy="0 ${pi/2} 0" />
       </xacro:cylinder_inertial>
     </link>
@@ -173,11 +191,17 @@
       <parent link="${prefix}forearm_link" />
       <child link = "${prefix}wrist_1_link" />
-      <origin xyz="0.0 0.0 ${forearm_length}" rpy="0.0 ${pi / 2.0} 0.0" />
-      <axis xyz="0 1 0" />
+      <origin xyz="${__kinematics['wrist_1']['x']} ${__kinematics['wrist_1']['y']} ${__kinematics['wrist_1']['z']}" rpy="${__kinematics['wrist_1']['roll']} ${__kinematics['wrist_1']['pitch']} ${__kinematics['wrist_1']['yaw']}" />
+      <axis xyz="0 0 1" />
       <xacro:unless value="${joint_limited}">
         <limit lower="${-2.0 * pi}" upper="${2.0 * pi}" effort="54.0" velocity="3.2"/>
-      </xacro:unless>
-      <xacro:if value="${joint_limited}">
-        <limit lower="${-1.3 * pi}" upper="${1.3 * pi}" effort="54.0" velocity="3.2"/>
+        <xacro:if value="${safety_limits}">
+          <safety_controller soft_lower_limit="${-2.0 * pi + safety_pos_margin}" soft_upper_limit="${2.0 * pi - safety_pos_margin}" k_position="${safety_k_position}" k_velocity="0.0"/>
+        </xacro:if>
+      </xacro:unless>
+      <xacro:if value="${joint_limited}">
+        <limit lower="${wrist_1_lower_limit}" upper="${wrist_1_upper_limit}" effort="54.0" velocity="3.2"/>
+        <xacro:if value="${safety_limits}">
+          <safety_controller soft_lower_limit="${wrist_1_lower_limit + safety_pos_margin}" soft_upper_limit="${wrist_1_upper_limit - safety_pos_margin}" k_position="${safety_k_position}" k_velocity="0.0"/>
+        </xacro:if>
       </xacro:if>
       <dynamics damping="0.0" friction="0.0"/>
@@ -185,4 +209,5 @@
     <link name="${prefix}wrist_1_link">
       <visual>
+        <origin xyz="0 0 -0.085" rpy="${pi/2} 0 0"/>
         <geometry>
           <mesh filename="package://iai_ur_description/meshes/ur3/visual/wrist1.dae"/>
@@ -193,9 +218,10 @@
       </visual>
       <collision>
+        <origin xyz="0 0 -0.085" rpy="${pi/2} 0 0"/>
         <geometry>
           <mesh filename="package://iai_ur_description/meshes/ur3/collision/wrist1.stl"/>
         </geometry>
       </collision>
-      <xacro:cylinder_inertial radius="0.075" length="0.12" mass="${wrist_1_mass}">
+      <xacro:cylinder_inertial radius="0.075" length="${-1*__kinematics['wrist_2']['y']}" mass="${wrist_1_mass}">
         <origin xyz="0.0 0.0 0.0" rpy="0 0 0" />
       </xacro:cylinder_inertial>
@@ -204,11 +230,17 @@
       <parent link="${prefix}wrist_1_link" />
       <child link = "${prefix}wrist_2_link" />
-      <origin xyz="0.0 ${wrist_1_length} 0.0" rpy="0.0 0.0 0.0" />
+      <origin xyz="${__kinematics['wrist_2']['x']} ${__kinematics['wrist_2']['y']} ${__kinematics['wrist_2']['z']}" rpy="${__kinematics['wrist_2']['roll']} ${__kinematics['wrist_2']['pitch']} ${__kinematics['wrist_2']['yaw']}" />
       <axis xyz="0 0 1" />
       <xacro:unless value="${joint_limited}">
         <limit lower="${-2.0 * pi}" upper="${2.0 * pi}" effort="54.0" velocity="3.2"/>
-      </xacro:unless>
-      <xacro:if value="${joint_limited}">
-        <limit lower="${-1.3 * pi}" upper="${1.3 * pi}" effort="54.0" velocity="3.2"/>
+        <xacro:if value="${safety_limits}">
+          <safety_controller soft_lower_limit="${-2.0 * pi + safety_pos_margin}" soft_upper_limit="${2.0 * pi - safety_pos_margin}" k_position="${safety_k_position}" k_velocity="0.0"/>
+        </xacro:if>
+      </xacro:unless>
+      <xacro:if value="${joint_limited}">
+        <limit lower="${wrist_2_lower_limit}" upper="${wrist_2_upper_limit}" effort="54.0" velocity="3.2"/>
+        <xacro:if value="${safety_limits}">
+          <safety_controller soft_lower_limit="${wrist_2_lower_limit + safety_pos_margin}" soft_upper_limit="${wrist_2_upper_limit - safety_pos_margin}" k_position="${safety_k_position}" k_velocity="0.0"/>
+        </xacro:if>
       </xacro:if>
       <dynamics damping="0.0" friction="0.0"/>
@@ -216,4 +248,5 @@
     <link name="${prefix}wrist_2_link">
       <visual>
+        <origin xyz="0 0 -0.085" rpy="0 0 0"/>
         <geometry>
           <mesh filename="package://iai_ur_description/meshes/ur3/visual/wrist2.dae"/>
@@ -224,9 +257,10 @@
       </visual>
       <collision>
+        <origin xyz="0 0 -0.085" rpy="0 0 0"/>
         <geometry>
           <mesh filename="package://iai_ur_description/meshes/ur3/collision/wrist2.stl"/>
         </geometry>
       </collision>
-      <xacro:cylinder_inertial radius="0.075" length="0.12" mass="${wrist_2_mass}">
+      <xacro:cylinder_inertial radius="0.075" length="${__kinematics['wrist_3']['y']}" mass="${wrist_2_mass}">
         <origin xyz="0.0 0.0 0.0" rpy="0 0 0" />
       </xacro:cylinder_inertial>
@@ -235,11 +269,17 @@
       <parent link="${prefix}wrist_2_link" />
       <child link = "${prefix}wrist_3_link" />
-      <origin xyz="0.0 0.0 ${wrist_2_length}" rpy="0.0 0.0 0.0" />
-      <axis xyz="0 1 0" />
+      <origin xyz="${__kinematics['wrist_3']['x']} ${__kinematics['wrist_3']['y']} ${__kinematics['wrist_3']['z']}" rpy="${__kinematics['wrist_3']['roll']} ${__kinematics['wrist_3']['pitch']} ${__kinematics['wrist_3']['yaw']}" />
+      <axis xyz="0 0 1" />
       <xacro:unless value="${joint_limited}">
         <limit lower="${-2.0 * pi}" upper="${2.0 * pi}" effort="54.0" velocity="3.2"/>
-      </xacro:unless>
-      <xacro:if value="${joint_limited}">
-				<limit lower="${-1 * pi}" upper="${1 * pi}" effort="54.0" velocity="3.2"/>
+        <xacro:if value="${safety_limits}">
+          <safety_controller soft_lower_limit="${-2.0 * pi + safety_pos_margin}" soft_upper_limit="${2.0 * pi - safety_pos_margin}" k_position="${safety_k_position}" k_velocity="0.0"/>
+        </xacro:if>
+      </xacro:unless>
+      <xacro:if value="${joint_limited}">
+        <limit lower="${wrist_3_lower_limit}" upper="${wrist_3_upper_limit}" effort="54.0" velocity="3.2"/>
+        <xacro:if value="${safety_limits}">
+          <safety_controller soft_lower_limit="${wrist_3_lower_limit + safety_pos_margin}" soft_upper_limit="${wrist_3_upper_limit - safety_pos_margin}" k_position="${safety_k_position}" k_velocity="0.0"/>
+        </xacro:if>
       </xacro:if>
       <dynamics damping="0.0" friction="0.0"/>
@@ -247,4 +287,5 @@
     <link name="${prefix}wrist_3_link">
       <visual>
+        <origin xyz="0 0 -0.082" rpy="${pi/2} 0 0"/>
         <geometry>
           <mesh filename="package://iai_ur_description/meshes/ur3/visual/wrist3.dae"/>
@@ -255,10 +296,11 @@
       </visual>
       <collision>
+        <origin xyz="0 0 -0.082" rpy="${pi/2} 0 0"/>
         <geometry>
           <mesh filename="package://iai_ur_description/meshes/ur3/collision/wrist3.stl"/>
         </geometry>
       </collision>
-      <xacro:cylinder_inertial radius="0.075" length="0.12" mass="${wrist_3_mass}">
-        <origin xyz="0.0 0.0 0.0" rpy="0 0 0" />
+      <xacro:cylinder_inertial radius="0.045" length="0.0305" mass="${wrist_3_mass}">
+        <origin xyz="0.0 0.0 ${-0.0305/2}" rpy="0 0 0" />
       </xacro:cylinder_inertial>
     </link>
@@ -266,5 +308,5 @@
       <parent link="${prefix}wrist_3_link" />
       <child link = "${prefix}ee_link" />
-      <origin xyz="0.0 ${wrist_3_length} 0.0" rpy="0.0 0.0 ${pi/2.0}" />
+      <origin xyz="0.0 0.0 0.0" rpy="0.0 ${-pi/2.0} ${pi/2.0}" />
     </joint>
     <link name="${prefix}ee_link">
@@ -276,5 +318,10 @@
       </collision>
     </link>
-    <xacro:ur_arm_transmission prefix="${prefix}" />
+    <joint name="${prefix}wrist_3_passive_joint" type="fixed">
+      <origin xyz="0 0 0" rpy="0 0 0"/>
+      <parent link="${prefix}wrist_3_link"/>
+      <child link="${prefix}tool0"/>
+    </joint>
+    <xacro:ur_arm_transmission prefix="${prefix}" hw_interface="${transmission_hw_interface}" />
     <xacro:ur_arm_gazebo prefix="${prefix}" />
     <!-- ROS base_link to UR 'Base' Coordinates transform -->
@@ -285,5 +332,5 @@
                  degrees)
       -->
-      <origin xyz="0 0 0" rpy="0 0 ${-pi}"/>
+      <origin xyz="0 0 0" rpy="0 0 ${-base_correction}"/>
       <parent link="${prefix}base_link"/>
       <child link="${prefix}base"/>
@@ -291,9 +338,4 @@
     <!-- Frame coincident with all-zeros TCP on UR controller -->
     <link name="${prefix}tool0"/>
-    <joint name="${prefix}wrist_3_link-tool0_fixed_joint" type="fixed">
-      <origin xyz="0 ${wrist_3_length} 0" rpy="${pi/-2.0} 0 0"/>
-      <parent link="${prefix}wrist_3_link"/>
-      <child link="${prefix}tool0"/>
-    </joint>
   </xacro:macro>
 </robot>

File: iai_ur_description/urdf/ur3_robot.urdf.xacro (robot description, xacro)
@@ -1,5 +1,6 @@
 <?xml version="1.0"?>
-<robot xmlns:xacro="http://www.ros.org/wiki/xacro"
+<robot xmlns:xacro="http://wiki.ros.org/xacro"
        name="ur3" >
+  <xacro:arg name="transmission_hw_interface" default="hardware_interface/PositionJointInterface"/>
   <!-- common stuff -->
   <xacro:include filename="$(find iai_ur_description)/urdf/common.gazebo.xacro" />
@@ -7,5 +8,9 @@
   <xacro:include filename="$(find iai_ur_description)/urdf/ur3.urdf.xacro" />
   <!-- arm -->
-  <xacro:ur3_robot prefix="" joint_limited="false"/>
+  <xacro:arg name="kinematics_config" default="$(find iai_ur_description)/config/ur3_default.yaml"/>
+  <xacro:ur3_robot prefix="" joint_limited="false"
+    transmission_hw_interface="$(arg transmission_hw_interface)"
+    kinematics_file="${load_yaml('$(arg kinematics_config)')}"
+  />
   <link name="world" />
   <joint name="world_joint" type="fixed">
