Commit message: boxy noetic compatability

File: iai_boxy_description/urdf/boxy_description.urdf.xacro (robot description, xacro)
@@ -25,4 +25,5 @@
   <!-- /Property definitions e.g. constants -->
   <xacro:include filename="$(find iai_boxy_base)/robots/base.URDF"/>
+  <xacro:property name="M_PI" value="${pi}" />
   <xacro:macro name="boxy">
     <!-- virtual joints to model odometry -->
@@ -84,8 +85,8 @@
     <!-- mounting plate of UR3 -->
     <xacro:property name="ur3_prefix" value="neck_"/>
-    <adapter_boxy_ur3_xacro prefix="${ur3_prefix}" parent="base_link">
+    <xacro:adapter_boxy_ur3_xacro prefix="${ur3_prefix}" parent="base_link">
       <origin xyz="0.175 -0.227 1.48" rpy="0 0 0"/>
-    </adapter_boxy_ur3_xacro>
-    <xacro:ur3_robot prefix="${ur3_prefix}" joint_limited="true" transmission_hw_interface="$(arg transmission_hw_interface)" kinematics_file="${load_yaml('$(arg kinematics_config)')}"/>
+    </xacro:adapter_boxy_ur3_xacro>
+    <xacro:ur3_robot prefix="${ur3_prefix}" joint_limited="true" transmission_hw_interface="$(arg transmission_hw_interface)" kinematics_file="${xacro.load_yaml('$(arg kinematics_config)')}"/>
     <joint name="${ur3_prefix}base_mounting_joint" type="fixed">
       <parent link="${ur3_prefix}adapter_ur3_frame_out" />
@@ -94,10 +95,10 @@
     </joint>
     <!-- The following URDF has frame_in / frame_out, so it is placed at the parent -->
-    <adapter_iso50_kinect2_xacro parent="neck_tool0" prefix="neck">
+    <xacro:adapter_iso50_kinect2_xacro parent="neck_tool0" prefix="neck">
       <origin xyz="0 0 0" rpy="0 0 -1.570795"/>
-    </adapter_iso50_kinect2_xacro>
-    <kinect2_xacro parent="neck_adapter_iso50_kinect2_frame_out" prefix="head_mount">
+    </xacro:adapter_iso50_kinect2_xacro>
+    <xacro:kinect2_xacro parent="neck_adapter_iso50_kinect2_frame_out" prefix="head_mount">
       <origin xyz="-0.031284 0.098627 0.023544" rpy="4.728550 6.279385 1.578295"/>
-    </kinect2_xacro>
+    </xacro:kinect2_xacro>
     <!-- JOINT to connect the base with the torso -->
     <joint name="torso_joint" type="fixed">
@@ -109,30 +110,30 @@
     <xacro:include filename="$(find iai_boxy_torso)/robots/torso.URDF"/>
     <!--FIXME: triangle_left_arm_link should be rotated, and not the origin of the arm (which right now is calib_left_arm_base_link -->
-    <kuka_lwr_arm parent="triangle_left_arm_link" prefix="left_" color_postfix="">
+    <xacro:kuka_lwr_arm parent="triangle_left_arm_link" prefix="left_" color_postfix="">
       <!-- From CAD -->
       <!--origin xyz="0 0 0" rpy="0 0 1.047198"/-->
       <!-- from calibration on 20160903 -->
       <origin xyz="-0.006185 0.004080 -0.010726" rpy="6.276354 6.281653 1.074679"/>
-    </kuka_lwr_arm>
-    <lwr4_cabling_adaptor parent="left_arm_flange_link" prefix="left_arm_">
+    </xacro:kuka_lwr_arm>
+    <xacro:lwr4_cabling_adaptor parent="left_arm_flange_link" prefix="left_arm_">
       <origin xyz="0 0 0.01" rpy="0 0 0"/>
-    </lwr4_cabling_adaptor>
+    </xacro:lwr4_cabling_adaptor>
     <!-- The following URDFs have frame_in / frame_out, so they are simply placed at their parent -->
-    <kms_40_xacro parent="left_arm_cabling_adaptor_link" prefix="left_arm_">
+    <xacro:kms_40_xacro parent="left_arm_cabling_adaptor_link" prefix="left_arm_">
       <origin xyz="0 0 0" rpy="0 0 0"/>
       <!--places the kms40 frame 13mm from the parent -->
-    </kms_40_xacro>
-    <adapter_kms40_fwk050_xacro parent="left_arm_kms40_frame_out" prefix="left_arm_">
-      <origin xyz="0 0 0" rpy="0 0 0"/>
-    </adapter_kms40_fwk050_xacro>
-    <fwk_fwa_050_xacro parent="left_arm_adapter_kms40_fwk050_frame_out" prefix="left_arm_">
-      <origin xyz="0 0 0" rpy="0 0 0"/>
-    </fwk_fwa_050_xacro>
-    <adapter_fwa050_wsg50_xacro parent="left_arm_fwk_fwa_050_frame_out" prefix="left_arm_">
+    </xacro:kms_40_xacro>
+    <xacro:adapter_kms40_fwk050_xacro parent="left_arm_kms40_frame_out" prefix="left_arm_">
+      <origin xyz="0 0 0" rpy="0 0 0"/>
+    </xacro:adapter_kms40_fwk050_xacro>
+    <xacro:fwk_fwa_050_xacro parent="left_arm_adapter_kms40_fwk050_frame_out" prefix="left_arm_">
+      <origin xyz="0 0 0" rpy="0 0 0"/>
+    </xacro:fwk_fwa_050_xacro>
+    <xacro:adapter_fwa050_wsg50_xacro parent="left_arm_fwk_fwa_050_frame_out" prefix="left_arm_">
       <origin xyz="0 0 0.0" rpy="0 0 0"/>
-    </adapter_fwa050_wsg50_xacro>
-    <wsg_50_xacro name="left_gripper" parent="left_arm_adapter_fwa050_wsg50_frame_out">
-      <origin xyz="0 0 0" rpy="0 0 0"/>
-    </wsg_50_xacro>
+    </xacro:adapter_fwa050_wsg50_xacro>
+    <xacro:wsg_50_xacro name="left_gripper" parent="left_arm_adapter_fwa050_wsg50_frame_out">
+      <origin xyz="0 0 0" rpy="0 0 0"/>
+    </xacro:wsg_50_xacro>
     <link name="left_wrist_optical_frame_x">
       <inertial>
@@ -238,27 +239,29 @@
 	</wsg_50_xacro-->
     <!--This is a 60deg rotation to calib_right_arm_base_link -->
-    <kuka_lwr_arm parent="triangle_right_arm_link" prefix="right_" color_postfix="">
+    <xacro:kuka_lwr_arm parent="triangle_right_arm_link" prefix="right_" color_postfix="">
       <origin xyz="0 0 0" rpy="0 0 -1.047198"/>
-    </kuka_lwr_arm>
-    <lwr4_cabling_adaptor parent="right_arm_flange_link" prefix="right_arm_">
+    </xacro:kuka_lwr_arm>
+    <xacro:lwr4_cabling_adaptor parent="right_arm_flange_link" prefix="right_arm_">
       <origin xyz="0 0 0.01" rpy="0 0 0"/>
-    </lwr4_cabling_adaptor>
+    </xacro:lwr4_cabling_adaptor>
     <!-- The following URDFs have frame_in / frame_out, so they are simply placed at their parent -->
-    <kms_40_xacro parent="right_arm_cabling_adaptor_link" prefix="right_arm_">
+    <xacro:kms_40_xacro parent="right_arm_cabling_adaptor_link" prefix="right_arm_">
       <origin xyz="0 0 0" rpy="0 0 3.14159265359"/>
       <!--places the kms40 frame 13mm from the parent -->
-    </kms_40_xacro>
-    <adapter_kms40_fwk050_xacro parent="right_arm_kms40_frame_out" prefix="right_arm_">
-      <origin xyz="0 0 0" rpy="0 0 0"/>
-    </adapter_kms40_fwk050_xacro>
-    <fwk_fwa_050_xacro parent="right_arm_adapter_kms40_fwk050_frame_out" prefix="right_arm_">
-      <origin xyz="0 0 0" rpy="0 0 0"/>
-    </fwk_fwa_050_xacro>
-    <adapter_fwa050_wsg50_xacro parent="right_arm_fwk_fwa_050_frame_out" prefix="right_arm_">
+    </xacro:kms_40_xacro>
+    <xacro:adapter_kms40_fwk050_xacro parent="right_arm_kms40_frame_out" prefix="right_arm_">
+      <origin xyz="0 0 0" rpy="0 0 0"/>
+    </xacro:adapter_kms40_fwk050_xacro>
+    <xacro:fwk_fwa_050_xacro parent="right_arm_adapter_kms40_fwk050_frame_out" prefix="right_arm_">
+      <origin xyz="0 0 0" rpy="0 0 0"/>
+    </xacro:fwk_fwa_050_xacro>
+    <xacro:adapter_fwa050_wsg50_xacro parent="right_arm_fwk_fwa_050_frame_out" prefix="right_arm_">
       <origin xyz="0 0 0.0" rpy="0 0 0"/>
-    </adapter_fwa050_wsg50_xacro>
-    <wsg_50_xacro name="right_gripper" parent="right_arm_adapter_fwa050_wsg50_frame_out">
+    </xacro:adapter_fwa050_wsg50_xacro>
+    <xacro:wsg_50_xacro name="right_gripper" parent="right_arm_adapter_fwa050_wsg50_frame_out">
       <origin xyz="0 0 0" rpy="0 0 3.14159265359"/>
-    </wsg_50_xacro>
+    </xacro:wsg_50_xacro>
   </xacro:macro>
+  <xacro:boxy >
+  </xacro:boxy>
 </robot>

File: iai_kuka_lwr4_description/urdf/kuka_lwr_arm.urdf.xacro (robot description, xacro)
@@ -24,5 +24,5 @@
         <mass value="${arm_elem_base_mass}"/>
         <origin xyz="0 0 0.055" rpy="0 0 0"/>
-        <cylinder_inertia_def radius="0.06" length="0.11"
+        <xacro:cylinder_inertia_def radius="0.06" length="0.11"
                               mass="${arm_elem_base_mass}"/>
       </inertial>
@@ -64,5 +64,5 @@
         <mass value="${arm_elem_link_mass}"/>
         <origin rpy="0 0 0" xyz="0 0 0.130"/>
-        <cuboid_inertia_def length="0.12" width="0.06" height="0.260"
+        <xacro:cuboid_inertia_def length="0.12" width="0.06" height="0.260"
                             mass="${arm_elem_link_mass}"/>
       </inertial>
@@ -108,5 +108,5 @@
         <mass value="${arm_elem_link_mass}"/>
         <origin rpy="0 0 0" xyz="0 0.06 ${0.130 - 0.06}"/>
-        <cuboid_inertia_def length="0.12" width="0.06" height="0.260"
+        <xacro:cuboid_inertia_def length="0.12" width="0.06" height="0.260"
                             mass="${arm_elem_link_mass}"/>
       </inertial>
@@ -152,5 +152,5 @@
         <mass value="${arm_elem_link_mass}"/>
         <origin rpy="0 0 0" xyz="0 0.06 0.130"/>
-        <cuboid_inertia_def length="0.12" width="0.06" height="0.260"
+        <xacro:cuboid_inertia_def length="0.12" width="0.06" height="0.260"
                             mass="${arm_elem_link_mass}"/>
       </inertial>
@@ -196,5 +196,5 @@
         <mass value="${arm_elem_link_mass}"/>
         <origin rpy="0 0 0" xyz="0 -0.06 ${0.130 - 0.06}"/>
-        <cuboid_inertia_def length="0.12" width="0.06" height="0.2600"
+        <xacro:cuboid_inertia_def length="0.12" width="0.06" height="0.2600"
                             mass="${arm_elem_link_mass}"/>
       </inertial>
@@ -240,5 +240,5 @@
         <mass value="${arm_elem_link_mass}"/>
         <origin rpy="0 0 0" xyz="0 0 0.124"/>
-        <cuboid_inertia_def length="0.12" width="0.06" height="0.248"
+        <xacro:cuboid_inertia_def length="0.12" width="0.06" height="0.248"
                             mass="${arm_elem_link_mass}"/>
       </inertial>
@@ -284,5 +284,5 @@
         <mass value="${arm_elem_ball_link_mass}"/>
         <origin rpy="0 0 0" xyz="0 0 0.0625"/>
-        <cuboid_inertia_def length="0.125" width="0.125" height="0.125"
+        <xacro:cuboid_inertia_def length="0.125" width="0.125" height="0.125"
                             mass="${arm_elem_ball_link_mass}"/>
       </inertial>
@@ -328,5 +328,5 @@
         <mass value="${arm_elem_end_link_mass}"/>
         <origin xyz="0 0 0"/>
-        <cuboid_inertia_def length="1" width="1" height="1"
+        <xacro:cuboid_inertia_def length="1" width="1" height="1"
                             mass="${arm_elem_end_link_mass}"/>
       </inertial>
@@ -365,5 +365,5 @@
         <mass value="${arm_elem_flange_link_mass}"/>
         <origin xyz="0 0 0" rpy="0 0 0"/>
-        <cuboid_inertia_def length="1" width="1" height="1"
+        <xacro:cuboid_inertia_def length="1" width="1" height="1"
                             mass="${arm_elem_flange_link_mass}"/>
       </inertial>

File: iai_ur_description/urdf/ur3.urdf.xacro (robot description, xacro)
@@ -26,5 +26,5 @@
     safety_k_position:=20
     kinematics_file">
-    <xacro:property name="__kinematics" value="${kinematics_file['kinematics']}"/>
+    <xacro:property name="_kinematics" value="${kinematics_file['kinematics']}"/>
     <!-- Inertia parameters -->
     <xacro:property name="base_mass" value="2.0" />  <!-- This mass might be incorrect -->
@@ -74,5 +74,5 @@
       <parent link="${prefix}base_link" />
       <child link = "${prefix}shoulder_link" />
-      <origin xyz="${__kinematics['shoulder']['x']} ${__kinematics['shoulder']['y']} ${__kinematics['shoulder']['z']}" rpy="${__kinematics['shoulder']['roll']} ${__kinematics['shoulder']['pitch']} ${__kinematics['shoulder']['yaw'] + base_correction}" />
+      <origin xyz="${_kinematics['shoulder']['x']} ${_kinematics['shoulder']['y']} ${_kinematics['shoulder']['z']}" rpy="${_kinematics['shoulder']['roll']} ${_kinematics['shoulder']['pitch']} ${_kinematics['shoulder']['yaw'] + base_correction}" />
       <axis xyz="0 0 1" />
       <xacro:unless value="${joint_limited}">
@@ -113,5 +113,5 @@
       <parent link="${prefix}shoulder_link" />
       <child link = "${prefix}upper_arm_link" />
-      <origin xyz="${__kinematics['upper_arm']['x']} ${__kinematics['upper_arm']['y']} ${__kinematics['upper_arm']['z']}" rpy="${__kinematics['upper_arm']['roll']} ${__kinematics['upper_arm']['pitch']} ${__kinematics['upper_arm']['yaw']}" />
+      <origin xyz="${_kinematics['upper_arm']['x']} ${_kinematics['upper_arm']['y']} ${_kinematics['upper_arm']['z']}" rpy="${_kinematics['upper_arm']['roll']} ${_kinematics['upper_arm']['pitch']} ${_kinematics['upper_arm']['yaw']}" />
       <axis xyz="0 0 1" />
       <xacro:unless value="${joint_limited}">
@@ -145,6 +145,6 @@
         </geometry>
       </collision>
-      <xacro:cylinder_inertial radius="0.075" length="${-1*__kinematics['forearm']['x']}" mass="${upper_arm_mass}">
-        <origin xyz="${0.5*__kinematics['forearm']['x']} 0.0 ${upper_arm_inertia_offset}" rpy="0 ${pi/2} 0" />
+      <xacro:cylinder_inertial radius="0.075" length="${-1*_kinematics['forearm']['x']}" mass="${upper_arm_mass}">
+        <origin xyz="${0.5*_kinematics['forearm']['x']} 0.0 ${upper_arm_inertia_offset}" rpy="0 ${pi/2} 0" />
       </xacro:cylinder_inertial>
     </link>
@@ -152,5 +152,5 @@
       <parent link="${prefix}upper_arm_link" />
       <child link = "${prefix}forearm_link" />
-      <origin xyz="${__kinematics['forearm']['x']} ${__kinematics['forearm']['y']} ${__kinematics['forearm']['z']}" rpy="${__kinematics['forearm']['roll']} ${__kinematics['forearm']['pitch']} ${__kinematics['forearm']['yaw']}" />
+      <origin xyz="${_kinematics['forearm']['x']} ${_kinematics['forearm']['y']} ${_kinematics['forearm']['z']}" rpy="${_kinematics['forearm']['roll']} ${_kinematics['forearm']['pitch']} ${_kinematics['forearm']['yaw']}" />
       <axis xyz="0 0 1" />
       <xacro:unless value="${joint_limited}">
@@ -184,6 +184,6 @@
         </geometry>
       </collision>
-      <xacro:cylinder_inertial radius="0.075" length="${-1*__kinematics['wrist_1']['x']}" mass="${forearm_mass}">
-        <origin xyz="${0.5*__kinematics['forearm']['x']} 0.0 ${elbow_offset}" rpy="0 ${pi/2} 0" />
+      <xacro:cylinder_inertial radius="0.075" length="${-1*_kinematics['wrist_1']['x']}" mass="${forearm_mass}">
+        <origin xyz="${0.5*_kinematics['forearm']['x']} 0.0 ${elbow_offset}" rpy="0 ${pi/2} 0" />
       </xacro:cylinder_inertial>
     </link>
@@ -191,5 +191,5 @@
       <parent link="${prefix}forearm_link" />
       <child link = "${prefix}wrist_1_link" />
-      <origin xyz="${__kinematics['wrist_1']['x']} ${__kinematics['wrist_1']['y']} ${__kinematics['wrist_1']['z']}" rpy="${__kinematics['wrist_1']['roll']} ${__kinematics['wrist_1']['pitch']} ${__kinematics['wrist_1']['yaw']}" />
+      <origin xyz="${_kinematics['wrist_1']['x']} ${_kinematics['wrist_1']['y']} ${_kinematics['wrist_1']['z']}" rpy="${_kinematics['wrist_1']['roll']} ${_kinematics['wrist_1']['pitch']} ${_kinematics['wrist_1']['yaw']}" />
       <axis xyz="0 0 1" />
       <xacro:unless value="${joint_limited}">
@@ -223,5 +223,5 @@
         </geometry>
       </collision>
-      <xacro:cylinder_inertial radius="0.075" length="${-1*__kinematics['wrist_2']['y']}" mass="${wrist_1_mass}">
+      <xacro:cylinder_inertial radius="0.075" length="${-1*_kinematics['wrist_2']['y']}" mass="${wrist_1_mass}">
         <origin xyz="0.0 0.0 0.0" rpy="0 0 0" />
       </xacro:cylinder_inertial>
@@ -230,5 +230,5 @@
       <parent link="${prefix}wrist_1_link" />
       <child link = "${prefix}wrist_2_link" />
-      <origin xyz="${__kinematics['wrist_2']['x']} ${__kinematics['wrist_2']['y']} ${__kinematics['wrist_2']['z']}" rpy="${__kinematics['wrist_2']['roll']} ${__kinematics['wrist_2']['pitch']} ${__kinematics['wrist_2']['yaw']}" />
+      <origin xyz="${_kinematics['wrist_2']['x']} ${_kinematics['wrist_2']['y']} ${_kinematics['wrist_2']['z']}" rpy="${_kinematics['wrist_2']['roll']} ${_kinematics['wrist_2']['pitch']} ${_kinematics['wrist_2']['yaw']}" />
       <axis xyz="0 0 1" />
       <xacro:unless value="${joint_limited}">
@@ -262,5 +262,5 @@
         </geometry>
       </collision>
-      <xacro:cylinder_inertial radius="0.075" length="${__kinematics['wrist_3']['y']}" mass="${wrist_2_mass}">
+      <xacro:cylinder_inertial radius="0.075" length="${_kinematics['wrist_3']['y']}" mass="${wrist_2_mass}">
         <origin xyz="0.0 0.0 0.0" rpy="0 0 0" />
       </xacro:cylinder_inertial>
@@ -269,5 +269,5 @@
       <parent link="${prefix}wrist_2_link" />
       <child link = "${prefix}wrist_3_link" />
-      <origin xyz="${__kinematics['wrist_3']['x']} ${__kinematics['wrist_3']['y']} ${__kinematics['wrist_3']['z']}" rpy="${__kinematics['wrist_3']['roll']} ${__kinematics['wrist_3']['pitch']} ${__kinematics['wrist_3']['yaw']}" />
+      <origin xyz="${_kinematics['wrist_3']['x']} ${_kinematics['wrist_3']['y']} ${_kinematics['wrist_3']['z']}" rpy="${_kinematics['wrist_3']['roll']} ${_kinematics['wrist_3']['pitch']} ${_kinematics['wrist_3']['yaw']}" />
       <axis xyz="0 0 1" />
       <xacro:unless value="${joint_limited}">
