Commit message: [justin-urdf] fixed justin-urdf for pycram usage, and filled in package.xml

File: iai_dlr_rollin_justin/urdf/rollin_justin.urdf (robot description, URDF)
Before this commit: robot rollin-justin, 63 links, 62 joints
Links:
- added link base_footprint; collision box size=0.001 0.001 0.001; visual box size=0.01 0.01 0.01
- added link l_gripper_tool_frame, mass 0.1
- added link r_gripper_tool_frame, mass 0.1
- link base_link: geometry collision mesh filename=package://iai_dlr_rollin_justin/mjcf/rollin-justin/meshes/s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 scale=1 1 1; visual mesh filename=package://iai_dlr_rollin_justin/mjcf/rollin-justin/meshes/s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 scale=1 1 1
- link head1: geometry collision mesh filename=package://iai_dlr_rollin_justin/mjcf/rollin-justin/meshes/s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 scale=1 1 1; visual mesh filename=package://iai_dlr_rollin_justin/mjcf/rollin-justin/meshes/s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 scale=1 1 1
- link head2: geometry collision mesh filename=package://iai_dlr_rollin_justin/mjcf/rollin-justin/meshes/s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 scale=1 1 1; visual mesh filename=package://iai_dlr_rollin_justin/mjcf/rollin-justin/meshes/s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 scale=1 1 1
- link left_1thumb2: geometry collision mesh filename=package://iai_dlr_rollin_justin/mjcf/rollin-justin/meshes/s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 scale=1 1 1; visual mesh filename=package://iai_dlr_rollin_justin/mjcf/rollin-justin/meshes/s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 scale=1 1 1
- link left_1thumb3: geometry collision mesh filename=package://iai_dlr_rollin_justin/mjcf/rollin-justin/meshes/s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 scale=1 1 1; visual mesh filename=package://iai_dlr_rollin_justin/mjcf/rollin-justin/meshes/s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 scale=1 1 1
- link left_1thumb4: geometry collision mesh filename=package://iai_dlr_rollin_justin/mjcf/rollin-justin/meshes/s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 scale=1 1 1; visual mesh filename=package://iai_dlr_rollin_justin/mjcf/rollin-justin/meshes/s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 scale=1 1 1
- link left_1thumb_base: geometry visual mesh filename=package://iai_dlr_rollin_justin/mjcf/rollin-justin/meshes/s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 scale=1 1 1
- link left_2tip2: geometry collision mesh filename=package://iai_dlr_rollin_justin/mjcf/rollin-justin/meshes/s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 scale=1 1 1; visual mesh filename=package://iai_dlr_rollin_justin/mjcf/rollin-justin/meshes/s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 scale=1 1 1
- link left_2tip3: geometry collision mesh filename=package://iai_dlr_rollin_justin/mjcf/rollin-justin/meshes/s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 scale=1 1 1; visual mesh filename=package://iai_dlr_rollin_justin/mjcf/rollin-justin/meshes/s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 scale=1 1 1
- link left_2tip4: geometry collision mesh filename=package://iai_dlr_rollin_justin/mjcf/rollin-justin/meshes/s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 scale=1 1 1; visual mesh filename=package://iai_dlr_rollin_justin/mjcf/rollin-justin/meshes/s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 scale=1 1 1
- link left_2tip_base: geometry visual mesh filename=package://iai_dlr_rollin_justin/mjcf/rollin-justin/meshes/s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 scale=1 1 1
- link left_3middle2: geometry collision mesh filename=package://iai_dlr_rollin_justin/mjcf/rollin-justin/meshes/s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 scale=1 1 1; visual mesh filename=package://iai_dlr_rollin_justin/mjcf/rollin-justin/meshes/s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 scale=1 1 1
- link left_3middle3: geometry collision mesh filename=package://iai_dlr_rollin_justin/mjcf/rollin-justin/meshes/s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 scale=1 1 1; visual mesh filename=package://iai_dlr_rollin_justin/mjcf/rollin-justin/meshes/s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 scale=1 1 1
- link left_3middle4: geometry collision mesh filename=package://iai_dlr_rollin_justin/mjcf/rollin-justin/meshes/s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 scale=1 1 1; visual mesh filename=package://iai_dlr_rollin_justin/mjcf/rollin-justin/meshes/s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 scale=1 1 1
- link left_3middle_base: geometry collision mesh filename=package://iai_dlr_rollin_justin/mjcf/rollin-justin/meshes/s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 scale=1 1 1; visual mesh filename=package://iai_dlr_rollin_justin/mjcf/rollin-justin/meshes/s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 scale=1 1 1
- link left_4ring2: geometry collision mesh filename=package://iai_dlr_rollin_justin/mjcf/rollin-justin/meshes/s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 scale=1 1 1; visual mesh filename=package://iai_dlr_rollin_justin/mjcf/rollin-justin/meshes/s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 scale=1 1 1
- link left_4ring3: geometry collision mesh filename=package://iai_dlr_rollin_justin/mjcf/rollin-justin/meshes/s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 scale=1 1 1; visual mesh filename=package://iai_dlr_rollin_justin/mjcf/rollin-justin/meshes/s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 scale=1 1 1
- link left_4ring4: geometry collision mesh filename=package://iai_dlr_rollin_justin/mjcf/rollin-justin/meshes/s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 scale=1 1 1; visual mesh filename=package://iai_dlr_rollin_justin/mjcf/rollin-justin/meshes/s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 scale=1 1 1
- link left_4ring_base: geometry visual mesh filename=package://iai_dlr_rollin_justin/mjcf/rollin-justin/meshes/s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 scale=1 1 1
- link left_arm1: geometry collision mesh filename=package://iai_dlr_rollin_justin/mjcf/rollin-justin/meshes/s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 scale=1 1 1; visual mesh filename=package://iai_dlr_rollin_justin/mjcf/rollin-justin/meshes/s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 scale=1 1 1
- link left_arm2: geometry collision mesh filename=package://iai_dlr_rollin_justin/mjcf/rollin-justin/meshes/s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 scale=1 1 1; visual mesh filename=package://iai_dlr_rollin_justin/mjcf/rollin-justin/meshes/s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 scale=1 1 1
- link left_arm3: geometry collision mesh filename=package://iai_dlr_rollin_justin/mjcf/rollin-justin/meshes/s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 scale=1 1 1; visual mesh filename=package://iai_dlr_rollin_justin/mjcf/rollin-justin/meshes/s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 scale=1 1 1
- link left_arm4: geometry collision mesh filename=package://iai_dlr_rollin_justin/mjcf/rollin-justin/meshes/s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 scale=1 1 1; visual mesh filename=package://iai_dlr_rollin_justin/mjcf/rollin-justin/meshes/s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 scale=1 1 1
- link left_arm5: geometry collision mesh filename=package://iai_dlr_rollin_justin/mjcf/rollin-justin/meshes/s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 scale=1 1 1; visual mesh filename=package://iai_dlr_rollin_justin/mjcf/rollin-justin/meshes/s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 scale=1 1 1
- link left_arm6: geometry collision mesh filename=package://iai_dlr_rollin_justin/mjcf/rollin-justin/meshes/s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 scale=1 1 1; visual mesh filename=package://iai_dlr_rollin_justin/mjcf/rollin-justin/meshes/s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 scale=1 1 1
- link left_arm7: geometry collision mesh filename=package://iai_dlr_rollin_justin/mjcf/rollin-justin/meshes/s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 scale=1 1 1; visual mesh filename=package://iai_dlr_rollin_justin/mjcf/rollin-justin/meshes/s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 scale=1 1 1
- link right_1thumb2: geometry collision mesh filename=package://iai_dlr_rollin_justin/mjcf/rollin-justin/meshes/s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 scale=1 1 1; visual mesh filename=package://iai_dlr_rollin_justin/mjcf/rollin-justin/meshes/s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 scale=1 1 1
- link right_1thumb3: geometry collision mesh filename=package://iai_dlr_rollin_justin/mjcf/rollin-justin/meshes/s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 scale=1 1 1; visual mesh filename=package://iai_dlr_rollin_justin/mjcf/rollin-justin/meshes/s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 scale=1 1 1
- link right_1thumb4: geometry collision mesh filename=package://iai_dlr_rollin_justin/mjcf/rollin-justin/meshes/s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 scale=1 1 1; visual mesh filename=package://iai_dlr_rollin_justin/mjcf/rollin-justin/meshes/s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 scale=1 1 1
- link right_1thumb_base: geometry visual mesh filename=package://iai_dlr_rollin_justin/mjcf/rollin-justin/meshes/s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 scale=1 1 1
- link right_2tip2: geometry collision mesh filename=package://iai_dlr_rollin_justin/mjcf/rollin-justin/meshes/s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 scale=1 1 1; visual mesh filename=package://iai_dlr_rollin_justin/mjcf/rollin-justin/meshes/s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 scale=1 1 1
- link right_2tip3: geometry collision mesh filename=package://iai_dlr_rollin_justin/mjcf/rollin-justin/meshes/s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 scale=1 1 1; visual mesh filename=package://iai_dlr_rollin_justin/mjcf/rollin-justin/meshes/s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 scale=1 1 1
- link right_2tip4: geometry collision mesh filename=package://iai_dlr_rollin_justin/mjcf/rollin-justin/meshes/s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 scale=1 1 1; visual mesh filename=package://iai_dlr_rollin_justin/mjcf/rollin-justin/meshes/s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 scale=1 1 1
- link right_2tip_base: geometry visual mesh filename=package://iai_dlr_rollin_justin/mjcf/rollin-justin/meshes/s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 scale=1 1 1
- link right_3middle2: geometry collision mesh filename=package://iai_dlr_rollin_justin/mjcf/rollin-justin/meshes/s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 scale=1 1 1; visual mesh filename=package://iai_dlr_rollin_justin/mjcf/rollin-justin/meshes/s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 scale=1 1 1
- link right_3middle3: geometry collision mesh filename=package://iai_dlr_rollin_justin/mjcf/rollin-justin/meshes/s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 scale=1 1 1; visual mesh filename=package://iai_dlr_rollin_justin/mjcf/rollin-justin/meshes/s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 scale=1 1 1
- link right_3middle4: geometry collision mesh filename=package://iai_dlr_rollin_justin/mjcf/rollin-justin/meshes/s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 scale=1 1 1; visual mesh filename=package://iai_dlr_rollin_justin/mjcf/rollin-justin/meshes/s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 scale=1 1 1
- link right_3middle_base: geometry visual mesh filename=package://iai_dlr_rollin_justin/mjcf/rollin-justin/meshes/s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 scale=1 1 1
- link right_4ring2: geometry collision mesh filename=package://iai_dlr_rollin_justin/mjcf/rollin-justin/meshes/s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 scale=1 1 1; visual mesh filename=package://iai_dlr_rollin_justin/mjcf/rollin-justin/meshes/s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 scale=1 1 1
- link right_4ring3: geometry collision mesh filename=package://iai_dlr_rollin_justin/mjcf/rollin-justin/meshes/s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 scale=1 1 1; visual mesh filename=package://iai_dlr_rollin_justin/mjcf/rollin-justin/meshes/s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 scale=1 1 1
- link right_4ring4: geometry collision mesh filename=package://iai_dlr_rollin_justin/mjcf/rollin-justin/meshes/s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 scale=1 1 1; visual mesh filename=package://iai_dlr_rollin_justin/mjcf/rollin-justin/meshes/s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 scale=1 1 1
- link right_4ring_base: geometry visual mesh filename=package://iai_dlr_rollin_justin/mjcf/rollin-justin/meshes/s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 scale=1 1 1
- link right_arm1: geometry collision mesh filename=package://iai_dlr_rollin_justin/mjcf/rollin-justin/meshes/s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 scale=1 1 1; visual mesh filename=package://iai_dlr_rollin_justin/mjcf/rollin-justin/meshes/s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 scale=1 1 1
- link right_arm2: geometry collision mesh filename=package://iai_dlr_rollin_justin/mjcf/rollin-justin/meshes/s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 scale=1 1 1; visual mesh filename=package://iai_dlr_rollin_justin/mjcf/rollin-justin/meshes/s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 scale=1 1 1
- link right_arm3: geometry collision mesh filename=package://iai_dlr_rollin_justin/mjcf/rollin-justin/meshes/s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 scale=1 1 1; visual mesh filename=package://iai_dlr_rollin_justin/mjcf/rollin-justin/meshes/s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 scale=1 1 1
- link right_arm4: geometry collision mesh filename=package://iai_dlr_rollin_justin/mjcf/rollin-justin/meshes/s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 scale=1 1 1; visual mesh filename=package://iai_dlr_rollin_justin/mjcf/rollin-justin/meshes/s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 scale=1 1 1
- link right_arm5: geometry collision mesh filename=package://iai_dlr_rollin_justin/mjcf/rollin-justin/meshes/s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 scale=1 1 1; visual mesh filename=package://iai_dlr_rollin_justin/mjcf/rollin-justin/meshes/s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 scale=1 1 1
- link right_arm6: geometry collision mesh filename=package://iai_dlr_rollin_justin/mjcf/rollin-justin/meshes/s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 scale=1 1 1; visual mesh filename=package://iai_dlr_rollin_justin/mjcf/rollin-justin/meshes/s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 scale=1 1 1
- link right_arm7: geometry collision mesh filename=package://iai_dlr_rollin_justin/mjcf/rollin-justin/meshes/s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 scale=1 1 1; visual mesh filename=package://iai_dlr_rollin_justin/mjcf/rollin-justin/meshes/s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 scale=1 1 1
- link torso1: geometry collision mesh filename=package://iai_dlr_rollin_justin/mjcf/rollin-justin/meshes/s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 scale=1 1 1; visual mesh filename=package://iai_dlr_rollin_justin/mjcf/rollin-justin/meshes/s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 scale=1 1 1
- link torso2: geometry collision mesh filename=package://iai_dlr_rollin_justin/mjcf/rollin-justin/meshes/s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 scale=1 1 1; visual mesh filename=package://iai_dlr_rollin_justin/mjcf/rollin-justin/meshes/s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 scale=1 1 1
- link torso3: geometry collision mesh filename=package://iai_dlr_rollin_justin/mjcf/rollin-justin/meshes/s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 scale=1 1 1; visual mesh filename=package://iai_dlr_rollin_justin/mjcf/rollin-justin/meshes/s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 scale=1 1 1
- link torso4: geometry collision mesh filename=package://iai_dlr_rollin_justin/mjcf/rollin-justin/meshes/s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 scale=1 1 1; visual mesh filename=package://iai_dlr_rollin_justin/mjcf/rollin-justin/meshes/s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 scale=1 1 1
Joints:
- added joint base_footprint_joint: type fixed, parent base_footprint, child base_link, origin xyz=0.25525 0.225 0.1616 rpy=0 0 0
- added joint l_gripper_tool_joint: type fixed, parent left_palm, child l_gripper_tool_frame, origin xyz=0.0 0 0.13 rpy=0 0 0
- added joint r_gripper_tool_joint: type fixed, parent right_palm, child r_gripper_tool_frame, origin xyz=0.0 0.0 0.13 rpy=0 0 0
