Commit message: adjusted files for dualarm with table urdf

File: iai_dualarm_description/robots/dualarm_ur5s_one_gripper_table.urdf.xacro (robot description, xacro)
@@ -1,5 +1,6 @@
 <?xml version="1.0"?>
-<robot xmlns:xacro="http://wiki.ros.org/xacro"
-       name="ur5dualarm" >
+<robot xmlns:xacro="http://www.ros.org/wiki/xacro"
+       name="ur5dualarm">
+  <!-- Args -->
   <xacro:arg name="transmission_hw_interface" default="hardware_interface/PositionJointInterface"/>
   <material name="gray">
@@ -9,4 +10,8 @@
     <color rgba="1.0 1.0 1.0 1.0"/>
   </material>
+  <!-- Common stuff -->
+  <xacro:include filename="$(find iai_ur_description)/urdf/common.gazebo.xacro"/>
+  <!-- UR5 Arm -->
+  <xacro:include filename="$(find iai_ur_description)/urdf/ur5.urdf.xacro"/>
   <material name="Grey">
     <color rgba="0.7 0.7 0.7 1.0"/>
@@ -38,5 +43,5 @@
     kinematics_file="${xacro.load_yaml('$(arg kinematics_config_left)')}"
   />
-  <!-- arm right -->
+  <!-- Right arm -->
   <xacro:arg name="kinematics_config_right" default="$(find iai_ur_description)/config/ur5_default.yaml"/>
   <xacro:ur5_robot prefix="right_" joint_limited="false"
@@ -132,7 +137,8 @@
     <origin xyz="0 0 0" rpy="0 0 0" />
   </kms_40_xacro>
-<!--Gripper-->
-<xacro:include filename="$(find iai_wsg_50_description)/urdf/wsg_50.urdf.xacro"/>
-<link name="left_adapter">
+  <!-- Gripper -->
+  <xacro:include filename="$(find wpg_300_120_description)/urdf/wpg_300_120_meshed.urdf.xacro"/>
+  <!-- Adapter -->
+  <link name="left_adapter">
     <visual>
       <origin xyz="0 0 0" rpy="0 0 0"/>
@@ -148,8 +154,9 @@
     <parent link="left_wrist_3_link"/>
     <child link="left_adapter"/>
-    <origin xyz="0 0 0.005" rpy="0.0 0.0 3.14" />
+    <origin xyz="0 0 0.005" rpy="0 0 3.14"/>
   </joint>
-  <xacro:wsg_50_xacro parent="left_adapter" name="left_gripper">
+  <!-- WSG 300-120 gripper attached to adapter -->
+  <xacro:wsg_300_120_xacro parent="left_adapter" name="left_gripper">
     <origin xyz="0 0 0" rpy="0 0 -0.785"/>
-  </xacro:wsg_50_xacro>
+  </xacro:wsg_300_120_xacro>
 </robot>

Commit message: adjusted mounting plate locations for dualarm

File: iai_dualarm_description/robots/dualarm_ur5s_one_gripper_table.urdf.xacro (robot description, xacro)
@@ -23,6 +23,6 @@
   <xacro:property name="left_arm_mounting_plate_length" value="0.15" />
   <xacro:property name="left_arm_mounting_plate_height" value="0.006" />
-  <xacro:property name="left_arm_mounting_plate_x_offset" value="0.37" />
-  <xacro:property name="left_arm_mounting_plate_y_offset" value="0.22" />
+  <xacro:property name="left_arm_mounting_plate_x_offset" value="0.045" />
+  <xacro:property name="left_arm_mounting_plate_y_offset" value="0.368" />
   <xacro:property name="left_kms_mounting_plate_height" value="0.016" />
   <!-- right mounting location -->
@@ -30,6 +30,6 @@
   <xacro:property name="right_arm_mounting_plate_length" value="0.15" />
   <xacro:property name="right_arm_mounting_plate_height" value="0.006" />
-  <xacro:property name="right_arm_mounting_plate_x_offset" value="1.07" />
-  <xacro:property name="right_arm_mounting_plate_y_offset" value="0.22" />
+  <xacro:property name="right_arm_mounting_plate_x_offset" value="0.994" />
+  <xacro:property name="right_arm_mounting_plate_y_offset" value="0.368" />
   <xacro:property name="right_kms_mounting_plate_height" value="0.016" />
   <!-- common stuff -->
