Commit message: added second gripper and renamed urdfs/launchs to reflect that

File: iai_dualarm_description/robots/dualarm_ur5s_two_gripper_table.urdf.xacro (robot description, xacro)
@@ -156,7 +156,26 @@
     <origin xyz="0 0 0.005" rpy="0 0 3.14"/>
   </joint>
+  <link name="right_adapter">
+    <visual>
+      <origin xyz="0 0 0" rpy="0 0 0"/>
+      <geometry>
+        <cylinder radius="0.035" length="0.01"/>
+      </geometry>
+      <material name="Cyan">
+        <color rgba="0 1.0 1.0 1.0"/>
+      </material>
+    </visual>
+  </link>
+  <joint name="right_adapter_joint" type="fixed">
+    <parent link="right_wrist_3_link"/>
+    <child link="right_adapter"/>
+    <origin xyz="0 0 0.005" rpy="0 0 3.14"/>
+  </joint>
   <!-- WSG 300-120 gripper attached to adapter -->
   <xacro:wsg_300_120_xacro parent="left_adapter" name="left_gripper">
     <origin xyz="0 0 0" rpy="0 0 -0.785"/>
   </xacro:wsg_300_120_xacro>
+  <xacro:wsg_300_120_xacro parent="right_adapter" name="right_gripper">
+    <origin xyz="0 0 0" rpy="0 0 -0.785"/>
+  </xacro:wsg_300_120_xacro>
 </robot>
