Commit message: [Armar7] removed fake omni drive

File: iai_kit_armar7/urdf/Armar7.urdf (robot description, URDF)
Before this commit: robot Armar7, 189 links, 188 joints
Links:
- removed link X_Platform_link
- removed link Y_Platform_link
- removed link Yaw_Platform_link
Joints:
- removed joint Platform
- removed joint X_Platform
- removed joint Y_Platform
- removed joint Yaw_Platform
- joint Dummy_Platform: child Dummy_Platform_link -> Platform_link; parent root -> Dummy_Platform_link
