Commit message: [iai_daisy] removed kms40 mounting plate

File: iai_daisy_description/robots/daisy.urdf.xacro (robot description, xacro)
@@ -104,20 +104,4 @@
     <origin xyz="0.0 0.0 ${left_arm_mounting_plate_height}" rpy="0 0 -${pi/4}" />
   </xacro:ur_robot>
-  <link name="left_kms_mounting_plate">
-    <visual>
-      <geometry>
-        <mesh filename="package://iai_table_robot_description/meshes/adapter_plate_iso50_kms40_weiss.stl" scale="0.001 0.001 0.001"/>
-      </geometry>
-      <material name="gray"/>
-    </visual>
-  </link>
-  <joint name="left_kms_mounting_plate_joint" type="fixed">
-    <parent link="left_tool0" />
-    <child link="left_kms_mounting_plate" />
-    <origin xyz="0 0 0" rpy="0 ${pi/2} 0" />
-  </joint>
-  <kms_40_xacro parent="left_kms_mounting_plate" prefix="left_kms_">
-    <origin xyz="0 0 0" rpy="0 0 0" />
-  </kms_40_xacro>
   <link name="left_adapter">
     <visual>
@@ -164,20 +148,4 @@
     <origin xyz="0.0 0.0 ${right_arm_mounting_plate_height}" rpy="0 0 -${pi/4}" />
   </xacro:ur_robot>
-  <link name="right_kms_mounting_plate">
-    <visual>
-      <geometry>
-        <mesh filename="package://iai_table_robot_description/meshes/adapter_plate_iso50_kms40_weiss.stl" scale="0.001 0.001 0.001"/>
-      </geometry>
-      <material name="gray"/>
-    </visual>
-  </link>
-  <joint name="right_kms_mounting_plate_joint" type="fixed">
-    <parent link="right_tool0" />
-    <child link="right_kms_mounting_plate" />
-    <origin xyz="0 0 0" rpy="0 ${pi/2} 0" />
-  </joint>
-  <kms_40_xacro parent="right_kms_mounting_plate" prefix="right_kms_">
-    <origin xyz="0 0 0" rpy="0 0 0" />
-  </kms_40_xacro>
   <link name="right_adapter">
     <visual>

Commit message: [iai_daisy] adjusted left ur5 arm rotation to reflect real setup

File: iai_daisy_description/robots/daisy.urdf.xacro (robot description, xacro)
@@ -102,5 +102,5 @@
     safety_k_position="20"
     force_abs_paths="false">
-    <origin xyz="0.0 0.0 ${left_arm_mounting_plate_height}" rpy="0 0 -${pi/4}" />
+    <origin xyz="0.0 0.0 ${left_arm_mounting_plate_height}" rpy="0 0 ${pi/2}" />
   </xacro:ur_robot>
   <link name="left_adapter">

Commit message: [iai_daisy] adjusted gripper position on arm

File: iai_daisy_description/robots/daisy.urdf.xacro (robot description, xacro)
@@ -119,5 +119,5 @@
   </joint>
   <xacro:wsg_300_120_xacro parent="left_adapter" name="left_gripper">
-    <origin xyz="0 0 0" rpy="0 0 -0.785"/>
+    <origin xyz="0 0 0" rpy="0 0 -${pi/2}"/>
   </xacro:wsg_300_120_xacro>
   <joint name="right_arm_mounting_plate_joint" type="fixed">
@@ -163,5 +163,5 @@
   </joint>
   <xacro:wsg_300_120_xacro parent="right_adapter" name="right_gripper">
-    <origin xyz="0 0 0" rpy="0 0 -0.785"/>
+    <origin xyz="0 0 0" rpy="0 0 -${pi/2}"/>
   </xacro:wsg_300_120_xacro>
   <xacro:ur_ros2_control

Commit message: [DAiSy] fixed the gripper mounting rotations

File: iai_daisy_description/robots/daisy.urdf.xacro (robot description, xacro)
@@ -106,5 +106,5 @@
   <link name="left_gripper_mounting_plate">
     <visual>
-      <origin xyz="0 0 0" rpy="0 0 ${pi/2}"/>
+      <origin xyz="0 0 0" rpy="0 0 0"/>
       <geometry>
         <mesh filename="package://iai_daisy_description/meshes/FL-ISO50-WPG300_WITH_FILLET.stl" scale="0.001 0.001 0.001"/>
@@ -113,5 +113,5 @@
     </visual>
     <collision>
-      <origin xyz="0 0 0" rpy="0 0 ${pi/2}"/>
+      <origin xyz="0 0 0" rpy="0 0 0"/>
       <geometry>
         <mesh filename="package://iai_daisy_description/meshes/FL-ISO50-WPG300_WITH_FILLET.stl" scale="0.001 0.001 0.001"/>
@@ -122,8 +122,8 @@
     <parent link="left_flange"/>
     <child link="left_gripper_mounting_plate"/>
-    <origin xyz="0 0 0.005" rpy="${pi/2} 0 ${pi/2}"/>
+    <origin xyz="0 0 0.005" rpy="0 ${pi/2} 0"/>
   </joint>
   <xacro:wsg_300_120_xacro parent="left_gripper_mounting_plate" name="left_gripper">
-    <origin xyz="0 0 0" rpy="0 0 -${pi/2}"/>
+    <origin xyz="0 0 0" rpy="0 0 0"/>
   </xacro:wsg_300_120_xacro>
   <joint name="right_arm_mounting_plate_joint" type="fixed">
@@ -156,11 +156,11 @@
   <link name="right_gripper_mounting_plate">
     <visual>
-      <origin xyz="0 0 0" rpy="0 0 ${pi/2}"/>
-      <geometry>
-        <mesh filename="package://iai_daisy_description/meshes/FL-ISO50-WPG300_WITH_FILLET.stl" scale="0.001 0.001 0.001"/>
-      </geometry>
-    </visual>
-    <collision>
-      <origin xyz="0 0 0" rpy="0 0 ${pi/2}"/>
+      <origin xyz="0 0 0" rpy="0 0 0"/>
+      <geometry>
+        <mesh filename="package://iai_daisy_description/meshes/FL-ISO50-WPG300_WITH_FILLET.stl" scale="0.001 0.001 0.001"/>
+      </geometry>
+    </visual>
+    <collision>
+      <origin xyz="0 0 0" rpy="0 0 0"/>
       <geometry>
         <mesh filename="package://iai_daisy_description/meshes/FL-ISO50-WPG300_WITH_FILLET.stl" scale="0.001 0.001 0.001"/>
@@ -171,8 +171,8 @@
     <parent link="right_flange"/>
     <child link="right_gripper_mounting_plate"/>
-    <origin xyz="0 0 0.005" rpy="${pi/2} 0 ${pi/2}"/>
+    <origin xyz="0 0 0.005" rpy="0 ${pi/2} 0"/>
   </joint>
   <xacro:wsg_300_120_xacro parent="right_gripper_mounting_plate" name="right_gripper">
-    <origin xyz="0 0 0" rpy="0 0 -${pi/2}"/>
+    <origin xyz="0 0 0" rpy="0 0 0"/>
   </xacro:wsg_300_120_xacro>
   <link name="left_gripper_left_finger_tip_link">
