Commit message: [DAiSy] Added table_root link and adjusted orientation of the robot to work with LeftOf/RightOf in Semantic Digital Twin

File: iai_daisy_description/robots/daisy.urdf.xacro (robot description, xacro)
@@ -47,4 +47,5 @@
   <xacro:property name="table_height" value="0.6077" />
   <xacro:property name="table_length" value="1.19" />
+  <xacro:property name="table_width" value="0.60" />
   <xacro:property name="left_arm_mounting_plate_width" value="0.18" />
   <xacro:property name="left_arm_mounting_plate_length" value="0.15" />
@@ -58,4 +59,5 @@
   <xacro:property name="right_arm_mounting_plate_y_offset" value="0.368" />
   <link name="map" />
+  <link name="table"/>
   <joint name="table_joint" type="fixed">
       <parent link="map"/>
@@ -63,6 +65,7 @@
       <origin xyz="0.0 0.0 0.0" rpy="0.0 0.0 0.0" />
   </joint>
-  <link name="table">
-    <visual>
+  <link name="table_center">
+    <visual>
+      <origin xyz="${table_length/2} ${table_width/2} 0" rpy="0 0 0"/>
       <geometry>
         <mesh filename="package://iai_table_robot_description/meshes/complete_table.dae"/>
@@ -71,4 +74,5 @@
     </visual>
     <collision>
+      <origin xyz="${table_length/2} ${table_width/2} 0" rpy="0 0 0"/>
       <geometry>
         <mesh filename="package://iai_table_robot_description/meshes/complete_table.stl"/>
@@ -77,8 +81,13 @@
     </collision>
   </link>
+  <joint name="table_center_joint" type="fixed">
+      <parent link="table"/>
+      <child link="table_center"/>
+      <origin xyz="${table_width/2} ${table_length/2} 0" rpy="0 0 ${-pi/2}"/>
+  </joint>
   <joint name="left_arm_mounting_plate_joint" type="fixed">
-    <parent link="table"/>
+    <parent link="table_center"/>
     <child link="left_arm_mounting_plate"/>
-    <origin xyz="${-table_length+left_arm_mounting_plate_x_offset+left_arm_mounting_plate_length/2} ${-left_arm_mounting_plate_y_offset-left_arm_mounting_plate_width/2} ${table_height}"/>
+    <origin xyz="${-table_length/2+left_arm_mounting_plate_x_offset+left_arm_mounting_plate_length/2} ${+table_width/2-left_arm_mounting_plate_y_offset-left_arm_mounting_plate_width/2} ${table_height}"/>
   </joint>
   <link name="left_arm_mounting_plate">
@@ -128,7 +137,7 @@
   </xacro:wsg_300_120_xacro>
   <joint name="right_arm_mounting_plate_joint" type="fixed">
-    <parent link="table"/>
+    <parent link="table_center"/>
     <child link="right_arm_mounting_plate"/>
-    <origin xyz="${-table_length+right_arm_mounting_plate_x_offset+right_arm_mounting_plate_length/2} ${-right_arm_mounting_plate_y_offset-right_arm_mounting_plate_width/2} ${table_height}"/>
+    <origin xyz="${-table_length/2+right_arm_mounting_plate_x_offset+right_arm_mounting_plate_length/2} ${+table_width/2-right_arm_mounting_plate_y_offset-right_arm_mounting_plate_width/2} ${table_height}"/>
   </joint>
   <link name="right_arm_mounting_plate">

Commit message: [DAiSy] Added fake camera link to satisfy Semantic Digital Twin's requirements of having a default camera.

File: iai_daisy_description/robots/daisy.urdf.xacro (robot description, xacro)
@@ -86,4 +86,17 @@
       <origin xyz="${table_width/2} ${table_length/2} 0" rpy="0 0 ${-pi/2}"/>
   </joint>
+  <link name="camera_link">
+    <visual>
+      <geometry>
+        <box size="0.12 0.03 0.03"/>
+      </geometry>
+      <material name="gray"/>
+    </visual>
+  </link>
+  <joint name="camera_joint" type="fixed">
+      <parent link="table_center"/>
+      <child link="camera_link"/>
+      <origin xyz="0 -0.28 1.2" rpy="${-pi/3} 0 0"/>
+  </joint>
   <joint name="left_arm_mounting_plate_joint" type="fixed">
     <parent link="table_center"/>

Commit message: Set up dedicated network for DAiSy and add realtime parameters
DAiSy now has an isolated network with different IP addesses than before.
The realtime parameters decrease possibility of delay in the communication.

File: iai_daisy_description/robots/daisy.urdf.xacro (robot description, xacro)
@@ -24,4 +24,5 @@
   <xacro:arg name="left_mock_sensor_commands" default="false" />
   <xacro:arg name="left_robot_ip" default="192.168.57.101" />
+  <xacro:arg name="left_reverse_ip" default="192.168.250.1" />
   <xacro:arg name="left_reverse_port" default="50012" />
   <xacro:arg name="left_script_sender_port" default="50011" />
@@ -36,4 +37,5 @@
   <xacro:arg name="right_mock_sensor_commands" default="false" />
   <xacro:arg name="right_robot_ip" default="192.168.57.100" />
+  <xacro:arg name="right_reverse_ip" default="192.168.250.1" />
   <xacro:arg name="right_reverse_port" default="50001" />
   <xacro:arg name="right_script_sender_port" default="50002" />
@@ -44,8 +46,10 @@
   <xacro:arg name="ur_output_recipe_filename" default="$(find ur_robot_driver)/resources/rtde_output_recipe.txt" />
   <xacro:arg name="ur_input_recipe_filename" default="$(find ur_robot_driver)/resources/rtde_input_recipe.txt" />
+  <xacro:arg name="non_blocking_read" default="true" />
+  <xacro:arg name="robot_receive_timeout" default="0.1" />
   <xacro:property name="M_PI" value="3.1415926535897931"/>
   <xacro:property name="table_height" value="0.6077" />
   <xacro:property name="table_length" value="1.19" />
-  <xacro:property name="table_width" value="0.60" />
+<xacro:property name="table_width" value="0.60" />
   <xacro:property name="left_arm_mounting_plate_width" value="0.18" />
   <xacro:property name="left_arm_mounting_plate_length" value="0.15" />
@@ -279,4 +283,5 @@
     kinematics_parameters_file="$(arg left_kinematics_parameters_file)"
     robot_ip="$(arg left_robot_ip)"
+    reverse_ip="$(arg left_reverse_ip)"
     script_filename="$(arg ur_script_filename)"
     output_recipe_filename="$(arg ur_output_recipe_filename)"
@@ -285,4 +290,6 @@
     mock_sensor_commands="$(arg left_mock_sensor_commands)"
     headless_mode="$(arg headless_mode)"
+    non_blocking_read="$(arg non_blocking_read)"
+    robot_receive_timeout="$(arg robot_receive_timeout)"
     reverse_port="$(arg left_reverse_port)"
     script_sender_port="$(arg left_script_sender_port)"
@@ -295,4 +302,5 @@
     kinematics_parameters_file="$(arg right_kinematics_parameters_file)"
     robot_ip="$(arg right_robot_ip)"
+    reverse_ip="$(arg right_reverse_ip)"
     script_filename="$(arg ur_script_filename)"
     output_recipe_filename="$(arg ur_output_recipe_filename)"
@@ -301,4 +309,6 @@
     mock_sensor_commands="$(arg right_mock_sensor_commands)"
     headless_mode="$(arg headless_mode)"
+    non_blocking_read="$(arg non_blocking_read)"
+    robot_receive_timeout="$(arg robot_receive_timeout)"
     reverse_port="$(arg right_reverse_port)"
     script_sender_port="$(arg right_script_sender_port)"

Commit message: Add cable guide and additional collision body to URDF/XACRO
Both objects allow better self collision avoidance.

File: iai_daisy_description/robots/daisy.urdf.xacro (robot description, xacro)
@@ -62,4 +62,57 @@
   <xacro:property name="right_arm_mounting_plate_x_offset" value="0.994" />
   <xacro:property name="right_arm_mounting_plate_y_offset" value="0.368" />
+  <!-- Gripper cable guide properties + macro === -->
+  <xacro:property name="gripper_side_cylinder_length" value="0.10" />
+  <xacro:property name="gripper_side_cylinder_radius" value="0.0175" /> <!-- 3.5 cm diameter -->
+  <xacro:property name="gripper_side_cylinder_y_offset" value="0.075" /> <!-- adjust to clear the mounting plate edge -->
+  <xacro:macro name="gripper_side_cylinder" params="parent prefix">
+    <link name="${prefix}_side_cylinder_link">
+      <visual>
+        <origin xyz="0 0 0" rpy="0 0 0"/>
+        <geometry>
+          <cylinder length="${gripper_side_cylinder_length}" radius="${gripper_side_cylinder_radius}"/>
+        </geometry>
+        <material name="grey"/>
+      </visual>
+      <collision>
+        <origin xyz="0 0 0" rpy="0 0 0"/>
+        <geometry>
+          <cylinder length="${gripper_side_cylinder_length}" radius="${gripper_side_cylinder_radius}"/>
+        </geometry>
+      </collision>
+    </link>
+    <joint name="${prefix}_side_cylinder_joint" type="fixed">
+      <parent link="${parent}"/>
+      <child link="${prefix}_side_cylinder_link"/>
+      <!-- offset in +Y of the parent frame; rpy=0 keeps the cylinder's
+           native Z-axis aligned with the parent's Z-axis -->
+      <origin xyz="0 ${gripper_side_cylinder_y_offset} -${gripper_side_cylinder_length/2 - 0.02}" rpy="0 0 0"/>
+    </joint>
+  </xacro:macro>
+    <!-- Gripper Wrist 2 collision === -->
+  <xacro:property name="gripper_collision_cylinder_length" value="0.005" />
+  <xacro:property name="gripper_collision_cylinder_radius" value="0.034" /> <!-- 7.2 cm diameter -->
+  <xacro:macro name="wrist_collision_cylinder_macro" params="parent prefix">
+    <link name="${prefix}_wrist_collision_cylinder_link">
+      <visual>
+        <origin xyz="0 0 0" rpy="0 0 0"/>
+        <geometry>
+          <cylinder length="${gripper_collision_cylinder_length}" radius="${gripper_collision_cylinder_radius}"/>
+        </geometry>
+        <material name="grey"/>
+      </visual>
+      <collision>
+        <origin xyz="0 0 0" rpy="0 0 0"/>
+        <geometry>
+          <cylinder length="${gripper_collision_cylinder_length}" radius="${gripper_collision_cylinder_radius}"/>
+        </geometry>
+      </collision>
+    </link>
+    <joint name="${prefix}_wrist_collision_cylinder_joint" type="fixed">
+      <parent link="${parent}"/>
+      <child link="${prefix}_wrist_collision_cylinder_link"/>
+      <origin xyz="0 -0.051 -0.0028" rpy="${pi/2} 0 0"/>
+    </joint>
+  </xacro:macro>
   <link name="map" />
   <link name="table"/>
@@ -132,5 +185,5 @@
   <link name="left_gripper_mounting_plate">
     <visual>
-      <origin xyz="0 0 0" rpy="0 0 0"/>
+      <origin xyz="0 0 0" rpy="${pi} 0 0"/>
       <geometry>
         <mesh filename="package://iai_daisy_description/meshes/FL-ISO50-WPG300_WITH_FILLET.stl" scale="0.001 0.001 0.001"/>
@@ -139,5 +192,5 @@
     </visual>
     <collision>
-      <origin xyz="0 0 0" rpy="0 0 0"/>
+      <origin xyz="0 0 0" rpy="${pi} 0 0"/>
       <geometry>
         <mesh filename="package://iai_daisy_description/meshes/FL-ISO50-WPG300_WITH_FILLET.stl" scale="0.001 0.001 0.001"/>
@@ -148,8 +201,11 @@
     <parent link="left_flange"/>
     <child link="left_gripper_mounting_plate"/>
-    <origin xyz="0 0 0.005" rpy="0 ${pi/2} 0"/>
-  </joint>
+    <origin xyz="0.005 0 0" rpy="0 ${pi/2} 0"/>
+  </joint>
+  <!-- === Cable guide on the left gripper === -->
+  <xacro:gripper_side_cylinder parent="left_gripper_mounting_plate" prefix="left_gripper" />
+  <xacro:wrist_collision_cylinder_macro parent="left_wrist_2_link" prefix="left_gripper" />
   <xacro:wsg_300_120_xacro parent="left_gripper_mounting_plate" name="left_gripper">
-    <origin xyz="0 0 0" rpy="0 0 0"/>
+    <origin xyz="0 0 0.005" rpy="0 0 0"/>
   </xacro:wsg_300_120_xacro>
   <joint name="right_arm_mounting_plate_joint" type="fixed">
@@ -182,5 +238,5 @@
   <link name="right_gripper_mounting_plate">
     <visual>
-      <origin xyz="0 0 0" rpy="0 0 0"/>
+      <origin xyz="0 0 0" rpy="${pi} 0 0"/>
       <geometry>
         <mesh filename="package://iai_daisy_description/meshes/FL-ISO50-WPG300_WITH_FILLET.stl" scale="0.001 0.001 0.001"/>
@@ -188,5 +244,5 @@
     </visual>
     <collision>
-      <origin xyz="0 0 0" rpy="0 0 0"/>
+      <origin xyz="0 0 0" rpy="${pi} 0 0"/>
       <geometry>
         <mesh filename="package://iai_daisy_description/meshes/FL-ISO50-WPG300_WITH_FILLET.stl" scale="0.001 0.001 0.001"/>
@@ -197,8 +253,11 @@
     <parent link="right_flange"/>
     <child link="right_gripper_mounting_plate"/>
-    <origin xyz="0 0 0.005" rpy="0 ${pi/2} 0"/>
-  </joint>
+    <origin xyz="0.005 0 0" rpy="-${pi/2} 0 -${pi/2}"/>
+  </joint>
+  <!-- === Cable guide on the right gripper === -->
+  <xacro:gripper_side_cylinder parent="right_gripper_mounting_plate" prefix="right_gripper" />
+  <xacro:wrist_collision_cylinder_macro parent="right_wrist_2_link" prefix="right_gripper" />
   <xacro:wsg_300_120_xacro parent="right_gripper_mounting_plate" name="right_gripper">
-    <origin xyz="0 0 0" rpy="0 0 0"/>
+    <origin xyz="0 0 0.005" rpy="0 0 0"/>
   </xacro:wsg_300_120_xacro>
   <link name="left_gripper_left_finger_tip_link">

Commit message: Fix DAiSy URDF/XACRO
Change thickness of one of the adapter mounting
plates from 0.006 to 0.01 like on the real robot.

File: iai_daisy_description/robots/daisy.urdf.xacro (robot description, xacro)
@@ -59,5 +59,5 @@
   <xacro:property name="right_arm_mounting_plate_width" value="0.18" />
   <xacro:property name="right_arm_mounting_plate_length" value="0.15" />
-  <xacro:property name="right_arm_mounting_plate_height" value="0.006" />
+  <xacro:property name="right_arm_mounting_plate_height" value="0.01" />
   <xacro:property name="right_arm_mounting_plate_x_offset" value="0.994" />
   <xacro:property name="right_arm_mounting_plate_y_offset" value="0.368" />

Commit message: Rotate gripper to fix orientation
Fits with the real robot now.

File: iai_daisy_description/robots/daisy.urdf.xacro (robot description, xacro)
@@ -185,5 +185,5 @@
   <link name="left_gripper_mounting_plate">
     <visual>
-      <origin xyz="0 0 0" rpy="${pi} 0 0"/>
+      <origin xyz="0 0 0" rpy="${pi} 0 ${pi/2}"/>
       <geometry>
         <mesh filename="package://iai_daisy_description/meshes/FL-ISO50-WPG300_WITH_FILLET.stl" scale="0.001 0.001 0.001"/>
@@ -192,5 +192,5 @@
     </visual>
     <collision>
-      <origin xyz="0 0 0" rpy="${pi} 0 0"/>
+      <origin xyz="0 0 0" rpy="${pi} 0 ${pi/2}"/>
       <geometry>
         <mesh filename="package://iai_daisy_description/meshes/FL-ISO50-WPG300_WITH_FILLET.stl" scale="0.001 0.001 0.001"/>
@@ -201,5 +201,5 @@
     <parent link="left_flange"/>
     <child link="left_gripper_mounting_plate"/>
-    <origin xyz="0.005 0 0" rpy="0 ${pi/2} 0"/>
+    <origin xyz="0.005 0 0" rpy="${pi/2} 0 ${pi/2}"/>
   </joint>
   <!-- === Cable guide on the left gripper === -->
@@ -207,5 +207,5 @@
   <xacro:wrist_collision_cylinder_macro parent="left_wrist_2_link" prefix="left_gripper" />
   <xacro:wsg_300_120_xacro parent="left_gripper_mounting_plate" name="left_gripper">
-    <origin xyz="0 0 0.005" rpy="0 0 0"/>
+    <origin xyz="0 0 0.005" rpy="0 0 -${pi/2}"/>
   </xacro:wsg_300_120_xacro>
   <joint name="right_arm_mounting_plate_joint" type="fixed">
@@ -238,5 +238,5 @@
   <link name="right_gripper_mounting_plate">
     <visual>
-      <origin xyz="0 0 0" rpy="${pi} 0 0"/>
+      <origin xyz="0 0 0" rpy="${pi} 0 ${pi/2}"/>
       <geometry>
         <mesh filename="package://iai_daisy_description/meshes/FL-ISO50-WPG300_WITH_FILLET.stl" scale="0.001 0.001 0.001"/>
@@ -244,5 +244,5 @@
     </visual>
     <collision>
-      <origin xyz="0 0 0" rpy="${pi} 0 0"/>
+      <origin xyz="0 0 0" rpy="${pi} 0 ${pi/2}"/>
       <geometry>
         <mesh filename="package://iai_daisy_description/meshes/FL-ISO50-WPG300_WITH_FILLET.stl" scale="0.001 0.001 0.001"/>
@@ -259,5 +259,5 @@
   <xacro:wrist_collision_cylinder_macro parent="right_wrist_2_link" prefix="right_gripper" />
   <xacro:wsg_300_120_xacro parent="right_gripper_mounting_plate" name="right_gripper">
-    <origin xyz="0 0 0.005" rpy="0 0 0"/>
+    <origin xyz="0 0 0.005" rpy="0 0 -${pi/2}"/>
   </xacro:wsg_300_120_xacro>
   <link name="left_gripper_left_finger_tip_link">

Commit message: daisy table collision is now a box

File: iai_daisy_description/robots/daisy.urdf.xacro (robot description, xacro)
@@ -131,7 +131,7 @@
     </visual>
     <collision>
-      <origin xyz="${table_length/2} ${table_width/2} 0" rpy="0 0 0"/>
-      <geometry>
-        <mesh filename="package://iai_table_robot_description/meshes/complete_table.stl"/>
+      <origin xyz="0 0 ${table_height/2}" rpy="0 0 0"/>
+      <geometry>
+        <box size="${table_length} ${table_width} ${table_height}"/>
       </geometry>
       <material name="gray"/>
